File: State Sensing Board/State Sensing Board.sch (KiCad schematic (older format))
At the start: 14 parts, among them J1 HallSensor_Conn, U1 AH1815-P, U2 AH1815-P

Commit message: Partial Update
Parts:
- added TP999: TestPoint, Frequently Used:Pad_1.25-2.5, symbol Naquadah_Generator:TestPoint
- C1, C2, R1, R29: footprint Naquadah_Generator:0805_2012Metric_HandSolder -> Frequently Used:0805_2012Metric_HandSolder
- TP101, TP102, TP103, TP104: footprint Naquadah_Generator:Pad_1.25-2.5 -> Frequently Used:Pad_1.25-2.5
Connections:
- wire segments 44 -> 45
Changed lines of the file:
@@
 F 0 "R2" H 5120 1796 50  0000 L CNN
 F 1 "47K" H 5120 1705 50  0000 L CNN
-F 2 "Naquadah_Generator:0805_2012Metric_HandSolder" V 4980 1750 50  0001 C CNN
+F 2 "Frequently Used:0805_2012Metric_HandSolder" V 4980 1750 50  0001 C CNN
 F 3 "http://www.koaspeer.com/pdfs/RK73H.pdf" H 5050 1750 50  0001 C CNN
 F 4 "2019-RK73H2ATTD4702FCT-ND" H 5050 1750 50  0001 C CNN "Digikey Part No."
@@
 F 0 "C2" H 3565 2246 50  0000 L CNN
 F 1 "47nF" H 3565 2155 50  0000 L CNN
-F 2 "Naquadah_Generator:0805_2012Metric_HandSolder" H 3488 2050 50  0001 C CNN
+F 2 "Frequently Used:0805_2012Metric_HandSolder" H 3488 2050 50  0001 C CNN
 F 3 "https://media.digikey.com/pdf/Data%20Sheets/Samsung%20PDFs/CL_Series_MLCC_ds.pdf" H 3450 2200 50  0001 C CNN
 F 4 "1276-2527-1-ND" H 3450 2200 50  0001 C CNN "Digikey Part No."
@@
 F 0 "R1" H 7420 1796 50  0000 L CNN
 F 1 "47K" H 7420 1705 50  0000 L CNN
-F 2 "Naquadah_Generator:0805_2012Metric_HandSolder" V 7280 1750 50  0001 C CNN
+F 2 "Frequently Used:0805_2012Metric_HandSolder" V 7280 1750 50  0001 C CNN
 F 3 "http://www.koaspeer.com/pdfs/RK73H.pdf" H 7350 1750 50  0001 C CNN
 F 4 "2019-RK73H2ATTD4702FCT-ND" H 7350 1750 50  0001 C CNN "Digikey Part No."
@@
 F 0 "C1" H 6015 2246 50  0000 L CNN
 F 1 "47nF" H 6015 2155 50  0000 L CNN
-F 2 "Naquadah_Generator:0805_2012Metric_HandSolder" H 5938 2050 50  0001 C CNN
+F 2 "Frequently Used:0805_2012Metric_HandSolder" H 5938 2050 50  0001 C CNN
 F 3 "https://media.digikey.com/pdf/Data%20Sheets/Samsung%20PDFs/CL_Series_MLCC_ds.pdf" H 5900 2200 50  0001 C CNN
 F 4 "1276-2527-1-ND" H 5900 2200 50  0001 C CNN "Digikey Part No."
@@
 F 0 "TP101" H 5150 3350 50  0000 L BNN
 F 1 "TestPoint" H 5150 3250 50  0001 L BNN
-F 2 "Naquadah_Generator:Pad_1.25-2.5" H 5400 3050 50  0001 C CNN
+F 2 "Frequently Used:Pad_1.25-2.5" H 5400 3050 50  0001 C CNN
 F 3 "None" H 5400 3050 50  0001 C CNN
 F 4 "GND" H 5150 3250 50  0000 L BNN "Name"
@@
 F 0 "TP104" H 5250 2400 50  0000 R BNN
 F 1 "TestPoint" H 5250 2500 50  0001 R BNN
-F 2 "Naquadah_Generator:Pad_1.25-2.5" H 5400 2200 50  0001 C CNN
+F 2 "Frequently Used:Pad_1.25-2.5" H 5400 2200 50  0001 C CNN
 F 3 "None" H 5400 2200 50  0001 C CNN
 F 4 "S2" H 5150 2500 50  0000 L BNN "Name"
@@
 F 0 "TP103" H 7550 2400 50  0000 R BNN
 F 1 "TestPoint" H 7550 2500 50  0001 R BNN
-F 2 "Naquadah_Generator:Pad_1.25-2.5" H 7700 2200 50  0001 C CNN
+F 2 "Frequently Used:Pad_1.25-2.5" H 7700 2200 50  0001 C CNN
 F 3 "None" H 7700 2200 50  0001 C CNN
 F 4 "S1" H 7450 2500 50  0000 L BNN "Name"
@@
 F 0 "TP102" H 5150 1550 50  0000 L BNN
 F 1 "TestPoint" H 5150 1450 50  0001 L BNN
-F 2 "Naquadah_Generator:Pad_1.25-2.5" H 5400 1250 50  0001 C CNN
+F 2 "Frequently Used:Pad_1.25-2.5" H 5400 1250 50  0001 C CNN
 F 3 "None" H 5400 1250 50  0001 C CNN
 F 4 "PWR" H 5150 1450 50  0000 L BNN "Name"
@@
 Connection ~ 6950 2750
 Wire Wire Line
-	6950 2750 6950 3050
+	6950 2750 6950 2950
 Wire Wire Line
 	5900 2050 5900 1600
@@
 Wire Wire Line
 	5050 2200 5200 2200
+$Comp
+L Naquadah_Generator:TestPoint TP999
+U 1 1 5EC6781B
+P 6950 2950
+F 0 "TP999" H 6900 3250 50  0000 L BNN
+F 1 "TestPoint" H 6900 3150 50  0001 L BNN
+F 2 "Frequently Used:Pad_1.25-2.5" H 7150 2950 50  0001 C CNN
+F 3 "None" H 7150 2950 50  0001 C CNN
+F 4 "TPTEST" H 6900 3150 50  0000 L BNN "Name"
+F 5 "None" H 6950 2950 50  0001 C CNN "Digikey Part No."
+F 6 "None" H 6950 2950 50  0001 C CNN "Manufacturer Name"
+F 7 "None" H 6950 2950 50  0001 C CNN "Manufacturer Part No."
+	1    6950 2950
+	0    1    1    0
+$EndComp
+Connection ~ 6950 2950
+Wire Wire Line
+	6950 2950 6950 3050
 $EndSCHEMATC

Commit message: Resize to correct for scale
Parts:
- removed LG1: OSHW Logo, Naquadah_Generator:OSHW_3mm_No_Text, symbol Naquadah_Generator:Logo
- removed TP999: TestPoint, Frequently Used:Pad_1.25-2.5, symbol Naquadah_Generator:TestPoint
- H1: footprint Naquadah_Generator:MountingSlot_2.7mm_2.7mm_M2.5 -> Naquadah_Generator:MountingSlot_2.2mm_2.2mm_M2.0
- TP101, TP102, TP103, TP104: footprint Frequently Used:Pad_1.25-2.5 -> Naquadah_Generator:Pad_1.25-1.25
Connections:
- wire segments 45 -> 44
Changed lines of the file:
@@
 L Mechanical:MountingHole H1
 U 1 1 5EA2820E
-P 8900 5250
-F 0 "H1" H 9000 5296 50  0000 L CNN
-F 1 "MountingHole" H 9000 5205 50  0000 L CNN
-F 2 "Naquadah_Generator:MountingSlot_2.7mm_2.7mm_M2.5" H 8900 5250 50  0001 C CNN
-F 3 "None" H 8900 5250 50  0001 C CNN
-F 4 "None" H 8900 5250 50  0001 C CNN "Digikey Part No."
-F 5 "None" H 8900 5250 50  0001 C CNN "Manufacturer Name"
-F 6 "None" H 8900 5250 50  0001 C CNN "Manufacturer Part No."
-	1    8900 5250
+P 8900 5450
+F 0 "H1" H 9000 5496 50  0000 L CNN
+F 1 "MountingHole" H 9000 5405 50  0000 L CNN
+F 2 "Naquadah_Generator:MountingSlot_2.2mm_2.2mm_M2.0" H 8900 5450 50  0001 C CNN
+F 3 "None" H 8900 5450 50  0001 C CNN
+F 4 "None" H 8900 5450 50  0001 C CNN "Digikey Part No."
+F 5 "None" H 8900 5450 50  0001 C CNN "Manufacturer Name"
+F 6 "None" H 8900 5450 50  0001 C CNN "Manufacturer Part No."
+	1    8900 5450
 	1    0    0    1
 $EndComp
@@
 Additional Features
 $Comp
-L Naquadah_Generator:Logo LG1
-U 1 1 5EAA34E4
-P 8900 5500
-F 0 "LG1" V 8854 5415 50  0000 R CNN
-F 1 "OSHW Logo" V 8945 5415 50  0000 R CNN
-F 2 "Naquadah_Generator:OSHW_3mm_No_Text" H 8900 5500 50  0001 C CNN
-F 3 "None" H 8900 5500 50  0001 C CNN
-F 4 "None" H 8900 5500 50  0001 C CNN "Digikey Part No."
-F 5 "None" H 8900 5500 50  0001 C CNN "Manufacturer Part No."
-F 6 "None" H 8900 5500 50  0001 C CNN "Manufacturer Name"
-	1    8900 5500
-	0    -1   1    0
-$EndComp
-$Comp
 L Naquadah_Generator:WireAssembly WA101
 U 1 1 5EF2EBE6
@@
 F 0 "TP101" H 5150 3350 50  0000 L BNN
 F 1 "TestPoint" H 5150 3250 50  0001 L BNN
-F 2 "Frequently Used:Pad_1.25-2.5" H 5400 3050 50  0001 C CNN
+F 2 "Naquadah_Generator:Pad_1.25-1.25" H 5400 3050 50  0001 C CNN
 F 3 "None" H 5400 3050 50  0001 C CNN
 F 4 "GND" H 5150 3250 50  0000 L BNN "Name"
@@
 F 0 "TP104" H 5250 2400 50  0000 R BNN
 F 1 "TestPoint" H 5250 2500 50  0001 R BNN
-F 2 "Frequently Used:Pad_1.25-2.5" H 5400 2200 50  0001 C CNN
+F 2 "Naquadah_Generator:Pad_1.25-1.25" H 5400 2200 50  0001 C CNN
 F 3 "None" H 5400 2200 50  0001 C CNN
 F 4 "S2" H 5150 2500 50  0000 L BNN "Name"
@@
 F 0 "TP103" H 7550 2400 50  0000 R BNN
 F 1 "TestPoint" H 7550 2500 50  0001 R BNN
-F 2 "Frequently Used:Pad_1.25-2.5" H 7700 2200 50  0001 C CNN
+F 2 "Naquadah_Generator:Pad_1.25-1.25" H 7700 2200 50  0001 C CNN
 F 3 "None" H 7700 2200 50  0001 C CNN
 F 4 "S1" H 7450 2500 50  0000 L BNN "Name"
@@
 F 0 "TP102" H 5150 1550 50  0000 L BNN
 F 1 "TestPoint" H 5150 1450 50  0001 L BNN
-F 2 "Frequently Used:Pad_1.25-2.5" H 5400 1250 50  0001 C CNN
+F 2 "Naquadah_Generator:Pad_1.25-1.25" H 5400 1250 50  0001 C CNN
 F 3 "None" H 5400 1250 50  0001 C CNN
 F 4 "PWR" H 5150 1450 50  0000 L BNN "Name"
@@
 Connection ~ 6950 2750
 Wire Wire Line
-	6950 2750 6950 2950
-Wire Wire Line
 	5900 2050 5900 1600
 Wire Wire Line
@@
 Wire Wire Line
 	5050 2200 5200 2200
-$Comp
-L Naquadah_Generator:TestPoint TP999
-U 1 1 5EC6781B
-P 6950 2950
-F 0 "TP999" H 6900 3250 50  0000 L BNN
-F 1 "TestPoint" H 6900 3150 50  0001 L BNN
-F 2 "Frequently Used:Pad_1.25-2.5" H 7150 2950 50  0001 C CNN
-F 3 "None" H 7150 2950 50  0001 C CNN
-F 4 "TPTEST" H 6900 3150 50  0000 L BNN "Name"
-F 5 "None" H 6950 2950 50  0001 C CNN "Digikey Part No."
-F 6 "None" H 6950 2950 50  0001 C CNN "Manufacturer Name"
-F 7 "None" H 6950 2950 50  0001 C CNN "Manufacturer Part No."
-	1    6950 2950
-	0    1    1    0
-$EndComp
-Connection ~ 6950 2950
-Wire Wire Line
-	6950 2950 6950 3050
+Wire Wire Line
+	6950 2750 6950 3050
 $EndSCHEMATC

Commit message: Updates to PCB Mount
Parts:
- H1: symbol Mechanical:MountingHole -> Naquadah_Generator:MountingHole
Changed lines of the file:
@@
 $EndComp
 $Comp
-L Mechanical:MountingHole H1
+L Naquadah_Generator:MountingHole H1
 U 1 1 5EA2820E
 P 8900 5450

Commit message: Adding Power Daughter Board
Parts:
- C1, C2: Digikey Part No. 1276-2527-1-ND -> (none); Source (none) -> Digikey; Source Part No. (none) -> 1276-2527-1-ND
- H1, TP101, TP102, TP103, TP104: Digikey Part No. None -> (none); Source (none) -> Digikey; Source Part No. (none) -> None
- J1: Digikey Part No. 455-1804-1-ND -> (none); Source (none) -> Digikey; Source Part No. (none) -> 455-1804-1-ND
- R1, R29: Digikey Part No. 2019-RK73H2ATTD4702FCT-ND -> (none); Source (none) -> Digikey; Source Part No. (none) -> 2019-RK73H2ATTD4702FCT-ND
- U1, U2: Digikey Part No. AH1815-W-7DICT-ND -> (none); Source (none) -> Digikey; Source Part No. (none) -> AH1815-W-7DICT-ND
- WA101: Digikey Part No. 455-3010-ND -> (none); Source (none) -> Digikey; Source Part No. (none) -> 455-3010-ND
Other:
- moved on the sheet: J1
Changed lines of the file:
@@
 F 2 "Naquadah_Generator:SC-59_Hall_Sensor_Handsoldering" H 4500 2200 50  0001 C CNN
 F 3 "https://www.diodes.com/assets/Datasheets/AH1806.pdf" H 4500 2200 50  0001 C CNN
-F 4 "AH1815-W-7DICT-ND" H 4500 2200 50  0001 C CNN "Digikey Part No."
+F 4 "AH1815-W-7DICT-ND" H 4500 2200 50  0001 C CNN "Source Part No."
 F 5 "Diodes Incorporated" H 4500 2200 50  0001 C CNN "Manufacturer Name"
 F 6 "AH1815-W-7" H 4500 2200 50  0001 C CNN "Manufacturer Part No."
+F 7 "Digikey" H 4500 2200 50  0001 C CNN "Source"
 	1    4500 2200
 	1    0    0    -1
@@
 F 2 "Frequently Used:0805_2012Metric_HandSolder" V 4980 1750 50  0001 C CNN
 F 3 "http://www.koaspeer.com/pdfs/RK73H.pdf" H 5050 1750 50  0001 C CNN
-F 4 "2019-RK73H2ATTD4702FCT-ND" H 5050 1750 50  0001 C CNN "Digikey Part No."
+F 4 "2019-RK73H2ATTD4702FCT-ND" H 5050 1750 50  0001 C CNN "Source Part No."
 F 5 "KOA Speer Electronics" H 5050 1750 50  0001 C CNN "Manufacturer Name"
 F 6 "RK73H2ATTD4702F" H 5050 1750 50  0001 C CNN "Manufacturer Part No."
+F 7 "Digikey" H 5050 1750 50  0001 C CNN "Source"
 	1    5050 1750
 	1    0    0    -1
@@
 F 2 "Frequently Used:0805_2012Metric_HandSolder" H 3488 2050 50  0001 C CNN
 F 3 "https://media.digikey.com/pdf/Data%20Sheets/Samsung%20PDFs/CL_Series_MLCC_ds.pdf" H 3450 2200 50  0001 C CNN
-F 4 "1276-2527-1-ND" H 3450 2200 50  0001 C CNN "Digikey Part No."
+F 4 "1276-2527-1-ND" H 3450 2200 50  0001 C CNN "Source Part No."
 F 5 "	Samsung Electro-Mechanics" H 3450 2200 50  0001 C CNN "Manufacturer Name"
 F 6 "CL21B473KBANNNC" H 3450 2200 50  0001 C CNN "Manufacturer Part No."
+F 7 "Digikey" H 3450 2200 50  0001 C CNN "Source"
 	1    3450 2200
 	1    0    0    -1
@@
 F 2 "Naquadah_Generator:SC-59_Hall_Sensor_Handsoldering" H 6950 2200 50  0001 C CNN
 F 3 "https://www.diodes.com/assets/Datasheets/AH1806.pdf" H 6950 2200 50  0001 C CNN
-F 4 "AH1815-W-7DICT-ND" H 6950 2200 50  0001 C CNN "Digikey Part No."
+F 4 "AH1815-W-7DICT-ND" H 6950 2200 50  0001 C CNN "Source Part No."
 F 5 "Diodes Incorporated" H 6950 2200 50  0001 C CNN "Manufacturer Name"
 F 6 "AH1815-W-7" H 6950 2200 50  0001 C CNN "Manufacturer Part No."
+F 7 "Digikey" H 6950 2200 50  0001 C CNN "Source"
 	1    6950 2200
 	1    0    0    -1
@@
 F 2 "Frequently Used:0805_2012Metric_HandSolder" V 7280 1750 50  0001 C CNN
 F 3 "http://www.koaspeer.com/pdfs/RK73H.pdf" H 7350 1750 50  0001 C CNN
-F 4 "2019-RK73H2ATTD4702FCT-ND" H 7350 1750 50  0001 C CNN "Digikey Part No."
+F 4 "2019-RK73H2ATTD4702FCT-ND" H 7350 1750 50  0001 C CNN "Source Part No."
 F 5 "KOA Speer Electronics" H 7350 1750 50  0001 C CNN "Manufacturer Name"
 F 6 "RK73H2ATTD4702F" H 7350 1750 50  0001 C CNN "Manufacturer Part No."
+F 7 "Digikey" H 7350 1750 50  0001 C CNN "Source"
 	1    7350 1750
 	1    0    0    -1
@@
 F 2 "Frequently Used:0805_2012Metric_HandSolder" H 5938 2050 50  0001 C CNN
 F 3 "https://media.digikey.com/pdf/Data%20Sheets/Samsung%20PDFs/CL_Series_MLCC_ds.pdf" H 5900 2200 50  0001 C CNN
-F 4 "1276-2527-1-ND" H 5900 2200 50  0001 C CNN "Digikey Part No."
+F 4 "1276-2527-1-ND" H 5900 2200 50  0001 C CNN "Source Part No."
 F 5 "	Samsung Electro-Mechanics" H 5900 2200 50  0001 C CNN "Manufacturer Name"
 F 6 "CL21B473KBANNNC" H 5900 2200 50  0001 C CNN "Manufacturer Part No."
+F 7 "Digikey" H 5900 2200 50  0001 C CNN "Source"
 	1    5900 2200
 	1    0    0    -1
@@
 F 2 "Naquadah_Generator:MountingSlot_2.2mm_2.2mm_M2.0" H 8900 5450 50  0001 C CNN
 F 3 "None" H 8900 5450 50  0001 C CNN
-F 4 "None" H 8900 5450 50  0001 C CNN "Digikey Part No."
+F 4 "None" H 8900 5450 50  0001 C CNN "Source Part No."
 F 5 "None" H 8900 5450 50  0001 C CNN "Manufacturer Name"
 F 6 "None" H 8900 5450 50  0001 C CNN "Manufacturer Part No."
+F 7 "Digikey" H 8900 5450 50  0001 C CNN "Source"
 	1    8900 5450
 	1    0    0    1
@@
 L Naquadah_Generator:State_Sensing_Conn J1
 U 1 1 5EA677CD
-P 3150 6750
-F 0 "J1" H 3150 6300 50  0000 C CNN
-F 1 "HallSensor_Conn" H 3150 6400 50  0000 C CNN
-F 2 "Naquadah_Generator:State_Sensing_Daughter_Board_JST_Conn" H 3150 7050 50  0001 C CNN
-F 3 "http://www.jst-mfg.com/product/pdf/eng/eSH.pdf" H 3150 6750 50  0001 C CNN
-F 4 "455-1804-1-ND" H 3150 6750 50  0001 C CNN "Digikey Part No."
-F 5 "JST Sales America Inc." H 3150 6750 50  0001 C CNN "Manufacturer Name"
-F 6 "SM04B-SRSS-TB(LF)(SN)" H 3150 6750 50  0001 C CNN "Manufacturer Part No."
-	1    3150 6750
+P 3200 6750
+F 0 "J1" H 3200 6300 50  0000 C CNN
+F 1 "HallSensor_Conn" H 3200 6400 50  0000 C CNN
+F 2 "Naquadah_Generator:State_Sensing_Daughter_Board_JST_Conn" H 3200 7050 50  0001 C CNN
+F 3 "http://www.jst-mfg.com/product/pdf/eng/eSH.pdf" H 3200 6750 50  0001 C CNN
+F 4 "455-1804-1-ND" H 3200 6750 50  0001 C CNN "Source Part No."
+F 5 "JST Sales America Inc." H 3200 6750 50  0001 C CNN "Manufacturer Name"
+F 6 "SM04B-SRSS-TB(LF)(SN)" H 3200 6750 50  0001 C CNN "Manufacturer Part No."
+F 7 "Digikey" H 3200 6750 50  0001 C CNN "Source"
+	1    3200 6750
 	-1   0    0    1
 $EndComp
@@
 F 2 "Naquadah_Generator:Wire_Assembly_Four" H 8650 5950 50  0001 C CNN
 F 3 "http://www.jst-mfg.com/product/pdf/eng/eSR.pdf" H 8650 5950 50  0001 C CNN
-F 4 "455-3010-ND" H 8650 5850 50  0001 C CNN "Digikey Part No."
+F 4 "455-3010-ND" H 8650 5850 50  0001 C CNN "Source Part No."
 F 5 "JST Sales America Inc." H 8650 5850 50  0001 C CNN "Manufacturer Name"
 F 6 "A04SR04SR30K51B" H 8650 5850 50  0001 C CNN "Manufacturer Part No."
+F 7 "Digikey" H 8650 5850 50  0001 C CNN "Source"
 	1    8650 5850
 	1    0    0    -1
@@
 F 3 "None" H 5400 3050 50  0001 C CNN
 F 4 "GND" H 5150 3250 50  0000 L BNN "Name"
-F 5 "None" H 5200 3050 50  0001 C CNN "Digikey Part No."
+F 5 "None" H 5200 3050 50  0001 C CNN "Source Part No."
 F 6 "None" H 5200 3050 50  0001 C CNN "Manufacturer Name"
 F 7 "None" H 5200 3050 50  0001 C CNN "Manufacturer Part No."
+F 8 "Digikey" H 5200 3050 50  0001 C CNN "Source"
 	1    5200 3050
 	1    0    0    -1
@@
 F 3 "None" H 5400 2200 50  0001 C CNN
 F 4 "S2" H 5150 2500 50  0000 L BNN "Name"
-F 5 "None" H 5200 2200 50  0001 C CNN "Digikey Part No."
+F 5 "None" H 5200 2200 50  0001 C CNN "Source Part No."
 F 6 "None" H 5200 2200 50  0001 C CNN "Manufacturer Name"
 F 7 "None" H 5200 2200 50  0001 C CNN "Manufacturer Part No."
+F 8 "Digikey" H 5200 2200 50  0001 C CNN "Source"
 	1    5200 2200
 	-1   0    0    1
@@
 F 3 "None" H 7700 2200 50  0001 C CNN
 F 4 "S1" H 7450 2500 50  0000 L BNN "Name"
-F 5 "None" H 7500 2200 50  0001 C CNN "Digikey Part No."
+F 5 "None" H 7500 2200 50  0001 C CNN "Source Part No."
 F 6 "None" H 7500 2200 50  0001 C CNN "Manufacturer Name"
 F 7 "None" H 7500 2200 50  0001 C CNN "Manufacturer Part No."
+F 8 "Digikey" H 7500 2200 50  0001 C CNN "Source"
 	1    7500 2200
 	-1   0    0    1
@@
 F 3 "None" H 5400 1250 50  0001 C CNN
 F 4 "PWR" H 5150 1450 50  0000 L BNN "Name"
-F 5 "None" H 5200 1250 50  0001 C CNN "Digikey Part No."
+F 5 "None" H 5200 1250 50  0001 C CNN "Source Part No."
 F 6 "None" H 5200 1250 50  0001 C CNN "Manufacturer Part No."
 F 7 "None" H 5200 1250 50  0001 C CNN "Manufacturer Name"
+F 8 "Digikey" H 5200 1250 50  0001 C CNN "Source"
 	1    5200 1250
 	1    0    0    -1

Commit message: PCB preliminary version
Parts:
- TP101: footprint Naquadah_Generator:Pad_1.25-1.25 -> Frequently_Used:Pad_1.25-1.25; Source Digikey -> None
- TP102, TP103, TP104: footprint Naquadah_Generator:Pad_1.25-1.25 -> Frequently_Used:Pad_1.25-1.25
Changed lines of the file:
@@
 F 0 "TP101" H 5150 3350 50  0000 L BNN
 F 1 "TestPoint" H 5150 3250 50  0001 L BNN
-F 2 "Naquadah_Generator:Pad_1.25-1.25" H 5400 3050 50  0001 C CNN
+F 2 "Frequently_Used:Pad_1.25-1.25" H 5400 3050 50  0001 C CNN
 F 3 "None" H 5400 3050 50  0001 C CNN
 F 4 "GND" H 5150 3250 50  0000 L BNN "Name"
@@
 F 6 "None" H 5200 3050 50  0001 C CNN "Manufacturer Name"
 F 7 "None" H 5200 3050 50  0001 C CNN "Manufacturer Part No."
-F 8 "Digikey" H 5200 3050 50  0001 C CNN "Source"
+F 8 "None" H 5200 3050 50  0001 C CNN "Source"
 	1    5200 3050
 	1    0    0    -1
@@
 F 0 "TP104" H 5250 2400 50  0000 R BNN
 F 1 "TestPoint" H 5250 2500 50  0001 R BNN
-F 2 "Naquadah_Generator:Pad_1.25-1.25" H 5400 2200 50  0001 C CNN
+F 2 "Frequently_Used:Pad_1.25-1.25" H 5400 2200 50  0001 C CNN
 F 3 "None" H 5400 2200 50  0001 C CNN
 F 4 "S2" H 5150 2500 50  0000 L BNN "Name"
@@
 F 0 "TP103" H 7550 2400 50  0000 R BNN
 F 1 "TestPoint" H 7550 2500 50  0001 R BNN
-F 2 "Naquadah_Generator:Pad_1.25-1.25" H 7700 2200 50  0001 C CNN
+F 2 "Frequently_Used:Pad_1.25-1.25" H 7700 2200 50  0001 C CNN
 F 3 "None" H 7700 2200 50  0001 C CNN
 F 4 "S1" H 7450 2500 50  0000 L BNN "Name"
@@
 F 0 "TP102" H 5150 1550 50  0000 L BNN
 F 1 "TestPoint" H 5150 1450 50  0001 L BNN
-F 2 "Naquadah_Generator:Pad_1.25-1.25" H 5400 1250 50  0001 C CNN
+F 2 "Frequently_Used:Pad_1.25-1.25" H 5400 1250 50  0001 C CNN
 F 3 "None" H 5400 1250 50  0001 C CNN
 F 4 "PWR" H 5150 1450 50  0000 L BNN "Name"

Commit message: Switched to 4 pin power board connector
Parts:
- TP101, TP102, TP103, TP104: symbol Naquadah_Generator:TestPoint -> Frequently_Used:TestPoint
Changed lines of the file:
@@
 $EndComp
 $Comp
-L Naquadah_Generator:TestPoint TP101
+L Frequently_Used:TestPoint TP101
 U 1 1 5EF333AD
 P 5200 3050
@@
 $EndComp
 $Comp
-L Naquadah_Generator:TestPoint TP104
+L Frequently_Used:TestPoint TP104
 U 1 1 5EF79EC8
 P 5200 2200
@@
 $EndComp
 $Comp
-L Naquadah_Generator:TestPoint TP103
+L Frequently_Used:TestPoint TP103
 U 1 1 5EF7C130
 P 7500 2200
@@
 $EndComp
 $Comp
-L Naquadah_Generator:TestPoint TP102
+L Frequently_Used:TestPoint TP102
 U 1 1 5EF7C9EB
 P 5200 1250

Commit message: Updates
Parts:
- J1: footprint Naquadah_Generator:State_Sensing_Daughter_Board_JST_Conn -> Naquadah_Generator:Daughter_Board_Hor_4_Pin_JST_Conn
Changed lines of the file:
@@
 F 0 "J1" H 3200 6300 50  0000 C CNN
 F 1 "HallSensor_Conn" H 3200 6400 50  0000 C CNN
-F 2 "Naquadah_Generator:State_Sensing_Daughter_Board_JST_Conn" H 3200 7050 50  0001 C CNN
+F 2 "Naquadah_Generator:Daughter_Board_Hor_4_Pin_JST_Conn" H 3200 7050 50  0001 C CNN
 F 3 "http://www.jst-mfg.com/product/pdf/eng/eSH.pdf" H 3200 6750 50  0001 C CNN
 F 4 "455-1804-1-ND" H 3200 6750 50  0001 C CNN "Source Part No."

Commit message: Move libraries and added configuration path.
Moved Li-Ion library to common KiCad library.  Added variables to configuration paths to reference my KiCad libraries.  Moved all 3D components to my common library.
Parts:
- TP101, TP102, TP103, TP104: footprint Frequently_Used:Pad_1.25-1.25 -> FrequentlyUsed:Pad_1.25-1.25; symbol Frequently_Used:TestPoint -> Frequently_Used_LE:TestPoint
Changed lines of the file:
@@
 $EndComp
 $Comp
-L Frequently_Used:TestPoint TP101
+L Frequently_Used_LE:TestPoint TP101
 U 1 1 5EF333AD
 P 5200 3050
 F 0 "TP101" H 5150 3350 50  0000 L BNN
 F 1 "TestPoint" H 5150 3250 50  0001 L BNN
-F 2 "Frequently_Used:Pad_1.25-1.25" H 5400 3050 50  0001 C CNN
+F 2 "FrequentlyUsed:Pad_1.25-1.25" H 5400 3050 50  0001 C CNN
 F 3 "None" H 5400 3050 50  0001 C CNN
 F 4 "GND" H 5150 3250 50  0000 L BNN "Name"
@@
 $EndComp
 $Comp
-L Frequently_Used:TestPoint TP104
+L Frequently_Used_LE:TestPoint TP104
 U 1 1 5EF79EC8
 P 5200 2200
 F 0 "TP104" H 5250 2400 50  0000 R BNN
 F 1 "TestPoint" H 5250 2500 50  0001 R BNN
-F 2 "Frequently_Used:Pad_1.25-1.25" H 5400 2200 50  0001 C CNN
+F 2 "FrequentlyUsed:Pad_1.25-1.25" H 5400 2200 50  0001 C CNN
 F 3 "None" H 5400 2200 50  0001 C CNN
 F 4 "S2" H 5150 2500 50  0000 L BNN "Name"
@@
 $EndComp
 $Comp
-L Frequently_Used:TestPoint TP103
+L Frequently_Used_LE:TestPoint TP103
 U 1 1 5EF7C130
 P 7500 2200
 F 0 "TP103" H 7550 2400 50  0000 R BNN
 F 1 "TestPoint" H 7550 2500 50  0001 R BNN
-F 2 "Frequently_Used:Pad_1.25-1.25" H 7700 2200 50  0001 C CNN
+F 2 "FrequentlyUsed:Pad_1.25-1.25" H 7700 2200 50  0001 C CNN
 F 3 "None" H 7700 2200 50  0001 C CNN
 F 4 "S1" H 7450 2500 50  0000 L BNN "Name"
@@
 $EndComp
 $Comp
-L Frequently_Used:TestPoint TP102
+L Frequently_Used_LE:TestPoint TP102
 U 1 1 5EF7C9EB
 P 5200 1250
 F 0 "TP102" H 5150 1550 50  0000 L BNN
 F 1 "TestPoint" H 5150 1450 50  0001 L BNN
-F 2 "Frequently_Used:Pad_1.25-1.25" H 5400 1250 50  0001 C CNN
+F 2 "FrequentlyUsed:Pad_1.25-1.25" H 5400 1250 50  0001 C CNN
 F 3 "None" H 5400 1250 50  0001 C CNN
 F 4 "PWR" H 5150 1450 50  0000 L BNN "Name"
