File: State Sensing Board/State Sensing Board.sch (KiCad schematic (older format))
At the start: 13 parts, among them J1 HallSensor_Conn, U1 AH1815-P, U2 AH1815-P

Commit message: Audio update
Parts:
- TP101, TP102, TP103, TP104: footprint FrequentlyUsed:Pad_1.25-1.25 -> Frequently_Used_LE:Pad_1.25-1.25
Changed lines of the file:
@@
 F 0 "TP101" H 5150 3350 50  0000 L BNN
 F 1 "TestPoint" H 5150 3250 50  0001 L BNN
-F 2 "FrequentlyUsed:Pad_1.25-1.25" H 5400 3050 50  0001 C CNN
+F 2 "Frequently_Used_LE:Pad_1.25-1.25" H 5400 3050 50  0001 C CNN
 F 3 "None" H 5400 3050 50  0001 C CNN
 F 4 "GND" H 5150 3250 50  0000 L BNN "Name"
@@
 F 0 "TP104" H 5250 2400 50  0000 R BNN
 F 1 "TestPoint" H 5250 2500 50  0001 R BNN
-F 2 "FrequentlyUsed:Pad_1.25-1.25" H 5400 2200 50  0001 C CNN
+F 2 "Frequently_Used_LE:Pad_1.25-1.25" H 5400 2200 50  0001 C CNN
 F 3 "None" H 5400 2200 50  0001 C CNN
 F 4 "S2" H 5150 2500 50  0000 L BNN "Name"
@@
 F 0 "TP103" H 7550 2400 50  0000 R BNN
 F 1 "TestPoint" H 7550 2500 50  0001 R BNN
-F 2 "FrequentlyUsed:Pad_1.25-1.25" H 7700 2200 50  0001 C CNN
+F 2 "Frequently_Used_LE:Pad_1.25-1.25" H 7700 2200 50  0001 C CNN
 F 3 "None" H 7700 2200 50  0001 C CNN
 F 4 "S1" H 7450 2500 50  0000 L BNN "Name"
@@
 F 0 "TP102" H 5150 1550 50  0000 L BNN
 F 1 "TestPoint" H 5150 1450 50  0001 L BNN
-F 2 "FrequentlyUsed:Pad_1.25-1.25" H 5400 1250 50  0001 C CNN
+F 2 "Frequently_Used_LE:Pad_1.25-1.25" H 5400 1250 50  0001 C CNN
 F 3 "None" H 5400 1250 50  0001 C CNN
 F 4 "PWR" H 5150 1450 50  0000 L BNN "Name"

Commit message: Power updates
Parts:
- C1, C2: symbol Naquadah_Generator:C -> Frequently_Used_LE:C
- R1, R29: symbol Naquadah_Generator:R -> Frequently_Used_LE:R
- TP101, TP102, TP103, TP104: value TestPoint -> TestPoint_1; symbol Frequently_Used_LE:TestPoint -> Frequently_Used_LE:TestPoint_1
Changed lines of the file:
@@
 $EndComp
 $Comp
-L Naquadah_Generator:R R29
+L Frequently_Used_LE:R R29
 U 1 1 5E9F2F30
 P 5050 1750
@@
 $EndComp
 $Comp
-L Naquadah_Generator:C C2
+L Frequently_Used_LE:C C2
 U 1 1 5E9F46C8
 P 3450 2200
@@
 $EndComp
 $Comp
-L Naquadah_Generator:R R?
+L Frequently_Used_LE:R R?
 U 1 1 5EA0E7B8
 P 7350 1750
@@
 $EndComp
 $Comp
-L Naquadah_Generator:C C?
+L Frequently_Used_LE:C C?
 U 1 1 5EA0E7CD
 P 5900 2200
@@
 $EndComp
 $Comp
-L Frequently_Used_LE:TestPoint TP101
+L Frequently_Used_LE:TestPoint_1 TP101
 U 1 1 5EF333AD
 P 5200 3050
 F 0 "TP101" H 5150 3350 50  0000 L BNN
-F 1 "TestPoint" H 5150 3250 50  0001 L BNN
+F 1 "TestPoint_1" H 5150 3250 50  0001 L BNN
 F 2 "Frequently_Used_LE:Pad_1.25-1.25" H 5400 3050 50  0001 C CNN
 F 3 "None" H 5400 3050 50  0001 C CNN
@@
 $EndComp
 $Comp
-L Frequently_Used_LE:TestPoint TP104
+L Frequently_Used_LE:TestPoint_1 TP104
 U 1 1 5EF79EC8
 P 5200 2200
 F 0 "TP104" H 5250 2400 50  0000 R BNN
-F 1 "TestPoint" H 5250 2500 50  0001 R BNN
+F 1 "TestPoint_1" H 5250 2500 50  0001 R BNN
 F 2 "Frequently_Used_LE:Pad_1.25-1.25" H 5400 2200 50  0001 C CNN
 F 3 "None" H 5400 2200 50  0001 C CNN
@@
 $EndComp
 $Comp
-L Frequently_Used_LE:TestPoint TP103
+L Frequently_Used_LE:TestPoint_1 TP103
 U 1 1 5EF7C130
 P 7500 2200
 F 0 "TP103" H 7550 2400 50  0000 R BNN
-F 1 "TestPoint" H 7550 2500 50  0001 R BNN
+F 1 "TestPoint_1" H 7550 2500 50  0001 R BNN
 F 2 "Frequently_Used_LE:Pad_1.25-1.25" H 7700 2200 50  0001 C CNN
 F 3 "None" H 7700 2200 50  0001 C CNN
@@
 $EndComp
 $Comp
-L Frequently_Used_LE:TestPoint TP102
+L Frequently_Used_LE:TestPoint_1 TP102
 U 1 1 5EF7C9EB
 P 5200 1250
 F 0 "TP102" H 5150 1550 50  0000 L BNN
-F 1 "TestPoint" H 5150 1450 50  0001 L BNN
+F 1 "TestPoint_1" H 5150 1450 50  0001 L BNN
 F 2 "Frequently_Used_LE:Pad_1.25-1.25" H 5400 1250 50  0001 C CNN
 F 3 "None" H 5400 1250 50  0001 C CNN

Commit message: Switched to 0603_1608M size for passives
Other:
- moved on the sheet: H1, WA101
Changed lines of the file:
@@
 L Naquadah_Generator:MountingHole H1
 U 1 1 5EA2820E
-P 8900 5450
-F 0 "H1" H 9000 5496 50  0000 L CNN
-F 1 "MountingHole" H 9000 5405 50  0000 L CNN
-F 2 "Naquadah_Generator:MountingSlot_2.2mm_2.2mm_M2.0" H 8900 5450 50  0001 C CNN
-F 3 "None" H 8900 5450 50  0001 C CNN
-F 4 "None" H 8900 5450 50  0001 C CNN "Source Part No."
-F 5 "None" H 8900 5450 50  0001 C CNN "Manufacturer Name"
-F 6 "None" H 8900 5450 50  0001 C CNN "Manufacturer Part No."
-F 7 "Digikey" H 8900 5450 50  0001 C CNN "Source"
-	1    8900 5450
+P 9150 5450
+F 0 "H1" H 9250 5496 50  0000 L CNN
+F 1 "MountingHole" H 9250 5405 50  0000 L CNN
+F 2 "Naquadah_Generator:MountingSlot_2.2mm_2.2mm_M2.0" H 9150 5450 50  0001 C CNN
+F 3 "None" H 9150 5450 50  0001 C CNN
+F 4 "None" H 9150 5450 50  0001 C CNN "Source Part No."
+F 5 "None" H 9150 5450 50  0001 C CNN "Manufacturer Name"
+F 6 "None" H 9150 5450 50  0001 C CNN "Manufacturer Part No."
+F 7 "Digikey" H 9150 5450 50  0001 C CNN "Source"
+	1    9150 5450
 	1    0    0    1
 $EndComp
@@
 Text Notes 4900 3500 0    98   ~ 20
 Hall Sensor Schematic
-Text Notes 3000 7700 0    98   ~ 20
+Text Notes 3000 7500 0    98   ~ 20
 Connectors
 Wire Notes Line
@@
 L Naquadah_Generator:WireAssembly WA101
 U 1 1 5EF2EBE6
-P 8650 5850
-F 0 "WA101" H 9028 5896 50  0000 L CNN
-F 1 "WireAssembly" H 9028 5805 50  0000 L CNN
-F 2 "Naquadah_Generator:Wire_Assembly_Four" H 8650 5950 50  0001 C CNN
-F 3 "http://www.jst-mfg.com/product/pdf/eng/eSR.pdf" H 8650 5950 50  0001 C CNN
-F 4 "455-3010-ND" H 8650 5850 50  0001 C CNN "Source Part No."
-F 5 "JST Sales America Inc." H 8650 5850 50  0001 C CNN "Manufacturer Name"
-F 6 "A04SR04SR30K51B" H 8650 5850 50  0001 C CNN "Manufacturer Part No."
-F 7 "Digikey" H 8650 5850 50  0001 C CNN "Source"
-	1    8650 5850
+P 8850 5850
+F 0 "WA101" H 9228 5896 50  0000 L CNN
+F 1 "WireAssembly" H 9228 5805 50  0000 L CNN
+F 2 "Naquadah_Generator:Wire_Assembly_Four" H 8850 5950 50  0001 C CNN
+F 3 "http://www.jst-mfg.com/product/pdf/eng/eSR.pdf" H 8850 5950 50  0001 C CNN
+F 4 "455-3010-ND" H 8850 5850 50  0001 C CNN "Source Part No."
+F 5 "JST Sales America Inc." H 8850 5850 50  0001 C CNN "Manufacturer Name"
+F 6 "A04SR04SR30K51B" H 8850 5850 50  0001 C CNN "Manufacturer Part No."
+F 7 "Digikey" H 8850 5850 50  0001 C CNN "Source"
+	1    8850 5850
 	1    0    0    -1
 $EndComp

Commit message: Update JST connectors
Parts:
- J1: footprint Naquadah_Generator:Daughter_Board_Hor_4_Pin_JST_Conn -> Connector_JST:JST_SH_SM04B-SRSS-TB_1x04-1MP_P1.00mm_Horizontal
- WA1: renamed from WA101; footprint Naquadah_Generator:Wire_Assembly_Four -> Mechanical_LE:Wire_Assembly; symbol Naquadah_Generator:WireAssembly -> Mechanical_LE:WireAssembly; Manufacturer Part No. A04SR04SR30K51B -> A04SR04SR30K152A; Source Part No. 455-3010-ND -> 455-3002-ND
Other:
- note added: "6 pin at 1 mm spacing cable assembly.\nThe cable is reversed.\nThe mother board and daughter board\nuse the same foot prints."
- moved on the sheet: H1, WA1
Changed lines of the file:
@@
 L Naquadah_Generator:MountingHole H1
 U 1 1 5EA2820E
-P 9150 5450
-F 0 "H1" H 9250 5496 50  0000 L CNN
-F 1 "MountingHole" H 9250 5405 50  0000 L CNN
-F 2 "Naquadah_Generator:MountingSlot_2.2mm_2.2mm_M2.0" H 9150 5450 50  0001 C CNN
-F 3 "None" H 9150 5450 50  0001 C CNN
-F 4 "None" H 9150 5450 50  0001 C CNN "Source Part No."
-F 5 "None" H 9150 5450 50  0001 C CNN "Manufacturer Name"
-F 6 "None" H 9150 5450 50  0001 C CNN "Manufacturer Part No."
-F 7 "Digikey" H 9150 5450 50  0001 C CNN "Source"
-	1    9150 5450
+P 8450 5600
+F 0 "H1" H 8550 5646 50  0000 L CNN
+F 1 "MountingHole" H 8550 5555 50  0000 L CNN
+F 2 "Naquadah_Generator:MountingSlot_2.2mm_2.2mm_M2.0" H 8450 5600 50  0001 C CNN
+F 3 "None" H 8450 5600 50  0001 C CNN
+F 4 "None" H 8450 5600 50  0001 C CNN "Source Part No."
+F 5 "None" H 8450 5600 50  0001 C CNN "Manufacturer Name"
+F 6 "None" H 8450 5600 50  0001 C CNN "Manufacturer Part No."
+F 7 "Digikey" H 8450 5600 50  0001 C CNN "Source"
+	1    8450 5600
 	1    0    0    1
 $EndComp
@@
 F 0 "J1" H 3200 6300 50  0000 C CNN
 F 1 "HallSensor_Conn" H 3200 6400 50  0000 C CNN
-F 2 "Naquadah_Generator:Daughter_Board_Hor_4_Pin_JST_Conn" H 3200 7050 50  0001 C CNN
+F 2 "Connector_JST:JST_SH_SM04B-SRSS-TB_1x04-1MP_P1.00mm_Horizontal" H 3200 7050 50  0001 C CNN
 F 3 "http://www.jst-mfg.com/product/pdf/eng/eSH.pdf" H 3200 6750 50  0001 C CNN
 F 4 "455-1804-1-ND" H 3200 6750 50  0001 C CNN "Source Part No."
@@
 Additional Features
 $Comp
-L Naquadah_Generator:WireAssembly WA101
+L Mechanical_LE:WireAssembly WA1
 U 1 1 5EF2EBE6
-P 8850 5850
-F 0 "WA101" H 9228 5896 50  0000 L CNN
-F 1 "WireAssembly" H 9228 5805 50  0000 L CNN
-F 2 "Naquadah_Generator:Wire_Assembly_Four" H 8850 5950 50  0001 C CNN
-F 3 "http://www.jst-mfg.com/product/pdf/eng/eSR.pdf" H 8850 5950 50  0001 C CNN
-F 4 "455-3010-ND" H 8850 5850 50  0001 C CNN "Source Part No."
-F 5 "JST Sales America Inc." H 8850 5850 50  0001 C CNN "Manufacturer Name"
-F 6 "A04SR04SR30K51B" H 8850 5850 50  0001 C CNN "Manufacturer Part No."
-F 7 "Digikey" H 8850 5850 50  0001 C CNN "Source"
-	1    8850 5850
+P 9850 5600
+F 0 "WA1" H 10100 5650 50  0000 L CNN
+F 1 "WireAssembly" H 10100 5550 50  0000 L CNN
+F 2 "Mechanical_LE:Wire_Assembly" H 9850 5700 50  0001 C CNN
+F 3 "https://www.digikey.com/htmldatasheets/production/1917075/0/0/1/axxsrxxsr30k152a-drawing.html" H 9850 5700 50  0001 C CNN
+F 4 "455-3002-ND" H 9850 5600 50  0001 C CNN "Source Part No."
+F 5 "JST Sales America Inc." H 9850 5600 50  0001 C CNN "Manufacturer Name"
+F 6 "A04SR04SR30K152A" H 9850 5600 50  0001 C CNN "Manufacturer Part No."
+F 7 "Digikey" H 9850 5600 50  0001 C CNN "Source"
+	1    9850 5600
 	1    0    0    -1
 $EndComp
@@
 Wire Wire Line
 	6950 2750 6950 3050
+Text Notes 9600 6100 0    50   ~ 0
+6 pin at 1 mm spacing cable assembly.\nThe cable is reversed.\nThe mother board and daughter board\nuse the same foot prints.
 $EndSCHEMATC

Commit message: Updated fiducials.
Parts:
- added FID1, FID2, FID3, FID4, FID5, FID6: Fiducial, Fiducial_LE:Fiducial_0.5mm_Mask1mm, symbol Mechanical_LE:Fiducial
- J1: footprint Connector_JST:JST_SH_SM04B-SRSS-TB_1x04-1MP_P1.00mm_Horizontal -> Connector_LE:JST_SH_SM04B-SRSS-TB_1x04-1MP_P1.00mm_Horizontal
Other:
- moved on the sheet: H1
Changed lines of the file:
@@
 L Naquadah_Generator:MountingHole H1
 U 1 1 5EA2820E
-P 8450 5600
-F 0 "H1" H 8550 5646 50  0000 L CNN
-F 1 "MountingHole" H 8550 5555 50  0000 L CNN
-F 2 "Naquadah_Generator:MountingSlot_2.2mm_2.2mm_M2.0" H 8450 5600 50  0001 C CNN
-F 3 "None" H 8450 5600 50  0001 C CNN
-F 4 "None" H 8450 5600 50  0001 C CNN "Source Part No."
-F 5 "None" H 8450 5600 50  0001 C CNN "Manufacturer Name"
-F 6 "None" H 8450 5600 50  0001 C CNN "Manufacturer Part No."
-F 7 "Digikey" H 8450 5600 50  0001 C CNN "Source"
-	1    8450 5600
+P 8700 5750
+F 0 "H1" H 8800 5796 50  0000 L CNN
+F 1 "MountingHole" H 8800 5705 50  0000 L CNN
+F 2 "Naquadah_Generator:MountingSlot_2.2mm_2.2mm_M2.0" H 8700 5750 50  0001 C CNN
+F 3 "None" H 8700 5750 50  0001 C CNN
+F 4 "None" H 8700 5750 50  0001 C CNN "Source Part No."
+F 5 "None" H 8700 5750 50  0001 C CNN "Manufacturer Name"
+F 6 "None" H 8700 5750 50  0001 C CNN "Manufacturer Part No."
+F 7 "Digikey" H 8700 5750 50  0001 C CNN "Source"
+	1    8700 5750
 	1    0    0    1
 $EndComp
@@
 F 0 "J1" H 3200 6300 50  0000 C CNN
 F 1 "HallSensor_Conn" H 3200 6400 50  0000 C CNN
-F 2 "Connector_JST:JST_SH_SM04B-SRSS-TB_1x04-1MP_P1.00mm_Horizontal" H 3200 7050 50  0001 C CNN
+F 2 "Connector_LE:JST_SH_SM04B-SRSS-TB_1x04-1MP_P1.00mm_Horizontal" H 3200 7050 50  0001 C CNN
 F 3 "http://www.jst-mfg.com/product/pdf/eng/eSH.pdf" H 3200 6750 50  0001 C CNN
 F 4 "455-1804-1-ND" H 3200 6750 50  0001 C CNN "Source Part No."
@@
 Text Notes 9600 6100 0    50   ~ 0
 6 pin at 1 mm spacing cable assembly.\nThe cable is reversed.\nThe mother board and daughter board\nuse the same foot prints.
+$Comp
+L Mechanical_LE:Fiducial FID1
+U 1 1 5F6AA7A9
+P 7550 5450
+F 0 "FID1" H 7635 5496 50  0000 L CNN
+F 1 "Fiducial" H 7550 5100 50  0001 C CNN
+F 2 "Fiducial_LE:Fiducial_0.5mm_Mask1mm" H 7550 5300 50  0001 C CNN
+F 3 "None" H 7500 5450 50  0001 C CNN
+F 4 "TOP1" H 7635 5405 50  0000 L CNN "Name"
+F 5 "None" H 7550 5000 50  0001 C CNN "Manufacturer Name"
+F 6 "None" H 7550 4900 50  0001 C CNN "Manufacturer Part No."
+F 7 "None" H 7550 4700 50  0001 C CNN "Source"
+F 8 "None" H 7550 4800 50  0001 C CNN "Source Part No."
+F 9 "Fiducial mark" H 7550 5200 50  0001 C CNN "Description"
+	1    7550 5450
+	1    0    0    -1
+$EndComp
+$Comp
+L Mechanical_LE:Fiducial FID2
+U 1 1 5F674B67
+P 7550 5700
+F 0 "FID2" H 7635 5746 50  0000 L CNN
+F 1 "Fiducial" H 7550 5350 50  0001 C CNN
+F 2 "Fiducial_LE:Fiducial_0.5mm_Mask1mm" H 7550 5550 50  0001 C CNN
+F 3 "None" H 7500 5700 50  0001 C CNN
+F 4 "TOP2" H 7635 5655 50  0000 L CNN "Name"
+F 5 "None" H 7550 5250 50  0001 C CNN "Manufacturer Name"
+F 6 "None" H 7550 5150 50  0001 C CNN "Manufacturer Part No."
+F 7 "None" H 7550 4950 50  0001 C CNN "Source"
+F 8 "None" H 7550 5050 50  0001 C CNN "Source Part No."
+F 9 "Fiducial mark" H 7550 5450 50  0001 C CNN "Description"
+	1    7550 5700
+	1    0    0    -1
+$EndComp
+$Comp
+L Mechanical_LE:Fiducial FID3
+U 1 1 5F675665
+P 7550 5950
+F 0 "FID3" H 7635 5996 50  0000 L CNN
+F 1 "Fiducial" H 7550 5600 50  0001 C CNN
+F 2 "Fiducial_LE:Fiducial_0.5mm_Mask1mm" H 7550 5800 50  0001 C CNN
+F 3 "None" H 7500 5950 50  0001 C CNN
+F 4 "TOP3" H 7635 5905 50  0000 L CNN "Name"
+F 5 "None" H 7550 5500 50  0001 C CNN "Manufacturer Name"
+F 6 "None" H 7550 5400 50  0001 C CNN "Manufacturer Part No."
+F 7 "None" H 7550 5200 50  0001 C CNN "Source"
+F 8 "None" H 7550 5300 50  0001 C CNN "Source Part No."
+F 9 "Fiducial mark" H 7550 5700 50  0001 C CNN "Description"
+	1    7550 5950
+	1    0    0    -1
+$EndComp
+$Comp
+L Mechanical_LE:Fiducial FID4
+U 1 1 5F677F81
+P 8050 5450
+F 0 "FID4" H 8135 5496 50  0000 L CNN
+F 1 "Fiducial" H 8050 5100 50  0001 C CNN
+F 2 "Fiducial_LE:Fiducial_0.5mm_Mask1mm" H 8050 5300 50  0001 C CNN
+F 3 "None" H 8000 5450 50  0001 C CNN
+F 4 "BOT1" H 8135 5405 50  0000 L CNN "Name"
+F 5 "None" H 8050 5000 50  0001 C CNN "Manufacturer Name"
+F 6 "None" H 8050 4900 50  0001 C CNN "Manufacturer Part No."
+F 7 "None" H 8050 4700 50  0001 C CNN "Source"
+F 8 "None" H 8050 4800 50  0001 C CNN "Source Part No."
+F 9 "Fiducial mark" H 8050 5200 50  0001 C CNN "Description"
+	1    8050 5450
+	1    0    0    -1
+$EndComp
+$Comp
+L Mechanical_LE:Fiducial FID5
+U 1 1 5F677F8D
+P 8050 5700
+F 0 "FID5" H 8135 5746 50  0000 L CNN
+F 1 "Fiducial" H 8050 5350 50  0001 C CNN
+F 2 "Fiducial_LE:Fiducial_0.5mm_Mask1mm" H 8050 5550 50  0001 C CNN
+F 3 "None" H 8000 5700 50  0001 C CNN
+F 4 "BOT2" H 8135 5655 50  0000 L CNN "Name"
+F 5 "None" H 8050 5250 50  0001 C CNN "Manufacturer Name"
+F 6 "None" H 8050 5150 50  0001 C CNN "Manufacturer Part No."
+F 7 "None" H 8050 4950 50  0001 C CNN "Source"
+F 8 "None" H 8050 5050 50  0001 C CNN "Source Part No."
+F 9 "Fiducial mark" H 8050 5450 50  0001 C CNN "Description"
+	1    8050 5700
+	1    0    0    -1
+$EndComp
+$Comp
+L Mechanical_LE:Fiducial FID6
+U 1 1 5F677F99
+P 8050 5950
+F 0 "FID6" H 8135 5996 50  0000 L CNN
+F 1 "Fiducial" H 8050 5600 50  0001 C CNN
+F 2 "Fiducial_LE:Fiducial_0.5mm_Mask1mm" H 8050 5800 50  0001 C CNN
+F 3 "None" H 8000 5950 50  0001 C CNN
+F 4 "BOT3" H 8135 5905 50  0000 L CNN "Name"
+F 5 "None" H 8050 5500 50  0001 C CNN "Manufacturer Name"
+F 6 "None" H 8050 5400 50  0001 C CNN "Manufacturer Part No."
+F 7 "None" H 8050 5200 50  0001 C CNN "Source"
+F 8 "None" H 8050 5300 50  0001 C CNN "Source Part No."
+F 9 "Fiducial mark" H 8050 5700 50  0001 C CNN "Description"
+	1    8050 5950
+	1    0    0    -1
+$EndComp
 $EndSCHEMATC
