File: State Sensing Board/State Sensing Board - Copy.sch (KiCad schematic (older format))
At the start: 14 parts, among them J1 HallSensor_Conn, U1 AH1815-P, U2 AH1815-P

Commit message: Changed name of libraries to remove underscore
Parts:
- C1, C2: Digikey Part No. 1276-2527-1-ND -> (none); Manufacturer Name Samsung Electro-Mechanics -> (none); Manufacturer Part No. CL21B473KBANNNC -> (none)
- H1: Digikey Part No. None -> (none); Manufacturer Name None -> (none); Manufacturer Part No. None -> (none)
- J1: value HallSensor_Conn -> HallSensor_Conn_T4; footprint Naquadah_Generator:State_Sensing_Daughter_Board_JST_Conn -> Naquadah_Generator:JST_SH_SM04B-SRSS-TB_1x04-1MP_P1.00mm_Horizontal; symbol Naquadah_Generator:State_Sensing_Conn -> Naquadah_Generator:HallSensor_Conn_T4; Digikey Part No. 455-1804-1-ND -> (none); Manufacturer Name JST Sales America Inc. -> (none); Manufacturer Part No. SM04B-SRSS-TB(LF)(SN) -> (none)
- LG1: Manufacturer Name None -> (none)
- R1, R29: Digikey Part No. 2019-RK73H2ATTD4702FCT-ND -> (none); Manufacturer Name KOA Speer Electronics -> (none); Manufacturer Part No. RK73H2ATTD4702F -> (none)
Changed lines of the file:
@@
 F 3 "https://www.diodes.com/assets/Datasheets/AH1806.pdf" H 4500 2200 50  0001 C CNN
 F 4 "AH1815-W-7DICT-ND" H 4500 2200 50  0001 C CNN "Digikey Part No."
-F 5 "Diodes Incorporated" H 4500 2200 50  0001 C CNN "Manufacturer Name"
-F 6 "AH1815-W-7" H 4500 2200 50  0001 C CNN "Manufacturer Part No."
+F 5 "" H 4500 2200 50  0001 C CNN "Manfacturer Part No."
+F 6 "Diodes Incorporated" H 4500 2200 50  0001 C CNN "Manufacturer Name"
+F 7 "AH1815-W-7" H 4500 2200 50  0001 C CNN "Manufacturer Part No."
 	1    4500 2200
 	1    0    0    -1
@@
 F 1 "47K" H 5120 1705 50  0000 L CNN
 F 2 "Naquadah_Generator:0805_2012Metric_HandSolder" V 4980 1750 50  0001 C CNN
-F 3 "http://www.koaspeer.com/pdfs/RK73H.pdf" H 5050 1750 50  0001 C CNN
-F 4 "2019-RK73H2ATTD4702FCT-ND" H 5050 1750 50  0001 C CNN "Digikey Part No."
-F 5 "KOA Speer Electronics" H 5050 1750 50  0001 C CNN "Manufacturer Name"
-F 6 "RK73H2ATTD4702F" H 5050 1750 50  0001 C CNN "Manufacturer Part No."
+F 3 "~" H 5050 1750 50  0001 C CNN
 	1    5050 1750
 	1    0    0    -1
@@
 F 1 "47nF" H 3565 2155 50  0000 L CNN
 F 2 "Naquadah_Generator:0805_2012Metric_HandSolder" H 3488 2050 50  0001 C CNN
-F 3 "https://media.digikey.com/pdf/Data%20Sheets/Samsung%20PDFs/CL_Series_MLCC_ds.pdf" H 3450 2200 50  0001 C CNN
-F 4 "1276-2527-1-ND" H 3450 2200 50  0001 C CNN "Digikey Part No."
-F 5 "	Samsung Electro-Mechanics" H 3450 2200 50  0001 C CNN "Manufacturer Name"
-F 6 "CL21B473KBANNNC" H 3450 2200 50  0001 C CNN "Manufacturer Part No."
+F 3 "~" H 3450 2200 50  0001 C CNN
 	1    3450 2200
 	1    0    0    -1
@@
 F 3 "https://www.diodes.com/assets/Datasheets/AH1806.pdf" H 6950 2200 50  0001 C CNN
 F 4 "AH1815-W-7DICT-ND" H 6950 2200 50  0001 C CNN "Digikey Part No."
-F 5 "Diodes Incorporated" H 6950 2200 50  0001 C CNN "Manufacturer Name"
-F 6 "AH1815-W-7" H 6950 2200 50  0001 C CNN "Manufacturer Part No."
+F 5 "" H 6950 2200 50  0001 C CNN "Manfacturer Part No."
+F 6 "Diodes Incorporated" H 6950 2200 50  0001 C CNN "Manufacturer Name"
+F 7 "AH1815-W-7" H 6950 2200 50  0001 C CNN "Manufacturer Part No."
 	1    6950 2200
 	1    0    0    -1
@@
 F 1 "47K" H 7420 1705 50  0000 L CNN
 F 2 "Naquadah_Generator:0805_2012Metric_HandSolder" V 7280 1750 50  0001 C CNN
-F 3 "http://www.koaspeer.com/pdfs/RK73H.pdf" H 7350 1750 50  0001 C CNN
-F 4 "2019-RK73H2ATTD4702FCT-ND" H 7350 1750 50  0001 C CNN "Digikey Part No."
-F 5 "KOA Speer Electronics" H 7350 1750 50  0001 C CNN "Manufacturer Name"
-F 6 "RK73H2ATTD4702F" H 7350 1750 50  0001 C CNN "Manufacturer Part No."
+F 3 "~" H 7350 1750 50  0001 C CNN
 	1    7350 1750
 	1    0    0    -1
@@
 F 1 "47nF" H 6015 2155 50  0000 L CNN
 F 2 "Naquadah_Generator:0805_2012Metric_HandSolder" H 5938 2050 50  0001 C CNN
-F 3 "https://media.digikey.com/pdf/Data%20Sheets/Samsung%20PDFs/CL_Series_MLCC_ds.pdf" H 5900 2200 50  0001 C CNN
-F 4 "1276-2527-1-ND" H 5900 2200 50  0001 C CNN "Digikey Part No."
-F 5 "	Samsung Electro-Mechanics" H 5900 2200 50  0001 C CNN "Manufacturer Name"
-F 6 "CL21B473KBANNNC" H 5900 2200 50  0001 C CNN "Manufacturer Part No."
+F 3 "~" H 5900 2200 50  0001 C CNN
 	1    5900 2200
 	1    0    0    -1
@@
 F 1 "MountingHole" H 9000 5205 50  0000 L CNN
 F 2 "Naquadah_Generator:MountingSlot_2.7mm_2.7mm_M2.5" H 8900 5250 50  0001 C CNN
-F 3 "None" H 8900 5250 50  0001 C CNN
-F 4 "None" H 8900 5250 50  0001 C CNN "Digikey Part No."
-F 5 "None" H 8900 5250 50  0001 C CNN "Manufacturer Name"
-F 6 "None" H 8900 5250 50  0001 C CNN "Manufacturer Part No."
+F 3 "~" H 8900 5250 50  0001 C CNN
 	1    8900 5250
 	1    0    0    1
 $EndComp
 $Comp
-L Naquadah_Generator:State_Sensing_Conn J1
+L Naquadah_Generator:HallSensor_Conn_T4 J1
 U 1 1 5EA677CD
-P 3150 6750
-F 0 "J1" H 3150 6300 50  0000 C CNN
-F 1 "HallSensor_Conn" H 3150 6400 50  0000 C CNN
-F 2 "Naquadah_Generator:State_Sensing_Daughter_Board_JST_Conn" H 3150 7050 50  0001 C CNN
-F 3 "http://www.jst-mfg.com/product/pdf/eng/eSH.pdf" H 3150 6750 50  0001 C CNN
-F 4 "455-1804-1-ND" H 3150 6750 50  0001 C CNN "Digikey Part No."
-F 5 "JST Sales America Inc." H 3150 6750 50  0001 C CNN "Manufacturer Name"
-F 6 "SM04B-SRSS-TB(LF)(SN)" H 3150 6750 50  0001 C CNN "Manufacturer Part No."
-	1    3150 6750
+P 3150 6800
+F 0 "J1" H 3227 6383 50  0000 C CNN
+F 1 "HallSensor_Conn_T4" H 3227 6474 50  0000 C CNN
+F 2 "Naquadah_Generator:JST_SH_SM04B-SRSS-TB_1x04-1MP_P1.00mm_Horizontal" H 3150 7100 50  0001 C CNN
+F 3 "~" H 3150 6800 50  0001 C CNN
+	1    3150 6800
 	-1   0    0    1
 $EndComp
@@
 F 3 "None" H 8900 5500 50  0001 C CNN
 F 4 "None" H 8900 5500 50  0001 C CNN "Digikey Part No."
-F 5 "None" H 8900 5500 50  0001 C CNN "Manufacturer Part No."
-F 6 "None" H 8900 5500 50  0001 C CNN "Manufacturer Name"
+F 5 "" H 8900 5500 50  0001 C CNN "Manfacturer Part No."
+F 6 "None" H 8900 5500 50  0001 C CNN "Manufacturer Part No."
 	1    8900 5500
 	0    -1   1    0
@@
 F 3 "http://www.jst-mfg.com/product/pdf/eng/eSR.pdf" H 8650 5950 50  0001 C CNN
 F 4 "455-3010-ND" H 8650 5850 50  0001 C CNN "Digikey Part No."
-F 5 "JST Sales America Inc." H 8650 5850 50  0001 C CNN "Manufacturer Name"
-F 6 "A04SR04SR30K51B" H 8650 5850 50  0001 C CNN "Manufacturer Part No."
+F 5 "" H 8650 5850 50  0001 C CNN "Manfacturer Part No."
+F 6 "JST Sales America Inc." H 8650 5850 50  0001 C CNN "Manufacturer Name"
+F 7 "A04SR04SR30K51B" H 8650 5850 50  0001 C CNN "Manufacturer Part No."
 	1    8650 5850
 	1    0    0    -1
@@
 F 4 "GND" H 5150 3250 50  0000 L BNN "Name"
 F 5 "None" H 5200 3050 50  0001 C CNN "Digikey Part No."
-F 6 "None" H 5200 3050 50  0001 C CNN "Manufacturer Name"
-F 7 "None" H 5200 3050 50  0001 C CNN "Manufacturer Part No."
+F 6 "" H 5200 3050 50  0001 C CNN "Manfacturer Part No."
+F 7 "None" H 5200 3050 50  0001 C CNN "Manufacturer Name"
+F 8 "None" H 5200 3050 50  0001 C CNN "Manufacturer Part No."
 	1    5200 3050
 	1    0    0    -1
@@
 F 4 "S2" H 5150 2500 50  0000 L BNN "Name"
 F 5 "None" H 5200 2200 50  0001 C CNN "Digikey Part No."
-F 6 "None" H 5200 2200 50  0001 C CNN "Manufacturer Name"
-F 7 "None" H 5200 2200 50  0001 C CNN "Manufacturer Part No."
+F 6 "" H 5200 2200 50  0001 C CNN "Manfacturer Part No."
+F 7 "None" H 5200 2200 50  0001 C CNN "Manufacturer Name"
+F 8 "None" H 5200 2200 50  0001 C CNN "Manufacturer Part No."
 	1    5200 2200
 	-1   0    0    1
@@
 F 4 "S1" H 7450 2500 50  0000 L BNN "Name"
 F 5 "None" H 7500 2200 50  0001 C CNN "Digikey Part No."
-F 6 "None" H 7500 2200 50  0001 C CNN "Manufacturer Name"
-F 7 "None" H 7500 2200 50  0001 C CNN "Manufacturer Part No."
+F 6 "" H 7500 2200 50  0001 C CNN "Manfacturer Part No."
+F 7 "None" H 7500 2200 50  0001 C CNN "Manufacturer Name"
+F 8 "None" H 7500 2200 50  0001 C CNN "Manufacturer Part No."
 	1    7500 2200
 	-1   0    0    1
