File: State Sensing Board/State Sensing Board.kicad_pcb (KiCad board)
At the start: 2 copper layers, 30.4 x 8.9 mm, 7 parts, among them J1 HallSensor_Conn, U1 AH1815-P, U2 AH1815-P

Commit message: Update State Sensing Board.kicad_pcb
Parts:
- C1, C2, R1, R2: moved to F.Cu
- moved R1 8.70 mm to (157.6, 89.4)
- moved C2 7.70 mm to (131.1, 89.4)
- moved C1 2.80 mm to (149.8, 89.4)
- moved R2 2.00 mm to (138.7, 89.4)
- moved U2 1.77 mm to (134.9, 89.4)
- moved U1 0.30 mm to (153.7, 89.4)
Routing:
- net /VCC: track 15.2 -> 45.9 mm
- net /GND: track 17.4 -> 36.6 mm
- net /OUT1: track 20.7 -> 5.78 mm
- net /OUT2: track 29.1 -> 25.2 mm, vias 3 -> 1
Other:
- board text added: "GND"
- board text added: "OUT1"
- board text added: "OUT2"
- board text added: "SENSOR 1"
- board text added: "SENSOR 2"
- board text added: "VCC"

Commit message: Update hall sensor board.
Parts:
- added H1: MountingHole, Naquadah_Generator:MountingSlot_2.7mm_2.7mm_M2.5, F.Cu at (139.6, 89.4)
- J1: footprint Naquadah_Generator:WireSoldPads -> Naquadah_Generator:WireSoldPads_1x4_NOL
- moved U2 10.7 mm to (124.2, 89.4)
- moved C2 10.7 mm to (120.4, 89.3)
- moved R2 10.7 mm to (128.0, 89.3)
- moved J1 3.49 mm to (155.5, 89.4), turned to 90 degrees
Connections:
- J1 pad 1: /VCC -> /OUT1
- J1 pad 2: /OUT1 -> /OUT2
- J1 pad 3: /OUT2 -> /GND
- J1 pad 4: /GND -> /VCC
Routing:
- net /VCC: track 45.9 -> 11.1 mm, vias 2 -> 1
- net /GND: track 36.6 -> 10.5 mm
- net /OUT2: track 25.2 -> 31.1 mm
- net /OUT1: track 5.78 -> 7.51 mm
- added copper zone on B.Cu, net /GND
- added copper zone on F.Cu, net /VCC
Other:
- board size 30.4 x 8.9 mm -> 39.2 x 9 mm
- net class Power added: clearance 0.4, trace_width 0.5, via_dia 1.6, via_drill 0.8

Commit message: Update component values
Parts:
- added G***: LOGO, Logos:OSHW_3mm_No_Text, B.Cu at (121.3, 89.3)
Other:
- board text added: "NQH-PCB-002"
- board text added: "V1.0.0"

Commit message: State sensing board revisions
Moved everything except hall sensors to back of state sensing board.
Parts:
- removed G***: LOGO, Logos:OSHW_3mm_No_Text
- C1, C2: value 50n -> 47n; footprint Capacitor_SMD:C_0603_1608Metric_Pad1.05x0.95mm_HandSolder -> Capacitor_SMD:C_1206_3216Metric_Pad1.42x1.75mm_HandSolder; moved to B.Cu
- J1: value HallSensor_Conn -> HallSensor_Conn_T4; footprint Naquadah_Generator:WireSoldPads_1x4_NOL -> Connector_JST:JST_SH_SM04B-SRSS-TB_1x04-1MP_P1.00mm_Horizontal
- R1, R2: value 50K -> 47K; footprint Resistor_SMD:R_0603_1608Metric_Pad1.05x0.95mm_HandSolder -> Resistor_SMD:R_1206_3216Metric_Pad1.42x1.75mm_HandSolder; moved to B.Cu
- U1, U2: footprint Package_TO_SOT_SMD:SC-59_Handsoldering -> Naquadah_Generator:SC-59_Hall_Sensor_Handsoldering
- moved R1 36.2 mm to (124.7, 104.5)
- moved H1 28.6 mm to (115.3, 104.5)
- moved J1 26.9 mm to (133.2, 104.5), turned to 270 degrees
- moved C1 26.6 mm to (128.0, 104.5)
- moved R2 26.5 mm to (106.2, 104.5)
- moved U2 25.3 mm to (103.8, 104.4)
- moved U1 25.3 mm to (133.3, 104.4)
- moved C2 23.1 mm to (103.0, 104.5)
Connections:
- C1 pad 1: /VCC -> +5V
- C1 pad 2: /GND -> GND
- C2 pad 1: /VCC -> +5V
- C2 pad 2: /GND -> GND
- J1 pad 1: /OUT1 -> GND
- J1 pad 2: /OUT2 -> +5V
- J1 pad 3: /GND -> OUT1
- J1 pad 4: /VCC -> OUT2
- R1 pad 1: /VCC -> +5V
- R1 pad 2: /OUT1 -> OUT1
- R2 pad 1: /VCC -> +5V
- R2 pad 2: /OUT2 -> OUT2
- U1 pad 1: /VCC -> +5V
- U1 pad 2: /GND -> GND
- U1 pad 3: /OUT1 -> OUT1
- U2 pad 1: /VCC -> +5V
- U2 pad 2: /GND -> GND
- U2 pad 3: /OUT2 -> OUT2
Routing:
- net OUT2: track 0.00 -> 31.4 mm, vias 0 -> 2
- net /OUT2: track 31.1 -> 0.00 mm, vias 1 -> 0
- net OUT1: track 0.00 -> 14.5 mm, vias 0 -> 1
- net /VCC: track 11.1 -> 0.00 mm, vias 1 -> 0
- net /GND: track 10.5 -> 0.00 mm, vias 2 -> 0
- net +5V: track 0.00 -> 8.05 mm, vias 0 -> 3
- net /OUT1: track 7.51 -> 0.00 mm, vias 1 -> 0
- net GND: track 0.00 -> 5.41 mm, vias 0 -> 2
- added copper zone on F.Cu, net +5V
- added copper zone on B.Cu, net GND
- removed copper zone on B.Cu, net /GND
- removed copper zone on F.Cu, net /VCC
Other:
- board size 39.2 x 9 mm -> 37.1 x 9 mm
- board text added: "1"
- board text added: "2"
- board text added: "G"
- board text added: "V"
- board text removed: "GND"
- board text removed: "OUT1"
- board text removed: "OUT2"
- board text removed: "VCC"

Commit message: Updates to State Sensing Board
Parts:
- added L1: OSHW Logo, Logos:OSHW_3mm_No_Text, B.Cu at (109.5, 104.5)

Commit message: Update State Sensing Board.kicad_pcb
Routing:
- net +5V: track 8.21 -> 10.2 mm, vias 3 -> 2
Changed lines of the file:
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@@
     (thickness 1.6)
     (drawings 19)
-    (tracks 44)
+    (tracks 45)
     (zones 0)
     (modules 9)
@@
   (page A4)
   (layers
-    (0 F.Cu signal hide)
+    (0 F.Cu signal)
     (31 B.Cu signal)
     (32 B.Adhes user)
-    (33 F.Adhes user hide)
+    (33 F.Adhes user)
     (34 B.Paste user)
     (35 F.Paste user)
@@
     (effects (font (size 1 1) (thickness 0.15)))
   )
-  (via (at 126.32 103.0125) (size 0.8) (drill 0.4) (layers F.Cu B.Cu) (net 1))
   (segment (start 102.393999 105.204999) (end 102.51 105.321) (width 0.25) (layer F.Cu) (net 2))
   (segment (start 127.96 103.0125) (end 126.32 103.0125) (width 0.25) (layer B.Cu) (net 1))
@@
   (segment (start 129.52 104) (end 129.51 103.99) (width 0.5) (layer B.Cu) (net 1))
   (segment (start 131.19 104) (end 129.52 104) (width 0.5) (layer B.Cu) (net 1))
+  (segment (start 128.5325 103.0125) (end 129.51 103.99) (width 0.25) (layer B.Cu) (net 1))
+  (segment (start 127.96 103.0125) (end 128.5325 103.0125) (width 0.25) (layer B.Cu) (net 1))
   (via (at 100.97 104.39) (size 0.8) (drill 0.4) (layers F.Cu B.Cu) (net 2))
   (segment (start 102.15 105.349999) (end 101 105.349999) (width 0.25) (layer F.Cu) (net 2))

Commit message: Before changing BOM
Parts:
- added TP101: GND, Naquadah_Generator:Pad_1.25-2.5, B.Cu at (121.1, 101.4)
- added TP102: PWR, Naquadah_Generator:Pad_1.25-2.5, B.Cu at (121.1, 104.0)
- added TP103: S1, Naquadah_Generator:Pad_1.25-2.5, B.Cu at (121.1, 105.8)
- added TP104: S2, Naquadah_Generator:Pad_1.25-2.5, B.Cu at (121.1, 107.6)
- added WA101: WireAssembly, Naquadah_Generator:Wire_Assembly_Four, F.Cu at (151.0, 104.5)
- C1, C2: footprint Capacitor_SMD:C_1206_3216Metric_Pad1.42x1.75mm_HandSolder -> Naquadah_Generator:C_1206_3216Metric_Pad1.42x1.75mm_HandSolder
- J1: footprint Connector_JST:JST_SH_SM04B-SRSS-TB_1x04-1MP_P1.00mm_Horizontal -> Naquadah_Generator:JST_SH_SM04B-SRSS-TB_1x04-1MP_P1.00mm_Horizontal
- LG1: renamed from L1; footprint Logos:OSHW_3mm_No_Text -> Naquadah_Generator:OSHW_3mm_No_Text
- R1, R2: footprint Resistor_SMD:R_1206_3216Metric_Pad1.42x1.75mm_HandSolder -> Naquadah_Generator:R_1206_3216Metric_Pad1.42x1.75mm_HandSolder
- moved H1 1.54 mm to (113.8, 104.5)
- moved LG1 0.47 mm to (109.0, 104.5)
Connections:
- net OUT1 renamed SENS1
- net OUT2 renamed SENS2
Routing:
- net SENS1: track 14.5 -> 18.5 mm
- net +5V: track 10.2 -> 13.5 mm, vias 2 -> 3
- net SENS2: track 31.4 -> 34.5 mm, vias 2 -> 3
- net GND: track 5.41 -> 4.71 mm

Commit message: Changed name of libraries to remove underscore
Parts:
- C1, C2: value 47n -> 47nF; footprint Naquadah_Generator:C_1206_3216Metric_Pad1.42x1.75mm_HandSolder -> Naquadah_Generator:0805_2012Metric_HandSolder
- J1: value HallSensor_Conn_T4 -> HallSensor_Conn; footprint Naquadah_Generator:JST_SH_SM04B-SRSS-TB_1x04-1MP_P1.00mm_Horizontal -> Naquadah_Generator:State_Sensing_Daughter_Board_JST_Conn
- R1, R2: footprint Naquadah_Generator:R_1206_3216Metric_Pad1.42x1.75mm_HandSolder -> Naquadah_Generator:0805_2012Metric_HandSolder
- TP101: value GND -> TestPoint
- TP102: value PWR -> TestPoint
- TP103: value S1 -> TestPoint
- TP104: value S2 -> TestPoint
Routing:
- net SENS1: track 18.5 -> 17.3 mm
