File: State Sensing Board/State Sensing Board.kicad_pcb (KiCad board)
At the start: 2 copper layers, 29.7 x 7.5 mm, 13 parts, among them J1 HallSensor_Conn, U1 AH1815-P, U2 AH1815-P

Commit message: Power board 2 switch V1
Changed lines of the file:
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@@
   )
   (gr_text NQH-PCB-002 (at 122.475 101.65 180) (layer F.SilkS)
-    (effects (font (size 1.25 1.25) (thickness 0.25)))
+    (effects (font (size 1.25 1.25) (thickness 0.2)))
   )
   (gr_text G (at 122.11 101.65) (layer B.SilkS)
@@
   (gr_line (start 133.3 103.999999) (end 133.3 104.999999) (layer Dwgs.User) (width 0.05))
   (gr_text V1.0.0 (at 122.475 107.25 180) (layer F.SilkS)
-    (effects (font (size 1.25 1.25) (thickness 0.25)))
+    (effects (font (size 1.25 1.25) (thickness 0.2)))
   )
   (gr_text 1 (at 130.48 106.746189 90) (layer B.SilkS)

Commit message: Move libraries and added configuration path.
Moved Li-Ion library to common KiCad library.  Added variables to configuration paths to reference my KiCad libraries.  Moved all 3D components to my common library.
Parts:
- J1: footprint Naquadah_Generator:State_Sensing_Daughter_Board_JST_Conn -> Naquadah_Generator:Daughter_Board_Hor_4_Pin_JST_Conn
- TP101, TP102, TP103, TP104: footprint Naquadah_Generator:Pad_1.25-1.25 -> FrequentlyUsed:Pad_1.25-1.25

Commit message: Update JST connectors
Parts:
- J1: footprint Naquadah_Generator:Daughter_Board_Hor_4_Pin_JST_Conn -> Connector_JST:JST_SH_SM04B-SRSS-TB_1x04-1MP_P1.00mm_Horizontal
- TP101, TP102, TP103, TP104: value TestPoint -> TestPoint_1; footprint FrequentlyUsed:Pad_1.25-1.25 -> Frequently_Used_LE:Pad_1.25-1.25
- WA1: renamed from WA101; footprint Naquadah_Generator:Wire_Assembly_Four -> Mechanical_LE:Wire_Assembly

Commit message: Updated fiducials.
Parts:
- added FID1: Fiducial, Fiducial_LE:Fiducial_0.5mm_Mask1mm, F.Cu at (114.3, 101.6)
- added FID2: Fiducial, Fiducial_LE:Fiducial_0.5mm_Mask1mm, F.Cu at (124.8, 104.5)
- added FID3: Fiducial, Fiducial_LE:Fiducial_0.5mm_Mask1mm, F.Cu at (136.3, 101.6)
- added FID4: Fiducial, Fiducial_LE:Fiducial_0.5mm_Mask1mm, B.Cu at (128.8, 107.5)
- added FID5: Fiducial, Fiducial_LE:Fiducial_0.5mm_Mask1mm, B.Cu at (120.4, 107.5)
- added FID6: Fiducial, Fiducial_LE:Fiducial_0.5mm_Mask1mm, B.Cu at (117.2, 107.5)
- J1: footprint Connector_JST:JST_SH_SM04B-SRSS-TB_1x04-1MP_P1.00mm_Horizontal -> Connector_LE:JST_SH_SM04B-SRSS-TB_1x04-1MP_P1.00mm_Horizontal
