File: Li-ion 5A Boost 1A Charge Protect/Li-ion 5A Boost 1A Charge Protect.kicad_pcb (KiCad board)
At the start: 2 copper layers, 78 x 22.7 mm, 38 parts, among them J1 USB_MICRO-B_FEMALE-SMT, U101 AP9101CK6, U102 ECH8695R-TL-W

Commit message: Updates before converting to 0805_2012
Parts:
- removed J1: USB_MICRO-B_FEMALE-SMT, Li-ion 5A Boost 1A Charge Protect:USB-B-MICRO-SMD
- added J101: USB_C_FEMALE, Li-ion 5A Boost 1A Charge Protect:GCT_USB4110-GF-A, F.Cu at (212.0, 94.4)
- added SW101: SW_SPST, Li-ion 5A Boost 1A Charge Protect:GF1230054, F.Cu at (214.8, 85.3)
- added U103: MCP73833T, Li-ion 5A Boost 1A Charge Protect:MCP73833, F.Cu at (213.4, 58.8)
- added U104: PAM2423AECADJR, Li-ion 5A Boost 1A Charge Protect:PAM2423AECADJR, F.Cu at (214.0, 52.7)
- added W103: 2.5x5.0, Li-ion 5A Boost 1A Charge Protect:Pad_2.5-5.0, F.Cu at (226.3, 95.3)
- added W104: 2.5x5.0, Li-ion 5A Boost 1A Charge Protect:Pad_2.5-5.0, F.Cu at (220.7, 95.0)
- added W107: 2.5x5.0, Li-ion 5A Boost 1A Charge Protect:Pad_2.5-5.0, F.Cu at (220.0, 52.4)
- C101, C102, C103, C104, C105, C106, C107, C108, C109, C110, C111: footprint Li-ion 5A Boost 1A Charge Protect:C_0603_1608Metric_HandSolder -> Li-ion 5A Boost 1A Charge Protect:0805_2012Metric_HandSolder
- D101: renamed from D1; value SS34 -> NTS12120EMFST1G; footprint Li-ion 5A Boost 1A Charge Protect:DO-214AC -> Li-ion 5A Boost 1A Charge Protect:NTS12120EMFST1G
- L101: value 6.8pH -> 6.8uH; footprint Li-ion 5A Boost 1A Charge Protect:CD75 -> Li-ion 5A Boost 1A Charge Protect:L_MGV1004
- LED101, LED102: value LED -> GREEN
- LED103: value LED -> RED
- R101, R103, R104, R105, R106, R107, R108, R109, R110, R111, TH101: footprint Li-ion 5A Boost 1A Charge Protect:R_0603_1608Metric_HandSolder -> Li-ion 5A Boost 1A Charge Protect:0805_2012Metric_HandSolder
- R102: value 2k7 -> 2.7k; footprint Li-ion 5A Boost 1A Charge Protect:R_0603_1608Metric_HandSolder -> Li-ion 5A Boost 1A Charge Protect:0805_2012Metric_HandSolder
- R112: value 1K -> 1k; footprint Li-ion 5A Boost 1A Charge Protect:R_0603_1608Metric_HandSolder -> Li-ion 5A Boost 1A Charge Protect:0805_2012Metric_HandSolder
- U101: footprint Package_TO_SOT_SMD:SOT-23-6 -> Li-ion 5A Boost 1A Charge Protect:SOT-23-6
- W101: value POW+ -> 2.5x5.0; footprint Li-ion 5A Boost 1A Charge Protect:Pad_2.54-5.08 -> Li-ion 5A Boost 1A Charge Protect:Pad_2.5-5.0
- W102: value POW- -> 2.5x5.0; footprint Li-ion 5A Boost 1A Charge Protect:Pad_2.54-5.08 -> Li-ion 5A Boost 1A Charge Protect:Pad_2.5-5.0
- W105: renamed from W103; value BATT+ -> 2.5x5.0; footprint Li-ion 5A Boost 1A Charge Protect:Pad_2.54-5.08 -> Li-ion 5A Boost 1A Charge Protect:Pad_2.5-5.0
- W106: renamed from W104; value BATT- -> 2.5x5.0; footprint Li-ion 5A Boost 1A Charge Protect:Pad_2.54-5.08 -> Li-ion 5A Boost 1A Charge Protect:Pad_2.5-5.0
- W108: renamed from W106; value GND -> 2.5x5.0; footprint Li-ion 5A Boost 1A Charge Protect:Pad_2.54-5.08 -> Li-ion 5A Boost 1A Charge Protect:Pad_2.5-5.0
- moved R111 102.3 mm to (243.0, 80.2), turned to 0 degrees
- moved L101 81.7 mm to (232.6, 85.2)
- moved D101 27.6 mm to (157.5, 58.8)
- moved R110 26.3 mm to (149.0, 61.0), turned to 270 degrees
- moved R112 23.9 mm to (170.2, 63.3)
- moved LED104 20.6 mm to (165.2, 61.1)
- moved R104 14.8 mm to (190.0, 58.2)
- moved C101 14.8 mm to (190.0, 55.6)
- moved C102 14.8 mm to (199.3, 44.5)
- moved C111 14.8 mm to (193.8, 50.1)
- moved LED102 14.8 mm to (190.4, 44.8)
- moved LED103 14.8 mm to (181.1, 55.9)
- moved R102 14.8 mm to (190.0, 53.1)
- moved R103 14.8 mm to (198.2, 50.1)
- moved R105 14.8 mm to (194.3, 52.6)
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Connections:
- C109 pad 1: (no net) -> Net-(C109-Pad1)
- D101 pad 2: (no net) -> Net-(D101-Pad2)
- L101 pad 2: (no net) -> Net-(D101-Pad2)
- R103 pad 1: (no net) -> /PG
- R104 pad 1: (no net) -> /ST2
- R105 pad 1: (no net) -> /ST1
- R106 pad 1: (no net) -> /PROG
Routing:
- net /BATT+: track 105.6 -> 0.00 mm, vias 1 -> 0
- net /GND: track 31.3 -> 0.00 mm, vias 53 -> 0
- net /VUSB: track 27.5 -> 0.00 mm, vias 2 -> 0
- net /5V_BOOST: track 19.5 -> 0.00 mm
- net Net-(IC1-Pad6): track 12.0 -> 0.00 mm
- net Net-(C1-Pad2): track 11.3 -> 0.00 mm
- net Net-(IC1-Pad7): track 8.69 -> 0.00 mm
- net Net-(U$1-Pad3): track 8.37 -> 0.00 mm
- net /FEEDBACK12V: track 7.07 -> 0.00 mm
- net /FEEDBACK5V: track 6.43 -> 0.00 mm
- net Net-(R4-Pad2): track 5.97 -> 0.00 mm
- net /BATT-: track 5.56 -> 0.00 mm
- net Net-(LED3-PadC): track 4.29 -> 0.00 mm
- net /PROG: track 3.08 -> 0.00 mm
- net Net-(U$1-Pad1): track 2.80 -> 0.00 mm
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- removed copper zone on F.Cu, net /12VBOOST
- removed copper zone on F.Cu, net /5V_BOOST
- removed copper zone on F.Cu, net /BATT+
- removed copper zone on F.Cu, net /BATT-
- removed copper zone on B.Cu, net /GND
- removed copper zone on F.Cu, net /GND
- removed copper zone on F.Cu, net /SWITCH12V
- removed copper zone on F.Cu, net /V-IN-BOOST
- removed copper zone on F.Cu, net /VUSB
Other:
- board text removed: "1k"
- board text removed: "22uF"
- board text removed: "22uH"
- board text removed: "7k5"
- board text removed: "MT3608"
- board text removed: "PvdW(2018)"
- board text removed: "SS34"

Commit message: Moved Li-Ion Libraries
Parts:
- C103, C111: footprint Li-ion 5A Boost 1A Charge Protect:0805_2012Metric_HandSolder -> Li-ion 5A Boost 1A Charge Protect:UCD1E471MNL1GS
- moved L101 101.0 mm to (132.1, 75.9)
- moved R111 96.6 mm to (147.0, 90.5)
- moved U104 82.0 mm to (141.0, 89.9)
- moved C107 77.8 mm to (136.1, 95.5), turned to 270 degrees
- moved R109 73.7 mm to (135.1, 92.5), turned to 180 degrees
- moved C105 71.3 mm to (134.1, 95.5), turned to 270 degrees
- moved C104 69.9 mm to (133.9, 89.2), turned to 270 degrees
- moved C109 67.3 mm to (139.2, 85.9), turned to 180 degrees
- moved C103 65.6 mm to (127.2, 89.4), turned to 270 degrees
- moved C106 54.1 mm to (136.1, 89.2), turned to 270 degrees
- moved C111 48.0 mm to (161.8, 85.9), turned to 270 degrees
- moved LED104 36.0 mm to (193.2, 83.7), turned to 270 degrees
- moved R112 34.0 mm to (193.2, 88.4)
- moved R110 27.5 mm to (147.0, 88.4), turned to 180 degrees
- moved W104 26.1 mm to (246.4, 99.3)
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Connections:
- net /FDBK renamed /FB
- net /V-IN-BOOST renamed /BOOSTVIN
- net Net-(C107-Pad1) renamed /COMP
- net Net-(C109-Pad1) renamed /SS
- C110 pad 1: /5V_BOOST -> /BOOSTVOUT
- C111 pad 1: /5V_BOOST -> /BOOSTVOUT
- D101 pad 1: /5V_BOOST -> /SW
- D101 pad 2: Net-(D101-Pad2) -> (no net)
- D101 pad 5: (no net) -> /BOOSTVOUT
- L101 pad 2: Net-(D101-Pad2) -> /SW
- LED104 pad 2: /5V_BOOST -> /BOOSTVOUT
- R110 pad 1: /5V_BOOST -> /BOOSTVOUT
- U104 pad 8: Net-(D101-Pad2) -> /SW
- W107 pad 1: /5V_BOOST -> /BOOSTVOUT

Commit message: Start of PCB Layout
Parts:
- W101, W102, W103, W104, W105, W106, W107, W108: footprint Li-ion 5A Boost 1A Charge Protect:Pad_2.5-5.0 -> Li-ion 5A Boost 1A Charge Protect:Pad_3.0-5.0
- moved J101 187.8 mm to (57.5, 45.8), turned to 270 degrees
- moved W103 139.6 mm to (119.5, 55.5), turned to 90 degrees
- moved W104 135.8 mm to (119.5, 51.0), turned to 90 degrees
- moved W101 129.7 mm to (56.8, 54.2), turned to 90 degrees
- moved W102 126.0 mm to (57.0, 37.0), turned to 90 degrees
- moved R101 121.7 mm to (81.1, 77.8), turned to 180 degrees
- moved C102 121.5 mm to (77.8, 43.3), turned to 270 degrees
- moved U103 120.9 mm to (93.6, 43.2)
- moved SW101 117.3 mm to (126.0, 64.0)
- moved R105 113.4 mm to (81.1, 47.5), turned to 90 degrees
- moved C101 111.6 mm to (81.1, 80.4), turned to 180 degrees
- moved R103 110.5 mm to (87.7, 47.5), turned to 90 degrees
- moved R108 107.8 mm to (91.0, 47.5), turned to 270 degrees
- moved R104 106.1 mm to (84.4, 47.5), turned to 90 degrees
- moved LED102 106.0 mm to (84.4, 43.2), turned to 90 degrees
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Connections:
- C101 pad 1: Net-(C101-Pad1) -> /BATT+
- R101 pad 1: Net-(C101-Pad1) -> /BATT+
- R107 pad 1: /THERM -> /THRM
- R107 pad 2: /THERM -> /THRMIC
- R108 pad 1: /THERM -> /THRM
- TH101 pad 1: /THERM -> /THRM
- U101 pad 5: Net-(C101-Pad1) -> /BATT+
- U102 pad 6: Net-(U102-Pad6) -> (no net)
- U102 pad 7: Net-(U102-Pad6) -> (no net)
- U102 pad 8: Net-(U102-Pad6) -> (no net)
- U103 pad 2: (no net) -> /VUSB
- U103 pad 8: /THERM -> /THRMIC
- U103 pad 9: (no net) -> /BATT+
Routing:
- net GND: track 0.00 -> 6.50 mm
- net Net-(LED101-Pad1): track 0.00 -> 2.39 mm
- net Net-(LED102-Pad1): track 0.00 -> 2.20 mm
- net Net-(LED103-Pad1): track 0.00 -> 2.12 mm

Commit message: Updates
Parts:
- removed C101: 100nF, Li-ion 5A Boost 1A Charge Protect:0805_2012Metric_HandSolder
- removed C103: 470uF, Li-ion 5A Boost 1A Charge Protect:UCD1E471MNL1GS
- removed C105: 2.2nF, Li-ion 5A Boost 1A Charge Protect:0805_2012Metric_HandSolder
- removed LED103: RED, Li-ion 5A Boost 1A Charge Protect:LED_0805_2012Metric_HandSolder
- removed R109: 51k, Li-ion 5A Boost 1A Charge Protect:0805_2012Metric_HandSolder
- added C1: 100nF, Li-ion 5A Boost 1A Charge Protect:0805_2012Metric_HandSolder, F.Cu at (81.1, 80.4)
- added C3: 470uF, Li-ion 5A Boost 1A Charge Protect:UCD1E471MNL1GS, F.Cu at (124.0, 76.9)
- added C5: 2.2nF, Li-ion 5A Boost 1A Charge Protect:0805_2012Metric_HandSolder, F.Cu at (122.8, 85.4)
- added LED3: RED, Li-ion 5A Boost 1A Charge Protect:LED_0805_2012Metric_HandSolder, F.Cu at (81.1, 43.2)
- added R9: 51k, Li-ion 5A Boost 1A Charge Protect:0805_2012Metric_HandSolder, F.Cu at (127.1, 87.0)
- moved W8 1.44 mm to (166.4, 86.9)
- moved LED4 0.80 mm to (155.4, 82.5)
- moved R12 0.80 mm to (155.4, 87.9)
- moved C11 0.50 mm to (162.5, 76.9)
- moved C10 0.40 mm to (152.1, 82.5)
- moved C9 0.40 mm to (152.1, 87.9)
- moved U4 0.40 mm to (140.1, 87.0)
- moved W7 0.35 mm to (160.0, 86.9)
- moved D1 0.32 mm to (151.2, 73.7)
- renumbered C110 to C10, C111 to C11, C102 to C2, C104 to C4, C106 to C6, C107 to C7, C108 to C8, C109 to C9, D101 to D1, J101 to J1, L101 to L1, LED101 to LED1, LED102 to LED2, LED104 to LED4, R101 to R1, R110 to R10, R111 to R11, R112 to R12, R102 to R2, R103 to R3, R104 to R4, R105 to R5, R106 to R6, R107 to R7, R108 to R8, SW101 to SW1, TH101 to TH1, U101 to U1, U102 to U2, U103 to U3, U104 to U4, W101 to W1, W102 to W2, W103 to W3, W104 to W4, W105 to W5, W106 to W6, W107 to W7, W108 to W8
