File: Li-ion 5A Boost 1A Charge Protect/Li-ion 5A Boost 1A Charge Protect.kicad_pcb (KiCad board)
At the start: 2 copper layers, 78 x 22.7 mm, 44 parts, among them J1 USB_C_FEMALE, SW1 SW_SPST, U1 AP9101CK6, U2 ECH8695R-TL-W, U3 MCP73833T, U4 PAM2423AECADJR

Commit message: Preliminary PCB layout 1
Parts:
- moved W5 86.3 mm to (167.2, 62.4), turned to 270 degrees
- moved J1 76.7 mm to (131.3, 66.6), turned to 180 degrees
- moved C8 69.9 mm to (166.6, 67.9)
- moved U3 69.1 mm to (159.9, 62.7)
- moved C2 68.1 mm to (143.1, 62.8)
- moved LED1 68.1 mm to (153.0, 62.8)
- moved LED2 68.1 mm to (149.7, 62.8)
- moved LED3 68.1 mm to (146.4, 62.8)
- moved W1 65.7 mm to (121.9, 62.9), turned to 0 degrees
- moved W2 65.4 mm to (117.0, 62.9), turned to 0 degrees
- moved R7 65.3 mm to (159.8, 67.9)
- moved R4 65.3 mm to (146.4, 67.9)
- moved R5 65.3 mm to (143.1, 67.9)
- moved R8 65.3 mm to (153.0, 67.9)
- moved TH1 65.3 mm to (156.5, 67.9)
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Connections:
- C1 pad 1: /BATT+ -> /PVDD
- R1 pad 1: /BATT+ -> /PVDD
- U1 pad 5: /BATT+ -> /PVDD
Routing:
- net /BATT-: track 0.00 -> 17.3 mm
- net Net-(U1-Pad3): track 0.00 -> 9.62 mm, vias 0 -> 2
- net /PVDD: track 0.00 -> 6.91 mm
- net GND: track 6.50 -> 0.00 mm
- net Net-(U1-Pad1): track 0.00 -> 6.47 mm, vias 0 -> 2
- net Net-(R2-Pad1): track 0.00 -> 4.86 mm
- net Net-(LED1-Pad1): track 2.39 -> 0.14 mm
- net Net-(LED3-Pad1): track 2.12 -> 0.00 mm
- net Net-(LED2-Pad1): track 2.20 -> 0.57 mm
- added copper zone on F.Cu, net /BATT-
- added copper zone on F.Cu, net GND
Other:
- net class High Power added: clearance 0.1524, trace_width 0.5, via_dia 1.2, via_drill 0.6

Commit message: Updates  to PCB
Parts:
- moved R2 6.86 mm to (116.3, 84.2), turned to 270 degrees
- moved J1 2.35 mm to (133.5, 67.4)
- moved W4 2.07 mm to (111.7, 63.7)
- moved W3 1.89 mm to (106.5, 63.7)
- moved W1 1.89 mm to (123.6, 63.7)
- moved W2 1.63 mm to (118.4, 63.7)
- moved U4 1.00 mm to (141.1, 87.0)
- moved SW1 0.99 mm to (109.0, 70.2)
- moved C1 0.70 mm to (105.8, 84.7)
- moved R1 0.70 mm to (105.8, 81.3)
- moved U1 0.70 mm to (112.2, 81.8)
- moved U2 0.70 mm to (112.2, 86.8)
- moved W6 0.70 mm to (106.8, 87.8)
- moved W5 0.51 mm to (166.8, 62.7)
- moved D1 0.30 mm to (151.2, 74.0)
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Routing:
- net /COMP: track 0.00 -> 16.0 mm
- net Net-(U1-Pad1): track 6.47 -> 0.01 mm, vias 2 -> 0
- net /PVDD: track 6.91 -> 8.09 mm
- net Net-(R2-Pad1): track 4.86 -> 4.14 mm
- net Net-(LED2-Pad1): track 0.57 -> 0.00 mm
- added copper zone on F.Cu, net /BATT+
- added copper zone on F.Cu, net /BOOSTVIN
- added copper zone on F.Cu, net /VUSB
Other:
- board text added: "ST1"
- board text added: "ST2"

Commit message: PCB Updates
Parts:
- moved R10 3.30 mm to (152.1, 82.5)
- moved R11 3.30 mm to (152.1, 87.9)
- moved C9 3.28 mm to (148.9, 87.9)
- moved C10 3.23 mm to (148.9, 82.5)
Routing:
- net GND: track 0.00 -> 58.3 mm, vias 0 -> 11
- net /PG: track 0.00 -> 19.5 mm
- net /FB: track 0.00 -> 12.4 mm
- net /THRM: track 0.00 -> 8.38 mm
- net Net-(U1-Pad1): track 0.01 -> 6.68 mm, vias 0 -> 2
- net /THRMIC: track 0.00 -> 5.87 mm
- net Net-(LED2-Pad1): track 0.00 -> 5.72 mm
- net Net-(LED1-Pad1): track 0.14 -> 5.84 mm
- net Net-(LED3-Pad1): track 0.00 -> 5.52 mm
- net /SS: track 0.00 -> 5.48 mm
- net /PROG: track 0.00 -> 3.57 mm
- net Net-(LED4-Pad1): track 0.00 -> 3.42 mm
- net Net-(C5-Pad1): track 0.00 -> 3.33 mm
- added copper zone on F.Cu, net /BOOSTVOUT
- added copper zone on B.Cu, net GND
Other:
- board text added: "1"
- board text added: "2"
- board text added: "P"
- board text added: "POWER"

Commit message: Updated diode footprint
Routing:
- net GND: track 58.3 -> 59.7 mm, vias 11 -> 12
Other:
- board text added: "1 - STAT 1"
- board text added: "2 - STAT 2"
- board text added: "P - PWR GD"
- board text removed: "STAT1"
- board text removed: "STAT2"
Changed lines of the file:
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@@
     (thickness 1.6)
     (drawings 63)
-    (tracks 148)
+    (tracks 151)
     (zones 0)
     (modules 44)
@@
     (effects (font (size 0.9652 0.9652) (thickness 0.13208)) (justify left bottom))
   )
-  (gr_circle (center 178.5 125) (end 179 125) (layer F.SilkS) (width 1))
-  (gr_text "SYSTEM TEST" (at 186.5 125) (layer F.SilkS)
+  (gr_circle (center 172.89 118.63) (end 173.39 118.63) (layer F.SilkS) (width 1))
+  (gr_text "SYSTEM TEST" (at 180.89 118.63) (layer F.SilkS)
     (effects (font (size 1.25 1.25) (thickness 0.2)) (justify left))
   )
-  (gr_circle (center 181.5 125) (end 182 125) (layer F.SilkS) (width 1))
-  (gr_circle (center 184.5 125) (end 185 125) (layer F.SilkS) (width 1))
-  (gr_circle (center 178.5 120) (end 179 120) (layer F.SilkS) (width 1))
-  (gr_circle (center 181.5 122.5) (end 182 122.5) (layer F.SilkS) (width 1))
-  (gr_text "CHARGE COMPLETE" (at 186.5 122.5) (layer F.SilkS)
+  (gr_circle (center 175.89 118.63) (end 176.39 118.63) (layer F.SilkS) (width 1))
+  (gr_circle (center 178.89 118.63) (end 179.39 118.63) (layer F.SilkS) (width 1))
+  (gr_circle (center 172.89 113.63) (end 173.39 113.63) (layer F.SilkS) (width 1))
+  (gr_circle (center 175.89 116.13) (end 176.39 116.13) (layer F.SilkS) (width 1))
+  (gr_text "CHARGE COMPLETE" (at 180.89 116.13) (layer F.SilkS)
     (effects (font (size 1.25 1.25) (thickness 0.2)) (justify left))
   )
-  (gr_circle (center 178.5 122.5) (end 179.5 122.5) (layer F.SilkS) (width 0.15))
-  (gr_circle (center 184.5 122.5) (end 185 122.5) (layer F.SilkS) (width 1))
-  (gr_text CHARGING (at 186.5 120) (layer F.SilkS)
+  (gr_circle (center 172.89 116.13) (end 173.89 116.13) (layer F.SilkS) (width 0.15))
+  (gr_circle (center 178.89 116.13) (end 179.39 116.13) (layer F.SilkS) (width 1))
+  (gr_text CHARGING (at 180.89 113.63) (layer F.SilkS)
     (effects (font (size 1.25 1.25) (thickness 0.2)) (justify left))
   )
-  (gr_circle (center 184.5 120) (end 185 120) (layer F.SilkS) (width 1))
-  (gr_circle (center 181.5 120) (end 182.5 120) (layer F.SilkS) (width 0.15))
-  (gr_text "STANDBY / FAULT" (at 186.5 117.5) (layer F.SilkS)
+  (gr_circle (center 178.89 113.63) (end 179.39 113.63) (layer F.SilkS) (width 1))
+  (gr_circle (center 175.89 113.63) (end 176.89 113.63) (layer F.SilkS) (width 0.15))
+  (gr_text "STANDBY / FAULT" (at 180.89 111.13) (layer F.SilkS)
     (effects (font (size 1.25 1.25) (thickness 0.2)) (justify left))
   )
-  (gr_circle (center 184.5 117.5) (end 185 117.5) (layer F.SilkS) (width 1))
-  (gr_circle (center 181.5 117.5) (end 182.5 117.5) (layer F.SilkS) (width 0.15))
-  (gr_circle (center 178.5 117.5) (end 179.5 117.5) (layer F.SilkS) (width 0.15))
-  (gr_text PG (at 184.5 113 90) (layer F.SilkS)
+  (gr_circle (center 178.89 111.13) (end 179.39 111.13) (layer F.SilkS) (width 1))
+  (gr_circle (center 175.89 111.13) (end 176.89 111.13) (layer F.SilkS) (width 0.15))
+  (gr_circle (center 172.89 111.13) (end 173.89 111.13) (layer F.SilkS) (width 0.15))
+  (gr_text "P - PWR GD" (at 178.89 106.63 90) (layer F.SilkS)
     (effects (font (size 1.25 1.25) (thickness 0.2)) (justify left))
   )
-  (gr_text STAT2 (at 181.5 113 90) (layer F.SilkS)
+  (gr_text "2 - STAT 2" (at 175.89 106.63 90) (layer F.SilkS)
     (effects (font (size 1.25 1.25) (thickness 0.2)) (justify left))
   )
-  (gr_text STAT1 (at 178.5 113 90) (layer F.SilkS)
+  (gr_text "1 - STAT 1" (at 172.89 106.63 90) (layer F.SilkS)
     (effects (font (size 1.25 1.25) (thickness 0.2)) (justify left))
   )
-  (gr_text SHUTDOWN (at 186.5 115) (layer F.SilkS)
+  (gr_text SHUTDOWN (at 180.89 108.63) (layer F.SilkS)
     (effects (font (size 1.25 1.25) (thickness 0.2)) (justify left))
   )
-  (gr_circle (center 184.5 115) (end 185.5 115) (layer F.SilkS) (width 0.15))
-  (gr_circle (center 181.5 115) (end 182.5 115) (layer F.SilkS) (width 0.15))
-  (gr_circle (center 178.5 115) (end 179.5 115) (layer F.SilkS) (width 0.15))
+  (gr_circle (center 178.89 108.63) (end 179.89 108.63) (layer F.SilkS) (width 0.15))
+  (gr_circle (center 175.89 108.63) (end 176.89 108.63) (layer F.SilkS) (width 0.15))
+  (gr_circle (center 172.89 108.63) (end 173.89 108.63) (layer F.SilkS) (width 0.15))
   (gr_text BATT- (at 137.49 141.888771 90) (layer F.SilkS)
     (effects (font (size 1.2065 1.2065) (thickness 0.1651)) (justify left bottom))
@@
   (segment (start 141.075 86.7) (end 141.075 87.425) (width 0.25) (layer Top) (net 5))
   (segment (start 139.454 85.079) (end 141.075 86.7) (width 0.25) (layer Top) (net 5))
+  (segment (start 157.8553 63.700001) (end 157.8553 64.2947) (width 0.25) (layer Top) (net 5))
+  (via (at 157.34 64.81) (size 0.8) (drill 0.4) (layers Top Bottom) (net 5))
+  (segment (start 157.8553 64.2947) (end 157.34 64.81) (width 0.25) (layer Top) (net 5))
   (segment (start 149.65 69.675) (end 149.65 69.1) (width 0.25) (layer Top) (net 6))
   (segment (start 150.025 70.05) (end 149.65 69.675) (width 0.25) (layer Top) (net 6))
@@
     (connect_pads (clearance 0.000001))
     (min_thickness 0.254)
-    (fill yes (arc_segments 32) (thermal_gap 0.508) (thermal_bridge_width 1) (smoothing fillet) (radius 0.25))
+    (fill yes (arc_segments 32) (thermal_gap 0.508) (thermal_bridge_width 0.5) (smoothing fillet) (radius 0.25))
     (polygon
       (pts
-        (xy 123.75 89.75) (xy 112.2 89.75) (xy 112.25 73.25) (xy 123.75 73.25)
+        (xy 123.75 89.75) (xy 112.2 89.75) (xy 112.25 79.5) (xy 123.75 79.5)
       )
     )
@@
     (connect_pads (clearance 0.000001))
     (min_thickness 0.254)
-    (fill yes (arc_segments 32) (thermal_gap 0.508) (thermal_bridge_width 1) (smoothing fillet) (radius 0.25))
+    (fill yes (arc_segments 32) (thermal_gap 0.508) (thermal_bridge_width 0.5) (smoothing fillet) (radius 0.25))
     (polygon
       (pts
-        (xy 139.75 89.75) (xy 124.25 89.75) (xy 124.25 73.25) (xy 139.75 73.25)
+        (xy 139.75 89.75) (xy 124.25 89.75) (xy 124.25 82.75) (xy 139.75 82.75)
       )
     )
@@
     (connect_pads (clearance 0.000001))
     (min_thickness 0.254)
-    (fill yes (arc_segments 32) (thermal_gap 0.508) (thermal_bridge_width 1) (smoothing fillet) (radius 0.25))
+    (fill yes (arc_segments 32) (thermal_gap 0.508) (thermal_bridge_width 1.5) (smoothing fillet) (radius 0.25))
     (polygon
       (pts
-        (xy 162.25 75) (xy 162.25 80.25) (xy 164.5 82.75) (xy 164.5 90.75) (xy 157.75 90.75)
-        (xy 157.75 83.5) (xy 156.5 82) (xy 147.75 82) (xy 147.53 73.78) (xy 161 73.75)
+        (xy 162.25 75) (xy 162.25 80.25) (xy 164.5 82.75) (xy 164.5 91.25) (xy 157.75 91.25)
+        (xy 157.75 83.5) (xy 157.75 80.25) (xy 147.5 80.25) (xy 147.53 73.78) (xy 161 73.75)
       )
     )
+  )
+  (zone (net 9) (net_name /BOOSTVIN) (layer Top) (hatch edge 0.508)
+    (connect_pads (clearance 0.000001))
+    (min_thickness 0.254)
+    (fill yes (arc_segments 32) (thermal_gap 0.508) (thermal_bridge_width 1.5) (smoothing fillet) (radius 0.25))
+    (polygon
+      (pts
+        (xy 139.75 83) (xy 124.25 83) (xy 124.25 73.25) (xy 139.75 73.25)
+      )
+    )
+  )
+  (zone (net 5) (net_name GND) (layer Top) (hatch edge 0.508)
+    (connect_pads (clearance 0.000001))
+    (min_thickness 0.254)
+    (fill yes (arc_segments 32) (thermal_gap 0.508) (thermal_bridge_width 1.5) (smoothing fillet) (radius 0.25))
+    (polygon
+      (pts
+        (xy 123.75 80) (xy 112.25 80) (xy 112.25 73.25) (xy 123.75 73.25)
+      )
+    )
+  )
+  (zone (net 14) (net_name /BOOSTVOUT) (layer Top) (hatch edge 0.508)
+    (connect_pads (clearance 0.000001))
+    (min_thickness 0.254)
+    (fill yes (arc_segments 32) (thermal_gap 0.508) (thermal_bridge_width 0.5) (smoothing fillet) (radius 0.25))
+    (polygon
+      (pts
+        (xy 158 81.75) (xy 147.5 81.75) (xy 147.5 79.75) (xy 158 79.75)
+      )
+    )

Commit message: Updates to Boost out on PCB
Parts:
- moved LED4 5.43 mm to (155.4, 87.9)
- moved R12 5.42 mm to (155.4, 82.5)
- moved C11 3.00 mm to (165.5, 76.9)
- moved W8 2.10 mm to (169.9, 86.9)
- moved D1 1.74 mm to (151.5, 75.8), turned to 90 degrees
Connections:
- D1 pad 2: (no net) -> /SW
- D1 pad 3: (no net) -> /SW
- D1 pad 5: /BOOSTVOUT -> (no net)
- LED4 pad 1: Net-(LED4-Pad1) -> GND
- LED4 pad 2: /BOOSTVOUT -> Net-(LED4-Pad2)
- R12 pad 1: Net-(LED4-Pad1) -> /BOOSTVOUT
- R12 pad 2: GND -> Net-(LED4-Pad2)
Routing:
- net /SW: track 0.00 -> 3.50 mm
- net Net-(LED4-Pad2): track 0.00 -> 3.42 mm
- net Net-(LED4-Pad1): track 3.42 -> 0.00 mm
- added copper zone on F.Cu, net /SW
Other:
- board text added: "POWER OUT"
- board text removed: "POWER"

Commit message: PCB Updates
Parts:
- moved J1 2.00 mm to (133.5, 65.4)
- moved W5 1.79 mm to (168.5, 63.2)
- moved W7 1.06 mm to (161.8, 85.9)
- moved W8 1.00 mm to (169.9, 85.9)
Routing:
- net GND: track 59.7 -> 63.0 mm, vias 12 -> 20
- net Net-(LED3-Pad1): track 5.52 -> 4.83 mm
Other:
- board size 78 x 22.7 mm -> 71 x 31 mm
- board text added: "5V OUT"
- board text removed: "5Vout"
- board text removed: "BATT-"
- board text removed: "CHRG"
- board text removed: "GND"
- board text removed: "OFF"
- board text removed: "POWER OUT"
- board text removed: "VOUT"
- board text removed: "boost"
- board text removed: "charger"
- board text removed: "protection"

Commit message: PCB Update
Parts:
- moved W3 11.0 mm to (105.8, 74.7)
- moved W4 5.92 mm to (105.9, 64.8)
- moved C2 2.21 mm to (145.3, 62.8)
- moved C8 2.21 mm to (168.8, 67.9)
- moved J1 2.21 mm to (135.7, 65.4)
- moved LED2 2.21 mm to (151.9, 62.8)
- moved LED3 2.21 mm to (148.6, 62.8)
- moved R3 2.21 mm to (151.9, 67.9)
- moved R4 2.21 mm to (148.6, 67.9)
- moved R5 2.21 mm to (145.3, 67.9)
- moved R6 2.21 mm to (165.4, 67.9)
- moved R8 2.21 mm to (155.2, 67.9)
- moved TH1 2.21 mm to (158.7, 67.9)
- moved U3 2.21 mm to (162.1, 62.7)
- moved W1 2.21 mm to (125.8, 63.7)
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Connections:
- net Net-(R2-Pad1) renamed /PVM
Routing:
- net /ST1: track 0.00 -> 17.2 mm
- net /ST2: track 0.00 -> 14.2 mm
- net /BATT-: track 17.3 -> 6.15 mm
- net /SW: track 3.50 -> 0.01 mm
- net /PVDD: track 8.09 -> 6.62 mm
Other:
- board text added: "BATT-"

Commit message: Update Li-ion 5A Boost 1A Charge Protect.kicad_pcb
Connections:
- SW1 pad 1: /BATT+ -> /BOOSTVIN
- SW1 pad 2: /BOOSTVIN -> /BATT+
Changed lines of the file:
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@@
     )
     (pad 2 thru_hole circle (at 0 -1.09 270) (size 2.75 2.75) (drill 1.75) (layers *.Cu *.Mask)
+      (net 2 /BATT+))
+    (pad 1 thru_hole circle (at -4.6 -1.09 270) (size 2.75 2.75) (drill 1.75) (layers *.Cu *.Mask)
       (net 9 /BOOSTVIN))
-    (pad 1 thru_hole circle (at -4.6 -1.09 270) (size 2.75 2.75) (drill 1.75) (layers *.Cu *.Mask)
-      (net 2 /BATT+))
     (model GF-123-0054.stp
       (at (xyz 0 0 0))
