File: Li-ion 5A Boost 1A Charge Protect/Li-ion 5A Boost 1A Charge Protect.kicad_pcb (KiCad board)
At the start: 2 copper layers, 71 x 31 mm, 44 parts, among them J1 USB_C_FEMALE, SW1 SW_SPST, U1 AP9101CK6, U2 ECH8695R-TL-W, U3 MCP73833T, U4 PAM2423AECADJR

Commit message: PCB Update
Working layout with repositioned charge and protect sections.  Still work to be done on labeling, 3D models, and copper pours on bottom.
Parts:
- removed LED1, LED2: GREEN, Li-ion 5A Boost 1A Charge Protect:LED_0805_2012Metric_HandSolder
- removed LED3: RED, Li-ion 5A Boost 1A Charge Protect:LED_0805_2012Metric_HandSolder
- added LD1: GREEN, Li-ion 5A Boost 1A Charge Protect:LED_0805_2012Metric_HandSolder, F.Cu at (162.9, 69.1)
- added LD2: GREEN, Li-ion 5A Boost 1A Charge Protect:LED_0805_2012Metric_HandSolder, F.Cu at (162.9, 62.2)
- added LD3: RED, Li-ion 5A Boost 1A Charge Protect:LED_0805_2012Metric_HandSolder, F.Cu at (162.9, 65.7)
- moved W2 49.9 mm to (170.2, 68.8), turned to 270 degrees
- moved W1 44.4 mm to (170.2, 62.9), turned to 90 degrees
- moved W6 34.7 mm to (119.5, 56.0), turned to 180 degrees
- moved W4 34.6 mm to (140.3, 67.1)
- moved J1 31.9 mm to (166.4, 57.0)
- moved W5 30.6 mm to (140.3, 55.9), turned to 0 degrees
- moved SW1 29.0 mm to (136.7, 61.5), turned to 90 degrees
- moved W3 28.3 mm to (127.0, 56.0), turned to 0 degrees
- moved R1 26.7 mm to (126.5, 63.0), turned to 0 degrees
- moved C1 25.8 mm to (121.0, 63.0)
- moved C8 22.4 mm to (148.3, 58.8), turned to 0 degrees
- moved U2 20.8 mm to (119.1, 67.2), turned to 0 degrees
- moved R2 20.7 mm to (128.3, 67.2)
- moved R6 19.5 mm to (145.9, 67.4), turned to 0 degrees
- moved U1 18.8 mm to (124.2, 67.2), turned to 90 degrees
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- renumbered LED4 to LD4
Routing:
- net /PROG: track 3.57 -> 16.3 mm, vias 0 -> 2
- net GND: track 63.0 -> 53.2 mm, vias 20 -> 25
- net /BATT-: track 6.15 -> 0.00 mm
- net /THRMIC: track 5.87 -> 11.8 mm, vias 0 -> 2
- net /ST2: track 14.2 -> 10.9 mm, vias 0 -> 2
- net /ST1: track 17.2 -> 14.0 mm, vias 0 -> 2
- net Net-(LD1-Pad1): track 5.84 -> 3.42 mm
- net Net-(LD2-Pad1): track 5.72 -> 3.37 mm
- net /THRM: track 8.38 -> 6.42 mm
- net /PVM: track 4.14 -> 5.92 mm
- net Net-(LD3-Pad1): track 4.83 -> 3.34 mm
- net /PG: track 19.5 -> 18.6 mm, vias 0 -> 2
- net /BOOSTVOUT: vias 0 -> 3
- net /BOOSTVIN: vias 0 -> 2
- added copper zone on B.Cu, net /BATT+
- added copper zone on B.Cu, net /BATT-
- added copper zone on B.Cu, net /BOOSTVIN
- added copper zone on B.Cu, net /BOOSTVOUT
- added copper zone on B.Cu, net /SW
Other:
- board size 71 x 31 mm -> 58 x 39 mm
- board text added: "1-STAT 1"
- board text added: "2-STAT 2"
- board text added: "5V IN"
- board text added: "B+"
- board text added: "B-"
- board text added: "BOOST"
- board text added: "CHARGE"
- board text added: "P-POWER GOOD"
- board text added: "PROTECT"
- board text added: "SWI"
- board text added: "SWITCH"
- board text added: "SWO"
- board text removed: "1 - STAT 1"
- board text removed: "10K=130mA 5K=250mA 4K=300mA 3K=400mA 2K=580mA 1K66=690mA 1K5=780mA 1K33=900mA 1K2=1000mA"
- board text removed: "2 - STAT 2"
- board text removed: "BATT+"
- board text removed: "BATT-"
- board text removed: "CHRG RATE"
- board text removed: "P - PWR GD"
- board text removed: "PG"
- board text removed: "ST1"
- board text removed: "ST2"

Commit message: PCB Before Solder Footprint Switch
Before switching wire solder points to foot prints with through holes.
Connections:
- D1 pad 5: (no net) -> /BOOSTVOUT
Routing:
- net GND: track 53.2 -> 59.0 mm, vias 25 -> 22
- net /VUSB: vias 0 -> 2
- net /SW: vias 0 -> 3
- net /BATT-: vias 0 -> 2
- added copper zone on B.Cu, net /VUSB
Changed lines of the file:
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@@
     (34 B.Paste user)
     (35 F.Paste user)
-    (36 B.SilkS user)
+    (36 B.SilkS user hide)
     (37 F.SilkS user)
     (38 B.Mask user)
@@
   )
   (setup
-    (last_trace_width 0.25)
+    (last_trace_width 0.8)
     (user_trace_width 0.25)
     (user_trace_width 0.5)
@@
     (trace_clearance 0.1524)
     (zone_clearance 0.000001)
-    (zone_45_only no)
+    (zone_45_only yes)
     (trace_min 0.2)
     (via_size 0.8)
@@
     (pad 5C smd rect (at 1.905 4.2925 90) (size 0.75 0.475) (layers Top F.Paste F.Mask)
       (net 14 /BOOSTVOUT))
-    (pad 5 smd rect (at 0 2.0275 90) (size 4 3.5) (layers Top F.Paste F.Mask))
+    (pad 5 smd rect (at 0 2.0275 90) (size 4 3.5) (layers Top F.Paste F.Mask)
+      (net 14 /BOOSTVOUT))
     (pad 4 smd rect (at 1.905 -1.465 90) (size 0.75 1) (layers Top F.Paste F.Mask))
     (pad 3 smd rect (at 0.635 -1.465 90) (size 0.75 1) (layers Top F.Paste F.Mask)
@@
     (effects (font (size 3.6195 3.6195) (thickness 0.3048)) (justify left bottom))
   )
+  (via (at 144.5 77.75) (size 1) (drill 0.6) (layers Top Bottom) (net 12))
+  (via (at 117.5 60.5) (size 1) (drill 0.6) (layers Top Bottom) (net 1))
+  (via (at 121.5 60.5) (size 1) (drill 0.6) (layers Top Bottom) (net 1))
+  (via (at 153.5 75.75) (size 1) (drill 0.6) (layers Top Bottom) (net 14))
   (segment (start 149.1453 55.92) (end 149.14 55.539999) (width 1) (layer Top) (net 2))
   (segment (start 153.2347 55.950001) (end 153.2347 55.56) (width 1) (layer Top) (net 3))
+  (via (at 166.5 55.25) (size 1) (drill 0.6) (layers Top Bottom) (net 3))
+  (via (at 160.25 60.25) (size 1) (drill 0.6) (layers Top Bottom) (net 3))
   (via (at 144.89 65.64) (size 0.8) (drill 0.4) (layers Top Bottom) (net 4))
   (segment (start 144.89 65.64) (end 144.89 66.205685) (width 0.25) (layer Top) (net 4))
@@
   (via (at 169.64 59.51) (size 0.8) (drill 0.4) (layers Top Bottom) (net 5))
   (segment (start 169.64 58.045) (end 169.64 59.51) (width 0.5) (layer Top) (net 5))
-  (segment (start 170.057401 55.897401) (end 170.02 55.86) (width 0.5) (layer Top) (net 5))
-  (via (at 170.02 55.86) (size 0.8) (drill 0.4) (layers Top Bottom) (net 5))
-  (segment (start 169.64 58.045) (end 170.057401 57.627599) (width 0.5) (layer Top) (net 5))
-  (segment (start 170.057401 57.627599) (end 170.057401 55.897401) (width 0.5) (layer Top) (net 5))
-  (via (at 162.86 55.85) (size 0.8) (drill 0.4) (layers Top Bottom) (net 5))
-  (segment (start 162.822599 55.887401) (end 162.86 55.85) (width 0.5) (layer Top) (net 5))
-  (segment (start 163.24 58.045) (end 162.822599 57.627599) (width 0.5) (layer Top) (net 5))
-  (segment (start 162.822599 57.627599) (end 162.822599 55.887401) (width 0.5) (layer Top) (net 5))
   (via (at 131.925 88) (size 0.8) (drill 0.4) (layers Top Bottom) (net 5))
   (segment (start 130.345 88.009) (end 131.916 88.009) (width 0.25) (layer Top) (net 5))
@@
   (segment (start 139.454 85.079) (end 141.075 86.7) (width 0.25) (layer Top) (net 5))
   (via (at 167 73) (size 1) (drill 0.6) (layers Top Bottom) (net 5))
-  (via (at 173 73) (size 1) (drill 0.6) (layers Top Bottom) (net 5))
-  (via (at 173 81) (size 1) (drill 0.6) (layers Top Bottom) (net 5))
+  (via (at 172.5 73) (size 1) (drill 0.6) (layers Top Bottom) (net 5))
+  (via (at 172.5 81) (size 1) (drill 0.6) (layers Top Bottom) (net 5))
   (via (at 167 81) (size 1) (drill 0.6) (layers Top Bottom) (net 5))
-  (via (at 172.75 87.75) (size 1) (drill 0.6) (layers Top Bottom) (net 5))
   (via (at 167 87.75) (size 1) (drill 0.6) (layers Top Bottom) (net 5))
   (via (at 155.150002 53.18) (size 0.8) (drill 0.4) (layers Top Bottom) (net 5))
@@
   (segment (start 117.75 67.575) (end 118.425 67.575) (width 0.25) (layer Top) (net 5))
   (segment (start 118.425 67.575) (end 119.1 68.25) (width 0.25) (layer Top) (net 5))
+  (segment (start 169.64 59.51) (end 169.64 65.06) (width 0.8) (layer Bottom) (net 5))
+  (segment (start 163.24 59.51) (end 163.24 64.52) (width 0.8) (layer Bottom) (net 5))
   (via (at 151.5 55.67) (size 0.8) (drill 0.4) (layers Top Bottom) (net 6))
   (segment (start 151.5 55.532701) (end 151.5 55.67) (width 0.25) (layer Top) (net 6))
@@
   (segment (start 143.575 86.349) (end 146.024 86.349) (width 0.25) (layer Top) (net 11))
   (segment (start 146.024 86.349) (end 146.575 86.9) (width 0.25) (layer Top) (net 11))
+  (via (at 142 73.25) (size 1) (drill 0.6) (layers Top Bottom) (net 12))
+  (via (at 147.25 73.25) (size 1) (drill 0.6) (layers Top Bottom) (net 12))
   (segment (start 152.14375 84.059) (end 152.15 84.06525) (width 0.25) (layer Top) (net 13))
   (segment (start 152.14375 83.484) (end 152.14375 84.059) (width 0.25) (layer Top) (net 13))
@@
   (segment (start 152.14375 86.859) (end 151.016 86.859) (width 0.25) (layer Top) (net 13))
   (segment (start 151.016 86.859) (end 150 87.875) (width 0.25) (layer Top) (net 13))
-  (via (at 161.25 89.75) (size 1) (drill 0.6) (layers Top Bottom) (net 14))
-  (via (at 161.25 81.5) (size 1) (drill 0.6) (layers Top Bottom) (net 14))
-  (via (at 161.25 74) (size 1) (drill 0.6) (layers Top Bottom) (net 14))
+  (via (at 163.25 79.5) (size 1) (drill 0.6) (layers Top Bottom) (net 14))
+  (via (at 163.25 73) (size 1) (drill 0.6) (layers Top Bottom) (net 14))
   (segment (start 147.51 63.89) (end 147.52 63.9) (width 0.25) (layer Top) (net 15))
   (segment (start 146.935 63.89) (end 147.51 63.89) (width 0.25) (layer Top) (net 15))
@@
     )
   )
-  (zone (net 5) (net_name GND) (layer Bottom) (hatch edge 0.508)
+  (zone (net 3) (net_name /VUSB) (layer Bottom) (hatch edge 0.508)
     (connect_pads (clearance 0.000001))
     (min_thickness 0.254)
@@
     (polygon
       (pts
-        (xy 175 63.5) (xy 143.75 63.5) (xy 143.75 51) (xy 175 51)
+        (xy 175 63.5) (xy 157.5 63.5) (xy 157.5 51) (xy 175 51)
       )
     )
@@
       (pts
         (xy 165.5 72.25) (xy 165.5 81.5) (xy 165.5 83) (xy 165.5 91.25) (xy 157.75 91.25)
-        (xy 157.75 83.5) (xy 157.75 80.25) (xy 151.8 80.2) (xy 151.8 71.25) (xy 165.5 71.25)
+        (xy 157.75 83.5) (xy 157.75 80.25) (xy 151.75 80.2) (xy 151.75 71.25) (xy 165.5 71.25)
       )
     )
@@
     )
   )
-  (zone (net 12) (net_name /SW) (layer Top) (hatch edge 0.508)
-    (connect_pads (clearance 0.000001))
-    (min_thickness 0.254)
-    (fill yes (arc_segments 32) (thermal_gap 0.5) (thermal_bridge_width 0.5) (smoothing fillet) (radius 0.25))
-    (polygon
-      (pts
-        (xy 148.25 91.25) (xy 140 91.25) (xy 140 80.5) (xy 148.25 80.5)
-      )
-    )
-  )
   (zone (net 3) (net_name /VUSB) (layer Top) (hatch edge 0.508)
     (connect_pads (clearance 0.000001))
@@
     )
   )
+  (zone (net 14) (net_name /BOOSTVOUT) (layer Bottom) (hatch edge 0.508)
+    (connect_pads (clearance 0.000001))
+    (min_thickness 0.254)
+    (fill yes (arc_segments 32) (thermal_gap 0.5) (thermal_bridge_width 1.5) (smoothing fillet) (radius 0.25))
+    (polygon
+      (pts
+        (xy 165.5 80.5) (xy 151.75 80.5) (xy 151.75 71.25) (xy 165.5 71.25)
+      )
+    )
+  )
+  (zone (net 12) (net_name /SW) (layer Top) (hatch edge 0.508)
+    (connect_pads (clearance 0.000001))
+    (min_thickness 0.254)
+    (fill yes (arc_segments 32) (thermal_gap 0.5) (thermal_bridge_width 0.5) (smoothing fillet) (radius 0.25))
+    (polygon
+      (pts
+        (xy 148.25 91.25) (xy 140 91.25) (xy 140 80.5) (xy 148.25 80.5)
+      )
+    )
+  )
   (zone (net 12) (net_name /SW) (layer Bottom) (hatch edge 0.508)
     (connect_pads (clearance 0.000001))
     (min_thickness 0.254)
-    (fill yes (arc_segments 32) (thermal_gap 0.5) (thermal_bridge_width 1.5) (smoothing fillet) (radius 0.25))
-    (polygon
-      (pts
-        (xy 151 80.5) (xy 140 80.5) (xy 140 71.25) (xy 151 71.25)
-      )
-    )
-  )
-  (zone (net 14) (net_name /BOOSTVOUT) (layer Bottom) (hatch edge 0.508)
-    (connect_pads (clearance 0.000001))
-    (min_thickness 0.254)
-    (fill yes (arc_segments 32) (thermal_gap 0.5) (thermal_bridge_width 1.5) (smoothing fillet) (radius 0.25))
-    (polygon
-      (pts
-        (xy 165.5 92.25) (xy 158 92.25) (xy 158 71.25) (xy 165.5 71.25)
-      )
-    )
+    (fill yes (arc_segments 32) (thermal_gap 0.5) (thermal_bridge_width 0.5) (smoothing fillet) (radius 0.25))
+    (polygon
+      (pts
+        (xy 151.5 80.5) (xy 140 80.5) (xy 140 71.25) (xy 151.5 71.25)
+      )
+    )
+  )
+  (zone (net 5) (net_name GND) (layer Bottom) (hatch edge 0.508)
+    (connect_pads (clearance 0.000001))
+    (min_thickness 0.254)
+    (fill yes (arc_segments 32) (thermal_gap 0.5) (thermal_bridge_width 0.5) (smoothing fillet) (radius 0.25))
+    (polygon
+      (pts
+        (xy 175 91.75) (xy 123.5 91.75) (xy 123.5 80.75) (xy 175 80.75)
+      )
+    )
+  )
+  (zone (net 5) (net_name GND) (layer Bottom) (hatch edge 0.508)
+    (connect_pads (clearance 0.000001))
+    (min_thickness 0.254)
+    (fill yes (arc_segments 32) (thermal_gap 0.5) (thermal_bridge_width 0.5) (smoothing fillet) (radius 0.25))
+    (polygon
+      (pts
+        (xy 175 81.75) (xy 165.75 81.75) (xy 165.75 71) (xy 143.75 71) (xy 143.75 63.75)
+        (xy 175 63.75)
+      )
+    )
+  )
+  (zone (net 5) (net_name GND) (layer Bottom) (hatch edge 0.508)
+    (connect_pads (clearance 0.000001))
+    (min_thickness 0.254)
+    (fill yes (arc_segments 32) (thermal_gap 0.5) (thermal_bridge_width 0.5) (smoothing fillet) (radius 0.25))
+    (polygon
+      (pts
+        (xy 157.25 67.75) (xy 143.75 67.75) (xy 143.75 51) (xy 157.25 51)
+      )
+    )

Commit message: PCB Update
Parts:
- W1, W2, W3, W4, W5, W6, W7, W8: footprint Li-ion 5A Boost 1A Charge Protect:Pad_3.0-5.0 -> Li-ion 5A Boost 1A Charge Protect:Pad_3.0-5.0_w_TH
- moved C1 3.22 mm to (124.2, 62.6)
- moved R1 1.84 mm to (128.3, 62.6), turned to 90 degrees
- moved W7 1.20 mm to (161.8, 87.1)
- moved W8 1.20 mm to (169.9, 87.1)
- moved C11 0.75 mm to (165.5, 77.6)
- moved C3 0.75 mm to (124.0, 77.6)
- moved R2 0.45 mm to (128.3, 67.7)
- moved U1 0.45 mm to (124.2, 67.7)
- moved U2 0.45 mm to (119.1, 67.7)
Routing:
- net GND: track 59.0 -> 64.2 mm, vias 22 -> 21
- net /PVDD: track 6.96 -> 7.89 mm
- net /SW: vias 3 -> 4
- net /BOOSTVOUT: vias 3 -> 4
- net /BOOSTVIN: vias 2 -> 4

Commit message: PCB Update, back silk screen
Parts:
- moved R6 1.09 mm to (147.0, 67.4)
- moved R7 1.09 mm to (147.0, 63.9)
- moved R8 1.09 mm to (152.2, 67.4)
- moved TH1 1.09 mm to (152.2, 63.9)
Routing:
- net /THRMIC: track 11.8 -> 11.2 mm
Other:
- board text added: "+ BATT -"
- board text added: "- 5V OUT +"
- board text added: "5V"
- board text added: "COMPLETE"
- board text added: "FAULT"
- board text added: "IN"
- board text added: "Li-Ion 5V 5A Output 1A Charge"
- board text added: "OFF"
- board text added: "OUT"
- board text added: "STANDBY"
- board text added: "TEST"
- board text added: "V1.0.0"
- board text removed: "1-STAT 1"
- board text removed: "2-STAT 2"
- board text removed: "5V OUT"
- board text removed: "CHARGE COMPLETE"
- board text removed: "P-POWER GOOD"
- board text removed: "STANDBY / FAULT"
- board text removed: "SYSTEM TEST"

Commit message: PCB and 3D model updates
Other:
- board text removed: "+ BATT -"

Commit message: PCB Cleanup and corrections
Parts:
- removed W3, W6: 2.5x5.0, Li-ion 5A Boost 1A Charge Protect:Pad_3.0-5.0_w_TH
- added B+: 2.5x5.0, Li-ion 5A Boost 1A Charge Protect:Pad_3.0-5.0_w_TH, F.Cu at (127.0, 56.0)
- added B-: 2.5x5.0, Li-ion 5A Boost 1A Charge Protect:Pad_3.0-5.0_w_TH, F.Cu at (119.5, 56.0)
- renumbered W7 to +, W1 to +, W8 to -, W2 to -, W5 to SWI, W4 to SWO
Routing:
- net /VUSB: track 0.39 -> 3.09 mm
- net GND: track 64.2 -> 65.9 mm
- net /SW: vias 4 -> 3
- net /BOOSTVIN: vias 4 -> 3
Other:
- board text added: "+ 5V OUT -"
- board text removed: "- 5V OUT +"
- board text removed: "SWI"
- board text removed: "SWO"
