File: Li-ion 5A Boost 1A Charge Protect/Li-ion 5A Boost 1A Charge Protect.kicad_pcb (KiCad board)
At the start: 2 copper layers, 58 x 39 mm, 44 parts, among them J1 USB_C_FEMALE, SW1 SW_SPST, U1 AP9101CK6, U2 ECH8695R-TL-W, U3 MCP73833T, U4 PAM2423AECADJR

Commit message: PCB Tweaks
Routing:
- net GND: track 65.9 -> 62.8 mm
- net /VUSB: track 3.09 -> 3.66 mm
Changed lines of the file:
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@@
     (thickness 1.6)
     (drawings 63)
-    (tracks 199)
+    (tracks 197)
     (zones 0)
     (modules 44)
@@
   (page A)
   (layers
-    (0 Top signal hide)
+    (0 Top signal)
     (31 Bottom signal)
     (32 B.Adhes user hide)
@@
     (34 B.Paste user)
     (35 F.Paste user)
-    (36 B.SilkS user)
+    (36 B.SilkS user hide)
     (37 F.SilkS user hide)
     (38 B.Mask user)
@@
     (47 F.CrtYd user)
     (48 B.Fab user)
-    (49 F.Fab user)
+    (49 F.Fab user hide)
   )
   (setup
-    (last_trace_width 0.25)
+    (last_trace_width 0.5)
     (user_trace_width 0.25)
     (user_trace_width 0.5)
     (user_trace_width 0.8)
     (user_trace_width 1)
-    (user_trace_width 1.6)
+    (user_trace_width 1.5)
     (trace_clearance 0.1524)
     (zone_clearance 0.000001)
@@
     (solder_mask_min_width 0.25)
     (aux_axis_origin 0 0)
-    (visible_elements 7FFE7FFF)
+    (visible_elements 7FFFFFFF)
     (pcbplotparams
       (layerselection 0x010fc_ffffffff)
@@
   (via (at 119.5 60.92) (size 1) (drill 0.6) (layers Top Bottom) (net 1))
   (via (at 119.5 64.44) (size 1) (drill 0.6) (layers Top Bottom) (net 1))
-  (segment (start 149.1453 55.92) (end 149.14 55.539999) (width 1) (layer Top) (net 2))
-  (segment (start 153.2347 55.950001) (end 153.2347 55.56) (width 1) (layer Top) (net 3))
+  (segment (start 149.1553 56.190001) (end 149.15 55.81) (width 1.5) (layer Top) (net 2))
   (via (at 165 54) (size 1) (drill 0.6) (layers Top Bottom) (net 3))
   (via (at 159.99 60.42) (size 1) (drill 0.6) (layers Top Bottom) (net 3))
@@
   (segment (start 168.84 58.045) (end 168.84 57.74) (width 0.25) (layer Top) (net 3))
   (segment (start 168.84 57.74) (end 168.727599 57.627599) (width 0.25) (layer Top) (net 3))
+  (segment (start 153.2347 56.7453) (end 153.2347 55.794999) (width 1.5) (layer Top) (net 3))
+  (segment (start 153.23 56.75) (end 153.2347 56.7453) (width 1.5) (layer Top) (net 3))
   (via (at 145.98 65.61) (size 0.8) (drill 0.4) (layers Top Bottom) (net 4))
   (segment (start 145.98 67.42) (end 146 67.44) (width 0.25) (layer Top) (net 4))
   (segment (start 145.98 65.61) (end 145.98 67.42) (width 0.25) (layer Top) (net 4))
-  (segment (start 147.671997 53.689999) (end 146.730998 54.630998) (width 0.25) (layer Top) (net 4))
-  (segment (start 145.98 55.381996) (end 146.730998 54.630998) (width 0.25) (layer Bottom) (net 4))
-  (segment (start 149.1453 53.689999) (end 147.671997 53.689999) (width 0.25) (layer Top) (net 4))
-  (via (at 146.730998 54.630998) (size 0.8) (drill 0.4) (layers Top Bottom) (net 4))
-  (segment (start 145.98 65.61) (end 145.98 55.381996) (width 0.25) (layer Bottom) (net 4))
+  (segment (start 145.98 65.61) (end 145.98 54.816346) (width 0.25) (layer Bottom) (net 4))
+  (segment (start 147.106347 53.689999) (end 146.673897 54.122449) (width 0.25) (layer Top) (net 4))
+  (segment (start 149.1453 53.689999) (end 147.106347 53.689999) (width 0.25) (layer Top) (net 4))
+  (via (at 146.673897 54.122449) (size 0.8) (drill 0.4) (layers Top Bottom) (net 4))
+  (segment (start 145.98 54.816346) (end 146.673897 54.122449) (width 0.25) (layer Bottom) (net 4))
   (via (at 131.925 88) (size 0.8) (drill 0.4) (layers Top Bottom) (net 5))
   (segment (start 130.345 88.009) (end 131.916 88.009) (width 0.25) (layer Top) (net 5))
@@
   (via (at 118 82.5) (size 1) (drill 0.6) (layers Top Bottom) (net 5))
   (via (at 122 82.5) (size 1) (drill 0.6) (layers Top Bottom) (net 5))
-  (via (at 151.21 57.400002) (size 1) (drill 0.6) (layers Top Bottom) (net 5))
-  (via (at 151.209998 60.31) (size 1) (drill 0.6) (layers Top Bottom) (net 5))
-  (segment (start 149.81 60.31) (end 150.502892 60.31) (width 0.5) (layer Top) (net 5))
-  (segment (start 150.502892 60.31) (end 151.209998 60.31) (width 0.5) (layer Top) (net 5))
-  (segment (start 149.325 58.84) (end 149.325 59.825) (width 0.5) (layer Top) (net 5))
-  (segment (start 149.325 59.825) (end 149.81 60.31) (width 0.5) (layer Top) (net 5))
-  (segment (start 152.59 60.31) (end 151.209998 60.31) (width 0.5) (layer Top) (net 5))
-  (segment (start 153.065 58.84) (end 153.065 59.835) (width 0.5) (layer Top) (net 5))
-  (segment (start 153.065 59.835) (end 152.59 60.31) (width 0.5) (layer Top) (net 5))
-  (segment (start 152.590002 57.400002) (end 151.21 57.400002) (width 0.5) (layer Top) (net 5))
-  (segment (start 153.065 58.84) (end 153.065 57.875) (width 0.5) (layer Top) (net 5))
-  (segment (start 153.065 57.875) (end 152.590002 57.400002) (width 0.5) (layer Top) (net 5))
-  (segment (start 149.829998 57.400002) (end 151.21 57.400002) (width 0.5) (layer Top) (net 5))
-  (segment (start 149.325 58.84) (end 149.325 57.905) (width 0.5) (layer Top) (net 5))
-  (segment (start 149.325 57.905) (end 149.829998 57.400002) (width 0.5) (layer Top) (net 5))
   (segment (start 117.75 68.025) (end 118.425 68.025) (width 0.25) (layer Top) (net 5))
   (segment (start 118.425 68.025) (end 119.1 68.7) (width 0.25) (layer Top) (net 5))
@@
   (segment (start 169.514315 55.979999) (end 170.08 55.979999) (width 0.8) (layer Bottom) (net 5))
   (segment (start 166.770001 55.979999) (end 169.514315 55.979999) (width 0.8) (layer Bottom) (net 5))
+  (via (at 151.240002 57.88) (size 0.8) (drill 0.4) (layers Top Bottom) (net 5))
+  (via (at 151.21 59.78) (size 0.8) (drill 0.4) (layers Top Bottom) (net 5))
+  (segment (start 149.325 58.84) (end 149.33 58.84) (width 0.5) (layer Top) (net 5))
+  (segment (start 150.29 57.88) (end 151.240002 57.88) (width 0.5) (layer Top) (net 5))
+  (segment (start 149.33 58.84) (end 150.29 57.88) (width 0.5) (layer Top) (net 5))
+  (segment (start 152.11 57.88) (end 151.240002 57.88) (width 0.5) (layer Top) (net 5))
+  (segment (start 153.065 58.84) (end 153.065 58.835) (width 0.5) (layer Top) (net 5))
+  (segment (start 153.065 58.835) (end 152.11 57.88) (width 0.5) (layer Top) (net 5))
+  (segment (start 152.1 59.78) (end 151.21 59.78) (width 0.5) (layer Top) (net 5))
+  (segment (start 153.065 58.84) (end 153.04 58.84) (width 0.5) (layer Top) (net 5))
+  (segment (start 153.04 58.84) (end 152.1 59.78) (width 0.5) (layer Top) (net 5))
+  (segment (start 150.3 59.78) (end 151.21 59.78) (width 0.5) (layer Top) (net 5))
+  (segment (start 150.12 59.6) (end 150.3 59.78) (width 0.5) (layer Top) (net 5))
+  (segment (start 149.325 58.84) (end 150.085 59.6) (width 0.5) (layer Top) (net 5))
+  (segment (start 150.085 59.6) (end 150.12 59.6) (width 0.5) (layer Top) (net 5))
   (via (at 151.5 55.67) (size 0.8) (drill 0.4) (layers Top Bottom) (net 6))
   (segment (start 151.5 55.532701) (end 151.5 55.67) (width 0.25) (layer Top) (net 6))
@@
   (segment (start 151.15 63.87) (end 151.15 67.42) (width 0.25) (layer Top) (net 15))
   (via (at 146.81 61.39) (size 0.8) (drill 0.4) (layers Top Bottom) (net 16))
-  (via (at 146.789998 56.46) (size 0.8) (drill 0.4) (layers Top Bottom) (net 16))
-  (segment (start 147.63 54.69) (end 146.789998 55.530002) (width 0.25) (layer Top) (net 16))
-  (segment (start 149.1453 54.69) (end 147.63 54.69) (width 0.25) (layer Top) (net 16))
-  (segment (start 146.789998 55.530002) (end 146.789998 56.46) (width 0.25) (layer Top) (net 16))
   (segment (start 146.81 62.96) (end 146.81 61.39) (width 0.25) (layer Top) (net 16))
   (segment (start 146.040001 63.729999) (end 146.81 62.96) (width 0.25) (layer Top) (net 16))
-  (segment (start 146.789998 57.025685) (end 146.789998 56.46) (width 0.25) (layer Bottom) (net 16))
-  (segment (start 146.81 61.39) (end 146.789998 61.369998) (width 0.25) (layer Bottom) (net 16))
-  (segment (start 146.789998 61.369998) (end 146.789998 57.025685) (width 0.25) (layer Bottom) (net 16))
+  (segment (start 149.1453 54.69) (end 147.19 54.69) (width 0.25) (layer Top) (net 16))
+  (segment (start 147.19 54.69) (end 146.81 55.07) (width 0.25) (layer Top) (net 16))
+  (segment (start 146.81 61.39) (end 146.81 55.07) (width 0.25) (layer Bottom) (net 16))
+  (via (at 146.81 55.07) (size 0.8) (drill 0.4) (layers Top Bottom) (net 16))
   (segment (start 125.125 85.4) (end 123.975 85.4) (width 0.25) (layer Top) (net 17))
   (segment (start 127.078 85.959) (end 125.684 85.959) (width 0.25) (layer Top) (net 17))
@@
     )
   )
-  (zone (net 2) (net_name /BATT+) (layer Top) (hatch edge 0.508)
-    (connect_pads (clearance 0.000001))
-    (min_thickness 0.254)
-    (fill yes (arc_segments 32) (thermal_gap 0.5) (thermal_bridge_width 1.5) (smoothing fillet) (radius 0.25))
-    (polygon
-      (pts
-        (xy 124 51.5) (xy 151.120864 51.5) (xy 151.120864 63.5) (xy 124 63.5)
-      )
-    )
-  )
-  (zone (net 3) (net_name /VUSB) (layer Top) (hatch edge 0.508)
-    (connect_pads (clearance 0.000001))
-    (min_thickness 0.254)
-    (fill yes (arc_segments 32) (thermal_gap 0.5) (thermal_bridge_width 0.5) (smoothing fillet) (radius 0.25))
-    (polygon
-      (pts
-        (xy 174.5 53) (xy 174.5 60.5) (xy 165.5 60.5) (xy 165.5 71) (xy 151.5 71)
-        (xy 151.5 51.5) (xy 174.5 51.5)
-      )
-    )
-  )
   (zone (net 3) (net_name /VUSB) (layer Bottom) (hatch edge 0.508)
     (connect_pads (clearance 0.000001))
@@
       )
     )
+  )
+  (zone (net 2) (net_name /BATT+) (layer Top) (hatch edge 0.508)
+    (connect_pads (clearance 0.000001))
+    (min_thickness 0.254)
+    (fill yes (arc_segments 32) (thermal_gap 0.5) (thermal_bridge_width 1.5) (smoothing fillet) (radius 0.25))
+    (polygon
+      (pts
+        (xy 124 51.5) (xy 151.120864 51.5) (xy 151.120864 63.5) (xy 124 63.5)
+      )
+    )
+  )
+  (zone (net 3) (net_name /VUSB) (layer Top) (hatch edge 0.508)
+    (connect_pads (clearance 0.000001))
+    (min_thickness 0.254)
+    (fill yes (arc_segments 32) (thermal_gap 0.5) (thermal_bridge_width 0.5) (smoothing fillet) (radius 0.25))
+    (polygon
+      (pts
+        (xy 174.5 53) (xy 174.5 60.5) (xy 165.5 60.5) (xy 165.5 71) (xy 151.5 71)
+        (xy 151.5 51.5) (xy 174.5 51.5)
+      )
+    )

Commit message: PCB Tweaks
Parts:
- moved C2 0.20 mm to (154.1, 59.0)
- moved C8 0.20 mm to (148.3, 59.0)
Routing:
- net GND: track 62.8 -> 59.7 mm
- net /ST2: track 10.9 -> 11.8 mm
- net /ST1: track 14.0 -> 13.3 mm
- net /VUSB: vias 2 -> 3
