File: Li-ion 5A Boost 1A Charge Protect/Li-ion 5A Boost 1A Charge Protect.sch (KiCad schematic (older format))
At the start: 42 parts, among them J101 USB_C_FEMALE, SW101 SW_SPST, U101 AP9101CK6, U102 ECH8695R-TL-W, U103 MCP73833T, U104 PAM2423AECADJR

Commit message: Updates before converting to 0805_2012
Parts:
- added W103, W104: 2.5x5.0, Li-ion 5A Boost 1A Charge Protect:Pad_2.5-5.0, symbol Li-ion_5A_Boost_1A_Charge_Protect:TestPoint
- L101: value 6.8pH -> 6.8uH; footprint Li-ion 5A Boost 1A Charge Protect:CD75 -> Li-ion 5A Boost 1A Charge Protect:L_MGV1004; Description (none) -> 6.8µH Shielded Molded Inductor 8A 23.3mOhm; Digikey Part No. (none) -> 240-2938-1-ND; Manfacturer Part No. (none) -> MGV10046R8M-10
- SW101: footprint (none) -> Li-ion 5A Boost 1A Charge Protect:GF1230054; Description (none) -> Slide Switch SPST Through Hole 8.5A 125V; Digikey Part No. (none) -> CWI333-ND; Manfacturer Part No. (none) -> GF-123-0054
- TH101: Description (none) -> NTC Thermistor 10k; Digikey Part No. (none) -> 445-175460-1-ND; Manfacturer Part No. (none) -> NTCG203NH103JT1
- U103: footprint Li-ion 5A Boost 1A Charge Protect:Charger_MCP73833 -> Li-ion 5A Boost 1A Charge Protect:MCP73833
- U104: footprint Li-ion 5A Boost 1A Charge Protect:Boost_PAM242x -> Li-ion 5A Boost 1A Charge Protect:PAM2423AECADJR
- renumbered W103 to W105, W104 to W106, W105 to W107, W106 to W108
Connections:
- wire segments 135 -> 151
Other:
- moved on the sheet: C101, C103, C104, C110, C111, J101, R101, R102, SW101, U101, U102

Commit message: Moved Li-Ion Libraries
Parts:
- C101: Description (none) -> 0.1µF ±20% 50V Ceramic Capacitor X7R 0805 (2012 Metric); Digikey Part No. (none) -> 1276-2450-1-ND; Manfacturer Part No. (none) -> CL21B104MBCNNNC
- C102, C108: Description (none) -> 22µF ±10% 6.3V Ceramic Capacitor X5R 0805 (2012 Metric); Digikey Part No. (none) -> 1276-6687-1-ND; Manfacturer Part No. (none) -> CL21A226KQCLRNC
- C103, C111: footprint Li-ion 5A Boost 1A Charge Protect:0805_2012Metric_HandSolder -> Li-ion 5A Boost 1A Charge Protect:UCD1E471MNL1GS; Description (none) -> 470µF 25V Aluminum Electrolytic Capacitors Radial, Can - SMD; Digikey Part No. (none) -> 493-6386-1-ND; Manfacturer Part No. (none) -> UCD1E471MNL1GS
- C104, C110: Description (none) -> 10µF ±10% 6.3V Ceramic Capacitor X5R 0805 (2012 Metric); Digikey Part No. (none) -> 1276-2405-1-ND; Manfacturer Part No. (none) -> CL21A106KQCLRNC
- C105: Description (none) -> 2200pF ±10% 50V Ceramic Capacitor X7R 0805 (2012 Metric); Digikey Part No. (none) -> 1276-1171-1-ND; Manfacturer Part No. (none) -> CL21B222KBANNNC
- C106: Description (none) -> 1µF ±10% 16V Ceramic Capacitor X7R 0805 (2012 Metric); Digikey Part No. (none) -> 1276-2931-1-ND; Manfacturer Part No. (none) -> CL21B105KOFNNWE
- C107: Description (none) -> 47pF ±5% 50V Ceramic Capacitor C0G, NP0 0805 (2012 Metric); Digikey Part No. (none) -> 1276-1156-1-ND; Manfacturer Part No. (none) -> CL21C470JBANNNC
- C109: Description (none) -> 10000pF ±10% 50V Ceramic Capacitor X7R 0805 (2012 Metric); Digikey Part No. (none) -> 1276-1015-1-ND; Manfacturer Part No. (none) -> CL21B103KBANNNC
- D101: symbol Li-ion_5A_Boost_1A_Charge_Protect:D -> Li-ion_5A_Boost_1A_Charge_Protect:D_NTS12120EMFST1G
- R101: Digikey Part No. 311-330FRCT-ND -> 2019-RK73H2ATTD3300FCT-ND; Manfacturer Part No. RC1206FR-07330RL -> RK73H2ATTD3300F
- R102: Digikey Part No. YAG3855CT-ND -> 2019-RK73H2ATTD2701FCT-ND; Manfacturer Part No. AC1206FR-072K7L -> RK73H2ATTD2701F
- R103, R104, R105, R106, R112: Digikey Part No. 311-1.00KFRCT-ND -> 2019-RK73H2ATTD1001FCT-ND; Manfacturer Part No. RC1206FR-071KL -> RK73H2ATTD1001F
- R107: Digikey Part No. 311-1.54KFRCT-ND -> 2019-RK73H2ATTD1541FCT-ND; Manfacturer Part No. RC1206FR-071K54L -> RK73H2ATTD1541F
- R108: Digikey Part No. 311-69.8KFRCT-ND -> 2019-RK73H2ATTD6982FCT-ND; Manfacturer Part No. RC1206FR-0769K8L -> RK73H2ATTD6982F
- R109: Digikey Part No. 311-51.0KFRCT-ND -> 2019-RK73H2ATTD5102FCT-ND; Manfacturer Part No. RC1206FR-0751KL -> RK73H2ATTD5102F
- R110: Digikey Part No. 311-30.0KFRCT-ND -> 2019-RK73H2ATTD3002FCT-ND; Manfacturer Part No. RC1206FR-0730KL -> RK73H2ATTD3002F
- R111: Digikey Part No. 311-10.0KFRCT-ND -> 2019-RK73H2ATTD1002FCT-ND; Manfacturer Part No. RC1206FR-0710KL -> RK73H2ATTD1002F
- W101, W102, W103, W104, W105, W106, W107, W108: Digikey Part No. - -> None; Manfacturer Part No. - -> None
Connections:
- net labels added: BOOSTVIN, BOOSTVOUT, COMP, FB, SS, SW
- net labels removed: 5V_BOOST, FDBK, V-IN-BOOST

Commit message: Start of PCB Layout
Parts:
- W101, W102, W103, W104, W105, W106, W107, W108: footprint Li-ion 5A Boost 1A Charge Protect:Pad_2.5-5.0 -> Li-ion 5A Boost 1A Charge Protect:Pad_3.0-5.0
Connections:
- net labels added: THRM, THRMIC
- net labels removed: THERM
- wire segments 151 -> 167
- no-connect marks 9 -> 12
Other:
- moved on the sheet: J101, W101, W102

Commit message: Preliminary PCB layout 1
Parts:
- renumbered C101 to C1, C110 to C10, C111 to C11, C102 to C2, C103 to C3, C104 to C4, C105 to C5, C106 to C6, C107 to C7, C108 to C8, C109 to C9, D101 to D1, J101 to J1, L101 to L1, LED101 to LED1, LED102 to LED2, LED103 to LED3, LED104 to LED4, R101 to R1, R110 to R10, R111 to R11, R112 to R12, R102 to R2, R103 to R3, R104 to R4, R105 to R5, R106 to R6, R107 to R7, R108 to R8, R109 to R9, SW101 to SW1, TH101 to TH1, U101 to U1, U102 to U2, U103 to U3, U104 to U4, W101 to W1, W102 to W2, W103 to W3, W104 to W4, W105 to W5, W106 to W6, W107 to W7, W108 to W8
Connections:
- net labels added: PVDD

Commit message: Updates to Boost out on PCB
Connections:
- wire segments 167 -> 177
Other:
- moved on the sheet: LED4, R12
Changed lines of the file:
@@
 L Li-ion_5A_Boost_1A_Charge_Protect:R R12
 U 1 1 44057106
-P 11550 5900
-F 0 "R12" V 11450 5800 59  0000 L CNN
-F 1 "1k" V 11650 5800 59  0000 L CNN
-F 2 "Li-ion 5A Boost 1A Charge Protect:0805_2012Metric_HandSolder" H 11550 5900 50  0001 C CNN
-F 3 "http://www.koaspeer.com/pdfs/RK73H.pdf" H 11550 5900 50  0001 C CNN
-F 4 "1 kOhms ±1% 0.25W, 1/4W Chip Resistor 1206 (3216 Metric) " H 11550 5900 50  0001 C CNN "Description"
-F 5 "2019-RK73H2ATTD1001FCT-ND" H 11550 5900 50  0001 C CNN "Digikey Part No."
-F 6 "RK73H2ATTD1001F" H 11550 5900 50  0001 C CNN "Manfacturer Part No."
-	1    11550 5900
+P 11550 5300
+F 0 "R12" V 11450 5200 59  0000 L CNN
+F 1 "1k" V 11650 5200 59  0000 L CNN
+F 2 "Li-ion 5A Boost 1A Charge Protect:0805_2012Metric_HandSolder" H 11550 5300 50  0001 C CNN
+F 3 "http://www.koaspeer.com/pdfs/RK73H.pdf" H 11550 5300 50  0001 C CNN
+F 4 "1 kOhms ±1% 0.25W, 1/4W Chip Resistor 1206 (3216 Metric) " H 11550 5300 50  0001 C CNN "Description"
+F 5 "2019-RK73H2ATTD1001FCT-ND" H 11550 5300 50  0001 C CNN "Digikey Part No."
+F 6 "RK73H2ATTD1001F" H 11550 5300 50  0001 C CNN "Manfacturer Part No."
+	1    11550 5300
 	1    0    0    -1
 $EndComp
@@
 Wire Wire Line
 	9950 6200 10150 6200
-Connection ~ 10550 5000
 Connection ~ 10550 6200
 Connection ~ 10900 5000
@@
 L Li-ion_5A_Boost_1A_Charge_Protect:LED LED4
 U 1 1 602B6D8A
-P 11550 5300
-F 0 "LED4" H 11400 5400 59  0000 L CNN
-F 1 "RED" H 11450 5150 59  0000 L BNN
-F 2 "Li-ion 5A Boost 1A Charge Protect:LED_0805_2012Metric_HandSolder" H 11550 5300 50  0001 C CNN
-F 3 "https://www.we-online.de/katalog/datasheet/150080RS75000.pdf" H 11550 5300 50  0001 C CNN
-F 4 "Red 625nm LED Indication - Discrete 2V 0805 (2012 Metric)" H 11550 5300 50  0001 C CNN "Description"
-F 5 "732-4984-1-ND" H 11550 5300 50  0001 C CNN "Digikey Part No."
-F 6 "150080RS75000" H 11550 5300 50  0001 C CNN "Manfacturer Part No."
-	1    11550 5300
+P 11550 5900
+F 0 "LED4" H 11400 6000 59  0000 L CNN
+F 1 "RED" H 11450 5750 59  0000 L BNN
+F 2 "Li-ion 5A Boost 1A Charge Protect:LED_0805_2012Metric_HandSolder" H 11550 5900 50  0001 C CNN
+F 3 "https://www.we-online.de/katalog/datasheet/150080RS75000.pdf" H 11550 5900 50  0001 C CNN
+F 4 "Red 625nm LED Indication - Discrete 2V 0805 (2012 Metric)" H 11550 5900 50  0001 C CNN "Description"
+F 5 "732-4984-1-ND" H 11550 5900 50  0001 C CNN "Digikey Part No."
+F 6 "150080RS75000" H 11550 5900 50  0001 C CNN "Manfacturer Part No."
+	1    11550 5900
 	0    -1   -1   0
 $EndComp
@@
 	7550 1900 9200 1900
 Wire Wire Line
-	10350 5000 10550 5000
-Wire Wire Line
 	9950 5000 10050 5000
 $Comp
@@
 	4050 5950 4150 5950
 Connection ~ 4150 5950
+Wire Wire Line
+	10050 4950 10050 5000
+Connection ~ 10050 5000
+Wire Wire Line
+	10050 5000 10050 5050
+Connection ~ 10550 5000
+Wire Wire Line
+	10350 5050 10400 5050
+Wire Wire Line
+	10350 4950 10400 4950
+Wire Wire Line
+	10350 4900 10400 4900
+Wire Wire Line
+	10400 4950 10400 5000
+Wire Wire Line
+	10350 5100 10400 5100
+Wire Wire Line
+	10400 5050 10400 5000
+Connection ~ 10400 5000
+Wire Wire Line
+	10400 5000 10550 5000
+Wire Wire Line
+	10400 5050 10400 5100
+Connection ~ 10400 5050
+Wire Wire Line
+	10400 4950 10400 4900
+Connection ~ 10400 4950
 $EndSCHEMATC

Commit message: PCB Update
Connections:
- net labels added: PVM
Other:
- moved on the sheet: SW1
Changed lines of the file:
@@
 F 1 "MCP73833T" H 7025 2481 60  0000 C CNN
 F 2 "Li-ion 5A Boost 1A Charge Protect:MCP73833" H 7050 1500 60  0001 C CNN
-F 3 "http://ww1.microchip.com/downloads/en/Li-ion_5A_Boost_1A_Charge_ProtectDoc/22005b.pdf" H 7025 2481 60  0001 C CNN
+F 3 "http://ww1.microchip.com/downloads/en/DeviceDoc/22005b.pdf" H 7025 2481 60  0000 C CNN
 F 4 "Charger IC" H 7050 2100 50  0001 C CNN "Description"
 F 5 "	MCP73833T-AMI/UNCT-ND" H 7050 2100 50  0001 C CNN "Digikey Part No."
@@
 U 1 1 5EE83AA5
 P 7250 5000
-F 0 "SW1" H 7250 4850 50  0000 C CNN
-F 1 "SW_SPST" H 7250 4750 50  0000 C CNN
+F 0 "SW1" H 7250 5150 50  0000 C CNN
+F 1 "SW_SPST" H 7250 5250 50  0000 C CNN
 F 2 "Li-ion 5A Boost 1A Charge Protect:GF1230054" H 7250 5000 50  0001 C CNN
 F 3 "https://media.digikey.com/pdf/Data%20Sheets/CW%20Industries%20PDFs/GF-123-0054_Dwg.pdf" H 7250 5000 50  0001 C CNN
@@
 F 6 "GF-123-0054" H 7250 5000 50  0001 C CNN "Manfacturer Part No."
 	1    7250 5000
-	1    0    0    -1
+	-1   0    0    1
 $EndComp
 $Comp
@@
 	10400 4950 10400 4900
 Connection ~ 10400 4950
+Text Label 4000 5150 0    50   ~ 0
+PVM
 $EndSCHEMATC

Commit message: PCB Update
Working layout with repositioned charge and protect sections.  Still work to be done on labeling, 3D models, and copper pours on bottom.
Parts:
- renumbered LED1 to LD1, LED2 to LD2, LED3 to LD3, LED4 to LD4
Changed lines of the file:
@@
 F 1 "MCP73833T" H 7025 2481 60  0000 C CNN
 F 2 "Li-ion 5A Boost 1A Charge Protect:MCP73833" H 7050 1500 60  0001 C CNN
-F 3 "http://ww1.microchip.com/downloads/en/DeviceDoc/22005b.pdf" H 7025 2481 60  0000 C CNN
+F 3 "http://ww1.microchip.com/downloads/en/DeviceDoc/22005b.pdf" H 7025 2481 60  0001 C CNN
 F 4 "Charger IC" H 7050 2100 50  0001 C CNN "Description"
 F 5 "	MCP73833T-AMI/UNCT-ND" H 7050 2100 50  0001 C CNN "Digikey Part No."
@@
 PROG
 $Comp
-L Li-ion_5A_Boost_1A_Charge_Protect:LED LED1
+L Li-ion_5A_Boost_1A_Charge_Protect:LED LD1
 U 1 1 5EBA65E2
 P 4750 2050
-F 0 "LED1" H 4600 2150 50  0000 L CNN
+F 0 "LD1" H 4650 2150 50  0000 L CNN
 F 1 "GREEN" H 4650 1950 50  0000 L CNN
 F 2 "Li-ion 5A Boost 1A Charge Protect:LED_0805_2012Metric_HandSolder" H 4750 2050 50  0001 C CNN
@@
 $EndComp
 $Comp
-L Li-ion_5A_Boost_1A_Charge_Protect:LED LED2
+L Li-ion_5A_Boost_1A_Charge_Protect:LED LD2
 U 1 1 5EBA8419
 P 5100 2050
-F 0 "LED2" H 4950 2150 50  0000 L CNN
+F 0 "LD2" H 5000 2150 50  0000 L CNN
 F 1 "GREEN" H 5000 1950 50  0000 L CNN
 F 2 "Li-ion 5A Boost 1A Charge Protect:LED_0805_2012Metric_HandSolder" H 5100 2050 50  0001 C CNN
@@
 $EndComp
 $Comp
-L Li-ion_5A_Boost_1A_Charge_Protect:LED LED3
+L Li-ion_5A_Boost_1A_Charge_Protect:LED LD3
 U 1 1 5EBA883B
 P 5450 2050
-F 0 "LED3" H 5300 2150 50  0000 L CNN
+F 0 "LD3" H 5350 2150 50  0000 L CNN
 F 1 "RED" H 5350 1950 50  0000 L CNN
 F 2 "Li-ion 5A Boost 1A Charge Protect:LED_0805_2012Metric_HandSolder" H 5450 2050 50  0001 C CNN
@@
 	11550 5000 11550 5150
 $Comp
-L Li-ion_5A_Boost_1A_Charge_Protect:LED LED4
+L Li-ion_5A_Boost_1A_Charge_Protect:LED LD4
 U 1 1 602B6D8A
 P 11550 5900
-F 0 "LED4" H 11400 6000 59  0000 L CNN
+F 0 "LD4" H 11450 6000 59  0000 L CNN
 F 1 "RED" H 11450 5750 59  0000 L BNN
 F 2 "Li-ion 5A Boost 1A Charge Protect:LED_0805_2012Metric_HandSolder" H 11550 5900 50  0001 C CNN

Commit message: PCB Before Solder Footprint Switch
Before switching wire solder points to foot prints with through holes.
Connections:
- wire segments 177 -> 178
Changed lines of the file:
@@
 Wire Wire Line
 	10050 5000 10050 5050
-Connection ~ 10550 5000
 Wire Wire Line
 	10350 5050 10400 5050
-Wire Wire Line
-	10350 4950 10400 4950
-Wire Wire Line
-	10350 4900 10400 4900
-Wire Wire Line
-	10400 4950 10400 5000
 Wire Wire Line
 	10350 5100 10400 5100
 Wire Wire Line
 	10400 5050 10400 5000
-Connection ~ 10400 5000
-Wire Wire Line
-	10400 5000 10550 5000
 Wire Wire Line
 	10400 5050 10400 5100
 Connection ~ 10400 5050
+Text Label 4000 5150 0    50   ~ 0
+PVM
+Wire Wire Line
+	10400 5000 10350 5000
+Connection ~ 10400 5000
+Connection ~ 10550 5000
+Wire Wire Line
+	10400 5000 10550 5000
+Connection ~ 10400 4950
+Wire Wire Line
+	10400 4950 10400 5000
+Wire Wire Line
+	10350 4950 10400 4950
 Wire Wire Line
 	10400 4950 10400 4900
-Connection ~ 10400 4950
-Text Label 4000 5150 0    50   ~ 0
-PVM
+Wire Wire Line
+	10350 4900 10400 4900
 $EndSCHEMATC
