File: Li-ion 5A Boost 1A Charge Protect/Li-ion 5A Boost 1A Charge Protect.sch (KiCad schematic (older format))
At the start: 44 parts, among them J1 USB_C_FEMALE, SW1 SW_SPST, U1 AP9101CK6, U2 ECH8695R-TL-W, U3 MCP73833T, U4 PAM2423AECADJR

Commit message: PCB and 3D model updates
Other:
- moved on the sheet: C1, C10, C11, C2, C3, C4, C5, C6, C7, C8, C9, D1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

Commit message: PCB Cleanup and corrections
Parts:
- W1, W2, W3, W4, W5, W6, W7, W8: footprint Li-ion 5A Boost 1A Charge Protect:Pad_3.0-5.0 -> Li-ion 5A Boost 1A Charge Protect:Pad_3.0-5.0_w_TH
Changed lines of the file:
@@
 Rev "1.0.0"
 Comp ""
-Comment1 ""
+Comment1 "Designed by Lance A. Endres"
 Comment2 ""
 Comment3 ""
@@
 F 0 "W7" V 9850 3550 59  0000 L CNN
 F 1 "2.5x5.0" V 10050 3550 59  0000 L CNN
-F 2 "Li-ion 5A Boost 1A Charge Protect:Pad_3.0-5.0" H 9950 3500 50  0001 C CNN
+F 2 "Li-ion 5A Boost 1A Charge Protect:Pad_3.0-5.0_w_TH" H 9950 3500 50  0001 C CNN
 F 3 "None" H 9950 3500 50  0001 C CNN
 F 4 "Wire solder point" H 9950 3500 50  0001 C CNN "Description"
@@
 F 0 "W8" V 9850 4750 59  0000 L CNN
 F 1 "2.5x5.0" V 10050 4750 59  0000 L CNN
-F 2 "Li-ion 5A Boost 1A Charge Protect:Pad_3.0-5.0" H 9950 4700 50  0001 C CNN
+F 2 "Li-ion 5A Boost 1A Charge Protect:Pad_3.0-5.0_w_TH" H 9950 4700 50  0001 C CNN
 F 3 "None" H 9950 4700 50  0001 C CNN
 F 4 "Wire solder point" H 9950 4700 50  0001 C CNN "Description"
@@
 F 0 "W5" V 5200 6950 59  0000 R CNN
 F 1 "2.5x5.0" V 5000 6950 59  0000 R CNN
-F 2 "Li-ion 5A Boost 1A Charge Protect:Pad_3.0-5.0" H 5100 6750 50  0001 C CNN
+F 2 "Li-ion 5A Boost 1A Charge Protect:Pad_3.0-5.0_w_TH" H 5100 6750 50  0001 C CNN
 F 3 "None" H 5100 6750 50  0001 C CNN
 F 4 "Wire solder point" H 5100 6750 50  0001 C CNN "Description"
@@
 F 0 "W6" V 5200 7300 59  0000 R CNN
 F 1 "2.5x5.0" V 5000 7300 59  0000 R CNN
-F 2 "Li-ion 5A Boost 1A Charge Protect:Pad_3.0-5.0" H 5100 7100 50  0001 C CNN
+F 2 "Li-ion 5A Boost 1A Charge Protect:Pad_3.0-5.0_w_TH" H 5100 7100 50  0001 C CNN
 F 3 "None" H 5100 7100 50  0001 C CNN
 F 4 "Wire solder point" H 5100 7100 50  0001 C CNN "Description"
@@
 F 0 "W1" V 3300 6950 59  0000 R CNN
 F 1 "2.5x5.0" V 3100 6950 59  0000 R CNN
-F 2 "Li-ion 5A Boost 1A Charge Protect:Pad_3.0-5.0" H 3200 6750 50  0001 C CNN
+F 2 "Li-ion 5A Boost 1A Charge Protect:Pad_3.0-5.0_w_TH" H 3200 6750 50  0001 C CNN
 F 3 "None" H 3200 6750 50  0001 C CNN
 F 4 "Wire solder point" H 3200 6750 50  0001 C CNN "Description"
@@
 F 0 "W2" V 3300 7300 59  0000 R CNN
 F 1 "2.5x5.0" V 3100 7300 59  0000 R CNN
-F 2 "Li-ion 5A Boost 1A Charge Protect:Pad_3.0-5.0" H 3200 7100 50  0001 C CNN
+F 2 "Li-ion 5A Boost 1A Charge Protect:Pad_3.0-5.0_w_TH" H 3200 7100 50  0001 C CNN
 F 3 "None" H 3200 7100 50  0001 C CNN
 F 4 "Wire solder point" H 3200 7100 50  0001 C CNN "Description"
@@
 F 0 "W4" V 5400 3350 59  0000 L CNN
 F 1 "2.5x5.0" V 5550 3350 59  0000 L TNN
-F 2 "Li-ion 5A Boost 1A Charge Protect:Pad_3.0-5.0" H 5500 3300 50  0001 C CNN
+F 2 "Li-ion 5A Boost 1A Charge Protect:Pad_3.0-5.0_w_TH" H 5500 3300 50  0001 C CNN
 F 3 "None" H 5500 3300 50  0001 C CNN
 F 4 "Wire solder point" H 5500 3300 50  0001 C CNN "Description"
@@
 F 0 "W3" V 5000 3350 59  0000 L CNN
 F 1 "2.5x5.0" V 5150 3350 59  0000 L TNN
-F 2 "Li-ion 5A Boost 1A Charge Protect:Pad_3.0-5.0" H 5100 3300 50  0001 C CNN
+F 2 "Li-ion 5A Boost 1A Charge Protect:Pad_3.0-5.0_w_TH" H 5100 3300 50  0001 C CNN
 F 3 "None" H 5100 3300 50  0001 C CNN
 F 4 "Wire solder point" H 5100 3300 50  0001 C CNN "Description"

Commit message: Changed name of libraries to remove underscore
Parts:
- C10, C2, C4, C5, C6, C7, C8, C9: Manufacturer Name (none) -> Samsung Electro-Mechanics
Changed lines of the file:
@@
 F 5 "1276-2405-1-ND" H 6050 4150 50  0001 C CNN "Digikey Part No."
 F 6 "CL21A106KQCLRNC" H 6050 4150 50  0001 C CNN "Manfacturer Part No."
+F 7 "	Samsung Electro-Mechanics" H 6050 4150 50  0001 C CNN "Manufacturer Name"
 	1    6050 4150
 	1    0    0    -1
@@
 F 5 "1276-2405-1-ND" H 8950 4150 50  0001 C CNN "Digikey Part No."
 F 6 "CL21A106KQCLRNC" H 8950 4150 50  0001 C CNN "Manfacturer Part No."
+F 7 "	Samsung Electro-Mechanics" H 8950 4150 50  0001 C CNN "Manufacturer Name"
 	1    8950 4150
 	1    0    0    -1
@@
 U 1 1 5ECFE4F0
 P 6650 4200
-F 0 "R9" V 6750 4100 59  0000 L CNN
-F 1 "51k" V 6550 4100 59  0000 L CNN
+F 0 "R9" V 6550 4100 59  0000 L CNN
+F 1 "51k" V 6750 4100 59  0000 L CNN
 F 2 "Li-ion 5A Boost 1A Charge Protect:0805_2012Metric_HandSolder" H 6650 4200 50  0001 C CNN
 F 3 "http://www.koaspeer.com/pdfs/RK73H.pdf" H 6650 4200 50  0001 C CNN
@@
 F 5 "1276-1171-1-ND" H 6450 4400 50  0001 C CNN "Digikey Part No."
 F 6 "CL21B222KBANNNC" H 6450 4400 50  0001 C CNN "Manfacturer Part No."
+F 7 "	Samsung Electro-Mechanics" H 6450 4400 50  0001 C CNN "Manufacturer Name"
 	1    6450 4400
 	1    0    0    -1
@@
 F 5 "1276-1156-1-ND" H 6900 4400 50  0001 C CNN "Digikey Part No."
 F 6 "CL21C470JBANNNC" H 6900 4400 50  0001 C CNN "Manfacturer Part No."
+F 7 "Samsung Electro-Mechanics" H 6900 4400 50  0001 C CNN "Manufacturer Name"
 	1    6900 4400
 	1    0    0    -1
@@
 F 5 "1276-2931-1-ND" H 6800 3800 50  0001 C CNN "Digikey Part No."
 F 6 "CL21B105KOFNNWE" H 6800 3800 50  0001 C CNN "Manfacturer Part No."
+F 7 "Samsung Electro-Mechanics" H 6800 3800 50  0001 C CNN "Manufacturer Name"
 	1    6800 3800
 	0    1    1    0
@@
 F 5 "1276-1015-1-ND" H 8200 4500 50  0001 C CNN "Digikey Part No."
 F 6 "CL21B103KBANNNC" H 8200 4500 50  0001 C CNN "Manfacturer Part No."
+F 7 "Samsung Electro-Mechanics" H 8200 4500 50  0001 C CNN "Manufacturer Name"
 	1    8200 4500
 	1    0    0    -1
@@
 F 5 "1276-6687-1-ND" H 7550 1350 50  0001 C CNN "Digikey Part No."
 F 6 "CL21A226KQCLRNC" H 7550 1350 50  0001 C CNN "Manfacturer Part No."
+F 7 "Samsung Electro-Mechanics" H 7550 1350 50  0001 C CNN "Manufacturer Name"
 	1    7550 1350
 	1    0    0    -1
@@
 F 5 "1276-6687-1-ND" H 2700 1350 50  0001 C CNN "Digikey Part No."
 F 6 "CL21A226KQCLRNC" H 2700 1350 50  0001 C CNN "Manfacturer Part No."
+F 7 "Samsung Electro-Mechanics" H 2700 1350 50  0001 C CNN "Manufacturer Name"
 	1    2700 1350
 	1    0    0    -1

Commit message: Partial Update
Parts:
- W1, W2, W3, W4, W5, W6, W7, W8: Manufacturer Name (none) -> None
Changed lines of the file:
@@
 F 5 "None" H 9950 3500 50  0001 C CNN "Digikey Part No."
 F 6 "None" H 9950 3500 50  0001 C CNN "Manfacturer Part No."
+F 7 "None" H 9950 3500 50  0001 C CNN "Manufacturer Name"
 	1    9950 3500
 	0    1    1    0
@@
 F 5 "None" H 9950 4700 50  0001 C CNN "Digikey Part No."
 F 6 "None" H 9950 4700 50  0001 C CNN "Manfacturer Part No."
+F 7 "None" H 9950 4700 50  0001 C CNN "Manufacturer Name"
 	1    9950 4700
 	0    1    1    0
@@
 F 5 "None" H 5100 6750 50  0001 C CNN "Digikey Part No."
 F 6 "None" H 5100 6750 50  0001 C CNN "Manfacturer Part No."
+F 7 "None" H 5100 6750 50  0001 C CNN "Manufacturer Name"
 	1    5100 6750
 	0    -1   -1   0
@@
 F 5 "None" H 5100 7100 50  0001 C CNN "Digikey Part No."
 F 6 "None" H 5100 7100 50  0001 C CNN "Manfacturer Part No."
+F 7 "None" H 5100 7100 50  0001 C CNN "Manufacturer Name"
 	1    5100 7100
 	0    -1   -1   0
@@
 F 5 "None" H 3200 6750 50  0001 C CNN "Digikey Part No."
 F 6 "None" H 3200 6750 50  0001 C CNN "Manfacturer Part No."
+F 7 "None" H 3200 6750 50  0001 C CNN "Manufacturer Name"
 	1    3200 6750
 	0    -1   -1   0
@@
 F 5 "None" H 3200 7100 50  0001 C CNN "Digikey Part No."
 F 6 "None" H 3200 7100 50  0001 C CNN "Manfacturer Part No."
+F 7 "None" H 3200 7100 50  0001 C CNN "Manufacturer Name"
 	1    3200 7100
 	0    -1   -1   0
@@
 F 5 "None" H 5500 3300 50  0001 C CNN "Digikey Part No."
 F 6 "None" H 5500 3300 50  0001 C CNN "Manfacturer Part No."
+F 7 "None" H 5500 3300 50  0001 C CNN "Manufacturer Name"
 	1    5500 3300
 	1    0    0    -1
@@
 F 5 "None" H 5100 3300 50  0001 C CNN "Digikey Part No."
 F 6 "None" H 5100 3300 50  0001 C CNN "Manfacturer Part No."
+F 7 "None" H 5100 3300 50  0001 C CNN "Manufacturer Name"
 	1    5100 3300
 	1    0    0    -1

Commit message: Updates
Parts:
- J1: symbol Li-ion_5A_Boost_1A_Charge_Protect:USB_C_Plug_USB2.0 -> Connectors_LE:USB_C_Plug_USB2.0; Manufacturer Name (none) -> GCT
- LD1, LD2, LD3, LD4: Manufacturer Name (none) -> Würth Elektronik
Connections:
- no-connect marks 12 -> 16
Other:
- moved on the sheet: W1, W2, W5, W6

Commit message: Symbol field corrections and additions
Parts:
- C1: Manfacturer Part No. CL21B104MBCNNNC -> (none); Manufacturer Name (none) -> Samsung Electro-Mechanics; Manufacturer Part No. (none) -> CL21B104MBCNNNC
- C10, C4: Manfacturer Part No. CL21A106KQCLRNC -> (none); Manufacturer Name Samsung Electro-Mechanics -> Samsung Electro-Mechanics; Manufacturer Part No. (none) -> CL21A106KQCLRNC
- C11, C3: Manfacturer Part No. UCD1E471MNL1GS -> (none); Manufacturer Name (none) -> Nichicon; Manufacturer Part No. (none) -> UCD1E471MNL1GS
- C2, C8: Manfacturer Part No. CL21A226KQCLRNC -> (none); Manufacturer Part No. (none) -> CL21A226KQCLRNC
- C5: Manfacturer Part No. CL21B222KBANNNC -> (none); Manufacturer Name Samsung Electro-Mechanics -> Samsung Electro-Mechanics; Manufacturer Part No. (none) -> CL21B222KBANNNC
- C6: Manfacturer Part No. CL21B105KOFNNWE -> (none); Manufacturer Part No. (none) -> CL21B105KOFNNWE
- C7: Manfacturer Part No. CL21C470JBANNNC -> (none); Manufacturer Part No. (none) -> CL21C470JBANNNC
- C9: Manfacturer Part No. CL21B103KBANNNC -> (none); Manufacturer Part No. (none) -> CL21B103KBANNNC
- D1: Manfacturer Part No. NTS12120EMFST1G -> (none); Manufacturer Name (none) -> ON Semiconductor; Manufacturer Part No. (none) -> NTS12120EMFST1G
- J1: Manfacturer Part No. USB4110-GF-A -> (none); Manufacturer Part No. (none) -> USB4110-GF-A
- L1: Manfacturer Part No. MGV10046R8M-10 -> (none); Manufacturer Name (none) -> Laird-Signal Integrity Products; Manufacturer Part No. (none) -> MGV10046R8M-10
- LD1, LD2: Manfacturer Part No. 150080VS75000 -> (none); Manufacturer Part No. (none) -> 150080VS75000
- LD3, LD4: Manfacturer Part No. 150080RS75000 -> (none); Manufacturer Part No. (none) -> 150080RS75000
- R1: Manfacturer Part No. RK73H2ATTD3300F -> (none); Manufacturer Name (none) -> KOA Speer Electronics, Inc.; Manufacturer Part No. (none) -> RK73H2ATTD3300F
- R10: Manfacturer Part No. RK73H2ATTD3002F -> (none); Manufacturer Name (none) -> KOA Speer Electronics, Inc.; Manufacturer Part No. (none) -> RK73H2ATTD3002F
- R11: Manfacturer Part No. RK73H2ATTD1002F -> (none); Manufacturer Name (none) -> KOA Speer Electronics, Inc.; Manufacturer Part No. (none) -> RK73H2ATTD1002F
- R12, R3, R4, R5, R6: Manfacturer Part No. RK73H2ATTD1001F -> (none); Manufacturer Name (none) -> KOA Speer Electronics, Inc.; Manufacturer Part No. (none) -> RK73H2ATTD1001F
- R2: Manfacturer Part No. RK73H2ATTD2701F -> (none); Manufacturer Name (none) -> KOA Speer Electronics, Inc.; Manufacturer Part No. (none) -> RK73H2ATTD2701F
- R7: Manfacturer Part No. RK73H2ATTD1541F -> (none); Manufacturer Name (none) -> KOA Speer Electronics, Inc.; Manufacturer Part No. (none) -> RK73H2ATTD1541F
- R8: Manfacturer Part No. RK73H2ATTD6982F -> (none); Manufacturer Name (none) -> KOA Speer Electronics, Inc.; Manufacturer Part No. (none) -> RK73H2ATTD6982F
- R9: Manfacturer Part No. RK73H2ATTD5102F -> (none); Manufacturer Name (none) -> KOA Speer Electronics, Inc.; Manufacturer Part No. (none) -> RK73H2ATTD5102F
- SW1: Manfacturer Part No. GF-123-0054 -> (none); Manufacturer Name (none) -> CW Industries; Manufacturer Part No. (none) -> GF-123-0054
- TH1: Manfacturer Part No. NTCG203NH103JT1 -> (none); Manufacturer Name (none) -> TDK Corporation; Manufacturer Part No. (none) -> NTCG203NH103JT1
- U1: Manfacturer Part No. AP9101CK6-AYTRG1 -> (none); Manufacturer Name (none) -> Diodes Incorporated; Manufacturer Part No. (none) -> AP9101CK6-AYTRG1
- U2: Manfacturer Part No. ECH8695R-TL-W -> (none); Manufacturer Name (none) -> ON Semiconductor; Manufacturer Part No. (none) -> ECH8695R-TL-W
- U3: Digikey Part No. MCP73833T-AMI/UNCT-ND -> MCP73833T-AMI/UNCT-ND; Manfacturer Part No. MCP73833T-AMI/UN -> (none); Manufacturer Name (none) -> Microchip Technology; Manufacturer Part No. (none) -> MCP73833T-AMI/UN
- U4: Manfacturer Part No. PAM2423AECADJR -> (none); Manufacturer Name (none) -> Diodes Incorporated; Manufacturer Part No. (none) -> PAM2423AECADJR
- W1, W2, W3, W4, W5, W6, W7, W8: Manfacturer Part No. None -> (none); Manufacturer Part No. (none) -> None

Commit message: Adding Power Daughter Board
Parts:
- C1: Digikey Part No. 1276-2450-1-ND -> (none); Source (none) -> Digikey; Source Part No. (none) -> 1276-2450-1-ND
- C10, C4: Digikey Part No. 1276-2405-1-ND -> (none); Source (none) -> Digikey; Source Part No. (none) -> 1276-2405-1-ND
- C11, C3: Digikey Part No. 493-6386-1-ND -> (none); Source (none) -> Digikey; Source Part No. (none) -> 493-6386-1-ND
- C2, C8: Digikey Part No. 1276-6687-1-ND -> (none); Source (none) -> Digikey; Source Part No. (none) -> 1276-6687-1-ND
- C5: Digikey Part No. 1276-1171-1-ND -> (none); Source (none) -> Digikey; Source Part No. (none) -> 1276-1171-1-ND
- C6: Digikey Part No. 1276-2931-1-ND -> (none); Source (none) -> Digikey; Source Part No. (none) -> 1276-2931-1-ND
- C7: Digikey Part No. 1276-1156-1-ND -> (none); Source (none) -> Digikey; Source Part No. (none) -> 1276-1156-1-ND
- C9: Digikey Part No. 1276-1015-1-ND -> (none); Source (none) -> Digikey; Source Part No. (none) -> 1276-1015-1-ND
- D1: Digikey Part No. NTS12120EMFST1GOSCT-ND -> (none); Source (none) -> Digikey; Source Part No. (none) -> NTS12120EMFST1GOSCT-ND
- J1: Digikey Part No. 2073-USB4110-GF-A-1-ND -> (none); Source (none) -> Digikey; Source Part No. (none) -> 2073-USB4110-GF-A-1-ND
- L1: Digikey Part No. 240-2938-1-ND -> (none); Source (none) -> Digikey; Source Part No. (none) -> 240-2938-1-ND
- LD1, LD2: Digikey Part No. 732-4986-1-ND -> (none); Source (none) -> Digikey; Source Part No. (none) -> 732-4986-1-ND
- LD3, LD4: Digikey Part No. 732-4984-1-ND -> (none); Source (none) -> Digikey; Source Part No. (none) -> 732-4984-1-ND
- R1: Digikey Part No. 2019-RK73H2ATTD3300FCT-ND -> (none); Source (none) -> Digikey; Source Part No. (none) -> 2019-RK73H2ATTD3300FCT-ND
- R10: Digikey Part No. 2019-RK73H2ATTD3002FCT-ND -> (none); Source (none) -> Digikey; Source Part No. (none) -> 2019-RK73H2ATTD3002FCT-ND
- R11: Digikey Part No. 2019-RK73H2ATTD1002FCT-ND -> (none); Source (none) -> Digikey; Source Part No. (none) -> 2019-RK73H2ATTD1002FCT-ND
- R12, R3, R4, R5, R6: Digikey Part No. 2019-RK73H2ATTD1001FCT-ND -> (none); Source (none) -> Digikey; Source Part No. (none) -> 2019-RK73H2ATTD1001FCT-ND
- R2: Digikey Part No. 2019-RK73H2ATTD2701FCT-ND -> (none); Source (none) -> Digikey; Source Part No. (none) -> 2019-RK73H2ATTD2701FCT-ND
- R7: Digikey Part No. 2019-RK73H2ATTD1541FCT-ND -> (none); Source (none) -> Digikey; Source Part No. (none) -> 2019-RK73H2ATTD1541FCT-ND
- R8: Digikey Part No. 2019-RK73H2ATTD6982FCT-ND -> (none); Source (none) -> Digikey; Source Part No. (none) -> 2019-RK73H2ATTD6982FCT-ND
- R9: Digikey Part No. 2019-RK73H2ATTD5102FCT-ND -> (none); Source (none) -> Digikey; Source Part No. (none) -> 2019-RK73H2ATTD5102FCT-ND
- SW1: Digikey Part No. CWI333-ND -> (none); Source (none) -> Digikey; Source Part No. (none) -> CWI333-ND
- TH1: Digikey Part No. 445-175460-1-ND -> (none); Source (none) -> Digikey; Source Part No. (none) -> 445-175460-1-ND
- U1: Digikey Part No. AP9101CK6-AYTRG1DICT-ND -> (none); Source (none) -> Digikey; Source Part No. (none) -> AP9101CK6-AYTRG1DICT-ND
- U2: Digikey Part No. ECH8695R-TL-WOSCT-ND -> (none); Source (none) -> Digikey; Source Part No. (none) -> ECH8695R-TL-WOSCT-ND
- U3: Digikey Part No. MCP73833T-AMI/UNCT-ND -> (none); Source (none) -> Digikey; Source Part No. (none) -> MCP73833T-AMI/UNCT-ND
- U4: Digikey Part No. PAM2423AECADJRDICT-ND -> (none); Source (none) -> Digikey; Source Part No. (none) -> PAM2423AECADJRDICT-ND
- W1, W2, W3, W4, W5, W6, W7, W8: Digikey Part No. None -> (none); Source (none) -> None; Source Part No. (none) -> None
