File: Naquadah Generator Main/Naquadah Generator Main.sch (KiCad schematic (older format))
At the start: 12 parts, among them J1 Conn_01x03, SW1 SW_SPST, U1 74HC595, U2 74HC595

Commit message: Before changing BOM
Parts:
- removed J? (x2): Conn_01x04, symbol Connector_Generic:Conn_01x04
- added J101, J102: HallSensor_Conn_T4, Connector_JST:JST_SH_SM04B-SRSS-TB_1x04-1MP_P1.00mm_Horizontal, symbol Naquadah_Generator:HallSensor_Conn_T4
- renumbered U2 to U102
Connections:
- net labels added: +5V, SRCLK, SRDATA1IN, SRDATA1OUT, SRLATCH
- net labels removed: 5V, VGND
- wire segments 95 -> 97
Other:
- moved on the sheet: D1, R1

Commit message: Changed name of libraries to remove underscore
Parts:
- removed A1: ArduinoProMini, Arduino:Arduino-Pro-Mini, symbol Arduino:ArduinoProMini
- removed D2: LED, LED_THT:LED_D5.0mm, symbol Device:LED
- removed J1: Conn_01x03, Connector_Wire:SolderWirePad_1x03_P3.81mm_Drill1.2mm, symbol Connector_Generic:Conn_01x03
- removed J101, J102: HallSensor_Conn_T4, Connector_JST:JST_SH_SM04B-SRSS-TB_1x04-1MP_P1.00mm_Horizontal, symbol Naquadah_Generator:HallSensor_Conn_T4
- removed R2: 330, Resistor_THT:R_Axial_DIN0207_L6.3mm_D2.5mm_P10.16mm_Horizontal, symbol Device:R
- removed U1, U102: 74HC595, Package_DIP:DIP-16_W7.62mm, symbol 74xx:74HC595
- added C? (x2): 22pF, symbol Naquadah_Generator:C
- added C?: 0.1uF, symbol Naquadah_Generator:C
- added C? (x4): 1.0uF, symbol Naquadah_Generator:C
- added J101, J102: State_Sensing_Conn, Naquadah_Generator:State_Sensing_Mother_Board_JST_Conn, symbol Naquadah_Generator:State_Sensing_Conn
- added U: ATmega32U4-AU, Package_QFP:TQFP-44_10x10mm_P0.8mm, symbol Naquadah_Generator:ATmega32U4-AU
- added Y?: 16MHz, symbol Naquadah_Generator:Crystal
- R1: footprint Resistor_THT:R_Axial_DIN0207_L6.3mm_D2.5mm_P10.16mm_Horizontal -> Naquadah_Generator:0805_2012Metric_HandSolder
- SW1: symbol Switch:SW_SPST -> Naquadah_Generator:SW_SPST
Connections:
- net labels added: AREF, D+, D-, HALLEFF1, HALLEFF2, HALLEFF3, HALLEFF4, MODESEL, SRDATA, UCAP, VBUS, nRESET
- net labels removed: BL1, BL2, BL3, BL4, BL5, GL, HE1, HE2, HE3, HE4, IND, RL, SRDATA1IN, SRDATA1OUT, WL
- wire segments 97 -> 84
- no-connect marks 31 -> 0
Other:
- moved on the sheet: BT1, D1, R1

Commit message: Partial Update
Parts:
- added R1: 10k, Frequently_Used:0805_2012Metric_HandSolder, symbol Frequently_Used:R
- added SW1: RESET, Naquadah_Generator:PTS526SMG15SMTR2LFS_Hand_Solder, symbol Naquadah_Generator:PTS526_SMG15
- C1, C2, C3, C4, C5, C6, C7: renamed from C?; footprint (none) -> Frequently_Used:0805_2012Metric_HandSolder; symbol Naquadah_Generator:C -> Frequently_Used:C
- D1: symbol Device:LED -> Frequently_Used:LED
- R2: renamed from R1; footprint Naquadah_Generator:0805_2012Metric_HandSolder -> Frequently_Used:0805_2012Metric_HandSolder; symbol Device:R -> Frequently_Used:R
- SW2: renamed from SW1; symbol Naquadah_Generator:SW_SPST -> Frequently_Used:SW_SPST
- Y1: renamed from Y?; footprint (none) -> Naquadah_Generator:Oscillator_ABM3-16.000MHZ-B2-T; symbol Naquadah_Generator:Crystal -> Frequently_Used:Crystal; Digikey Part No. (none) -> 535-9103-1-ND; Manufacturer Name (none) -> Abracon; Manufacturer Part No. (none) -> ABM3-16.000MHZ-B2-T
- renumbered J101 to J1, J102 to J2, U to U1
Connections:
- net labels added: RXLED, TXLED, XTAL1, XTAL2
- wire segments 84 -> 98
Other:
- moved on the sheet: BT1, D1, R2, U1

Commit message: Resize to correct for scale
Parts:
- added J?: Conn_ISP, symbol Naquadah_Generator:Conn_ISP
Connections:
- net labels added: MISO, MOSI, SCK
- wire segments 98 -> 109
Other:
- note added: "ATmega34U4"
- note added: "ISP Breakout"
- note added: "Lights"
- note added: "Sensing Board 1"
- note added: "Sensing Board 2"
- moved on the sheet: C2, C3, J1, J2, R1, SW1, Y1

Commit message: Updates to PCB Mount
Parts:
- added H1, H2, H3, H4: PCB Mounting Hole, Naquadah_Generator:MountingHole_2.2mm_M2, symbol Naquadah_Generator:MountingHole
- added H5, H6, H7, H8: Top Through Hole, Naquadah_Generator:MountingHole_Top_Conn_M6, symbol Naquadah_Generator:MountingHole
- J8: renamed from J?; value Conn_ISP -> Conn_ISP_Prog; footprint (none) -> Naquadah_Generator:PinHeader_2x03_P2.54mm_Vertical; Digikey Part No. (none) -> None; Manufacturer Name (none) -> None; Manufacturer Part No. (none) -> None
- U1: Digikey Part No. (none) -> ATMEGA32U4-AU-ND; Manufacturer Name (none) -> Microchip Technology; Manufacturer Part No. (none) -> ATMEGA32U4-AU
Other:
- note added: "Cover Mounting"
- note added: "PCB Mounting"
- note added: "Power"
- moved on the sheet: C1, C2, C3, C4, C5, C6, C7, R1, SW1, U1, Y1

Commit message: Library Updates
Parts:
- renumbered J8 to J0
Connections:
- no-connect marks 0 -> 9
Other:
- moved on the sheet: H1, H2, H3, H4, H5, H6, H7, H8, J0, J1, J2

Commit message: Updates
Parts:
- removed H1, H2, H3, H4: PCB Mounting Hole, Naquadah_Generator:MountingHole_2.2mm_M2, symbol Naquadah_Generator:MountingHole
- removed H5, H6, H7, H8: Top Through Hole, Naquadah_Generator:MountingHole_Top_Conn_M6, symbol Naquadah_Generator:MountingHole
- removed J0: Conn_ISP_Prog, Naquadah_Generator:PinHeader_2x03_P2.54mm_Vertical, symbol Naquadah_Generator:Conn_ISP
- removed J1, J2: State_Sensing_Conn, Naquadah_Generator:State_Sensing_Mother_Board_JST_Conn, symbol Naquadah_Generator:State_Sensing_Conn
- added D23: GREEN, Frequently_Used:LED_0805_2012Metric_HandSolder, symbol Frequently_Used:LED
- added D24: YELLOW, Frequently_Used:LED_0805_2012Metric_HandSolder, symbol Frequently_Used:LED
- added R4, R9: 1k, Frequently_Used:0805_2012Metric_HandSolder, symbol Frequently_Used:R
- C1, C4, C5, C6: Description (none) -> 1µF ±10% 16V Ceramic Capacitor X7R 0805 (2012 Metric); Digikey Part No. (none) -> 1276-2931-1-ND; Manufacturer Name (none) -> Samsung Electro-Mechanics; Manufacturer Part No. (none) -> CL21B105KOFNNWE
- C2, C3: value 22pF -> 18pF; Digikey Part No. (none) -> 399-1052-1-ND; Manufacturer Name (none) -> Kemet; Manufacturer Part No. (none) -> C0603C180J5GACTU
- D25: renamed from D1; value LED -> RED; footprint LED_THT:LED_D5.0mm -> Frequently_Used:LED_0805_2012Metric_HandSolder; Description (none) -> Red 625nm LED Indication- Discrete 2V 0805 (2012 Metric); Digikey Part No. (none) -> 732-4984-1-ND; Manufacturer Name (none) -> Würth Elektronik; Manufacturer Part No. (none) -> 150080RS75000
- U1: Description (none) -> ATmega Microcontroller IC 8-Bit 16MHz 32KB (16K x 16) FLASH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; Digikey Part No. ATMEGA32U4-AU-ND -> ATMEGA32U4-AU-ND
- Y1: Description (none) -> Abracon LLC
Connections:
- net labels added: A3, D10, D7, D8, D9, RXI, TXO
- wire segments 109 -> 113
- no-connect marks 9 -> 5
Other:
- note added: "A0"
- note added: "A1"
- note added: "A2"
- note added: "A3"
- note added: "Connectors"
- note added: "D0/RXI"
- note added: "D1/TXO"
- note added: "D10"
- note added: "D2/SDA"
- note added: "D3/SCL"
- note added: "D4"
- note added: "D5"
- note added: "D6"
- note added: "D7"
- note added: "D8"
- note added: "D9"
- note removed: "Cover Mounting"
- note removed: "ISP Breakout"
- note removed: "PCB Mounting"
- note removed: "Sensing Board 1"
- note removed: "Sensing Board 2"
- moved on the sheet: BT1, D25, R2, SW2

Commit message: Symbol field corrections and additions
Parts:
- removed BT1: Battery_Cell, Connector_Wire:SolderWirePad_1x02_P3.81mm_Drill1mm, symbol Device:Battery_Cell
- removed D25: RED, Frequently_Used:LED_0805_2012Metric_HandSolder, symbol Frequently_Used:LED
- removed R2: 330, Frequently_Used:0805_2012Metric_HandSolder, symbol Frequently_Used:R
- removed SW2: SW_SPST, Connector_Wire:SolderWirePad_1x02_P3.81mm_Drill1mm, symbol Frequently_Used:SW_SPST
Connections:
- wire segments 113 -> 89
Changed lines of the file:
@@
 Comment4 ""
 $EndDescr
-$Comp
-L Device:Battery_Cell BT1
-U 1 1 5E9EA00B
-P 7850 5800
-F 0 "BT1" V 7595 5850 50  0000 C CNN
-F 1 "Battery_Cell" V 7686 5850 50  0000 C CNN
-F 2 "Connector_Wire:SolderWirePad_1x02_P3.81mm_Drill1mm" V 7850 5860 50  0001 C CNN
-F 3 "~" V 7850 5860 50  0001 C CNN
-	1    7850 5800
-	1    0    0    -1
-$EndComp
 Wire Wire Line
 	6400 4050 5900 4050
@@
 Wire Wire Line
 	6400 3850 5900 3850
-$Comp
-L Frequently_Used:GND #PWR020
-U 1 1 5E9CE7F6
-P 9500 5600
-F 0 "#PWR020" H 9500 5350 50  0001 C CNN
-F 1 "GND" H 9505 5427 50  0000 C CNN
-F 2 "" H 9500 5600 50  0001 C CNN
-F 3 "" H 9500 5600 50  0001 C CNN
-	1    9500 5600
-	1    0    0    -1
-$EndComp
 Wire Wire Line
 	4100 2300 4600 2300
@@
 Wire Wire Line
 	5900 3050 6400 3050
-$Comp
-L Frequently_Used:R R2
-U 1 1 5EA5504B
-P 10400 5150
-F 0 "R2" V 10500 5150 50  0000 C CNN
-F 1 "330" V 10300 5150 50  0000 C CNN
-F 2 "Frequently_Used:0805_2012Metric_HandSolder" V 10330 5150 50  0001 C CNN
-F 3 "~" H 10400 5150 50  0001 C CNN
-	1    10400 5150
-	0    -1   -1   0
-$EndComp
-$Comp
-L Frequently_Used:LED D25
-U 1 1 5EA55051
-P 10000 5150
-F 0 "D25" H 10000 5250 50  0000 C CNN
-F 1 "RED" H 10000 5050 50  0000 C CNN
-F 2 "Frequently_Used:LED_0805_2012Metric_HandSolder" H 10000 5150 50  0001 C CNN
-F 3 "https://www.we-online.de/katalog/datasheet/150080VS75000.pdf" H 10000 5150 50  0001 C CNN
-F 4 "Red 625nm LED Indication- Discrete 2V 0805 (2012 Metric)" H 10000 5150 50  0001 C CNN "Description"
-F 5 "732-4984-1-ND" H 10000 5150 50  0001 C CNN "Digikey Part No."
-F 6 "Würth Elektronik" H 10000 5150 50  0001 C CNN "Manufacturer Name"
-F 7 "150080RS75000" H 10000 5150 50  0001 C CNN "Manufacturer Part No."
-	1    10000 5150
-	1    0    0    -1
-$EndComp
-Wire Wire Line
-	10250 5150 10150 5150
-Wire Wire Line
-	10550 5150 10650 5150
 $Sheet
 S 8350 5100 500  800
@@
 F7 "BATGND" I L 8350 5800 50
 $EndSheet
-Wire Wire Line
-	7850 5600 8100 5600
-Wire Wire Line
-	8100 5600 8100 5700
-Wire Wire Line
-	8100 5700 8350 5700
-Wire Wire Line
-	7850 5900 8100 5900
-Wire Wire Line
-	8100 5900 8100 5800
-Wire Wire Line
-	8100 5800 8350 5800
-Wire Wire Line
-	8850 5450 9150 5450
-Wire Wire Line
-	10650 5150 10650 5450
-Wire Wire Line
-	9850 5150 9700 5150
-Wire Wire Line
-	8850 5550 9150 5550
-$Comp
-L Frequently_Used:SW_SPST SW2
-U 1 1 5EA8DC70
-P 9350 5150
-F 0 "SW2" H 9350 5385 50  0000 C CNN
-F 1 "SW_SPST" H 9350 5294 50  0000 C CNN
-F 2 "Connector_Wire:SolderWirePad_1x02_P3.81mm_Drill1mm" H 9350 5150 50  0001 C CNN
-F 3 "~" H 9350 5150 50  0001 C CNN
-	1    9350 5150
-	1    0    0    -1
-$EndComp
-Wire Wire Line
-	9550 5150 9550 5450
-Connection ~ 10650 5450
-Wire Wire Line
-	10650 5450 10800 5450
-Wire Wire Line
-	9700 5150 9700 5550
 $Comp
 L Frequently_Used:GND #PWR017
@@
 	1    0    0    -1
 $EndComp
-Wire Wire Line
-	9150 5450 9150 5150
-$Comp
-L Frequently_Used:PWR_FLAG #FLG01
-U 1 1 5EA63242
-P 9150 5600
-F 0 "#FLG01" H 9150 5675 50  0001 C CNN
-F 1 "PWR_FLAG" H 9150 5773 50  0000 C CNN
-F 2 "" H 9150 5600 50  0001 C CNN
-F 3 "~" H 9150 5600 50  0001 C CNN
-	1    9150 5600
-	-1   0    0    1
-$EndComp
-Connection ~ 9150 5550
-$Comp
-L Frequently_Used:PWR_FLAG #FLG02
-U 1 1 5EA650D8
-P 10200 5500
-F 0 "#FLG02" H 10200 5575 50  0001 C CNN
-F 1 "PWR_FLAG" H 10200 5673 50  0000 C CNN
-F 2 "" H 10200 5500 50  0001 C CNN
-F 3 "~" H 10200 5500 50  0001 C CNN
-	1    10200 5500
-	-1   0    0    1
-$EndComp
 Text Label 5950 3050 0    50   ~ 0
 HALLEFF4
 Wire Wire Line
 	3850 4050 3850 4150
-Wire Wire Line
-	9550 5450 10200 5450
-Wire Wire Line
-	10200 5500 10200 5450
-Connection ~ 10200 5450
-Wire Wire Line
-	10200 5450 10650 5450
-Wire Wire Line
-	9150 5600 9150 5550
-Wire Wire Line
-	9150 5550 9500 5550
-Wire Wire Line
-	9500 5600 9500 5550
-Connection ~ 9500 5550
-Wire Wire Line
-	9500 5550 9700 5550
-$Comp
-L Frequently_Used:+5V #PWR021
-U 1 1 5EB7A803
-P 10800 5400
-F 0 "#PWR021" H 10800 5250 50  0001 C CNN
-F 1 "+5V" H 10815 5573 50  0000 C CNN
-F 2 "" H 10800 5400 50  0001 C CNN
-F 3 "" H 10800 5400 50  0001 C CNN
-	1    10800 5400
-	1    0    0    -1
-$EndComp
-Wire Wire Line
-	10800 5400 10800 5450
 Text Label 5950 4050 0    50   ~ 0
 SRDATA
