File: Naquadah Generator Main/Naquadah Generator Main.sch (KiCad schematic (older format))
At the start: 15 parts, among them SW1 RESET, U1 ATmega32U4-AU, Y1 16MHz

Commit message: Adding Power Daughter Board
Parts:
- added SW?: MODE, Naquadah_Generator:PTS526SMG15SMTR2LFS_Hand_Solder, symbol Naquadah_Generator:PTS526_SMG15
- C1, C4, C5, C6: Digikey Part No. 1276-2931-1-ND -> (none); Source (none) -> Digikey; Source Part No. (none) -> 1276-2931-1-ND
- C2, C3: Digikey Part No. 399-1052-1-ND -> (none); Source (none) -> Digikey; Source Part No. (none) -> 399-1052-1-ND
- D23: Digikey Part No. 732-4986-1-ND -> (none); Source (none) -> Digikey; Source Part No. (none) -> 732-4986-1-ND
- D24: Digikey Part No. 732-4987-1-ND -> (none); Source (none) -> Digikey; Source Part No. (none) -> 732-4987-1-ND
- SW1: Digikey Part No. CKN12220-1-ND -> (none); Source (none) -> Digikey; Source Part No. (none) -> CKN12220-1-ND
- U1: Digikey Part No. ATMEGA32U4-AU-ND -> (none); Source (none) -> Digikey; Source Part No. (none) -> ATMEGA32U4-AU-ND
- Y1: Digikey Part No. 535-9103-1-ND -> (none); Source (none) -> Digikey; Source Part No. (none) -> 535-9103-1-ND
Connections:
- wire segments 89 -> 95
Changed lines of the file:
@@
 F 2 "Frequently_Used:0805_2012Metric_HandSolder" H 1738 4100 50  0001 C CNN
 F 3 "https://content.kemet.com/datasheets/KEM_C1003_C0G_SMD.pdf" H 1700 4250 50  0001 C CNN
-F 4 "399-1052-1-ND" H 1700 4250 50  0001 C CNN "Digikey Part No."
+F 4 "399-1052-1-ND" H 1700 4250 50  0001 C CNN "Source Part No."
 F 5 "Kemet" H 1700 4250 50  0001 C CNN "Manufacturer Name"
 F 6 "C0603C180J5GACTU" H 1700 4250 50  0001 C CNN "Manufacturer Part No."
+F 7 "Digikey" H 1700 4250 50  0001 C CNN "Source"
 	1    1700 4250
 	0    1    1    0
@@
 F 2 "Frequently_Used:0805_2012Metric_HandSolder" H 1738 3800 50  0001 C CNN
 F 3 "https://content.kemet.com/datasheets/KEM_C1003_C0G_SMD.pdf" H 1700 3950 50  0001 C CNN
-F 4 "399-1052-1-ND" H 1700 3950 50  0001 C CNN "Digikey Part No."
+F 4 "399-1052-1-ND" H 1700 3950 50  0001 C CNN "Source Part No."
 F 5 "Kemet" H 1700 3950 50  0001 C CNN "Manufacturer Name"
 F 6 "C0603C180J5GACTU" H 1700 3950 50  0001 C CNN "Manufacturer Part No."
+F 7 "Digikey" H 1700 3950 50  0001 C CNN "Source"
 	1    1700 3950
 	0    1    1    0
@@
 F 2 "Naquadah_Generator:Oscillator_ABM3-16.000MHZ-B2-T" H 2000 4100 50  0001 C CNN
 F 3 "https://abracon.com/Resonators/abm3.pdf" H 2000 4100 50  0001 C CNN
-F 4 "535-9103-1-ND" H 2000 4100 50  0001 C CNN "Digikey Part No."
+F 4 "535-9103-1-ND" H 2000 4100 50  0001 C CNN "Source Part No."
 F 5 "Abracon " H 2000 4100 50  0001 C CNN "Manufacturer Name"
 F 6 "ABM3-16.000MHZ-B2-T" H 2000 4100 50  0001 C CNN "Manufacturer Part No."
 F 7 "Abracon LLC" H 2000 4100 50  0001 C CNN "Description"
+F 8 "Digikey" H 2000 4100 50  0001 C CNN "Source"
 	1    2000 4100
 	0    1    1    0
@@
 F 3 "https://media.digikey.com/pdf/Data%20Sheets/Samsung%20PDFs/CL_Series_MLCC_ds.pdf" H 2500 1250 50  0001 C CNN
 F 4 "1µF ±10% 16V Ceramic Capacitor X7R 0805 (2012 Metric)" H 2500 1250 50  0001 C CNN "Description"
-F 5 "1276-2931-1-ND" H 2500 1250 50  0001 C CNN "Digikey Part No."
+F 5 "1276-2931-1-ND" H 2500 1250 50  0001 C CNN "Source Part No."
 F 6 "Samsung Electro-Mechanics" H 2500 1250 50  0001 C CNN "Manufacturer Name"
 F 7 "CL21B105KOFNNWE" H 2500 1250 50  0001 C CNN "Manufacturer Part No."
+F 8 "Digikey" H 2500 1250 50  0001 C CNN "Source"
 	1    2500 1250
 	1    0    0    -1
@@
 F 3 "https://media.digikey.com/pdf/Data%20Sheets/Samsung%20PDFs/CL_Series_MLCC_ds.pdf" H 2000 1250 50  0001 C CNN
 F 4 "1µF ±10% 16V Ceramic Capacitor X7R 0805 (2012 Metric)" H 2000 1250 50  0001 C CNN "Description"
-F 5 "1276-2931-1-ND" H 2000 1250 50  0001 C CNN "Digikey Part No."
+F 5 "1276-2931-1-ND" H 2000 1250 50  0001 C CNN "Source Part No."
 F 6 "Samsung Electro-Mechanics" H 2000 1250 50  0001 C CNN "Manufacturer Name"
 F 7 "CL21B105KOFNNWE" H 2000 1250 50  0001 C CNN "Manufacturer Part No."
+F 8 "Digikey" H 2000 1250 50  0001 C CNN "Source"
 	1    2000 1250
 	1    0    0    -1
@@
 F 2 "Naquadah_Generator:PTS526SMG15SMTR2LFS_Hand_Solder" H 1850 3300 50  0001 C CNN
 F 3 "https://dznh3ojzb2azq.cloudfront.net/products/Tactile/PTS526/documents/datasheet.pdf" H 1850 3300 50  0001 C CNN
-F 4 "CKN12220-1-ND" H 1850 3100 50  0001 C CNN "Digikey Part No."
+F 4 "CKN12220-1-ND" H 1850 3100 50  0001 C CNN "Source Part No."
 F 5 "C&K" H 1850 3100 50  0001 C CNN "Manufacturer Name"
 F 6 "PTS526 SM15 SMTR2 LFS" H 1850 3100 50  0001 C CNN "Manufacturer Part No."
+F 7 "Digikey" H 1850 3100 50  0001 C CNN "Source"
 	1    1850 3100
 	0    -1   -1   0
@@
 F 3 "https://media.digikey.com/pdf/Data%20Sheets/Samsung%20PDFs/CL_Series_MLCC_ds.pdf" H 1000 1250 50  0001 C CNN
 F 4 "1µF ±10% 16V Ceramic Capacitor X7R 0805 (2012 Metric)" H 1000 1250 50  0001 C CNN "Description"
-F 5 "1276-2931-1-ND" H 1000 1250 50  0001 C CNN "Digikey Part No."
+F 5 "1276-2931-1-ND" H 1000 1250 50  0001 C CNN "Source Part No."
 F 6 "Samsung Electro-Mechanics" H 1000 1250 50  0001 C CNN "Manufacturer Name"
 F 7 "CL21B105KOFNNWE" H 1000 1250 50  0001 C CNN "Manufacturer Part No."
+F 8 "Digikey" H 1000 1250 50  0001 C CNN "Source"
 	1    1000 1250
 	1    0    0    -1
@@
 F 3 "https://media.digikey.com/pdf/Data%20Sheets/Samsung%20PDFs/CL_Series_MLCC_ds.pdf" H 1500 1250 50  0001 C CNN
 F 4 "1µF ±10% 16V Ceramic Capacitor X7R 0805 (2012 Metric)" H 1500 1250 50  0001 C CNN "Description"
-F 5 "1276-2931-1-ND" H 1500 1250 50  0001 C CNN "Digikey Part No."
+F 5 "1276-2931-1-ND" H 1500 1250 50  0001 C CNN "Source Part No."
 F 6 "Samsung Electro-Mechanics" H 1500 1250 50  0001 C CNN "Manufacturer Name"
 F 7 "CL21B105KOFNNWE" H 1500 1250 50  0001 C CNN "Manufacturer Part No."
+F 8 "Digikey" H 1500 1250 50  0001 C CNN "Source"
 	1    1500 1250
 	1    0    0    -1
@@
 F 3 "https://www.we-online.de/katalog/datasheet/150080VS75000.pdf" H 7400 1050 50  0001 C CNN
 F 4 "Green 570nm LED Indication - Discrete 2V 0805 (2012 Metric)" H 7400 1050 50  0001 C CNN "Description"
-F 5 "732-4986-1-ND" H 7400 1050 50  0001 C CNN "Digikey Part No."
+F 5 "732-4986-1-ND" H 7400 1050 50  0001 C CNN "Source Part No."
 F 6 "Würth Elektronik" H 7400 1050 50  0001 C CNN "Manufacturer Name"
 F 7 "150080VS75000" H 7400 1050 50  0001 C CNN "Manufacturer Part No."
+F 8 "Digikey" H 7400 1050 50  0001 C CNN "Source"
 	1    7400 1050
 	0    1    1    0
@@
 F 3 "https://www.we-online.de/katalog/datasheet/150080VS75000.pdf" H 8000 1050 50  0001 C CNN
 F 4 "	Yellow 590nm LED Indication - Discrete 2V 0805 (2012 Metric)" H 8000 1050 50  0001 C CNN "Description"
-F 5 "732-4987-1-ND" H 8000 1050 50  0001 C CNN "Digikey Part No."
+F 5 "732-4987-1-ND" H 8000 1050 50  0001 C CNN "Source Part No."
 F 6 "Würth Elektronik" H 8000 1050 50  0001 C CNN "Manufacturer Name"
 F 7 "150080YS75000" H 8000 1050 50  0001 C CNN "Manufacturer Part No."
+F 8 "Digikey" H 8000 1050 50  0001 C CNN "Source"
 	1    8000 1050
 	0    1    1    0
@@
 F 2 "Package_QFP:TQFP-44_10x10mm_P0.8mm" H 5250 400 50  0001 C CIN
 F 3 "http://ww1.microchip.com/downloads/en/DeviceDoc/Atmel-7766-8-bit-AVR-ATmega16U4-32U4_Datasheet.pdf" H 5250 2650 50  0001 C CNN
-F 4 "ATMEGA32U4-AU-ND" H 5250 2650 50  0001 C CNN "Digikey Part No."
+F 4 "ATMEGA32U4-AU-ND" H 5250 2650 50  0001 C CNN "Source Part No."
 F 5 "Microchip Technology" H 5250 2650 50  0001 C CNN "Manufacturer Name"
 F 6 "ATMEGA32U4-AU" H 5250 2650 50  0001 C CNN "Manufacturer Part No."
 F 7 "ATmega Microcontroller IC 8-Bit 16MHz 32KB (16K x 16) FLASH 44-TQFP (10x10)" H 5250 2650 50  0001 C CNN "Description"
+F 8 "Digikey" H 5250 2650 50  0001 C CNN "Source"
 	1    5250 2650
 	1    0    0    -1
@@
 Text Notes 6500 2650 0    50   ~ 0
 D1/TXO
+$Comp
+L Naquadah_Generator:PTS526_SMG15 SW?
+U 1 1 5F15836F
+P 8400 2500
+F 0 "SW?" V 8500 2850 50  0000 R CNN
+F 1 "MODE" V 8300 2850 50  0000 R CNN
+F 2 "Naquadah_Generator:PTS526SMG15SMTR2LFS_Hand_Solder" H 8400 2700 50  0001 C CNN
+F 3 "https://dznh3ojzb2azq.cloudfront.net/products/Tactile/PTS526/documents/datasheet.pdf" H 8400 2700 50  0001 C CNN
+F 4 "CKN12220-1-ND" H 8400 2500 50  0001 C CNN "Source Part No."
+F 5 "C&K" H 8400 2500 50  0001 C CNN "Manufacturer Name"
+F 6 "PTS526 SM15 SMTR2 LFS" H 8400 2500 50  0001 C CNN "Manufacturer Part No."
+F 7 "Digikey" H 8400 2500 50  0001 C CNN "Source"
+	1    8400 2500
+	0    -1   -1   0
+$EndComp
+Wire Wire Line
+	8400 2300 8500 2300
+Wire Wire Line
+	8400 2700 8500 2700
+Wire Wire Line
+	8500 2700 8500 2800
+Connection ~ 8500 2700
+Wire Wire Line
+	8500 2700 8600 2700
+Wire Wire Line
+	8500 2300 8500 1850
+Connection ~ 8500 2300
+Wire Wire Line
+	8500 2300 8600 2300
+Text Label 8500 2200 1    50   ~ 0
+MODESEL
+$Comp
+L Frequently_Used:GND #PWR?
+U 1 1 5F16B284
+P 8500 2800
+F 0 "#PWR?" H 8500 2550 50  0001 C CNN
+F 1 "GND" H 8500 2650 50  0000 C CNN
+F 2 "" H 8500 2800 50  0001 C CNN
+F 3 "" H 8500 2800 50  0001 C CNN
+	1    8500 2800
+	1    0    0    -1
+$EndComp
 $EndSCHEMATC

Commit message: Before updating to two switches
Parts:
- gave numbers to parts that had none: 1
Changed lines of the file:
@@
 D1/TXO
 $Comp
-L Naquadah_Generator:PTS526_SMG15 SW?
+L Naquadah_Generator:PTS526_SMG15 SW2
 U 1 1 5F15836F
 P 8400 2500
-F 0 "SW?" V 8500 2850 50  0000 R CNN
+F 0 "SW2" V 8500 2850 50  0000 R CNN
 F 1 "MODE" V 8300 2850 50  0000 R CNN
 F 2 "Naquadah_Generator:PTS526SMG15SMTR2LFS_Hand_Solder" H 8400 2700 50  0001 C CNN
@@
 MODESEL
 $Comp
-L Frequently_Used:GND #PWR?
+L Frequently_Used:GND #PWR012
 U 1 1 5F16B284
 P 8500 2800
-F 0 "#PWR?" H 8500 2550 50  0001 C CNN
+F 0 "#PWR012" H 8500 2550 50  0001 C CNN
 F 1 "GND" H 8500 2650 50  0000 C CNN
 F 2 "" H 8500 2800 50  0001 C CNN

Commit message: Updates
Parts:
- removed SW2: MODE, Naquadah_Generator:PTS526SMG15SMTR2LFS_Hand_Solder, symbol Naquadah_Generator:PTS526_SMG15
Connections:
- net labels added: READY
- net labels removed: D8
- wire segments 95 -> 91
Other:
- moved on the sheet: SW1

Commit message: Move libraries and added configuration path.
Moved Li-Ion library to common KiCad library.  Added variables to configuration paths to reference my KiCad libraries.  Moved all 3D components to my common library.
Parts:
- C1, C2, C3, C4, C5, C6, C7: footprint Frequently_Used:0805_2012Metric_HandSolder -> FrequentlyUsed:0805_2012Metric_HandSolder; symbol Frequently_Used:C -> Frequently_Used_LE:C
- D23, D24: footprint Frequently_Used:LED_0805_2012Metric_HandSolder -> FrequentlyUsed:LED_0805_2012Metric_HandSolder; symbol Frequently_Used:LED -> Frequently_Used_LE:LED
- R1, R4, R9: footprint Frequently_Used:0805_2012Metric_HandSolder -> FrequentlyUsed:0805_2012Metric_HandSolder; symbol Frequently_Used:R -> Frequently_Used_LE:R
- Y1: symbol Frequently_Used:Crystal -> Frequently_Used_LE:Crystal
Changed lines of the file:
@@
 	6550 3000 7050 3000
 $Comp
-L Frequently_Used:GND #PWR017
+L Frequently_Used_LE:GND #PWR017
 U 1 1 5EA1BAA4
 P 4500 4100
@@
 	4500 2100 4500 2200
 $Comp
-L Frequently_Used:GND #PWR016
+L Frequently_Used_LE:GND #PWR016
 U 1 1 5EDBAB65
 P 4500 2200
@@
 UCAP
 $Comp
-L Frequently_Used:C C3
+L Frequently_Used_LE:C C3
 U 1 1 5EDC471D
 P 2450 4150
 F 0 "C3" V 2500 4100 50  0000 R CNN
 F 1 "18pF" V 2500 4200 50  0000 L CNN
-F 2 "Frequently_Used:0805_2012Metric_HandSolder" H 2488 4000 50  0001 C CNN
+F 2 "FrequentlyUsed:0805_2012Metric_HandSolder" H 2488 4000 50  0001 C CNN
 F 3 "https://content.kemet.com/datasheets/KEM_C1003_C0G_SMD.pdf" H 2450 4150 50  0001 C CNN
 F 4 "399-1052-1-ND" H 2450 4150 50  0001 C CNN "Source Part No."
@@
 $EndComp
 $Comp
-L Frequently_Used:C C2
+L Frequently_Used_LE:C C2
 U 1 1 5EDC72C2
 P 2450 3850
 F 0 "C2" V 2400 3800 50  0000 R CNN
 F 1 "18pF" V 2400 3900 50  0000 L CNN
-F 2 "Frequently_Used:0805_2012Metric_HandSolder" H 2488 3700 50  0001 C CNN
+F 2 "FrequentlyUsed:0805_2012Metric_HandSolder" H 2488 3700 50  0001 C CNN
 F 3 "https://content.kemet.com/datasheets/KEM_C1003_C0G_SMD.pdf" H 2450 3850 50  0001 C CNN
 F 4 "399-1052-1-ND" H 2450 3850 50  0001 C CNN "Source Part No."
@@
 $EndComp
 $Comp
-L Frequently_Used:Crystal Y1
+L Frequently_Used_LE:Crystal Y1
 U 1 1 5EDC870C
 P 2750 4000
@@
 Connection ~ 4500 1500
 $Comp
-L Frequently_Used:VBUS #PWR015
+L Frequently_Used_LE:VBUS #PWR015
 U 1 1 5EE32C9A
 P 4500 1400
@@
 	4500 1100 4500 1000
 $Comp
-L Frequently_Used:+5V #PWR014
+L Frequently_Used_LE:+5V #PWR014
 U 1 1 5EE39D3A
 P 4500 1000
@@
 $EndComp
 $Comp
-L Frequently_Used:+5V #PWR010
+L Frequently_Used_LE:+5V #PWR010
 U 1 1 5EE3F918
 P 3650 1000
@@
 $EndComp
 $Comp
-L Frequently_Used:GND #PWR011
+L Frequently_Used_LE:GND #PWR011
 U 1 1 5EE3FE38
 P 3650 1500
@@
 $EndComp
 $Comp
-L Frequently_Used:C C7
+L Frequently_Used_LE:C C7
 U 1 1 5EE403A0
 P 3650 1250
 F 0 "C7" H 3700 1350 50  0000 L CNN
 F 1 "0.1uF" H 3700 1150 50  0000 L CNN
-F 2 "Frequently_Used:0805_2012Metric_HandSolder" H 3688 1100 50  0001 C CNN
+F 2 "FrequentlyUsed:0805_2012Metric_HandSolder" H 3688 1100 50  0001 C CNN
 F 3 "~" H 3650 1250 50  0001 C CNN
 	1    3650 1250
@@
 	3650 1000 3650 1100
 $Comp
-L Frequently_Used:+5V #PWR08
+L Frequently_Used_LE:+5V #PWR08
 U 1 1 5EE46087
 P 3150 1000
@@
 $EndComp
 $Comp
-L Frequently_Used:GND #PWR09
+L Frequently_Used_LE:GND #PWR09
 U 1 1 5EE4608D
 P 3150 1500
@@
 $EndComp
 $Comp
-L Frequently_Used:C C6
+L Frequently_Used_LE:C C6
 U 1 1 5EE46093
 P 3150 1250
 F 0 "C6" H 3200 1350 50  0000 L CNN
 F 1 "1.0uF" H 3200 1150 50  0000 L CNN
-F 2 "Frequently_Used:0805_2012Metric_HandSolder" H 3188 1100 50  0001 C CNN
+F 2 "FrequentlyUsed:0805_2012Metric_HandSolder" H 3188 1100 50  0001 C CNN
 F 3 "https://media.digikey.com/pdf/Data%20Sheets/Samsung%20PDFs/CL_Series_MLCC_ds.pdf" H 3150 1250 50  0001 C CNN
 F 4 "1µF ±10% 16V Ceramic Capacitor X7R 0805 (2012 Metric)" H 3150 1250 50  0001 C CNN "Description"
@@
 	3150 1000 3150 1100
 $Comp
-L Frequently_Used:GND #PWR07
+L Frequently_Used_LE:GND #PWR07
 U 1 1 5EE499D3
 P 2650 1500
@@
 $EndComp
 $Comp
-L Frequently_Used:C C5
+L Frequently_Used_LE:C C5
 U 1 1 5EE499D9
 P 2650 1250
 F 0 "C5" H 2700 1350 50  0000 L CNN
 F 1 "1.0uF" H 2700 1150 50  0000 L CNN
-F 2 "Frequently_Used:0805_2012Metric_HandSolder" H 2688 1100 50  0001 C CNN
+F 2 "FrequentlyUsed:0805_2012Metric_HandSolder" H 2688 1100 50  0001 C CNN
 F 3 "https://media.digikey.com/pdf/Data%20Sheets/Samsung%20PDFs/CL_Series_MLCC_ds.pdf" H 2650 1250 50  0001 C CNN
 F 4 "1µF ±10% 16V Ceramic Capacitor X7R 0805 (2012 Metric)" H 2650 1250 50  0001 C CNN "Description"
@@
 	2650 900  2650 1100
 $Comp
-L Frequently_Used:GND #PWR03
+L Frequently_Used_LE:GND #PWR03
 U 1 1 5EE4D88E
 P 1650 1500
@@
 	1650 1000 1650 1100
 $Comp
-L Frequently_Used:VBUS #PWR02
+L Frequently_Used_LE:VBUS #PWR02
 U 1 1 5EE4F542
 P 1650 1000
@@
 UCAP
 $Comp
-L Frequently_Used:GND #PWR06
+L Frequently_Used_LE:GND #PWR06
 U 1 1 5EE53061
 P 2150 1500
@@
 nRESET
 $Comp
-L Frequently_Used:R R1
+L Frequently_Used_LE:R R1
 U 1 1 5EE7AB0D
 P 2650 2450
 F 0 "R1" V 2550 2450 50  0000 C CNN
 F 1 "10k" V 2750 2450 50  0000 C CNN
-F 2 "Frequently_Used:0805_2012Metric_HandSolder" V 2580 2450 50  0001 C CNN
+F 2 "FrequentlyUsed:0805_2012Metric_HandSolder" V 2580 2450 50  0001 C CNN
 F 3 "~" H 2650 2450 50  0001 C CNN
 	1    2650 2450
@@
 $EndComp
 $Comp
-L Frequently_Used:+5V #PWR04
+L Frequently_Used_LE:+5V #PWR04
 U 1 1 5EE7B8E3
 P 2650 2200
@@
 Connection ~ 2650 2650
 $Comp
-L Frequently_Used:GND #PWR05
+L Frequently_Used_LE:GND #PWR05
 U 1 1 5EE8456D
 P 2650 3250
@@
 RXLED
 $Comp
-L Frequently_Used:C C1
+L Frequently_Used_LE:C C1
 U 1 1 5EE4D894
 P 1650 1250
 F 0 "C1" H 1700 1350 50  0000 L CNN
 F 1 "1.0uF" H 1700 1150 50  0000 L CNN
-F 2 "Frequently_Used:0805_2012Metric_HandSolder" H 1688 1100 50  0001 C CNN
+F 2 "FrequentlyUsed:0805_2012Metric_HandSolder" H 1688 1100 50  0001 C CNN
 F 3 "https://media.digikey.com/pdf/Data%20Sheets/Samsung%20PDFs/CL_Series_MLCC_ds.pdf" H 1650 1250 50  0001 C CNN
 F 4 "1µF ±10% 16V Ceramic Capacitor X7R 0805 (2012 Metric)" H 1650 1250 50  0001 C CNN "Description"
@@
 $EndComp
 $Comp
-L Frequently_Used:C C4
+L Frequently_Used_LE:C C4
 U 1 1 5EE53067
 P 2150 1250
 F 0 "C4" H 2200 1350 50  0000 L CNN
 F 1 "1.0uF" H 2200 1150 50  0000 L CNN
-F 2 "Frequently_Used:0805_2012Metric_HandSolder" H 2188 1100 50  0001 C CNN
+F 2 "FrequentlyUsed:0805_2012Metric_HandSolder" H 2188 1100 50  0001 C CNN
 F 3 "https://media.digikey.com/pdf/Data%20Sheets/Samsung%20PDFs/CL_Series_MLCC_ds.pdf" H 2150 1250 50  0001 C CNN
 F 4 "1µF ±10% 16V Ceramic Capacitor X7R 0805 (2012 Metric)" H 2150 1250 50  0001 C CNN "Description"
@@
 	2200 4000 2200 3850
 $Comp
-L Frequently_Used:GND #PWR01
+L Frequently_Used_LE:GND #PWR01
 U 1 1 5ECBCDF9
 P 2000 4100
@@
 	8000 1050 8000 1000
 $Comp
-L Frequently_Used:+5V #PWR0103
+L Frequently_Used_LE:+5V #PWR0103
 U 1 1 5EDE6C2F
 P 8000 1000
@@
 $EndComp
 $Comp
-L Frequently_Used:R R4
+L Frequently_Used_LE:R R4
 U 1 1 5EDE0168
 P 8000 1550
 F 0 "R4" V 7900 1550 50  0000 C CNN
 F 1 "1k" V 8100 1550 50  0000 C CNN
-F 2 "Frequently_Used:0805_2012Metric_HandSolder" V 7930 1550 50  0001 C CNN
+F 2 "FrequentlyUsed:0805_2012Metric_HandSolder" V 7930 1550 50  0001 C CNN
 F 3 "~" H 8000 1550 50  0001 C CNN
 	1    8000 1550
@@
 $EndComp
 $Comp
-L Frequently_Used:LED D23
+L Frequently_Used_LE:LED D23
 U 1 1 5EDE016E
 P 8000 1200
 F 0 "D23" H 8000 1100 50  0000 C CNN
 F 1 "GREEN" H 8000 1300 50  0000 C CNN
-F 2 "Frequently_Used:LED_0805_2012Metric_HandSolder" H 8000 1200 50  0001 C CNN
+F 2 "FrequentlyUsed:LED_0805_2012Metric_HandSolder" H 8000 1200 50  0001 C CNN
 F 3 "https://www.we-online.de/katalog/datasheet/150080VS75000.pdf" H 8000 1200 50  0001 C CNN
 F 4 "Green 570nm LED Indication - Discrete 2V 0805 (2012 Metric)" H 8000 1200 50  0001 C CNN "Description"
@@
 	8600 1050 8600 1000
 $Comp
-L Frequently_Used:+5V #PWR0104
+L Frequently_Used_LE:+5V #PWR0104
 U 1 1 5EDF2F7E
 P 8600 1000
@@
 $EndComp
 $Comp
-L Frequently_Used:R R9
+L Frequently_Used_LE:R R9
 U 1 1 5EDF2F84
 P 8600 1550
 F 0 "R9" V 8500 1550 50  0000 C CNN
 F 1 "1k" V 8700 1550 50  0000 C CNN
-F 2 "Frequently_Used:0805_2012Metric_HandSolder" V 8530 1550 50  0001 C CNN
+F 2 "FrequentlyUsed:0805_2012Metric_HandSolder" V 8530 1550 50  0001 C CNN
 F 3 "~" H 8600 1550 50  0001 C CNN
 	1    8600 1550
@@
 $EndComp
 $Comp
-L Frequently_Used:LED D24
+L Frequently_Used_LE:LED D24
 U 1 1 5EDF2F8A
 P 8600 1200
 F 0 "D24" H 8600 1100 50  0000 C CNN
 F 1 "YELLOW" H 8600 1300 50  0000 C CNN
-F 2 "Frequently_Used:LED_0805_2012Metric_HandSolder" H 8600 1200 50  0001 C CNN
+F 2 "FrequentlyUsed:LED_0805_2012Metric_HandSolder" H 8600 1200 50  0001 C CNN
 F 3 "https://www.we-online.de/katalog/datasheet/150080VS75000.pdf" H 8600 1200 50  0001 C CNN
 F 4 "	Yellow 590nm LED Indication - Discrete 2V 0805 (2012 Metric)" H 8600 1200 50  0001 C CNN "Description"
@@
 	7300 3200 6550 3200
 $Comp
-L Frequently_Used:GND #PWR0105
+L Frequently_Used_LE:GND #PWR0105
 U 1 1 5EE11E5E
 P 7300 3300
