File: Naquadah Generator Main/Naquadah Generator Main.kicad_pcb (KiCad board)
At the start: 2 copper layers, 83 parts, among them J1 Conn_01x03, J2 Conn_01x02, J3 Conn_01x02, J4 Conn_01x02, J5 Conn_01x02, J6 Conn_01x02, Q1 BC337, Q2 BC337, Q3 BC337, Q4 BC337, Q5 BC337, Q6 BC337, Q7 BC337, Q8 BC337, SW1 SW_SPST, U1 74HC595, U2 74HC595, U3 AH1815-P, U4 AH1815-P, U5 AH1815-P, U6 AH1815-P

Commit message: Before changing BOM
Parts:
- removed C1, C2, C3, C4: 50n, Capacitor_THT:CP_Radial_Tantal_D5.5mm_P5.00mm
- removed R28, R29, R30, R31: 50K, Resistor_THT:R_Axial_DIN0207_L6.3mm_D2.5mm_P10.16mm_Horizontal
- removed U3, U4, U5, U6: AH1815-P, Package_TO_SOT_SMD:SC-59_Handsoldering
- added J101: HallSensor_Conn_T4, Connector_JST:JST_SH_SM04B-SRSS-TB_1x04-1MP_P1.00mm_Horizontal, F.Cu at (235.2, 121.1)
- added J102: HallSensor_Conn_T4, Connector_JST:JST_SH_SM04B-SRSS-TB_1x04-1MP_P1.00mm_Horizontal, F.Cu at (244.1, 121.1)
- moved R19 10.2 mm to (201.9, 79.9)
- moved D15 10.2 mm to (208.7, 73.7)
- moved D17 8.28 mm to (211.0, 110.5)
- moved R21 8.28 mm to (204.3, 104.8)
- moved J2 7.53 mm to (211.3, 94.4)
- moved D12 6.86 mm to (200.3, 56.6)
- moved R15 6.86 mm to (193.6, 62.3)
- moved D8 5.37 mm to (189.9, 43.1)
- moved R10 5.37 mm to (183.3, 48.6)
- moved D3 4.99 mm to (101.1, 155.5)
- moved R4 4.99 mm to (108.0, 149.7)
- moved D11 4.56 mm to (204.8, 128.1)
- moved R14 4.56 mm to (198.1, 122.1)
- moved R7 4.44 mm to (170.7, 38.0)
- moved D6 4.44 mm to (177.3, 32.4)
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- renumbered U2 to U102
Connections:
- A1 pad 10: Net-(A1-Pad10) -> (no net)
- A1 pad 11: Net-(A1-Pad11) -> (no net)
- A1 pad 12: Net-(A1-Pad12) -> (no net)
- A1 pad 13: Net-(A1-Pad13) -> (no net)
- A1 pad 17: Net-(A1-Pad17) -> (no net)
- A1 pad 18: Net-(A1-Pad18) -> (no net)
- A1 pad 19: Net-(A1-Pad19) -> (no net)
- A1 pad 20: Net-(A1-Pad20) -> (no net)
- A1 pad 22: Net-(A1-Pad22) -> (no net)
- A1 pad 23: Net-(A1-Pad23) -> (no net)
- A1 pad 24: Net-(A1-Pad24) -> (no net)
- A1 pad 25: Net-(A1-Pad25) -> (no net)
- A1 pad 26: Net-(A1-Pad26) -> (no net)
- A1 pad 27: Net-(A1-Pad27) -> (no net)
- A1 pad 28: Net-(A1-Pad28) -> (no net)
- A1 pad 29: Net-(A1-Pad29) -> (no net)
- A1 pad 30: Net-(A1-Pad30) -> (no net)
- A1 pad 31: Net-(A1-Pad31) -> (no net)
- A1 pad 32: Net-(A1-Pad32) -> (no net)
- A1 pad 33: Net-(A1-Pad33) -> (no net)
- A1 pad 34: Net-(A1-Pad34) -> (no net)
- A1 pad 8: Net-(A1-Pad8) -> (no net)
- A1 pad 9: Net-(A1-Pad9) -> (no net)
- R10 pad 1: 5V -> +5V
- R11 pad 1: 5V -> +5V
- R12 pad 1: 5V -> +5V
- R14 pad 1: 5V -> +5V
- R15 pad 1: 5V -> +5V
- R16 pad 1: 5V -> +5V
- R17 pad 1: 5V -> +5V
- R19 pad 1: 5V -> +5V
- R20 pad 1: 5V -> +5V
- R21 pad 1: 5V -> +5V
- R22 pad 1: 5V -> +5V
- R24 pad 1: 5V -> +5V
- R25 pad 1: 5V -> +5V
- R26 pad 1: 5V -> +5V
- R27 pad 1: 5V -> +5V
- R4 pad 1: 5V -> +5V
- R5 pad 1: 5V -> +5V
- R6 pad 1: 5V -> +5V
- R7 pad 1: 5V -> +5V
- R9 pad 1: 5V -> +5V
- U1 pad 15: Net-(U1-Pad15) -> (no net)
- U1 pad 2: Net-(U1-Pad2) -> (no net)
- U1 pad 3: Net-(U1-Pad3) -> (no net)
- U1 pad 4: Net-(U1-Pad4) -> (no net)
- U1 pad 5: Net-(U1-Pad5) -> (no net)
- U1 pad 6: Net-(U1-Pad6) -> (no net)
- U1 pad 7: Net-(U1-Pad7) -> (no net)
- U1 pad 9: Net-(U1-Pad9) -> (no net)

Commit message: Partial Update
Parts:
- removed J101, J102: HallSensor_Conn_T4, Connector_JST:JST_SH_SM04B-SRSS-TB_1x04-1MP_P1.00mm_Horizontal
- removed R32, R33, R34: 2.7k, Resistor_THT:R_Axial_DIN0207_L6.3mm_D2.5mm_P10.16mm_Horizontal
- removed the U1 at (122.0, 108.0)
- added C1: 1.0uF, Frequently_Used:0805_2012Metric_HandSolder, F.Cu at (178.8, 81.8)
- added C2: 22pF, Frequently_Used:0805_2012Metric_HandSolder, F.Cu at (179.0, 71.0)
- added C3: 22pF, Frequently_Used:0805_2012Metric_HandSolder, F.Cu at (175.0, 71.0)
- added C4: 1.0uF, Frequently_Used:0805_2012Metric_HandSolder, F.Cu at (169.8, 90.2)
- added C5: 1.0uF, Frequently_Used:0805_2012Metric_HandSolder, F.Cu at (183.8, 81.8)
- added C6: 1.0uF, Frequently_Used:0805_2012Metric_HandSolder, F.Cu at (178.5, 86.2)
- added C7: 0.1uF, Frequently_Used:0805_2012Metric_HandSolder, F.Cu at (183.0, 86.8)
- added J7: Conn_01x02, Connector_Wire:SolderWirePad_1x02_P3.81mm_Drill1.2mm, F.Cu at (232.4, 13.3)
- added R28: 330, Frequently_Used:0805_2012Metric_HandSolder, F.Cu at (117.0, 30.2)
- added R29: 2.7k, Frequently_Used:0805_2012Metric_HandSolder, F.Cu at (232.3, 22.9)
- added R30: 2.7k, Frequently_Used:0805_2012Metric_HandSolder, F.Cu at (216.4, 27.2)
- added R31: 2.7k, Frequently_Used:0805_2012Metric_HandSolder, F.Cu at (241.2, 12.2)
- added SW2: SW_SPST, Connector_Wire:SolderWirePad_1x02_P3.81mm_Drill1mm, F.Cu at (207.8, 13.0)
- added U2: 74HC595, Package_DIP:DIP-16_W7.62mm, F.Cu at (123.2, 72.8)
- added Y1: 16MHz, Naquadah_Generator:Oscillator_ABM3-16.000MHZ-B2-T, F.Cu at (177.5, 67.3)
- J1: value Conn_01x03 -> State_Sensing_Conn; footprint Connector_Wire:SolderWirePad_1x03_P3.81mm_Drill1.2mm -> Naquadah_Generator:State_Sensing_Mother_Board_JST_Conn
- J2: value Conn_01x02 -> State_Sensing_Conn; footprint Connector_Wire:SolderWirePad_1x02_P3.81mm_Drill1.2mm -> Naquadah_Generator:State_Sensing_Mother_Board_JST_Conn
- Q1, Q2, Q3, Q4, Q5, Q6, Q7, Q8: value BC337 -> BCW65ALT1G; footprint Package_TO_SOT_THT:TO-92_Inline -> Package_TO_SOT_SMD:SOT-23
- R1: value 330 -> 10k; footprint Resistor_THT:R_Axial_DIN0207_L6.3mm_D2.5mm_P10.16mm_Horizontal -> Frequently_Used:0805_2012Metric_HandSolder
- R10, R11, R12, R15, R16, R17, R2, R20, R21, R22, R25, R26, R27, R5, R6, R7: footprint Resistor_THT:R_Axial_DIN0207_L6.3mm_D2.5mm_P10.16mm_Horizontal -> Frequently_Used:0805_2012Metric_HandSolder
- R13, R18, R23, R3, R8: value 2.7k -> 330; footprint Resistor_THT:R_Axial_DIN0207_L6.3mm_D2.5mm_P10.16mm_Horizontal -> Frequently_Used:0805_2012Metric_HandSolder
- R14, R19, R24, R4, R9: value 330 -> 2.7k; footprint Resistor_THT:R_Axial_DIN0207_L6.3mm_D2.5mm_P10.16mm_Horizontal -> Frequently_Used:0805_2012Metric_HandSolder
- SW1: value SW_SPST -> RESET; footprint Connector_Wire:SolderWirePad_1x02_P3.81mm_Drill1mm -> Naquadah_Generator:PTS526SMG15SMTR2LFS_Hand_Solder
- U1: renamed from A1; value ArduinoProMini -> ATmega32U4-AU; footprint Arduino:Arduino-Pro-Mini -> Package_QFP:TQFP-44_10x10mm_P0.8mm
- moved R22 141.5 mm to (212.5, 115.8)
- moved R20 135.5 mm to (208.8, 79.0)
- moved R27 134.7 mm to (162.0, 158.5)
- moved R25 133.8 mm to (163.0, 29.5)
- moved R21 131.3 mm to (73.2, 112.0)
- moved SW1 113.2 mm to (178.5, 99.2)
- moved R19 91.5 mm to (112.5, 60.5), turned to 90 degrees
- moved J1 88.9 mm to (229.0, 128.2)
- moved R23 68.9 mm to (74.2, 75.0)
- moved R26 37.7 mm to (116.5, 159.0)
- moved R18 37.3 mm to (79.2, 61.5)
- moved R24 35.9 mm to (139.5, 62.5), turned to 270 degrees
- moved J2 25.0 mm to (229.8, 111.2)
- moved U1 11.2 mm to (166.0, 80.5)
- moved U3 10.1 mm to (123.5, 90.8)
- renumbered U102 to U3
Connections:
- BT1 pad 2: VGND -> GND
- D1 pad 1: VGND -> GND
- D2 pad 1: VGND -> GND
- J1 pad 1: VGND -> GND
- J1 pad 2: Net-(A1-Pad7) -> +5V
- J1 pad 3: Net-(A1-Pad2) -> /HALLEFF1
- J2 pad 1: Net-(J2-Pad1) -> GND
- J2 pad 2: 5V -> +5V
- J3 pad 2: 5V -> +5V
- J4 pad 2: 5V -> +5V
- J5 pad 1: Net-(J2-Pad1) -> Net-(J4-Pad1)
- J5 pad 2: 5V -> +5V
- J6 pad 1: Net-(J3-Pad1) -> Net-(J6-Pad1)
- J6 pad 2: 5V -> +5V
- Q1 pad 1: Net-(J2-Pad1) -> Net-(Q1-Pad1)
- Q1 pad 2: Net-(Q1-Pad2) -> GND
- Q1 pad 3: VGND -> Net-(J6-Pad1)
- Q2 pad 1: Net-(J3-Pad1) -> Net-(Q2-Pad1)
- Q2 pad 2: Net-(Q2-Pad2) -> GND
- Q2 pad 3: VGND -> Net-(J4-Pad1)
- Q3 pad 1: Net-(J4-Pad1) -> Net-(Q3-Pad1)
- Q3 pad 2: Net-(Q3-Pad2) -> GND
- Q3 pad 3: VGND -> Net-(J3-Pad1)
- Q4 pad 1: Net-(D19-Pad1) -> Net-(Q4-Pad1)
- Q4 pad 2: Net-(Q4-Pad2) -> GND
- Q4 pad 3: VGND -> Net-(D19-Pad1)
- Q5 pad 1: Net-(D3-Pad1) -> Net-(Q5-Pad1)
- Q5 pad 2: Net-(Q5-Pad2) -> GND
- Q5 pad 3: VGND -> Net-(D3-Pad1)
- Q6 pad 1: Net-(D10-Pad1) -> Net-(Q6-Pad1)
- Q6 pad 2: Net-(Q6-Pad2) -> GND
- Q6 pad 3: VGND -> Net-(D10-Pad1)
- Q7 pad 1: Net-(D11-Pad1) -> Net-(Q7-Pad1)
- Q7 pad 2: Net-(Q7-Pad2) -> GND
- Q7 pad 3: VGND -> Net-(D11-Pad1)
- Q8 pad 1: Net-(D15-Pad1) -> Net-(Q8-Pad1)
- Q8 pad 2: Net-(Q8-Pad2) -> GND
- Q8 pad 3: VGND -> Net-(D15-Pad1)
- R1 pad 1: Net-(D1-Pad2) -> +5V
- R1 pad 2: 5V -> /nRESET
- R10 pad 2: Net-(D8-Pad2) -> Net-(D7-Pad2)
- R11 pad 2: Net-(D9-Pad2) -> Net-(D8-Pad2)
- R12 pad 2: Net-(D10-Pad2) -> Net-(D9-Pad2)
- R13 pad 1: Net-(Q7-Pad2) -> +5V
- R13 pad 2: /BL4 -> Net-(D10-Pad2)
- R14 pad 1: +5V -> Net-(Q7-Pad1)
- R14 pad 2: Net-(D11-Pad2) -> /Shift Registers/SRBLUELT4
- R15 pad 2: Net-(D12-Pad2) -> Net-(D11-Pad2)
- R16 pad 2: Net-(D13-Pad2) -> Net-(D12-Pad2)
- R17 pad 2: Net-(D14-Pad2) -> Net-(D13-Pad2)
- R18 pad 1: Net-(Q8-Pad2) -> +5V
- R18 pad 2: /BL5 -> Net-(D14-Pad2)
- R19 pad 1: +5V -> Net-(Q8-Pad1)
- R19 pad 2: Net-(D15-Pad2) -> /Shift Registers/SRBLUELT5
- R2 pad 1: Net-(D2-Pad2) -> Net-(D1-Pad2)
- R2 pad 2: /IND -> +5V
- R20 pad 2: Net-(D16-Pad2) -> Net-(D15-Pad2)
- R21 pad 2: Net-(D17-Pad2) -> Net-(D16-Pad2)
- R22 pad 2: Net-(D18-Pad2) -> Net-(D17-Pad2)
- R23 pad 1: Net-(Q4-Pad2) -> +5V
- R23 pad 2: /BL1 -> Net-(D18-Pad2)
- R24 pad 1: +5V -> Net-(Q4-Pad1)
- R24 pad 2: Net-(D19-Pad2) -> /Shift Registers/SRBLUELT1
- R25 pad 2: Net-(D20-Pad2) -> Net-(D19-Pad2)
- R26 pad 2: Net-(D21-Pad2) -> Net-(D20-Pad2)
- R27 pad 2: Net-(D22-Pad2) -> Net-(D21-Pad2)
- R3 pad 1: Net-(Q5-Pad2) -> Net-(D2-Pad2)
- R3 pad 2: /BL2 -> /Shift Registers/IND
- R4 pad 1: +5V -> Net-(Q5-Pad1)
- R4 pad 2: Net-(D3-Pad2) -> /Shift Registers/SRBLUELT2
- R5 pad 2: Net-(D4-Pad2) -> Net-(D3-Pad2)
- R6 pad 2: Net-(D5-Pad2) -> Net-(D4-Pad2)
- R7 pad 2: Net-(D6-Pad2) -> Net-(D5-Pad2)
- R8 pad 1: Net-(Q6-Pad2) -> +5V
- R8 pad 2: /BL3 -> Net-(D6-Pad2)
- R9 pad 1: +5V -> Net-(Q6-Pad1)
- R9 pad 2: Net-(D7-Pad2) -> /Shift Registers/SRBLUELT3
- SW1 pad 1: /Power/5VO -> GND
- SW1 pad 2: 5V -> GND
- U1 pad 1: VGND -> (no net)
- U1 pad 13: (no net) -> /nRESET
- U1 pad 14: Net-(A1-Pad14) -> +5V
- U1 pad 15: Net-(A1-Pad15) -> GND
- U1 pad 16: Net-(A1-Pad16) -> /XTAL2
- U1 pad 17: (no net) -> /XTAL1
- U1 pad 18: (no net) -> /HALLEFF1
- U1 pad 2: Net-(A1-Pad2) -> VBUS
- U1 pad 21: 5V -> (no net)
- U1 pad 23: (no net) -> GND
- U1 pad 24: (no net) -> +5V
- U1 pad 25: (no net) -> /HALLEFF2
- U1 pad 27: (no net) -> /HALLEFF4
- U1 pad 3: /HE1 -> (no net)
- U1 pad 31: (no net) -> /HALLEFF3
- U1 pad 34: (no net) -> +5V
- U1 pad 4: /HE2 -> (no net)
- U1 pad 5: /HE3 -> GND
- U1 pad 6: /HE4 -> /UCAP
- U1 pad 7: Net-(A1-Pad7) -> VBUS
- U3 pad 1: /RL -> /Shift Registers/IND
- U3 pad 10: 5V -> +5V
- U3 pad 11: Net-(A1-Pad15) -> /SRCLK
- U3 pad 12: Net-(A1-Pad16) -> /SRLATCH
- U3 pad 13: VGND -> GND
- U3 pad 14: Net-(A1-Pad14) -> /Shift Registers/SR1OUT2IN
- U3 pad 15: /GL -> (no net)
- U3 pad 16: 5V -> +5V
- U3 pad 2: /WL -> (no net)
- U3 pad 3: /BL1 -> (no net)
- U3 pad 4: /BL2 -> (no net)
- U3 pad 5: /BL3 -> (no net)
- U3 pad 6: /BL4 -> (no net)
- U3 pad 7: /BL5 -> (no net)
- U3 pad 8: VGND -> GND
- U3 pad 9: Net-(U1-Pad14) -> (no net)

Commit message: Resize to correct for scale
Parts:
- removed Q1, Q2, Q3, Q4, Q5, Q6, Q7, Q8: BCW65ALT1G, Package_TO_SOT_SMD:SOT-23
- removed R14, R19, R24, R29, R30, R31, R4, R9: 2.7k, Frequently_Used:0805_2012Metric_HandSolder
- added U4: ULN2803ADWRG4, Naquadah_Generator:SOIC127P1030X265-18N, F.Cu at (99.7, 92.3)
- U2, U3: footprint Package_DIP:DIP-16_W7.62mm -> Naquadah_Generator:SOIC-16_3.9x9.9mm_P1.27mm_Hand_Solder
- moved J7 208.2 mm to (103.2, 176.5)
- moved D1 182.7 mm to (229.6, 165.9)
- moved R6 146.1 mm to (70.4, 46.5), turned to 32.5 degrees
- moved R7 124.9 mm to (139.8, 159.0), turned to 212.5 degrees
- moved R5 123.8 mm to (70.4, 157.9), turned to 327.5 degrees
- moved R10 105.8 mm to (151.2, 149.5), turned to 225 degrees
- moved R11 102.4 mm to (151.7, 54.8), turned to 135 degrees
- moved J3 102.1 mm to (119.5, 64.8), turned to 90 degrees
- moved R12 102.0 mm to (58.8, 148.1), turned to 315 degrees
- moved R16 95.9 mm to (160.2, 65.9), turned to 122.5 degrees
- moved R2 87.5 mm to (234.0, 160.6)
- moved R15 83.4 mm to (160.5, 138.8), turned to 237.5 degrees
- moved R17 79.4 mm to (50.0, 138.0), turned to 302.5 degrees
- moved R13 63.6 mm to (59.0, 55.6), turned to 45 degrees
- moved D2 55.2 mm to (109.0, 112.6), turned to 90 degrees
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Connections:
- net Net-(D10-Pad1) renamed /Shift Registers/BLUELT3
- net Net-(D11-Pad1) renamed /Shift Registers/BLUELT4
- net Net-(D15-Pad1) renamed /Shift Registers/BLUELT5
- net Net-(D19-Pad1) renamed /Shift Registers/BLUELT1
- net Net-(D3-Pad1) renamed /Shift Registers/BLUELT2
- net Net-(J4-Pad1) renamed /Shift Registers/RDLT
- net Net-(J6-Pad1) renamed /Shift Registers/GRNLT
- J3 pad 1: Net-(J3-Pad1) -> /Shift Registers/WHTLT
Routing:
- net /Shift Registers/SRBLUELT5: track 0.00 -> 17.7 mm
- net /Shift Registers/SRBLUELT1: track 0.00 -> 16.1 mm
- net /Shift Registers/SRRDLT: track 0.00 -> 16.1 mm
- net /Shift Registers/SRBLUELT3: track 0.00 -> 16.0 mm
- net /Shift Registers/SRBLUELT2: track 0.00 -> 16.0 mm
- net /Shift Registers/SRWHTLT: track 0.00 -> 15.9 mm
- net /Shift Registers/SRBLUELT4: track 0.00 -> 15.8 mm
- net /Shift Registers/SRGRNLT: track 0.00 -> 14.2 mm
Other:
- board text added: "BUELT1"
- board text removed: "Blue Lights 1"

Commit message: Updates to PCB Mount
Parts:
- added H1: PCB Mounting Hole, Naquadah_Generator:MountingHole_2.2mm_M2, F.Cu at (53.7, 47.0)
- added H2: PCB Mounting Hole, Naquadah_Generator:MountingHole_2.2mm_M2, F.Cu at (66.5, 38.1)
- added H3: PCB Mounting Hole, Naquadah_Generator:MountingHole_2.2mm_M2, F.Cu at (53.7, 52.9)
- added H4: PCB Mounting Hole, Naquadah_Generator:MountingHole_2.2mm_M2, F.Cu at (59.6, 47.0)
- added H5: Top Through Hole, Naquadah_Generator:MountingHole_Top_Conn_M6, F.Cu at (37.4, 49.3)
- added H6: Top Through Hole, Naquadah_Generator:MountingHole_Top_Conn_M6, F.Cu at (50.3, 39.6)
- added H7: Top Through Hole, Naquadah_Generator:MountingHole_Top_Conn_M6, F.Cu at (46.3, 49.3)
- added H8: Top Through Hole, Naquadah_Generator:MountingHole_Top_Conn_M6, F.Cu at (59.1, 39.6)
- added J8: Conn_ISP_Prog, Naquadah_Generator:PinHeader_2x03_P2.54mm_Vertical, F.Cu at (39.4, 40.0)
- moved J3 106.5 mm to (217.3, 106.9)
- moved J2 83.9 mm to (124.3, 74.3)
- moved J1 62.2 mm to (133.2, 122.4), turned to 90 degrees
- moved C2 52.1 mm to (98.5, 106.5)
- moved C3 52.1 mm to (94.5, 106.5)
- moved Y1 52.1 mm to (97.0, 102.7)
- moved U3 40.5 mm to (88.8, 64.2)
- moved U1 36.6 mm to (93.9, 91.5)
- moved SW1 34.5 mm to (125.1, 138.1)
- moved C4 30.7 mm to (120.5, 129.8)
- moved U2 27.3 mm to (86.5, 74.0)
- moved U4 27.3 mm to (74.5, 81.8)
- moved D2 25.9 mm to (84.9, 103.2)
- moved R3 25.9 mm to (85.2, 95.3)
- moved D19 19.8 mm to (123.5, 52.4)
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Connections:
- J2 pad 3: /HALLEFF3 -> /HALLEFF4
- J2 pad 4: /HALLEFF4 -> /HALLEFF3
- U1 pad 10: (no net) -> /MOSI
- U1 pad 11: (no net) -> /MISO
- U1 pad 9: (no net) -> /SCK
Other:
- board outline added: 115.6 x 115.6 mm
- board text removed: "BUELT1"

Commit message: Library Updates
Parts:
- moved H5 110.5 mm to (104.9, 136.8)
- moved H6 108.7 mm to (138.1, 103.7)
- moved H4 102.3 mm to (138.1, 112.7)
- moved H3 93.9 mm to (95.9, 136.8)
- moved H7 60.0 mm to (71.7, 103.7)
- moved H2 57.4 mm to (113.9, 70.5)
- moved H8 55.2 mm to (104.9, 70.5)
- moved H1 51.0 mm to (71.7, 94.7)
- moved J1 2.88 mm to (135.9, 123.4), turned to 237.5 degrees
- moved J2 1.53 mm to (124.6, 72.8), turned to 327.5 degrees
- renumbered J8 to J0

Commit message: Updates
Parts:
- added C8: 4.7uF, Frequently_Used:0805_2012Metric_HandSolder, F.Cu at (166.4, 156.6)
- added D23: GREEN, LED_THT:LED_D5.0mm, F.Cu at (184.0, 149.4)
- added D24: YELLOW, LED_THT:LED_D5.0mm, F.Cu at (191.5, 149.4)
- added D25: PRTR5V0U2X, Package_TO_SOT_SMD:SOT-143, F.Cu at (170.3, 147.9)
- added J8: USB Solder Pads, Naquadah_Generator:WireSoldPads_1x4_WOL, F.Cu at (158.9, 157.3)
- added P1: USB_C_Plug_USB2.0, Connectors LE:GCT_USB4110-GF-A, F.Cu at (160.8, 148.1)
- added R14: 1M, Frequently_Used:0805_2012Metric_HandSolder, F.Cu at (175.3, 147.1)
- added R19: 5.1k, Frequently_Used:0805_2012Metric_HandSolder, F.Cu at (170.1, 151.6)
- added R24: 5.1k, Frequently_Used:0805_2012Metric_HandSolder, F.Cu at (175.3, 150.0)
- added R29: 5.1k, Frequently_Used:0805_2012Metric_HandSolder, F.Cu at (171.2, 154.6)
- added R30: 5.1k, Frequently_Used:0805_2012Metric_HandSolder, F.Cu at (171.2, 157.5)
- added R4: 1k, Frequently_Used:0805_2012Metric_HandSolder, F.Cu at (183.9, 154.6)
- added R9: 1k, Frequently_Used:0805_2012Metric_HandSolder, F.Cu at (188.7, 154.6)
- D1: value LED -> RED
- moved SW1 38.8 mm to (126.2, 99.3)
- moved U3 38.0 mm to (50.8, 64.7)
- moved U1 12.6 mm to (105.2, 85.9)
- moved U4 1.06 mm to (75.3, 81.1)
- moved U2 1.06 mm to (87.3, 73.3)
Connections:
- U1 pad 22: (no net) -> /TXLED
- U1 pad 3: (no net) -> /D-
- U1 pad 33: (no net) -> GND
- U1 pad 4: (no net) -> /D+
- U1 pad 8: (no net) -> /RXLED
Routing:
- net /Shift Registers/SRBLUELT5: track 17.7 -> 18.3 mm

Commit message: Added real power schematic
Parts:
- moved R3 94.0 mm to (176.9, 116.1)
- moved D2 94.0 mm to (176.6, 124.0)
- moved SW1 49.7 mm to (172.2, 80.3)
- moved BT1 45.5 mm to (154.9, 37.4)
- moved R1 45.5 mm to (154.2, 28.0)
- moved C4 34.6 mm to (111.7, 96.3)
- moved J6 33.7 mm to (138.2, 34.2)
- moved SW2 20.3 mm to (171.0, 42.6)
- moved Y1 12.3 mm to (93.3, 91.0)
- moved C2 12.3 mm to (94.8, 94.7)
- moved C3 12.3 mm to (90.8, 94.7)
- moved U2 6.38 mm to (86.1, 79.5)
- moved U4 3.17 mm to (72.5, 79.5), turned to 180 degrees
Routing:
- net (no net): track 0.00 -> 123.6 mm
- net /Shift Registers/SRBLUELT5: track 18.3 -> 7.60 mm
- net /Shift Registers/SRBLUELT4: track 15.7 -> 8.26 mm
- net /Shift Registers/SRBLUELT3: track 16.0 -> 9.45 mm
- net /Shift Registers/SRBLUELT2: track 15.9 -> 10.8 mm
- net /Shift Registers/SRBLUELT1: track 16.0 -> 12.3 mm
- net /Shift Registers/SRWHTLT: track 15.8 -> 13.9 mm
- net /Shift Registers/SRRDLT: track 15.7 -> 16.7 mm
Other:
- net class Default: trace_width 0.25 -> 0.2

Commit message: Adding Power Daughter Board
Parts:
- removed the D1 at (229.6, 165.9)
- removed R2: 330, Frequently_Used:0805_2012Metric_HandSolder
- added C10: 22uF, Li-ion 5A Boost 1A Charge Protect:0805_2012Metric_HandSolder, F.Cu at (43.3, 180.6)
- added C11: 470uF, Li-ion 5A Boost 1A Charge Protect:UCD1E471MNL1GS, F.Cu at (85.6, 141.8)
- added C12: 10uF, Li-ion 5A Boost 1A Charge Protect:0805_2012Metric_HandSolder, F.Cu at (47.2, 176.9)
- added C13: 2.2nF, Li-ion 5A Boost 1A Charge Protect:0805_2012Metric_HandSolder, F.Cu at (56.2, 167.0)
- added C14: 1uF, Li-ion 5A Boost 1A Charge Protect:0805_2012Metric_HandSolder, F.Cu at (60.8, 161.1)
- added C15: 47pF, Li-ion 5A Boost 1A Charge Protect:0805_2012Metric_HandSolder, F.Cu at (64.4, 157.5)
- added C16: 22uF, Li-ion 5A Boost 1A Charge Protect:0805_2012Metric_HandSolder, F.Cu at (48.7, 172.2)
- added C17: 10nF, Li-ion 5A Boost 1A Charge Protect:0805_2012Metric_HandSolder, F.Cu at (56.0, 164.1)
- added C18: 10uF, Li-ion 5A Boost 1A Charge Protect:0805_2012Metric_HandSolder, F.Cu at (42.4, 177.6)
- added C19: 470uF, Li-ion 5A Boost 1A Charge Protect:UCD1E471MNL1GS, F.Cu at (67.6, 121.7)
- added C9: 100nF, Li-ion 5A Boost 1A Charge Protect:0805_2012Metric_HandSolder, F.Cu at (60.8, 164.1)
- added D26: GREEN, Li-ion 5A Boost 1A Charge Protect:LED_0805_2012Metric_HandSolder, F.Cu at (29.1, 182.2)
- added D27: GREEN, Li-ion 5A Boost 1A Charge Protect:LED_0805_2012Metric_HandSolder, F.Cu at (64.4, 154.5)
- added D28: RED, Li-ion 5A Boost 1A Charge Protect:LED_0805_2012Metric_HandSolder, F.Cu at (33.8, 182.2)
- added D29: 5A 100V, Li-ion 5A Boost 1A Charge Protect:DO-214AC, F.Cu at (67.2, 132.4)
- added D30: RED, Li-ion 5A Boost 1A Charge Protect:LED_0805_2012Metric_HandSolder, F.Cu at (56.1, 161.1)
- added L1: 6.8uH, Li-ion 5A Boost 1A Charge Protect:L_MGV0605, F.Cu at (76.0, 132.7)
- added R31: 330, Li-ion 5A Boost 1A Charge Protect:0805_2012Metric_HandSolder, F.Cu at (37.7, 177.6)
- added R32: 2.7k, Li-ion 5A Boost 1A Charge Protect:0805_2012Metric_HandSolder, F.Cu at (51.4, 167.7)
- added R33: 1k, Li-ion 5A Boost 1A Charge Protect:0805_2012Metric_HandSolder, F.Cu at (38.6, 180.6)
- added R34: 1k, Li-ion 5A Boost 1A Charge Protect:0805_2012Metric_HandSolder, F.Cu at (53.4, 170.6)
- added R35: 1k, Li-ion 5A Boost 1A Charge Protect:0805_2012Metric_HandSolder, F.Cu at (62.9, 170.0)
- added R36: 1k, Li-ion 5A Boost 1A Charge Protect:0805_2012Metric_HandSolder, F.Cu at (56.7, 176.5)
- added R37: 1.54k, Li-ion 5A Boost 1A Charge Protect:0805_2012Metric_HandSolder, F.Cu at (52.8, 179.5)
- added R38: 51k, Li-ion 5A Boost 1A Charge Protect:0805_2012Metric_HandSolder, F.Cu at (58.2, 172.9)
- added R39: 69.8k, Li-ion 5A Boost 1A Charge Protect:0805_2012Metric_HandSolder, F.Cu at (58.2, 170.0)
- added R40: 30k, Li-ion 5A Boost 1A Charge Protect:0805_2012Metric_HandSolder, F.Cu at (48.1, 179.8)
- added R41: 10k, Li-ion 5A Boost 1A Charge Protect:0805_2012Metric_HandSolder, F.Cu at (51.9, 176.5)
- added R42: 1k, Li-ion 5A Boost 1A Charge Protect:0805_2012Metric_HandSolder, F.Cu at (53.4, 173.6)
- added TH1: 10k, Li-ion 5A Boost 1A Charge Protect:0805_2012Metric_HandSolder, F.Cu at (60.9, 167.0)
- added U5: AP9101CK6, Li-ion 5A Boost 1A Charge Protect:SOT-23-6, F.Cu at (43.9, 173.1)
- added U6: ECH8695R-TL-W, Li-ion 5A Boost 1A Charge Protect:SOT65P280X95-8N, F.Cu at (24.1, 180.3)
- added U7: MCP73833T, Li-ion 5A Boost 1A Charge Protect:MCP73833, F.Cu at (40.5, 167.3)
- added U8: PAM2423AECADJR, Li-ion 5A Boost 1A Charge Protect:PAM2423AECADJR, F.Cu at (32.6, 169.3)
- added W1: 2.5x5.0, Li-ion 5A Boost 1A Charge Protect:Pad_3.0-5.0_w_TH, F.Cu at (59.7, 156.3)
- added W2: 2.5x5.0, Li-ion 5A Boost 1A Charge Protect:Pad_3.0-5.0_w_TH, F.Cu at (51.4, 162.9)
- added W3: 2.5x5.0, Li-ion 5A Boost 1A Charge Protect:Pad_3.0-5.0_w_TH, F.Cu at (39.2, 172.9)
- added W4: 2.5x5.0, Li-ion 5A Boost 1A Charge Protect:Pad_3.0-5.0_w_TH, F.Cu at (46.8, 167.5)
- added W7: 2.5x5.0, Li-ion 5A Boost 1A Charge Protect:Pad_3.0-5.0_w_TH, F.Cu at (55.1, 156.3)
- added W8: 2.5x5.0, Li-ion 5A Boost 1A Charge Protect:Pad_3.0-5.0_w_TH, F.Cu at (46.8, 160.8)
- C2, C3: value 22pF -> 18pF
- D1: renamed from D25; value PRTR5V0U2X -> SDP
- D23, D24: footprint LED_THT:LED_D5.0mm -> Frequently_Used:LED_0805_2012Metric_HandSolder
- moved SW2 207.8 mm to (15.4, 180.3)
- moved BT1 160.0 mm to (46.7, 155.2)
- moved U2 75.9 mm to (14.3, 54.8)
- moved U4 75.9 mm to (0.75, 54.8)
- moved C2 73.0 mm to (156.8, 56.1)
- moved C3 73.0 mm to (152.8, 56.1)
- moved C4 73.0 mm to (173.7, 57.7)
- moved U1 73.0 mm to (167.2, 47.3)
- moved Y1 73.0 mm to (155.3, 52.4)
Connections:
- net /Power/5VO renamed Net-(BT1-Pad1)
- BT1 pad 2: GND -> /Power/BATT-
- SW2 pad 2: +5V -> /Power/BATT+
