File: Naquadah Generator Main/Naquadah Generator Main.kicad_pcb (KiCad board)
At the start: 2 copper layers, 115.6 x 115.6 mm, 122 parts, among them J0 Conn_ISP_Prog, J1 State_Sensing_Conn, J10 Power Board Conn, J2 State_Sensing_Conn, J3 Conn_01x02, J8 USB Solder Pads, J9 Power_Conn, P1 USB_C_Plug_USB2.0, Q1 30V 5A, SW1 RESET, U1 ATmega32U4-AU, U2 74HC595, U3 74HC595, U4 ULN2803ADWRG4, U5 AP9101CK6, U6 ECH8695R-TL-W, U8 PAM2423AECADJR, Y1 16MHz

Commit message: PCB Updates
Parts:
- J1, J2: footprint Naquadah_Generator:Mother_Board_Hor_4_Pin_JST_Conn -> Naquadah_Generator:Daughter_Board_Hor_4_Pin_JST_Conn
- J10: footprint Naquadah_Generator:Mother_Board_Vert_5_Pin_JST_Conn -> Naquadah_Generator:Daughter_Board_Vert_5_Pin_JST_Conn
- J8: moved to B.Cu
- P1: footprint Connectors LE:GCT_USB4110-GF-A -> Connectors_LE:2047110001
- moved J8 123.8 mm to (104.5, 62.4)
- moved D1 112.4 mm to (110.5, 77.5)
- moved C2 109.7 mm to (90.8, 104.6), turned to 180 degrees
- moved Y1 105.5 mm to (95.1, 102.5), turned to 90 degrees
- moved C3 104.2 mm to (90.8, 100.3), turned to 180 degrees
- moved P1 103.4 mm to (104.9, 51.2)
- moved SW1 101.5 mm to (93.1, 110.9), turned to 180 degrees
- moved J0 60.2 mm to (81.6, 103.6), turned to 0 degrees
- moved J2 52.3 mm to (136.3, 123.7), turned to 237.5 degrees
- moved J1 52.1 mm to (124.7, 72.5), turned to 327.5 degrees
- moved TP3 48.2 mm to (120.0, 75.8), turned to 57.5 degrees
- moved TP6 47.4 mm to (130.2, 121.9), turned to 237.5 degrees
- moved TP4 41.5 mm to (124.0, 78.3), turned to 57.5 degrees
- moved TP5 40.7 mm to (132.8, 117.9), turned to 237.5 degrees
- moved R4 24.0 mm to (193.8, 145.5)
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Connections:
- P1 pad S2: (no net) -> /Connectors/SHLD
- P1 pad S3: (no net) -> /Connectors/SHLD
- P1 pad S4: (no net) -> /Connectors/SHLD
- U1 pad 18: /HALLEFF1 -> (no net)
- U1 pad 19: /MODESEL -> (no net)
- U1 pad 25: /HALLEFF2 -> /SRDATA
- U1 pad 26: (no net) -> /SRLATCH
- U1 pad 27: /HALLEFF4 -> /SRCLK
- U1 pad 29: (no net) -> /MODESEL
- U1 pad 32: (no net) -> /HALLEFF4
- U1 pad 36: /SRDATA -> (no net)
- U1 pad 37: /SRCLK -> (no net)
- U1 pad 38: /SRLATCH -> (no net)
- U1 pad 40: (no net) -> /HALLEFF2
- U1 pad 41: (no net) -> /HALLEFF1
Routing:
- net /Shift Registers/BLUELT5: track 374.5 -> 240.1 mm, vias 2 -> 4
- net (no net): track 123.6 -> 0.00 mm, vias 0 -> 4
- net /Shift Registers/BLUELT4: track 383.1 -> 272.9 mm, vias 2 -> 4
- net /Shift Registers/BLUELT3: track 385.1 -> 298.3 mm, vias 2 -> 4
- net /Shift Registers/BLUELT2: track 390.6 -> 328.6 mm, vias 2 -> 4
- net /SRCLK: track 0.00 -> 49.6 mm, vias 0 -> 2
- net /SRLATCH: track 0.00 -> 46.2 mm, vias 0 -> 2
- net /HALLEFF3: track 0.00 -> 44.2 mm, vias 0 -> 3
- net /HALLEFF1: track 0.00 -> 44.1 mm, vias 0 -> 2
- net /HALLEFF4: track 0.00 -> 42.2 mm, vias 0 -> 3
- net /HALLEFF2: track 0.00 -> 41.3 mm, vias 0 -> 2
- net /SRDATA: track 0.00 -> 41.1 mm, vias 0 -> 2
- net /Shift Registers/BLUELT1: track 395.1 -> 359.3 mm, vias 2 -> 4
- net /SCK: track 0.00 -> 34.7 mm
- net /nRESET: track 0.00 -> 33.7 mm, vias 0 -> 2
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
Commit message: Updates
Parts:
- added U7: VS1000, Package_QFP:LQFP-48_7x7mm_P0.5mm, F.Cu at (126.3, 135.1)
Connections:
- U1 pad 30: (no net) -> /AUDRESET
- U1 pad 31: /HALLEFF3 -> /M_TX_A_RX
- U1 pad 32: /HALLEFF4 -> /M_RX_A_TX
- U1 pad 38: (no net) -> /HALLEFF3
- U1 pad 39: (no net) -> /HALLEFF4
Routing:
- net /HALLEFF1: track 44.1 -> 39.3 mm
- net /HALLEFF2: track 41.3 -> 39.6 mm
- net /HALLEFF3: track 44.2 -> 43.6 mm, vias 3 -> 2
- net /HALLEFF4: track 42.2 -> 41.7 mm, vias 3 -> 2
