File: Naquadah Generator Main/Naquadah Generator Main.kicad_pcb (KiCad board)
At the start: 2 copper layers, 115.6 x 115.6 mm, 210 parts, among them J0 Conn_ISP_Prog, J1 State_Sensing_Conn, J10 Power Board Conn, J2 State_Sensing_Conn, J3 Conn_01x02, J4 USB Solder Pads, J5 Conn_01x07, J6 Conn_01x07, J8 USB Solder Pads, J9 Power_Conn, P1 USB_C_Plug_USB2.0, P2 USB_C_Plug_USB2.0, Q1 30V 5A, SW1 RESET, U1 ATmega32U4-AU, U10 PAM8302AAD, U11 MIC5219-3.3YM5-TR, U12 CD74HC4050PWR, U2 74HC595, U3 74HC595, U4 ULN2803ADWRG4, U5 AP9101CK6, U6 ECH8695R-TL-W, U7 VS1000, U8 PAM2421AECADJR, U9 MX25L1606EM1I-12G, Y1 16MHz, Y2 12MHz

Commit message: Switched to 0603_1608M size for passives
Parts:
- added TP20: TestPoint, Frequently_Used_LE:Pad_2.5-2.5, B.Cu at (31.5, 127.3)
- C1, C20, C22, C28, C29, C4, C5, C6: value 1.0uF -> 1uF; footprint Frequently_Used_LE:0805_2012Metric_HandSolder -> Frequently_Used_LE:0603_1608Metric
- C10, C16, C2, C21, C3, C33, C34, C35, C36, C7, C8: footprint Frequently_Used_LE:0805_2012Metric_HandSolder -> Frequently_Used_LE:0603_1608Metric
- C12, C13, C14, C15, C17, C18, R1, R10, R11, R12, R13, R14, R15, R16, R17, R18, R19, R2, R20, R21, R22, R23, R24, R25, R26, R27, R28, R29, R3, R30, R31, R32, R33, R34, R35, R36, R37, R38, R4, R40, R41, R47, R48, R49, R5, R50, R51, R52, R58, R59, R6, R62, R63, R7, R8, R9: footprint Frequently_Used_LE:0805_2012Metric -> Frequently_Used_LE:0603_1608Metric
- C23, C24: value 1UF -> 1uF; footprint Frequently_Used_LE:0805_2012Metric_HandSolder -> Frequently_Used_LE:0603_1608Metric
- C25: value 1.0uF -> 10uF; footprint Frequently_Used_LE:0805_2012Metric_HandSolder -> Frequently_Used_LE:0603_1608Metric
- C26, C27: value 22pF -> 220pF; footprint Frequently_Used_LE:0805_2012Metric_HandSolder -> Frequently_Used_LE:0603_1608Metric
- C9: value 100nF -> 0.1uF; footprint Frequently_Used_LE:0805_2012Metric -> Frequently_Used_LE:0603_1608Metric
- D23, D24, D28: footprint Frequently_Used_LE:LED_0805_2012Metric_HandSolder -> Frequently_Used_LE:LED_0805_2012Metric
- FID1: value TOP1 -> Fiducial
- FID2: value TOP2 -> Fiducial
- FID3: value TOP3 -> Fiducial
- FID4: value BOT1 -> Fiducial
- FID5: value BOT2 -> Fiducial
- FID6: value BOT3 -> Fiducial
- J10: value Power Board Conn -> User_Interface_6_Pin_Conn; footprint Naquadah_Generator:Daughter_Board_Vert_5_Pin_JST_Conn -> Naquadah_Generator:Daughter_Board_Vert_6_Pin_JST_Conn
- J3: footprint Connector_Wire:SolderWirePad_1x02_P3.81mm_Drill1.2mm -> Connector_LE:JST_SH_BM02B-SRSS-TB_1x02-1MP_P1.00mm_Vertical
- P1, P2: footprint Connectors_LE:2047110001 -> Connector_LE:2047110001
- R60: value 100k -> 10k
- TP16: moved to B.Cu
- U11: footprint Package_TO_SOT_SMD:SOT-23-5_HandSoldering -> Package_TO_SOT_SMD:SOT-23-5
- moved FID3 127.4 mm to (104.8, 150.8)
- moved FID6 124.7 mm to (104.8, 150.8)
- moved FID4 93.8 mm to (101.9, 66.1)
- moved FID1 93.7 mm to (101.9, 66.1)
- moved FID2 77.0 mm to (138.1, 108.6)
- moved FID5 69.2 mm to (138.1, 108.6)
- moved C27 5.15 mm to (153.7, 180.4), turned to 180 degrees
- moved C26 4.84 mm to (153.7, 172.9), turned to 180 degrees
- moved C24 4.80 mm to (140.9, 180.4), turned to 0 degrees
- moved C23 4.58 mm to (140.9, 172.9)
- moved R40 1.23 mm to (74.8, 87.0)
- moved R41 1.23 mm to (69.3, 87.0)
- moved C13 1.21 mm to (65.4, 79.3)
- moved R58 0.81 mm to (140.9, 175.4)
- moved R1 0.54 mm to (57.9, 89.2)
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Connections:
- net /Shift Registers/WHTLT renamed /WHITELT
- net Net-(L4-Pad2) renamed /Audio/Mono Amplifier PAM8302A/OUT-
- net Net-(L5-Pad2) renamed /Audio/Mono Amplifier PAM8302A/OUT+
- net Net-(R58-Pad1) renamed /Audio/Mono Amplifier PAM8302A/IN+
- net Net-(R59-Pad1) renamed /Audio/Mono Amplifier PAM8302A/IN-
- net Net-(R60-Pad1) renamed /Audio/Mono Amplifier PAM8302A/~SD
- C25 pad 1: AVDD -> AGND
- C25 pad 2: AGND -> AVDD
- J10 pad 3: /MODESEL -> /VOLUME
- J10 pad 4: /READY -> /MODESEL
- J10 pad 5: /SWITCH -> /READY
Routing:
- net DGND: track 45.1 -> 43.5 mm
- net /Power/Boost 3.0A 5V 0805_2012/FB: track 14.8 -> 13.6 mm
- net Net-(C13-Pad1): track 3.99 -> 2.84 mm
- net /BATT-: track 21.8 -> 22.4 mm

Commit message: Removed schematic templates,  Added audio connection
Removed schematic templates,  Added audio connection
Parts:
- J3: moved to B.Cu
- turned J3 to 90 degrees
Changed lines of the file:
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@@
     (add_net +3V3)
     (add_net +5V)
-    (add_net /A0)
     (add_net /AREF)
-    (add_net /AUDIORESET)
     (add_net /AUDIORESET3V)
     (add_net /Audio/AO+)
     (add_net /Audio/AO-)
     (add_net /Audio/AUDIOLEFT)
-    (add_net /Audio/AUDIOPRE+)
     (add_net "/Audio/Audio USB/CC1")
     (add_net "/Audio/Audio USB/CC2")
@@
     (add_net /Audio/MISO)
     (add_net /Audio/MOSI)
-    (add_net "/Audio/Mono Amplifier PAM8302A/AUDIOPRE+")
     (add_net "/Audio/Mono Amplifier PAM8302A/IN+")
     (add_net "/Audio/Mono Amplifier PAM8302A/IN-")
@@
     (add_net /D+)
     (add_net /D-)
-    (add_net /D11)
-    (add_net /D7)
     (add_net /HALLEFF1)
     (add_net /HALLEFF2)
@@
     (add_net /Power/SWGATE)
     (add_net /READY)
-    (add_net /RX)
     (add_net /RXLED)
     (add_net /SCK)
-    (add_net /SCL)
-    (add_net /SDA)
     (add_net /SNDLATCH3V)
     (add_net /SNDON3V)
@@
     (add_net "/Shift Registers/SRRDLT")
     (add_net "/Shift Registers/SRWHTLT")
-    (add_net /TX)
     (add_net /TXLED)
     (add_net /UCAP)
@@
     (add_net "Net-(JP1-Pad2)")
     (add_net "Net-(JP5-Pad2)")
-    (add_net "Net-(P1-PadA10)")
-    (add_net "Net-(P1-PadA11)")
-    (add_net "Net-(P1-PadA2)")
-    (add_net "Net-(P1-PadA3)")
-    (add_net "Net-(P1-PadA8)")
-    (add_net "Net-(P1-PadB10)")
-    (add_net "Net-(P1-PadB11)")
-    (add_net "Net-(P1-PadB2)")
-    (add_net "Net-(P1-PadB3)")
-    (add_net "Net-(P1-PadB8)")
-    (add_net "Net-(P2-PadA10)")
-    (add_net "Net-(P2-PadA11)")
-    (add_net "Net-(P2-PadA2)")
-    (add_net "Net-(P2-PadA3)")
-    (add_net "Net-(P2-PadA8)")
-    (add_net "Net-(P2-PadB10)")
-    (add_net "Net-(P2-PadB11)")
-    (add_net "Net-(P2-PadB2)")
-    (add_net "Net-(P2-PadB3)")
-    (add_net "Net-(P2-PadB8)")
-    (add_net "Net-(U1-Pad28)")
-    (add_net "Net-(U10-Pad2)")
-    (add_net "Net-(U12-Pad11)")
-    (add_net "Net-(U12-Pad12)")
-    (add_net "Net-(U12-Pad13)")
-    (add_net "Net-(U12-Pad14)")
-    (add_net "Net-(U12-Pad15)")
-    (add_net "Net-(U12-Pad16)")
-    (add_net "Net-(U3-Pad5)")
-    (add_net "Net-(U3-Pad6)")
-    (add_net "Net-(U3-Pad7)")
-    (add_net "Net-(U3-Pad9)")
-    (add_net "Net-(U5-Pad4)")
-    (add_net "Net-(U6-Pad5)")
-    (add_net "Net-(U6-Pad6)")
-    (add_net "Net-(U6-Pad7)")
-    (add_net "Net-(U6-Pad8)")
-    (add_net "Net-(U7-Pad40)")
     (add_net VBUS)
   )
@@
     )
   )
-  (module Connector_LE:JST_SH_BM02B-SRSS-TB_1x02-1MP_P1.00mm_Vertical (layer F.Cu)
-    (at 175.856822 66.158727 270)
+  (module Connector_LE:JST_SH_BM02B-SRSS-TB_1x02-1MP_P1.00mm_Vertical (layer B.Cu)
+    (at 175.856822 66.158727 90)
     (descr "JST SH series connector, BM02B-SRSS-TB (http://www.jst-mfg.com/product/pdf/eng/eSH.pdf), generated with kicad-footprint-generator")
     (tags "connector JST SH side entry")
     (attr smd)
-    (fp_text reference J3 (at 0 -3.3 90) (layer F.SilkS)
-      (effects (font (size 1 1) (thickness 0.15)))
-    )
-    (fp_text value Conn_01x02 (at 0 3.3 90) (layer F.Fab)
-      (effects (font (size 1 1) (thickness 0.15)))
-    )
-    (fp_line (start -2 1) (end 2 1) (layer F.Fab) (width 0.1))
-    (fp_line (start -2.11 -0.04) (end -2.11 1.11) (layer F.SilkS) (width 0.12))
-    (fp_line (start -2.11 1.11) (end -1.06 1.11) (layer F.SilkS) (width 0.12))
-    (fp_line (start -1.06 1.11) (end -1.06 2.1) (layer F.SilkS) (width 0.12))
-    (fp_line (start 2.11 -0.04) (end 2.11 1.11) (layer F.SilkS) (width 0.12))
-    (fp_line (start 2.11 1.11) (end 1.06 1.11) (layer F.SilkS) (width 0.12))
-    (fp_line (start -0.94 -2.01) (end 0.94 -2.01) (layer F.SilkS) (width 0.12))
-    (fp_line (start -2 -1.9) (end 2 -1.9) (layer F.Fab) (width 0.1))
-    (fp_line (start -2 1) (end -2 -1.9) (layer F.Fab) (width 0.1))
-    (fp_line (start 2 1) (end 2 -1.9) (layer F.Fab) (width 0.1))
-    (fp_line (start -0.65 -1.55) (end -0.65 -0.95) (layer F.Fab) (width 0.1))
-    (fp_line (start -0.65 -0.95) (end -0.35 -0.95) (layer F.Fab) (width 0.1))
-    (fp_line (start -0.35 -0.95) (end -0.35 -1.55) (layer F.Fab) (width 0.1))
-    (fp_line (start -0.35 -1.55) (end -0.65 -1.55) (layer F.Fab) (width 0.1))
-    (fp_line (start 0.35 -1.55) (end 0.35 -0.95) (layer F.Fab) (width 0.1))
-    (fp_line (start 0.35 -0.95) (end 0.65 -0.95) (layer F.Fab) (width 0.1))
-    (fp_line (start 0.65 -0.95) (end 0.65 -1.55) (layer F.Fab) (width 0.1))
-    (fp_line (start 0.65 -1.55) (end 0.35 -1.55) (layer F.Fab) (width 0.1))
-    (fp_line (start -2.9 -2.6) (end -2.9 2.6) (layer F.CrtYd) (width 0.05))
-    (fp_line (start -2.9 2.6) (end 2.9 2.6) (layer F.CrtYd) (width 0.05))
-    (fp_line (start 2.9 2.6) (end 2.9 -2.6) (layer F.CrtYd) (width 0.05))
-    (fp_line (start 2.9 -2.6) (end -2.9 -2.6) (layer F.CrtYd) (width 0.05))
-    (fp_line (start -1 1) (end -0.5 0.292893) (layer F.Fab) (width 0.1))
-    (fp_line (start -0.5 0.292893) (end 0 1) (layer F.Fab) (width 0.1))
-    (fp_text user %R (at 0 -0.25 90) (layer F.Fab)
-      (effects (font (size 1 1) (thickness 0.15)))
-    )
-    (pad 1 smd roundrect (at -0.5 1.325 270) (size 0.6 1.55) (layers F.Cu F.Paste F.Mask) (roundrect_rratio 0.25)
+    (fp_text reference J3 (at 0 3.3 270) (layer B.SilkS)
+      (effects (font (size 1 1) (thickness 0.15)) (justify mirror))
+    )
+    (fp_text value Conn_01x02 (at 0 -3.3 270) (layer B.Fab)
+      (effects (font (size 1 1) (thickness 0.15)) (justify mirror))
+    )
+    (fp_line (start -2 -1) (end 2 -1) (layer B.Fab) (width 0.1))
+    (fp_line (start -2.11 0.04) (end -2.11 -1.11) (layer B.SilkS) (width 0.12))
+    (fp_line (start -2.11 -1.11) (end -1.06 -1.11) (layer B.SilkS) (width 0.12))
+    (fp_line (start -1.06 -1.11) (end -1.06 -2.1) (layer B.SilkS) (width 0.12))
+    (fp_line (start 2.11 0.04) (end 2.11 -1.11) (layer B.SilkS) (width 0.12))
+    (fp_line (start 2.11 -1.11) (end 1.06 -1.11) (layer B.SilkS) (width 0.12))
+    (fp_line (start -0.94 2.01) (end 0.94 2.01) (layer B.SilkS) (width 0.12))
+    (fp_line (start -2 1.9) (end 2 1.9) (layer B.Fab) (width 0.1))
+    (fp_line (start -2 -1) (end -2 1.9) (layer B.Fab) (width 0.1))
+    (fp_line (start 2 -1) (end 2 1.9) (layer B.Fab) (width 0.1))
+    (fp_line (start -0.65 1.55) (end -0.65 0.95) (layer B.Fab) (width 0.1))
+    (fp_line (start -0.65 0.95) (end -0.35 0.95) (layer B.Fab) (width 0.1))
+    (fp_line (start -0.35 0.95) (end -0.35 1.55) (layer B.Fab) (width 0.1))
+    (fp_line (start -0.35 1.55) (end -0.65 1.55) (layer B.Fab) (width 0.1))
+    (fp_line (start 0.35 1.55) (end 0.35 0.95) (layer B.Fab) (width 0.1))
+    (fp_line (start 0.35 0.95) (end 0.65 0.95) (layer B.Fab) (width 0.1))
+    (fp_line (start 0.65 0.95) (end 0.65 1.55) (layer B.Fab) (width 0.1))
+    (fp_line (start 0.65 1.55) (end 0.35 1.55) (layer B.Fab) (width 0.1))
+    (fp_line (start -2.9 2.6) (end -2.9 -2.6) (layer B.CrtYd) (width 0.05))
+    (fp_line (start -2.9 -2.6) (end 2.9 -2.6) (layer B.CrtYd) (width 0.05))
+    (fp_line (start 2.9 -2.6) (end 2.9 2.6) (layer B.CrtYd) (width 0.05))
+    (fp_line (start 2.9 2.6) (end -2.9 2.6) (layer B.CrtYd) (width 0.05))
+    (fp_line (start -1 -1) (end -0.5 -0.292893) (layer B.Fab) (width 0.1))
+    (fp_line (start -0.5 -0.292893) (end 0 -1) (layer B.Fab) (width 0.1))
+    (fp_text user %R (at 0 0.25 270) (layer B.Fab)
+      (effects (font (size 1 1) (thickness 0.15)) (justify mirror))
+    )
+    (pad 1 smd roundrect (at -0.5 -1.325 90) (size 0.6 1.55) (layers B.Cu B.Paste B.Mask) (roundrect_rratio 0.25)
       (net 137 /WHITELT))
-    (pad 2 smd roundrect (at 0.5 1.325 270) (size 0.6 1.55) (layers F.Cu F.Paste F.Mask) (roundrect_rratio 0.25)
+    (pad 2 smd roundrect (at 0.5 -1.325 90) (size 0.6 1.55) (layers B.Cu B.Paste B.Mask) (roundrect_rratio 0.25)
       (net 22 +5V))
-    (pad MP smd roundrect (at -1.8 -1.2 270) (size 1.2 1.8) (layers F.Cu F.Paste F.Mask) (roundrect_rratio 0.208333))
-    (pad MP smd roundrect (at 1.8 -1.2 270) (size 1.2 1.8) (layers F.Cu F.Paste F.Mask) (roundrect_rratio 0.208333))
+    (pad MP smd roundrect (at -1.8 1.2 90) (size 1.2 1.8) (layers B.Cu B.Paste B.Mask) (roundrect_rratio 0.208333))
+    (pad MP smd roundrect (at 1.8 1.2 90) (size 1.2 1.8) (layers B.Cu B.Paste B.Mask) (roundrect_rratio 0.208333))
     (model ${LE3DMOD}/BM02B-SRSS-TB.STEP
       (offset (xyz 0 1.15 0))

Commit message: Update JST connectors
Parts:
- added J7: Conn_01x04, Connector_PinHeader_2.54mm:PinHeader_1x04_P2.54mm_Vertical, F.Cu at (219.3, 92.2)
- added WA1: WireAssembly, Mechanical_LE:Wire_Assembly, F.Cu at (250.5, 92.7)
- J1, J2: footprint Naquadah_Generator:Daughter_Board_Hor_4_Pin_JST_Conn -> Connector_JST:JST_SH_SM04B-SRSS-TB_1x04-1MP_P1.00mm_Horizontal
- J10: footprint Naquadah_Generator:Daughter_Board_Vert_6_Pin_JST_Conn -> Connector_JST:JST_SH_BM06B-SRSS-TB_1x06-1MP_P1.00mm_Vertical
- moved J2 27.0 mm to (113.7, 108.9), turned to 57.5 degrees
- moved J1 21.8 mm to (112.9, 90.7), turned to 147.5 degrees
- moved C6 5.48 mm to (116.5, 97.1)
- moved C7 5.48 mm to (116.4, 100.2)
- moved C4 5.48 mm to (116.5, 103.3)
- moved J10 3.46 mm to (115.4, 103.8), turned to 270 degrees
Routing:
- net /HALLEFF4: track 52.8 -> 41.3 mm, vias 2 -> 1
- net /HALLEFF3: track 53.1 -> 43.4 mm, vias 2 -> 1
- net DGND: track 43.5 -> 42.2 mm, vias 32 -> 31

Commit message: Clean up of audio page
Routing:
- net /HALLEFF2: track 49.6 -> 0.03 mm, vias 2 -> 0
- net /HALLEFF1: track 48.6 -> 0.00 mm, vias 2 -> 0
- net /HALLEFF3: track 43.4 -> 0.00 mm, vias 1 -> 0
- net /HALLEFF4: track 41.3 -> 0.01 mm, vias 1 -> 0
- net DGND: track 42.2 -> 40.8 mm, vias 31 -> 30
Changed lines of the file:
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@@
     (thickness 1.6)
     (drawings 11050)
-    (tracks 783)
+    (tracks 748)
     (zones 0)
     (modules 213)
@@
     (add_net +3V3)
     (add_net +5V)
-    (add_net /A0)
     (add_net /AREF)
-    (add_net /AUDIORESET)
     (add_net /AUDIORESET3V)
     (add_net /Audio/AO+)
     (add_net /Audio/AO-)
     (add_net /Audio/AUDIOLEFT)
-    (add_net /Audio/AUDIOPRE+)
     (add_net "/Audio/Audio USB/CC1")
     (add_net "/Audio/Audio USB/CC2")
@@
     (add_net /Audio/MISO)
     (add_net /Audio/MOSI)
-    (add_net "/Audio/Mono Amplifier PAM8302A/AUDIOPRE+")
     (add_net "/Audio/Mono Amplifier PAM8302A/IN+")
     (add_net "/Audio/Mono Amplifier PAM8302A/IN-")
@@
     (add_net /D+)
     (add_net /D-)
-    (add_net /D11)
-    (add_net /D7)
     (add_net /HALLEFF1)
     (add_net /HALLEFF2)
@@
     (add_net /Power/SWGATE)
     (add_net /READY)
-    (add_net /RX)
     (add_net /RXLED)
     (add_net /SCK)
-    (add_net /SCL)
-    (add_net /SDA)
     (add_net /SNDLATCH3V)
     (add_net /SNDON3V)
@@
     (add_net "/Shift Registers/SRRDLT")
     (add_net "/Shift Registers/SRWHTLT")
-    (add_net /TX)
     (add_net /TXLED)
     (add_net /UCAP)
@@
     (add_net "Net-(JP1-Pad2)")
     (add_net "Net-(JP5-Pad2)")
-    (add_net "Net-(P1-PadA10)")
-    (add_net "Net-(P1-PadA11)")
-    (add_net "Net-(P1-PadA2)")
-    (add_net "Net-(P1-PadA3)")
-    (add_net "Net-(P1-PadA8)")
-    (add_net "Net-(P1-PadB10)")
-    (add_net "Net-(P1-PadB11)")
-    (add_net "Net-(P1-PadB2)")
-    (add_net "Net-(P1-PadB3)")
-    (add_net "Net-(P1-PadB8)")
-    (add_net "Net-(P2-PadA10)")
-    (add_net "Net-(P2-PadA11)")
-    (add_net "Net-(P2-PadA2)")
-    (add_net "Net-(P2-PadA3)")
-    (add_net "Net-(P2-PadA8)")
-    (add_net "Net-(P2-PadB10)")
-    (add_net "Net-(P2-PadB11)")
-    (add_net "Net-(P2-PadB2)")
-    (add_net "Net-(P2-PadB3)")
-    (add_net "Net-(P2-PadB8)")
-    (add_net "Net-(U1-Pad28)")
-    (add_net "Net-(U10-Pad2)")
-    (add_net "Net-(U12-Pad11)")
-    (add_net "Net-(U12-Pad12)")
-    (add_net "Net-(U12-Pad13)")
-    (add_net "Net-(U12-Pad14)")
-    (add_net "Net-(U12-Pad15)")
-    (add_net "Net-(U12-Pad16)")
-    (add_net "Net-(U3-Pad5)")
-    (add_net "Net-(U3-Pad6)")
-    (add_net "Net-(U3-Pad7)")
-    (add_net "Net-(U3-Pad9)")
-    (add_net "Net-(U5-Pad4)")
-    (add_net "Net-(U6-Pad5)")
-    (add_net "Net-(U6-Pad6)")
-    (add_net "Net-(U6-Pad7)")
-    (add_net "Net-(U6-Pad8)")
-    (add_net "Net-(U7-Pad40)")
     (add_net VBUS)
   )
@@
   (segment (start 81.668168 56.564989) (end 80.99056 56.564989) (width 0.2) (layer F.Cu) (net 22))
   (segment (start 80.99056 56.564989) (end 75.146822 62.408727) (width 0.2) (layer F.Cu) (net 22))
-  (segment (start 125.249769 70.803338) (end 125.249769 70.91578) (width 0.2) (layer F.Cu) (net 22))
   (segment (start 104.226822 98.388727) (end 104.206822 98.408727) (width 0.2) (layer F.Cu) (net 22))
   (segment (start 81.331822 104.018727) (end 84.606822 104.018727) (width 0.2) (layer F.Cu) (net 24))
@@
   (segment (start 92.516822 101.478727) (end 90.566822 101.478727) (width 0.2) (layer F.Cu) (net 25))
   (segment (start 86.776822 101.478727) (end 85.016822 99.718727) (width 0.2) (layer F.Cu) (net 25))
-  (via (at 123.89682 73.528727) (size 0.8) (drill 0.4) (layers F.Cu B.Cu) (net 28))
-  (segment (start 123.89682 73.518729) (end 123.89682 73.528727) (width 0.2) (layer F.Cu) (net 28))
-  (segment (start 126.173117 71.040594) (end 126.173117 71.242432) (width 0.2) (layer F.Cu) (net 28))
-  (segment (start 126.173117 71.242432) (end 123.89682 73.518729) (width 0.2) (layer F.Cu) (net 28))
-  (via (at 120.20682 100.698727) (size 0.8) (drill 0.4) (layers F.Cu B.Cu) (net 28))
-  (segment (start 120.17682 100.728727) (end 120.20682 100.698727) (width 0.2) (layer F.Cu) (net 28))
-  (segment (start 103.796822 100.728727) (end 120.17682 100.728727) (width 0.2) (layer F.Cu) (net 28))
-  (segment (start 120.227688 100.677859) (end 120.20682 100.698727) (width 0.2) (layer B.Cu) (net 28))
-  (segment (start 123.89682 73.528727) (end 120.227688 77.197859) (width 0.2) (layer B.Cu) (net 28))
-  (segment (start 120.227688 77.197859) (end 120.227688 100.677859) (width 0.2) (layer B.Cu) (net 28))
-  (via (at 125.706822 73.178727) (size 0.8) (drill 0.4) (layers F.Cu B.Cu) (net 29))
-  (segment (start 125.706822 73.158727) (end 125.706822 73.178727) (width 0.2) (layer F.Cu) (net 29))
-  (segment (start 127.016508 71.577894) (end 127.016508 71.849041) (width 0.2) (layer F.Cu) (net 29))
-  (segment (start 127.016508 71.849041) (end 125.706822 73.158727) (width 0.2) (layer F.Cu) (net 29))
-  (via (at 120.986822 101.498727) (size 0.8) (drill 0.4) (layers F.Cu B.Cu) (net 29))
-  (segment (start 120.956822 101.528727) (end 120.986822 101.498727) (width 0.2) (layer F.Cu) (net 29))
   (segment (start 103.856822 101.508727) (end 103.876822 101.528727) (width 0.2) (layer F.Cu) (net 29))
-  (segment (start 103.876822 101.528727) (end 120.956822 101.528727) (width 0.2) (layer F.Cu) (net 29))
-  (segment (start 125.696822 73.188727) (end 125.696822 76.668727) (width 0.2) (layer B.Cu) (net 29))
-  (segment (start 125.706822 73.178727) (end 125.696822 73.188727) (width 0.2) (layer B.Cu) (net 29))
-  (segment (start 125.696822 76.668727) (end 121.006822 81.358727) (width 0.2) (layer B.Cu) (net 29))
-  (segment (start 121.006822 81.358727) (end 121.006822 101.478727) (width 0.2) (layer B.Cu) (net 29))
-  (segment (start 121.006822 101.478727) (end 120.986822 101.498727) (width 0.2) (layer B.Cu) (net 29))
-  (via (at 129.826824 103.098727) (size 0.8) (drill 0.4) (layers F.Cu B.Cu) (net 30))
-  (segment (start 103.776822 103.098727) (end 129.826824 103.098727) (width 0.2) (layer F.Cu) (net 30))
-  (segment (start 129.826824 103.098727) (end 129.826822 103.098729) (width 0.2) (layer B.Cu) (net 30))
-  (segment (start 129.826822 103.098729) (end 129.826822 120.428727) (width 0.2) (layer B.Cu) (net 30))
-  (via (at 130.606823 102.348727) (size 0.8) (drill 0.4) (layers F.Cu B.Cu) (net 31))
-  (segment (start 130.586823 102.328727) (end 130.606823 102.348727) (width 0.2) (layer F.Cu) (net 31))
   (segment (start 103.726822 102.318727) (end 103.736822 102.328727) (width 0.2) (layer F.Cu) (net 31))
-  (segment (start 103.736822 102.328727) (end 130.586823 102.328727) (width 0.2) (layer F.Cu) (net 31))
-  (segment (start 130.596822 102.358728) (end 130.606823 102.348727) (width 0.2) (layer B.Cu) (net 31))
-  (segment (start 130.596822 116.768727) (end 130.596822 102.358728) (width 0.2) (layer B.Cu) (net 31))
   (via (at 78.366822 152.658737) (size 0.8) (drill 0.4) (layers F.Cu B.Cu) (net 33))
   (segment (start 77.266822 151.558737) (end 77.966823 152.258738) (width 0.3) (layer F.Cu) (net 33))
@@
   (segment (start 79.266822 99.778727) (end 79.266822 101.908727) (width 0.2) (layer F.Cu) (net 104))
   (segment (start 79.266822 104.278727) (end 79.266822 101.928727) (width 0.2) (layer F.Cu) (net 104))
-  (segment (start 124.486334 69.965995) (end 123.239554 69.965995) (width 0.2) (layer F.Cu) (net 104))
-  (via (at 123.166822 70.038727) (size 0.8) (drill 0.4) (layers F.Cu B.Cu) (net 104))
-  (segment (start 123.239554 69.965995) (end 123.166822 70.038727) (width 0.2) (layer F.Cu) (net 104))
   (segment (start 85.951822 121.013727) (end 85.926822 121.038727) (width 0.2) (layer F.Cu) (net 104))
   (via (at 77.456822 120.008727) (size 0.8) (drill 0.4) (layers F.Cu B.Cu) (net 104))
@@
     )
   )
-  (zone (net 104) (net_name DGND) (layer B.Cu) (hatch edge 0.508)
+  (zone (net 22) (net_name +5V) (layer F.Cu) (hatch edge 0.508)
     (connect_pads (clearance 0.35))
     (min_thickness 0.254)
@@
     (polygon
       (pts
-        (xy 172.396822 166.158727) (xy 42.396822 166.158727) (xy 42.396822 36.158727) (xy 172.396822 36.158727)
+        (xy 167.946822 168.787768) (xy 37.946822 168.787768) (xy 37.946822 38.787768) (xy 167.946822 38.787768)
       )
     )
     (polygon
       (pts
-        (xy 52.396822 137.158727) (xy 52.396822 165.658727) (xy 99.896822 165.658727) (xy 99.896822 137.158727)
+        (xy 83.396822 127.908881) (xy 83.396822 137.158727) (xy 74.896822 137.158727) (xy 74.896822 168.157768) (xy 99.896822 168.157768)
+        (xy 99.896822 127.908248)
       )
     )
     (polygon
       (pts
-        (xy 93.396822 82.658727) (xy 93.396822 45.408727) (xy 72.146822 45.408727) (xy 72.146822 82.658727)
+        (xy 72.146822 42.907768) (xy 72.146822 82.657768) (xy 87.896822 82.657768) (xy 87.896822 94.657768) (xy 99.371822 94.657768)
+        (xy 99.421822 42.907768)
       )
     )
   )
-  (zone (net 22) (net_name +5V) (layer F.Cu) (hatch edge 0.508)
+  (zone (net 104) (net_name DGND) (layer B.Cu) (hatch edge 0.508)
     (connect_pads (clearance 0.35))
     (min_thickness 0.254)
@@
     (polygon
       (pts
-        (xy 167.946822 168.787768) (xy 37.946822 168.787768) (xy 37.946822 38.787768) (xy 167.946822 38.787768)
+        (xy 172.396822 166.158727) (xy 42.396822 166.158727) (xy 42.396822 36.158727) (xy 172.396822 36.158727)
       )
     )
     (polygon
       (pts
-        (xy 83.396822 127.908881) (xy 83.396822 137.158727) (xy 74.896822 137.158727) (xy 74.896822 168.157768) (xy 99.896822 168.157768)
-        (xy 99.896822 127.908248)
+        (xy 52.396822 137.158727) (xy 52.396822 165.658727) (xy 99.896822 165.658727) (xy 99.896822 137.158727)
       )
     )
     (polygon
       (pts
-        (xy 72.146822 42.907768) (xy 72.146822 82.657768) (xy 87.896822 82.657768) (xy 87.896822 94.657768) (xy 99.371822 94.657768)
-        (xy 99.421822 42.907768)
+        (xy 93.396822 82.658727) (xy 93.396822 45.408727) (xy 72.146822 45.408727) (xy 72.146822 82.658727)
       )
     )

Commit message: Updated fiducials.
Parts:
- FID1, FID2, FID3, FID4, FID5, FID6: footprint Fiducial:Fiducial_1mm_Mask2mm -> Fiducial_LE:Fiducial_1mm_Mask2mm
Connections:
- C34 pad 1: Net-(C33-Pad1) -> (no net)
- C34 pad 2: (no net) -> Net-(C33-Pad1)
