File: Naquadah Generator Main/Power.sch (KiCad schematic (older format))
At the start: 0 parts

Commit message: Added real power schematic
Parts:
- added C10, C16: 22uF, Li-ion 5A Boost 1A Charge Protect:0805_2012Metric_HandSolder, symbol Li-ion_5A_Boost_1A_Charge_Protect:C
- added C11, C19: 470uF, Li-ion 5A Boost 1A Charge Protect:UCD1E471MNL1GS, symbol Li-ion_5A_Boost_1A_Charge_Protect:CP1
- added C12, C18: 10uF, Li-ion 5A Boost 1A Charge Protect:0805_2012Metric_HandSolder, symbol Li-ion_5A_Boost_1A_Charge_Protect:C
- added C13: 2.2nF, Li-ion 5A Boost 1A Charge Protect:0805_2012Metric_HandSolder, symbol Li-ion_5A_Boost_1A_Charge_Protect:C
- added C14: 1uF, Li-ion 5A Boost 1A Charge Protect:0805_2012Metric_HandSolder, symbol Li-ion_5A_Boost_1A_Charge_Protect:C
- added C15: 47pF, Li-ion 5A Boost 1A Charge Protect:0805_2012Metric_HandSolder, symbol Li-ion_5A_Boost_1A_Charge_Protect:C
- added C17: 10nF, Li-ion 5A Boost 1A Charge Protect:0805_2012Metric_HandSolder, symbol Li-ion_5A_Boost_1A_Charge_Protect:C
- added C9: 100nF, Li-ion 5A Boost 1A Charge Protect:0805_2012Metric_HandSolder, symbol Li-ion_5A_Boost_1A_Charge_Protect:C
- added D26, D27: GREEN, Li-ion 5A Boost 1A Charge Protect:LED_0805_2012Metric_HandSolder, symbol Li-ion_5A_Boost_1A_Charge_Protect:LED
- added D28, D30: RED, Li-ion 5A Boost 1A Charge Protect:LED_0805_2012Metric_HandSolder, symbol Li-ion_5A_Boost_1A_Charge_Protect:LED
- added D29: NTS12120EMFST1G, Li-ion 5A Boost 1A Charge Protect:NTS12120EMFST1G, symbol Li-ion_5A_Boost_1A_Charge_Protect:D_NTS12120EMFST1G
- added L1: 6.8uH, Li-ion 5A Boost 1A Charge Protect:L_MGV1004, symbol Li-ion_5A_Boost_1A_Charge_Protect:L
- added R31: 330, Li-ion 5A Boost 1A Charge Protect:0805_2012Metric_HandSolder, symbol Li-ion_5A_Boost_1A_Charge_Protect:R
- added R32: 2.7k, Li-ion 5A Boost 1A Charge Protect:0805_2012Metric_HandSolder, symbol Li-ion_5A_Boost_1A_Charge_Protect:R
- added R33, R34, R35, R36, R42: 1k, Li-ion 5A Boost 1A Charge Protect:0805_2012Metric_HandSolder, symbol Li-ion_5A_Boost_1A_Charge_Protect:R
- added R37: 1.54k, Li-ion 5A Boost 1A Charge Protect:0805_2012Metric_HandSolder, symbol Li-ion_5A_Boost_1A_Charge_Protect:R
- added R38: 51k, Li-ion 5A Boost 1A Charge Protect:0805_2012Metric_HandSolder, symbol Li-ion_5A_Boost_1A_Charge_Protect:R
- added R39: 69.8k, Li-ion 5A Boost 1A Charge Protect:0805_2012Metric_HandSolder, symbol Li-ion_5A_Boost_1A_Charge_Protect:R
- added R40: 30k, Li-ion 5A Boost 1A Charge Protect:0805_2012Metric_HandSolder, symbol Li-ion_5A_Boost_1A_Charge_Protect:R
- added R41: 10k, Li-ion 5A Boost 1A Charge Protect:0805_2012Metric_HandSolder, symbol Li-ion_5A_Boost_1A_Charge_Protect:R
- added SW3: SW_SPST, Li-ion 5A Boost 1A Charge Protect:GF1230054, symbol Li-ion_5A_Boost_1A_Charge_Protect:SW_SPST
- added TH1: 10k, Li-ion 5A Boost 1A Charge Protect:0805_2012Metric_HandSolder, symbol Li-ion_5A_Boost_1A_Charge_Protect:Thermistor_NTC
- added U5: AP9101CK6, Li-ion 5A Boost 1A Charge Protect:SOT-23-6, symbol Li-ion_5A_Boost_1A_Charge_Protect:AP9101CK6
- added U6: ECH8695R-TL-W, Li-ion 5A Boost 1A Charge Protect:SOT65P280X95-8N, symbol Li-ion_5A_Boost_1A_Charge_Protect:ECH8695R-TL-W_Gates_on_Top
- added U7: MCP73833T, Li-ion 5A Boost 1A Charge Protect:MCP73833, symbol Li-ion_5A_Boost_1A_Charge_Protect:MCP73833T
- added U8: PAM2423AECADJR, Li-ion 5A Boost 1A Charge Protect:PAM2423AECADJR, symbol Li-ion_5A_Boost_1A_Charge_Protect:PAM2423AECADJR
- added W1, W2, W3, W4, W5, W6, W7, W8: 2.5x5.0, Li-ion 5A Boost 1A Charge Protect:Pad_3.0-5.0_w_TH, symbol Li-ion_5A_Boost_1A_Charge_Protect:TestPoint
Connections:
- net labels added: BATT+, BATT-, BOOSTVIN, BOOSTVOUT, COMP, FB, PG, PROG, PVDD, PVM, SS, ST1, ST2, SW, THRM, THRMIC, VUSB
- net labels removed: 5VO, BATGND, BATV, GNDIN, GNDO, VIN
- wire segments 5 -> 167
- no-connect marks 0 -> 4
Other:
- note added: "+"
- note added: "-"
- note added: "5V Boost"
- note added: "Charge"
- note added: "Connectors"
- note added: "Protection"

Commit message: Symbol field corrections and additions
Parts:
- removed SW3: SW_SPST, Li-ion 5A Boost 1A Charge Protect:GF1230054, symbol Li-ion_5A_Boost_1A_Charge_Protect:SW_SPST
- removed W5, W6: 2.5x5.0, Li-ion 5A Boost 1A Charge Protect:Pad_3.0-5.0_w_TH, symbol Li-ion_5A_Boost_1A_Charge_Protect:TestPoint
- added BT?: Battery_Cell, Connector_Wire:SolderWirePad_1x02_P3.81mm_Drill1mm, symbol Device:Battery_Cell
- added SW?: SW_SPST, Connector_Wire:SolderWirePad_1x02_P3.81mm_Drill1mm, symbol Frequently_Used:SW_SPST
- C10, C16: Manfacturer Part No. CL21A226KQCLRNC -> (none); Manufacturer Part No. (none) -> CL21A226KQCLRNC
- C11, C19: Manfacturer Part No. UCD1E471MNL1GS -> (none); Manufacturer Name (none) -> Nichicon; Manufacturer Part No. (none) -> UCD1E471MNL1GS
- C12, C18: Manfacturer Part No. CL21A106KQCLRNC -> (none); Manufacturer Name Samsung Electro-Mechanics -> Samsung Electro-Mechanics; Manufacturer Part No. (none) -> CL21A106KQCLRNC
- C13: Manfacturer Part No. CL21B222KBANNNC -> (none); Manufacturer Name Samsung Electro-Mechanics -> Samsung Electro-Mechanics; Manufacturer Part No. (none) -> CL21B222KBANNNC
- C14: Manfacturer Part No. CL21B105KOFNNWE -> (none); Manufacturer Part No. (none) -> CL21B105KOFNNWE
- C15: Manfacturer Part No. CL21C470JBANNNC -> (none); Manufacturer Part No. (none) -> CL21C470JBANNNC
- C17: Manfacturer Part No. CL21B103KBANNNC -> (none); Manufacturer Part No. (none) -> CL21B103KBANNNC
- C9: Manfacturer Part No. CL21B104MBCNNNC -> (none); Manufacturer Name (none) -> Samsung Electro-Mechanics; Manufacturer Part No. (none) -> CL21B104MBCNNNC
- D26, D27: Manfacturer Part No. 150080VS75000 -> (none); Manufacturer Part No. (none) -> 150080VS75000
- D28, D30: Manfacturer Part No. 150080RS75000 -> (none); Manufacturer Part No. (none) -> 150080RS75000
- D29: Manfacturer Part No. NTS12120EMFST1G -> (none); Manufacturer Name (none) -> ON Semiconductor; Manufacturer Part No. (none) -> NTS12120EMFST1G
- L1: Manfacturer Part No. MGV10046R8M-10 -> (none); Manufacturer Name (none) -> Laird-Signal Integrity Products; Manufacturer Part No. (none) -> MGV10046R8M-10
- R31: Manfacturer Part No. RK73H2ATTD3300F -> (none); Manufacturer Name (none) -> KOA Speer Electronics, Inc.; Manufacturer Part No. (none) -> RK73H2ATTD3300F
- R32: Manfacturer Part No. RK73H2ATTD2701F -> (none); Manufacturer Name (none) -> KOA Speer Electronics, Inc.; Manufacturer Part No. (none) -> RK73H2ATTD2701F
- R33, R34, R35, R36, R42: Manfacturer Part No. RK73H2ATTD1001F -> (none); Manufacturer Name (none) -> KOA Speer Electronics, Inc.; Manufacturer Part No. (none) -> RK73H2ATTD1001F
- R37: Manfacturer Part No. RK73H2ATTD1541F -> (none); Manufacturer Name (none) -> KOA Speer Electronics, Inc.; Manufacturer Part No. (none) -> RK73H2ATTD1541F
- R38: Manfacturer Part No. RK73H2ATTD5102F -> (none); Manufacturer Name (none) -> KOA Speer Electronics, Inc.; Manufacturer Part No. (none) -> RK73H2ATTD5102F
- R39: Manfacturer Part No. RK73H2ATTD6982F -> (none); Manufacturer Name (none) -> KOA Speer Electronics, Inc.; Manufacturer Part No. (none) -> RK73H2ATTD6982F
- R40: Manfacturer Part No. RK73H2ATTD3002F -> (none); Manufacturer Name (none) -> KOA Speer Electronics, Inc.; Manufacturer Part No. (none) -> RK73H2ATTD3002F
- R41: Manfacturer Part No. RK73H2ATTD1002F -> (none); Manufacturer Name (none) -> KOA Speer Electronics, Inc.; Manufacturer Part No. (none) -> RK73H2ATTD1002F
- TH1: Manfacturer Part No. NTCG203NH103JT1 -> (none); Manufacturer Name (none) -> TDK Corporation; Manufacturer Part No. (none) -> NTCG203NH103JT1
- U5: Manfacturer Part No. AP9101CK6-AYTRG1 -> (none); Manufacturer Name (none) -> Diodes Incorporated; Manufacturer Part No. (none) -> AP9101CK6-AYTRG1
- U6: Manfacturer Part No. ECH8695R-TL-W -> (none); Manufacturer Name (none) -> ON Semiconductor; Manufacturer Part No. (none) -> ECH8695R-TL-W
- U7: Digikey Part No. MCP73833T-AMI/UNCT-ND -> MCP73833T-AMI/UNCT-ND; Manfacturer Part No. MCP73833T-AMI/UN -> (none); Manufacturer Name (none) -> Microchip Technology; Manufacturer Part No. (none) -> MCP73833T-AMI/UN
- U8: Manfacturer Part No. PAM2423AECADJR -> (none); Manufacturer Name (none) -> Diodes Incorporated; Manufacturer Part No. (none) -> PAM2423AECADJR
- W1, W2, W3, W4, W7, W8: Manfacturer Part No. None -> (none); Manufacturer Part No. (none) -> None
Other:
- moved on the sheet: C11, C12, C13, C14, C15, C17, C18, C19, C9, D29, D30, L1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

Commit message: Adding Power Daughter Board
Parts:
- added Q?: 30V 5A, Naquadah_Generator:SOT-23_Handsoldering, symbol Transistor_FET:BSS138
- added R?: 1k, Li-ion 5A Boost 1A Charge Protect:0805_2012Metric_HandSolder, symbol Li-ion_5A_Boost_1A_Charge_Protect:R
- added R?: 100, Li-ion 5A Boost 1A Charge Protect:0805_2012Metric_HandSolder, symbol Li-ion_5A_Boost_1A_Charge_Protect:R
- added TP? (x2): TestPoint, Frequently_Used:Pad_2.5-2.5, symbol Naquadah_Generator:TestPoint
- C10, C16: Digikey Part No. 1276-6687-1-ND -> (none); Source (none) -> Digikey; Source Part No. (none) -> 1276-6687-1-ND
- C11, C19: Digikey Part No. 493-6386-1-ND -> (none); Source (none) -> Digikey; Source Part No. (none) -> 493-6386-1-ND
- C12, C18: Digikey Part No. 1276-2405-1-ND -> (none); Source (none) -> Digikey; Source Part No. (none) -> 1276-2405-1-ND
- C13: Digikey Part No. 1276-1171-1-ND -> (none); Source (none) -> Digikey; Source Part No. (none) -> 1276-1171-1-ND
- C14: Digikey Part No. 1276-2931-1-ND -> (none); Source (none) -> Digikey; Source Part No. (none) -> 1276-2931-1-ND
- C15: Digikey Part No. 1276-1156-1-ND -> (none); Source (none) -> Digikey; Source Part No. (none) -> 1276-1156-1-ND
- C17: Digikey Part No. 1276-1015-1-ND -> (none); Source (none) -> Digikey; Source Part No. (none) -> 1276-1015-1-ND
- C9: Digikey Part No. 1276-2450-1-ND -> (none); Source (none) -> Digikey; Source Part No. (none) -> 1276-2450-1-ND
- D26, D27: Digikey Part No. 732-4986-1-ND -> (none); Source (none) -> Digikey; Source Part No. (none) -> 732-4986-1-ND
- D28, D30: Digikey Part No. 732-4984-1-ND -> (none); Source (none) -> Digikey; Source Part No. (none) -> 732-4984-1-ND
- D29: value NTS12120EMFST1G -> 5A 100V; footprint Li-ion 5A Boost 1A Charge Protect:NTS12120EMFST1G -> Li-ion 5A Boost 1A Charge Protect:DO-214AC; symbol Li-ion_5A_Boost_1A_Charge_Protect:D_NTS12120EMFST1G -> Li-ion_5A_Boost_1A_Charge_Protect:D; Description Diode Schottky 120V 12A -> Diode Schottky 100V 5A Surface Mount DO-221AC (SlimSMA); Digikey Part No. NTS12120EMFST1GOSCT-ND -> (none); Manufacturer Name ON Semiconductor -> Vishay Semiconductor Diodes Division; Manufacturer Part No. NTS12120EMFST1G -> VSSAF510-M3/H; Source (none) -> Digikey; Source Part No. (none) -> VSSAF510-M3/HGICT-ND
- L1: footprint Li-ion 5A Boost 1A Charge Protect:L_MGV1004 -> Li-ion 5A Boost 1A Charge Protect:L_MGV0605; Description 6.8µH Shielded Molded Inductor 8A 23.3mOhm -> 6.8µH Shielded Molded Inductor 5.5A 44.6mOhm Max Nonstandard; Digikey Part No. 240-2938-1-ND -> (none); Manufacturer Part No. MGV10046R8M-10 -> MGV06056R8M-10; Source (none) -> Digikey; Source Part No. (none) -> 240-2915-1-ND
- R31: Digikey Part No. 2019-RK73H2ATTD3300FCT-ND -> (none); Source (none) -> Digikey; Source Part No. (none) -> 2019-RK73H2ATTD3300FCT-ND
- R32: Digikey Part No. 2019-RK73H2ATTD2701FCT-ND -> (none); Source (none) -> Digikey; Source Part No. (none) -> 2019-RK73H2ATTD2701FCT-ND
- R33, R34, R35, R36, R42: Digikey Part No. 2019-RK73H2ATTD1001FCT-ND -> (none); Source (none) -> Digikey; Source Part No. (none) -> 2019-RK73H2ATTD1001FCT-ND
- R37: Digikey Part No. 2019-RK73H2ATTD1541FCT-ND -> (none); Source (none) -> Digikey; Source Part No. (none) -> 2019-RK73H2ATTD1541FCT-ND
- R38: Digikey Part No. 2019-RK73H2ATTD5102FCT-ND -> (none); Source (none) -> Digikey; Source Part No. (none) -> 2019-RK73H2ATTD5102FCT-ND
- R39: Digikey Part No. 2019-RK73H2ATTD6982FCT-ND -> (none); Source (none) -> Digikey; Source Part No. (none) -> 2019-RK73H2ATTD6982FCT-ND
- R40: Digikey Part No. 2019-RK73H2ATTD3002FCT-ND -> (none); Source (none) -> Digikey; Source Part No. (none) -> 2019-RK73H2ATTD3002FCT-ND
- R41: Digikey Part No. 2019-RK73H2ATTD1002FCT-ND -> (none); Source Part No. (none) -> 2019-RK73H2ATTD1002FCT-ND
- TH1: Digikey Part No. 445-175460-1-ND -> (none); Source (none) -> Digikey; Source Part No. (none) -> 445-175460-1-ND
- U5: Digikey Part No. AP9101CK6-AYTRG1DICT-ND -> (none); Source (none) -> Digikey; Source Part No. (none) -> AP9101CK6-AYTRG1DICT-ND
- U6: Digikey Part No. ECH8695R-TL-WOSCT-ND -> (none); Source (none) -> Digikey; Source Part No. (none) -> ECH8695R-TL-WOSCT-ND
- U7: Digikey Part No. MCP73833T-AMI/UNCT-ND -> (none); Source (none) -> Digikey; Source Part No. (none) -> MCP73833T-AMI/UNCT-ND
- U8: Description Boost Switching Regulator IC -> Boost Switching Regulator IC Positive Adjustable 2.7V 1 Out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; Digikey Part No. PAM2423AECADJRDICT-ND -> (none); Manufacturer Part No. PAM2423AECADJR -> PAM2421AECADJR; Source (none) -> Digikey; Source Part No. (none) -> PAM2421AECADJRDICT-ND
- W1, W2, W3, W4, W7, W8: Digikey Part No. None -> (none); Source (none) -> None; Source Part No. (none) -> None
- gave numbers to parts that had none: 2
Connections:
- net BATT+: now also BT1.1 (+), TP?.1
- net BATT-: now also Q?.3 (D); no longer BT1.2 (-)
- net BOOSTVOUT: now also D29.1 (K); no longer D29.5 (K), D29.5A (K), D29.5B (K), D29.5C (K), D29.5D (K)
- net SW: no longer D29.1 (A), D29.3 (A)
- net at SW2.1 (A): now also R?.1; no longer BT1.1 (+)
- new net: BT1.2 (-), Q?.2 (S), R?.1, TP?.1
- new net: Q?.1 (G), R?.2, R?.2
Other:
- moved on the sheet: BT1, SW2

Commit message: Clean up
Parts:
- removed C10, C16: 22uF, Li-ion 5A Boost 1A Charge Protect:0805_2012Metric_HandSolder, symbol Li-ion_5A_Boost_1A_Charge_Protect:C
- removed D26, D27: GREEN, Li-ion 5A Boost 1A Charge Protect:LED_0805_2012Metric_HandSolder, symbol Li-ion_5A_Boost_1A_Charge_Protect:LED
- removed D28: RED, Li-ion 5A Boost 1A Charge Protect:LED_0805_2012Metric_HandSolder, symbol Li-ion_5A_Boost_1A_Charge_Protect:LED
- removed R33, R34, R35, R36: 1k, Li-ion 5A Boost 1A Charge Protect:0805_2012Metric_HandSolder, symbol Li-ion_5A_Boost_1A_Charge_Protect:R
- removed R37: 1.54k, Li-ion 5A Boost 1A Charge Protect:0805_2012Metric_HandSolder, symbol Li-ion_5A_Boost_1A_Charge_Protect:R
- removed R39: 69.8k, Li-ion 5A Boost 1A Charge Protect:0805_2012Metric_HandSolder, symbol Li-ion_5A_Boost_1A_Charge_Protect:R
- removed SW2: SW_SPST, Connector_Wire:SolderWirePad_1x02_P3.81mm_Drill1mm, symbol Frequently_Used:SW_SPST
- removed TH1: 10k, Li-ion 5A Boost 1A Charge Protect:0805_2012Metric_HandSolder, symbol Li-ion_5A_Boost_1A_Charge_Protect:Thermistor_NTC
- removed U7: MCP73833T, Li-ion 5A Boost 1A Charge Protect:MCP73833, symbol Li-ion_5A_Boost_1A_Charge_Protect:MCP73833T
- removed W1, W2, W3, W4: 2.5x5.0, Li-ion 5A Boost 1A Charge Protect:Pad_3.0-5.0_w_TH, symbol Li-ion_5A_Boost_1A_Charge_Protect:TestPoint
- added J?: Power_Daughter_Conn, Naquadah_Generator:State_Sensing_Mother_Board_JST_Conn, symbol Naquadah_Generator:Power_Daughter_Conn
- added J?: Conn_XT, symbol Connectors_LE:Conn_XT
Connections:
- net BATT+: now also J?.2 (+), J?.3 (BATT+), J?.4 (BATT+)
- net BATT-: now also J?.1 (-)
- net GND: now also J?.1 (GND), J?.2 (GND)
- net at Q?.1 (G), R?.2: now also R?.1; no longer R?.2
- new net READY: J?.6 (RDY)
- new net SWITCH: J?.5 (SW), R?.2
Other:
- note removed: "Charge"
- moved on the sheet: C11, C12, C13, C14, C15, C17, C18, C19, C9, D29, D30, L1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

Commit message: Switched to 4 pin power board connector
Parts:
- removed BT1: Battery_Cell, Connector_Wire:SolderWirePad_1x02_P3.81mm_Drill1mm, symbol Device:Battery_Cell
- J?: footprint Naquadah_Generator:State_Sensing_Mother_Board_JST_Conn -> Naquadah_Generator:Power_Mother_Board_Conn
- TP? (x2): symbol Naquadah_Generator:TestPoint -> Frequently_Used:TestPoint
Connections:
- net BATT-: no longer J?.1 (-)
- net at Q?.2 (S), R?.1, TP?.1: now also J?.1 (-)
Other:
- note removed: "+"
- note removed: "-"
- moved on the sheet: J?, Q?, R?, TP?
