File: Naquadah Generator Main/Power.sch (KiCad schematic (older format))
At the start: 31 parts, among them J10 Power Board Conn, J9 Power_Conn, Q1 30V 5A, U5 AP9101CK6, U6 ECH8695R-TL-W, U8 PAM2423AECADJR

Commit message: Power updates
Parts:
- removed C11, C19: 470uF, Li-ion:UCD1E471MNL1GS, symbol Li_Ion_LE:CP1
- removed C12, C18: 10uF, Li-ion:0805_2012Metric_HandSolder, symbol Li_Ion_LE:C
- removed C13: 2.2nF, Li-ion:0805_2012Metric_HandSolder, symbol Li_Ion_LE:C
- removed C14: 1uF, Li-ion:0805_2012Metric_HandSolder, symbol Li_Ion_LE:C
- removed C15: 47pF, Li-ion:0805_2012Metric_HandSolder, symbol Li_Ion_LE:C
- removed C17: 10nF, Li-ion:0805_2012Metric_HandSolder, symbol Li_Ion_LE:C
- removed C9: 100nF, Li-ion:0805_2012Metric_HandSolder, symbol Li_Ion_LE:C
- removed D29: 5A 100V, Li-ion:DO-214AC, symbol Li_Ion_LE:D
- removed L1: 6.8uH, Li-ion:L_MGV0605, symbol Li_Ion_LE:L
- removed R31: 330, Frequently_Used_LE:0805_2012Metric_HandSolder, symbol Li_Ion_LE:R
- removed R32: 2.7k, Frequently_Used_LE:0805_2012Metric_HandSolder, symbol Li_Ion_LE:R
- removed R38: 51k, Frequently_Used_LE:0805_2012Metric_HandSolder, symbol Li_Ion_LE:R
- removed R40: 30k, Frequently_Used_LE:0805_2012Metric_HandSolder, symbol Li_Ion_LE:R
- removed R41: 10k, Frequently_Used_LE:0805_2012Metric_HandSolder, symbol Li_Ion_LE:R
- removed U5: AP9101CK6, Li-ion:SOT-23-6, symbol Li_Ion_LE:AP9101CK6
- removed U6: ECH8695R-TL-W, Li-ion:SOT65P280X95-8N, symbol Li_Ion_LE:ECH8695R-TL-W_Gates_on_Top
- removed U8: PAM2423AECADJR, Li-ion:PAM2423AECADJR, symbol Li_Ion_LE:PAM2423AECADJR
- R2, R33: symbol Li_Ion_LE:R -> Frequently_Used_LE:R
- TP1, TP10, TP11, TP2, TP7, TP8, TP9: symbol Frequently_Used_LE:TestPoint -> Frequently_Used_LE:TestPoint_1
Connections:
- net labels added: +3.3V
- net labels removed: COMP, FB, PG1, PG2, PVDD, PVM, SS, SW
- wire segments 124 -> 51
- no-connect marks 4 -> 0
Other:
- note added: "3.3V 500mA Buck"
- note added: "5V 3.0A Boost"
- note removed: "5V Boost"
- moved on the sheet: J10, J9, Q1

Commit message: Audio updates, switching to separate USB schematic
Audio updates, switching to separate USB schematic
Changed lines of the file:
@@
 $Descr A 11000 8500
 encoding utf-8
-Sheet 11 15
+Sheet 11 16
 Title "Li-ion 3A Boost 1A Charge Protect"
 Date ""
@@
 Text Label 4800 2250 0    50   ~ 0
 BATT+
-Text Label 4650 2350 0    50   ~ 0
+Text Label 4700 2350 0    50   ~ 0
 BOOSTVOUT
 $Comp
 L Frequently_Used_LE:+5V #PWR?
 U 1 1 5EE5FC65
-P 4650 2250
+P 4200 2250
 AR Path="/5EE5FC65" Ref="#PWR?"  Part="1"
 AR Path="/5EA6751D/5EE5FC65" Ref="#PWR021"  Part="1"
-F 0 "#PWR021" H 4650 2100 50  0001 C CNN
-F 1 "+5V" H 4665 2423 50  0000 C CNN
-F 2 "" H 4650 2250 50  0001 C CNN
-F 3 "" H 4650 2250 50  0001 C CNN
-	1    4650 2250
-	1    0    0    -1
-$EndComp
-Wire Wire Line
-	4650 2350 4650 2250
+F 0 "#PWR021" H 4200 2100 50  0001 C CNN
+F 1 "+5V" H 4215 2423 50  0000 C CNN
+F 2 "" H 4200 2250 50  0001 C CNN
+F 3 "" H 4200 2250 50  0001 C CNN
+	1    4200 2250
+	1    0    0    -1
+$EndComp
+Wire Wire Line
+	4200 2350 4200 2250
 $Comp
 L Frequently_Used_LE:DGND #PWR022
 U 1 1 5EE6F6B6
-P 4650 2550
-F 0 "#PWR022" H 4650 2300 50  0001 C CNN
-F 1 "DGND" H 4655 2377 50  0000 C CNN
-F 2 "" H 4650 2550 50  0001 C CNN
-F 3 "" H 4650 2550 50  0001 C CNN
-	1    4650 2550
-	1    0    0    -1
-$EndComp
-Wire Wire Line
-	4650 2450 4650 2550
-Wire Wire Line
-	4650 2350 5150 2350
+P 4200 2550
+F 0 "#PWR022" H 4200 2300 50  0001 C CNN
+F 1 "DGND" H 4205 2377 50  0000 C CNN
+F 2 "" H 4200 2550 50  0001 C CNN
+F 3 "" H 4200 2550 50  0001 C CNN
+	1    4200 2550
+	1    0    0    -1
+$EndComp
+Wire Wire Line
+	4200 2450 4200 2550
 Wire Wire Line
 	4800 2250 5150 2250
@@
 F4 "GND" I L 5150 2450 50
 $EndSheet
-Wire Wire Line
-	4650 2450 5150 2450
 $Sheet
 S 2750 2100 550  400
@@
 L Frequently_Used_LE:+3.3V #PWR0143
 U 1 1 5F3E6A42
-P 7450 2100
-F 0 "#PWR0143" H 7450 1950 50  0001 C CNN
-F 1 "+3.3V" H 7465 2273 50  0000 C CNN
-F 2 "" H 7450 2100 50  0001 C CNN
-F 3 "" H 7450 2100 50  0001 C CNN
-	1    7450 2100
-	1    0    0    -1
-$EndComp
-Wire Wire Line
-	7450 2300 7450 2100
-Wire Wire Line
-	7450 2300 7950 2300
+P 7050 2100
+F 0 "#PWR0143" H 7050 1950 50  0001 C CNN
+F 1 "+3.3V" H 7065 2273 50  0000 C CNN
+F 2 "" H 7050 2100 50  0001 C CNN
+F 3 "" H 7050 2100 50  0001 C CNN
+	1    7050 2100
+	1    0    0    -1
+$EndComp
+Wire Wire Line
+	7050 2300 7050 2100
 Text Notes 7700 3000 0    79   ~ 16
 3.3V 500mA Buck
+Text HLabel 7850 5200 2    50   Input ~ 0
+BATT+
+$Comp
+L Frequently_Used_LE:PWR_FLAG #FLG0101
+U 1 1 5F47F237
+P 4600 2250
+F 0 "#FLG0101" H 4600 2325 50  0001 C CNN
+F 1 "PWR_FLAG" H 4600 2423 50  0000 C CNN
+F 2 "" H 4600 2250 50  0001 C CNN
+F 3 "~" H 4600 2250 50  0001 C CNN
+	1    4600 2250
+	1    0    0    -1
+$EndComp
+Wire Wire Line
+	4600 2350 4600 2250
+Wire Wire Line
+	4200 2350 4600 2350
+Wire Wire Line
+	4600 2350 5150 2350
+Connection ~ 4600 2350
+$Comp
+L Frequently_Used_LE:PWR_FLAG #FLG0102
+U 1 1 5F4889FE
+P 4600 2550
+F 0 "#FLG0102" H 4600 2625 50  0001 C CNN
+F 1 "PWR_FLAG" H 4600 2723 50  0000 C CNN
+F 2 "" H 4600 2550 50  0001 C CNN
+F 3 "~" H 4600 2550 50  0001 C CNN
+	1    4600 2550
+	-1   0    0    1
+$EndComp
+Wire Wire Line
+	4200 2450 4600 2450
+Wire Wire Line
+	4600 2550 4600 2450
+Connection ~ 4600 2450
+Wire Wire Line
+	4600 2450 5150 2450
+Wire Wire Line
+	7050 2300 7950 2300
 $EndSCHEMATC

Commit message: Added level shifter, moved user interface connector location
Added level shifter, moved user interface connector location
Parts:
- removed J10: Power Board Conn, Naquadah_Generator:Daughter_Board_Vert_5_Pin_JST_Conn, symbol Naquadah_Generator:Power_Daughter_5_Pin_Conn
- removed TP10, TP2, TP7, TP8, TP9: TestPoint, Frequently_Used_LE:Pad_2.5-2.5, symbol Frequently_Used_LE:TestPoint_1
- R2: footprint Frequently_Used_LE:0805_2012Metric_HandSolder -> Frequently_Used_LE:0805_2012Metric
- R33: footprint Frequently_Used_LE:0805_2012Metric_HandSolder -> Frequently_Used_LE:0805_2012Metric; Description 1 kOhms ±1% 0.25W, 1/4W Chip Resistor 1206 (3216 Metric) -> 100 Ohms ±1% 0.25W, 1/4W Chip Resistor 0805 (2012 Metric) A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; Manufacturer Part No. RK73H2ATTD1001F -> RK73H2ATTD1000F; Source Part No. 2019-RK73H2ATTD1001FCT-ND -> 2019-RK73H2ATTD1000FCT-ND
Other:
- note added: "Battery Connector and Main Power Switch"
- note removed: "Battery Connector and Power Main Switch"
- note removed: "Daughter Board Connector"
- moved on the sheet: J9, Q1, R2, R33, TP1, TP11

Commit message: Switched to 0603_1608M size for passives
Parts:
- J9: symbol Connectors_LE:Power_Conn -> Connector_LE:Power_Conn; Description (none) -> Battery Holder (Open) 18650 1 Cell SMD (SMT) Tab; Manufacturer Name (none) -> Keystone Electronics; Manufacturer Part No. (none) -> 1042; Source (none) -> Digikey; Source Part No. (none) -> 36-1042-ND
- R2: footprint Frequently_Used_LE:0805_2012Metric -> Frequently_Used_LE:0603_1608Metric; Description 1 kOhms ±1% 0.25W, 1/4W Chip Resistor 1206 (3216 Metric) -> 1 kOhms ±1% 0.25W, 1/4W Chip Resistor 0603 (1608 Metric) Au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; Manufacturer Name KOA Speer Electronics, Inc. -> Rohm Semiconductor; Manufacturer Part No. RK73H2ATTD1001F -> ESR03EZPF1001; Source Part No. 2019-RK73H2ATTD1001FCT-ND -> RHM1.00KADCT-ND
- R33: footprint Frequently_Used_LE:0805_2012Metric -> Frequently_Used_LE:0603_1608Metric; Description 100 Ohms ±1% 0.25W, 1/4W Chip Resistor 0805 (2012 Metric) A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 -> 100 Ohms ±1% 0.25W, 1/4W Chip Resistor 0603 (1608 Metric) A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; Manufacturer Name KOA Speer Electronics, Inc. -> Panasonic Electronic Components; Manufacturer Part No. RK73H2ATTD1000F -> ERJ-PA3F1000V; Source Part No. 2019-RK73H2ATTD1000FCT-ND -> P100BYCT-ND
- TP1, TP11: Description None -> Test point
Changed lines of the file:
@@
 $Descr A 11000 8500
 encoding utf-8
-Sheet 10 17
+Sheet 10 18
 Title "Li-ion 3A Boost 1A Charge Protect"
 Date ""
@@
 F 0 "R33" V 4000 5250 59  0000 C CNN
 F 1 "100" V 3800 5250 59  0000 C CNN
-F 2 "Frequently_Used_LE:0805_2012Metric" H 3900 5250 50  0001 C CNN
-F 3 "http://www.koaspeer.com/pdfs/RK73H.pdf" H 3900 5250 50  0001 C CNN
-F 4 "100 Ohms ±1% 0.25W, 1/4W Chip Resistor 0805 (2012 Metric) Automotive AEC-Q200, Moisture Resistant Thick Film" H 3900 5250 50  0001 C CNN "Description"
-F 5 "2019-RK73H2ATTD1000FCT-ND" H 3900 5250 50  0001 C CNN "Source Part No."
-F 6 "RK73H2ATTD1000F" H 3900 5250 50  0001 C CNN "Manufacturer Part No."
-F 7 "KOA Speer Electronics, Inc." H 3900 5250 50  0001 C CNN "Manufacturer Name"
+F 2 "Frequently_Used_LE:0603_1608Metric" H 3900 5250 50  0001 C CNN
+F 3 "https://industrial.panasonic.com/cdbs/www-data/pdf/RDO0000/AOA0000C331.pdf" H 3900 5250 50  0001 C CNN
+F 4 "100 Ohms ±1% 0.25W, 1/4W Chip Resistor 0603 (1608 Metric) Automotive AEC-Q200, Pulse Withstanding Thick Film" H 3900 5250 50  0001 C CNN "Description"
+F 5 "P100BYCT-ND" H 3900 5250 50  0001 C CNN "Source Part No."
+F 6 "ERJ-PA3F1000V" H 3900 5250 50  0001 C CNN "Manufacturer Part No."
+F 7 "Panasonic Electronic Components" H 3900 5250 50  0001 C CNN "Manufacturer Name"
 F 8 "Digikey" H 3900 5250 50  0001 C CNN "Source"
 	1    3900 5250
@@
 F 0 "R2" V 3200 5000 59  0000 C CNN
 F 1 "1k" V 3400 5000 59  0000 C CNN
-F 2 "Frequently_Used_LE:0805_2012Metric" H 3300 5000 50  0001 C CNN
-F 3 "http://www.koaspeer.com/pdfs/RK73H.pdf" H 3300 5000 50  0001 C CNN
-F 4 "1 kOhms ±1% 0.25W, 1/4W Chip Resistor 1206 (3216 Metric) " H 3300 5000 50  0001 C CNN "Description"
-F 5 "2019-RK73H2ATTD1001FCT-ND" H 3300 5000 50  0001 C CNN "Source Part No."
-F 6 "RK73H2ATTD1001F" H 3300 5000 50  0001 C CNN "Manufacturer Part No."
-F 7 "KOA Speer Electronics, Inc." H 3300 5000 50  0001 C CNN "Manufacturer Name"
+F 2 "Frequently_Used_LE:0603_1608Metric" H 3300 5000 50  0001 C CNN
+F 3 "https://d1d2qsbl8m0m72.cloudfront.net/en/products/databook/datasheet/passive/resistor/chip_resistor/esr-e.pdf" H 3300 5000 50  0001 C CNN
+F 4 "1 kOhms ±1% 0.25W, 1/4W Chip Resistor 0603 (1608 Metric) Automotive AEC-Q200, Pulse Withstanding Thick Film" H 3300 5000 50  0001 C CNN "Description"
+F 5 "RHM1.00KADCT-ND" H 3300 5000 50  0001 C CNN "Source Part No."
+F 6 "ESR03EZPF1001" H 3300 5000 50  0001 C CNN "Manufacturer Part No."
+F 7 "Rohm Semiconductor" H 3300 5000 50  0001 C CNN "Manufacturer Name"
 F 8 "Digikey" H 3300 5000 50  0001 C CNN "Source"
 	1    3300 5000
@@
 	2500 4650 2700 4650
 $Comp
-L Connectors_LE:Power_Conn J9
+L Connector_LE:Power_Conn J9
 U 1 1 5EE056F1
 P 2350 4650
@@
 F 1 "Power_Conn" H 2350 4750 50  0000 C CNN
 F 2 "Naquadah_Generator:Keystone-1042" H 2350 4650 50  0001 C CNN
-F 3 "~" H 2350 4650 50  0001 C CNN
+F 3 "https://www.keyelco.com/userAssets/file/M65p27.pdf" H 2350 4650 50  0001 C CNN
+F 4 "Battery Holder (Open) 18650 1 Cell SMD (SMT) Tab" H 2350 4650 50  0001 C CNN "Description"
+F 5 "Keystone Electronics" H 2350 4650 50  0001 C CNN "Manufacturer Name"
+F 6 "1042" H 2350 4650 50  0001 C CNN "Manufacturer Part No."
+F 7 "Digikey" H 2350 4650 50  0001 C CNN "Source"
+F 8 "36-1042-ND" H 2350 4650 50  0001 C CNN "Source Part No."
 	1    2350 4650
 	-1   0    0    1
@@
 F 7 "None" H 7195 4845 50  0001 C CNN "Manufacturer Name"
 F 8 "None" H 7195 4845 50  0001 C CNN "Manufacturer Part No."
-F 9 "None" H 7200 5200 50  0001 C CNN "Description"
+F 9 "Test point" H 7200 5200 50  0001 C CNN "Description"
 	1    7200 5200
 	-1   0    0    1
@@
 F 3 "None" H 4600 4750 50  0001 C CNN
 F 4 "SWBATT-" H 4400 5050 50  0000 C CNN "Name"
-F 5 "None" H 4400 4750 50  0001 C CNN "Description"
+F 5 "Test point" H 4400 4750 50  0001 C CNN "Description"
 F 6 "None" H 4400 4750 50  0001 C CNN "Source Part No."
 F 7 "None" H 4400 4750 50  0001 C CNN "Manufacturer Name"
