File: Naquadah Generator Main/BlueLights.sch (KiCad schematic (older format))
At the start: 10 parts, among them Q6 BC337

Commit message: Before changing BOM
Connections:
- net labels added: +5V, GND
- net labels removed: 5V, VGND
Changed lines of the file:
@@
 $Descr A4 11693 8268
 encoding utf-8
-Sheet 2 14
+Sheet 6 10
 Title ""
 Date ""
@@
 $EndDescr
 Wire Wire Line
-	5450 4750 5400 4750
-Wire Wire Line
-	5450 4550 5450 4750
-Wire Wire Line
-	4650 4350 4850 4350
-Text HLabel 4650 4350 0    50   Input ~ 0
+	5450 4550 5450 4650
+Wire Wire Line
+	4750 4350 4850 4350
+Text HLabel 4750 4350 0    50   Input ~ 0
 SIGNAL
 $Comp
@@
 AR Path="/5E9E5DE1/5E9FDE71" Ref="R3"  Part="1"
 AR Path="/5E9E4A6B/5E9FDE71" Ref="R13"  Part="1"
-F 0 "R23" V 4793 4350 50  0000 C CNN
-F 1 "2.7k" V 4884 4350 50  0000 C CNN
+F 0 "R23" V 4900 4350 50  0000 C CNN
+F 1 "2.7k" V 5100 4350 50  0000 C CNN
 F 2 "Resistor_THT:R_Axial_DIN0207_L6.3mm_D2.5mm_P10.16mm_Horizontal" V 4930 4350 50  0001 C CNN
 F 3 "~" H 5000 4350 50  0001 C CNN
@@
 	0    1    1    0
 $EndComp
-Text GLabel 5400 4750 0    50   Input ~ 0
-VGND
 $Comp
 L Transistor_BJT:BC337 Q6
@@
 	1    0    0    -1
 $EndComp
-Text GLabel 5450 3550 0    50   Input ~ 0
-5V
 Wire Wire Line
 	5450 4150 5800 4150
@@
 	0    -1   -1   0
 $EndComp
+$Comp
+L power:GND #PWR0115
+U 1 1 5EB39A74
+P 5450 4650
+AR Path="/5E9E304D/5EB39A74" Ref="#PWR0115"  Part="1"
+AR Path="/5E9E5DE1/5EB39A74" Ref="#PWR0109"  Part="1"
+AR Path="/5E9E5DDE/5EB39A74" Ref="#PWR0111"  Part="1"
+AR Path="/5E9E4A6B/5EB39A74" Ref="#PWR0113"  Part="1"
+AR Path="/5E9D240B/5EB39A74" Ref="#PWR0117"  Part="1"
+F 0 "#PWR0117" H 5450 4400 50  0001 C CNN
+F 1 "GND" H 5455 4477 50  0000 C CNN
+F 2 "" H 5450 4650 50  0001 C CNN
+F 3 "" H 5450 4650 50  0001 C CNN
+	1    5450 4650
+	1    0    0    -1
+$EndComp
+$Comp
+L power:+5V #PWR0116
+U 1 1 5EB3A90A
+P 5450 3500
+AR Path="/5E9E304D/5EB3A90A" Ref="#PWR0116"  Part="1"
+AR Path="/5E9E5DE1/5EB3A90A" Ref="#PWR0110"  Part="1"
+AR Path="/5E9E5DDE/5EB3A90A" Ref="#PWR0112"  Part="1"
+AR Path="/5E9E4A6B/5EB3A90A" Ref="#PWR0114"  Part="1"
+AR Path="/5E9D240B/5EB3A90A" Ref="#PWR0118"  Part="1"
+F 0 "#PWR0118" H 5450 3350 50  0001 C CNN
+F 1 "+5V" H 5465 3673 50  0000 C CNN
+F 2 "" H 5450 3500 50  0001 C CNN
+F 3 "" H 5450 3500 50  0001 C CNN
+	1    5450 3500
+	1    0    0    -1
+$EndComp
+Wire Wire Line
+	5450 3500 5450 3550
 $EndSCHEMATC

Commit message: Changed name of libraries to remove underscore
Changed lines of the file:
@@
 $Descr A4 11693 8268
 encoding utf-8
-Sheet 6 10
+Sheet 6 11
 Title ""
 Date ""
@@
 AR Path="/5E9E5DE1/5E9FDE71" Ref="R3"  Part="1"
 AR Path="/5E9E4A6B/5E9FDE71" Ref="R13"  Part="1"
-F 0 "R23" V 4900 4350 50  0000 C CNN
+AR Path="/5ED17BA0/5ED2A301/5E9FDE71" Ref="R?"  Part="1"
+AR Path="/5ED17BA0/5ED2A304/5E9FDE71" Ref="R?"  Part="1"
+AR Path="/5ED17BA0/5ED2A307/5E9FDE71" Ref="R?"  Part="1"
+AR Path="/5ED17BA0/5ED2A30A/5E9FDE71" Ref="R?"  Part="1"
+AR Path="/5ED17BA0/5ED2A30D/5E9FDE71" Ref="R?"  Part="1"
+F 0 "R?" V 4900 4350 50  0000 C CNN
 F 1 "2.7k" V 5100 4350 50  0000 C CNN
 F 2 "Resistor_THT:R_Axial_DIN0207_L6.3mm_D2.5mm_P10.16mm_Horizontal" V 4930 4350 50  0001 C CNN
@@
 AR Path="/5E9E5DE1/5E9FDE70" Ref="Q5"  Part="1"
 AR Path="/5E9E4A6B/5E9FDE70" Ref="Q7"  Part="1"
-F 0 "Q4" H 5541 4396 50  0000 L CNN
+AR Path="/5ED17BA0/5ED2A301/5E9FDE70" Ref="Q?"  Part="1"
+AR Path="/5ED17BA0/5ED2A304/5E9FDE70" Ref="Q?"  Part="1"
+AR Path="/5ED17BA0/5ED2A307/5E9FDE70" Ref="Q?"  Part="1"
+AR Path="/5ED17BA0/5ED2A30A/5E9FDE70" Ref="Q?"  Part="1"
+AR Path="/5ED17BA0/5ED2A30D/5E9FDE70" Ref="Q?"  Part="1"
+F 0 "Q?" H 5541 4396 50  0000 L CNN
 F 1 "BC337" H 5541 4305 50  0000 L CNN
 F 2 "Package_TO_SOT_THT:TO-92_Inline" H 5550 4275 50  0001 L CIN
@@
 AR Path="/5E9E5DE1/5E9E70EC" Ref="D3"  Part="1"
 AR Path="/5E9E4A6B/5E9E70EC" Ref="D11"  Part="1"
-F 0 "D19" V 5839 3883 50  0000 R CNN
+AR Path="/5ED17BA0/5ED2A301/5E9E70EC" Ref="D?"  Part="1"
+AR Path="/5ED17BA0/5ED2A304/5E9E70EC" Ref="D?"  Part="1"
+AR Path="/5ED17BA0/5ED2A307/5E9E70EC" Ref="D?"  Part="1"
+AR Path="/5ED17BA0/5ED2A30A/5E9E70EC" Ref="D?"  Part="1"
+AR Path="/5ED17BA0/5ED2A30D/5E9E70EC" Ref="D?"  Part="1"
+F 0 "D?" V 5839 3883 50  0000 R CNN
 F 1 "LED" V 5748 3883 50  0000 R CNN
 F 2 "LED_THT:LED_D5.0mm" H 5800 4000 50  0001 C CNN
@@
 AR Path="/5E9E5DE1/5E9DC34C" Ref="R4"  Part="1"
 AR Path="/5E9E4A6B/5E9DC34C" Ref="R14"  Part="1"
-F 0 "R24" H 5870 3746 50  0000 L CNN
+AR Path="/5ED17BA0/5ED2A301/5E9DC34C" Ref="R?"  Part="1"
+AR Path="/5ED17BA0/5ED2A304/5E9DC34C" Ref="R?"  Part="1"
+AR Path="/5ED17BA0/5ED2A307/5E9DC34C" Ref="R?"  Part="1"
+AR Path="/5ED17BA0/5ED2A30A/5E9DC34C" Ref="R?"  Part="1"
+AR Path="/5ED17BA0/5ED2A30D/5E9DC34C" Ref="R?"  Part="1"
+F 0 "R?" H 5870 3746 50  0000 L CNN
 F 1 "330" H 5870 3655 50  0000 L CNN
 F 2 "Resistor_THT:R_Axial_DIN0207_L6.3mm_D2.5mm_P10.16mm_Horizontal" V 5730 3700 50  0001 C CNN
@@
 AR Path="/5E9E5DE1/5E9DC352" Ref="R5"  Part="1"
 AR Path="/5E9E4A6B/5E9DC352" Ref="R15"  Part="1"
-F 0 "R25" H 6270 3746 50  0000 L CNN
+AR Path="/5ED17BA0/5ED2A301/5E9DC352" Ref="R?"  Part="1"
+AR Path="/5ED17BA0/5ED2A304/5E9DC352" Ref="R?"  Part="1"
+AR Path="/5ED17BA0/5ED2A307/5E9DC352" Ref="R?"  Part="1"
+AR Path="/5ED17BA0/5ED2A30A/5E9DC352" Ref="R?"  Part="1"
+AR Path="/5ED17BA0/5ED2A30D/5E9DC352" Ref="R?"  Part="1"
+F 0 "R?" H 6270 3746 50  0000 L CNN
 F 1 "330" H 6270 3655 50  0000 L CNN
 F 2 "Resistor_THT:R_Axial_DIN0207_L6.3mm_D2.5mm_P10.16mm_Horizontal" V 6130 3700 50  0001 C CNN
@@
 AR Path="/5E9E5DE1/5E9E70F0" Ref="R6"  Part="1"
 AR Path="/5E9E4A6B/5E9E70F0" Ref="R16"  Part="1"
-F 0 "R26" H 6670 3746 50  0000 L CNN
+AR Path="/5ED17BA0/5ED2A301/5E9E70F0" Ref="R?"  Part="1"
+AR Path="/5ED17BA0/5ED2A304/5E9E70F0" Ref="R?"  Part="1"
+AR Path="/5ED17BA0/5ED2A307/5E9E70F0" Ref="R?"  Part="1"
+AR Path="/5ED17BA0/5ED2A30A/5E9E70F0" Ref="R?"  Part="1"
+AR Path="/5ED17BA0/5ED2A30D/5E9E70F0" Ref="R?"  Part="1"
+F 0 "R?" H 6670 3746 50  0000 L CNN
 F 1 "330" H 6670 3655 50  0000 L CNN
 F 2 "Resistor_THT:R_Axial_DIN0207_L6.3mm_D2.5mm_P10.16mm_Horizontal" V 6530 3700 50  0001 C CNN
@@
 AR Path="/5E9E5DE1/5E9E70F2" Ref="R7"  Part="1"
 AR Path="/5E9E4A6B/5E9E70F2" Ref="R17"  Part="1"
-F 0 "R27" H 7070 3746 50  0000 L CNN
+AR Path="/5ED17BA0/5ED2A301/5E9E70F2" Ref="R?"  Part="1"
+AR Path="/5ED17BA0/5ED2A304/5E9E70F2" Ref="R?"  Part="1"
+AR Path="/5ED17BA0/5ED2A307/5E9E70F2" Ref="R?"  Part="1"
+AR Path="/5ED17BA0/5ED2A30A/5E9E70F2" Ref="R?"  Part="1"
+AR Path="/5ED17BA0/5ED2A30D/5E9E70F2" Ref="R?"  Part="1"
+F 0 "R?" H 7070 3746 50  0000 L CNN
 F 1 "330" H 7070 3655 50  0000 L CNN
 F 2 "Resistor_THT:R_Axial_DIN0207_L6.3mm_D2.5mm_P10.16mm_Horizontal" V 6930 3700 50  0001 C CNN
@@
 AR Path="/5E9E5DE1/5E9E70F3" Ref="D6"  Part="1"
 AR Path="/5E9E4A6B/5E9E70F3" Ref="D14"  Part="1"
-F 0 "D22" V 7039 3883 50  0000 R CNN
+AR Path="/5ED17BA0/5ED2A301/5E9E70F3" Ref="D?"  Part="1"
+AR Path="/5ED17BA0/5ED2A304/5E9E70F3" Ref="D?"  Part="1"
+AR Path="/5ED17BA0/5ED2A307/5E9E70F3" Ref="D?"  Part="1"
+AR Path="/5ED17BA0/5ED2A30A/5E9E70F3" Ref="D?"  Part="1"
+AR Path="/5ED17BA0/5ED2A30D/5E9E70F3" Ref="D?"  Part="1"
+F 0 "D?" V 7039 3883 50  0000 R CNN
 F 1 "LED" V 6948 3883 50  0000 R CNN
 F 2 "LED_THT:LED_D5.0mm" H 7000 4000 50  0001 C CNN
@@
 AR Path="/5E9E5DE1/5E9E70F1" Ref="D5"  Part="1"
 AR Path="/5E9E4A6B/5E9E70F1" Ref="D13"  Part="1"
-F 0 "D21" V 6639 3883 50  0000 R CNN
+AR Path="/5ED17BA0/5ED2A301/5E9E70F1" Ref="D?"  Part="1"
+AR Path="/5ED17BA0/5ED2A304/5E9E70F1" Ref="D?"  Part="1"
+AR Path="/5ED17BA0/5ED2A307/5E9E70F1" Ref="D?"  Part="1"
+AR Path="/5ED17BA0/5ED2A30A/5E9E70F1" Ref="D?"  Part="1"
+AR Path="/5ED17BA0/5ED2A30D/5E9E70F1" Ref="D?"  Part="1"
+F 0 "D?" V 6639 3883 50  0000 R CNN
 F 1 "LED" V 6548 3883 50  0000 R CNN
 F 2 "LED_THT:LED_D5.0mm" H 6600 4000 50  0001 C CNN
@@
 AR Path="/5E9E5DE1/5E9E70EF" Ref="D4"  Part="1"
 AR Path="/5E9E4A6B/5E9E70EF" Ref="D12"  Part="1"
-F 0 "D20" V 6239 3883 50  0000 R CNN
+AR Path="/5ED17BA0/5ED2A301/5E9E70EF" Ref="D?"  Part="1"
+AR Path="/5ED17BA0/5ED2A304/5E9E70EF" Ref="D?"  Part="1"
+AR Path="/5ED17BA0/5ED2A307/5E9E70EF" Ref="D?"  Part="1"
+AR Path="/5ED17BA0/5ED2A30A/5E9E70EF" Ref="D?"  Part="1"
+AR Path="/5ED17BA0/5ED2A30D/5E9E70EF" Ref="D?"  Part="1"
+F 0 "D?" V 6239 3883 50  0000 R CNN
 F 1 "LED" V 6148 3883 50  0000 R CNN
 F 2 "LED_THT:LED_D5.0mm" H 6200 4000 50  0001 C CNN
@@
 AR Path="/5E9E4A6B/5EB39A74" Ref="#PWR0113"  Part="1"
 AR Path="/5E9D240B/5EB39A74" Ref="#PWR0117"  Part="1"
-F 0 "#PWR0117" H 5450 4400 50  0001 C CNN
+AR Path="/5ED17BA0/5ED2A301/5EB39A74" Ref="#PWR?"  Part="1"
+AR Path="/5ED17BA0/5ED2A304/5EB39A74" Ref="#PWR?"  Part="1"
+AR Path="/5ED17BA0/5ED2A307/5EB39A74" Ref="#PWR?"  Part="1"
+AR Path="/5ED17BA0/5ED2A30A/5EB39A74" Ref="#PWR?"  Part="1"
+AR Path="/5ED17BA0/5ED2A30D/5EB39A74" Ref="#PWR?"  Part="1"
+F 0 "#PWR?" H 5450 4400 50  0001 C CNN
 F 1 "GND" H 5455 4477 50  0000 C CNN
 F 2 "" H 5450 4650 50  0001 C CNN
@@
 AR Path="/5E9E4A6B/5EB3A90A" Ref="#PWR0114"  Part="1"
 AR Path="/5E9D240B/5EB3A90A" Ref="#PWR0118"  Part="1"
-F 0 "#PWR0118" H 5450 3350 50  0001 C CNN
+AR Path="/5ED17BA0/5ED2A301/5EB3A90A" Ref="#PWR?"  Part="1"
+AR Path="/5ED17BA0/5ED2A304/5EB3A90A" Ref="#PWR?"  Part="1"
+AR Path="/5ED17BA0/5ED2A307/5EB3A90A" Ref="#PWR?"  Part="1"
+AR Path="/5ED17BA0/5ED2A30A/5EB3A90A" Ref="#PWR?"  Part="1"
+AR Path="/5ED17BA0/5ED2A30D/5EB3A90A" Ref="#PWR?"  Part="1"
+F 0 "#PWR?" H 5450 3350 50  0001 C CNN
 F 1 "+5V" H 5465 3673 50  0000 C CNN
 F 2 "" H 5450 3500 50  0001 C CNN

Commit message: Partial Update
Parts:
- removed Q6: BC337, Package_TO_SOT_THT:TO-92_Inline, symbol Transistor_BJT:BC337
- added Q4: BCW65ALT1G, Package_TO_SOT_SMD:SOT-23, symbol Frequently_Used:BCW65ALT1G
- R4: renamed from R8; footprint Resistor_THT:R_Axial_DIN0207_L6.3mm_D2.5mm_P10.16mm_Horizontal -> Frequently_Used:0805_2012Metric_HandSolder
- R5: renamed from R9; footprint Resistor_THT:R_Axial_DIN0207_L6.3mm_D2.5mm_P10.16mm_Horizontal -> Frequently_Used:0805_2012Metric_HandSolder
- R6: renamed from R10; footprint Resistor_THT:R_Axial_DIN0207_L6.3mm_D2.5mm_P10.16mm_Horizontal -> Frequently_Used:0805_2012Metric_HandSolder
- R7: renamed from R11; footprint Resistor_THT:R_Axial_DIN0207_L6.3mm_D2.5mm_P10.16mm_Horizontal -> Frequently_Used:0805_2012Metric_HandSolder
- R8: renamed from R12; footprint Resistor_THT:R_Axial_DIN0207_L6.3mm_D2.5mm_P10.16mm_Horizontal -> Frequently_Used:0805_2012Metric_HandSolder
- renumbered D7 to D3, D8 to D4, D9 to D5, D10 to D6

Commit message: Resize to correct for scale
Parts:
- removed Q4: BCW65ALT1G, Package_TO_SOT_SMD:SOT-23, symbol Frequently_Used:BCW65ALT1G
- removed R4: 2.7k, Frequently_Used:0805_2012Metric_HandSolder, symbol Device:R
Connections:
- net labels added: COLLECTOR
- net labels removed: GND, SIGNAL
- wire segments 11 -> 9
Changed lines of the file:
@@
 $Descr A4 11693 8268
 encoding utf-8
-Sheet 8 11
+Sheet 8 10
 Title ""
 Date ""
@@
 Comment4 ""
 $EndDescr
-Wire Wire Line
-	5450 4550 5450 4650
-Wire Wire Line
-	4750 4350 4850 4350
-Text HLabel 4750 4350 0    50   Input ~ 0
-SIGNAL
-$Comp
-L Device:R R?
-U 1 1 5E9FDE71
-P 5000 4350
-AR Path="/5E9E5DDE/5E9FDE71" Ref="R?"  Part="1"
-AR Path="/5E9E304D/5E9FDE71" Ref="R?"  Part="1"
-AR Path="/5E9D240B/5E9FDE71" Ref="R?"  Part="1"
-AR Path="/5E9E5DE1/5E9FDE71" Ref="R?"  Part="1"
-AR Path="/5E9E4A6B/5E9FDE71" Ref="R?"  Part="1"
-AR Path="/5ED17BA0/5ED2A301/5E9FDE71" Ref="R4"  Part="1"
-AR Path="/5ED17BA0/5ED2A304/5E9FDE71" Ref="R9"  Part="1"
-AR Path="/5ED17BA0/5ED2A307/5E9FDE71" Ref="R14"  Part="1"
-AR Path="/5ED17BA0/5ED2A30A/5E9FDE71" Ref="R19"  Part="1"
-AR Path="/5ED17BA0/5ED2A30D/5E9FDE71" Ref="R24"  Part="1"
-F 0 "R24" V 4900 4350 50  0000 C CNN
-F 1 "2.7k" V 5100 4350 50  0000 C CNN
-F 2 "Frequently_Used:0805_2012Metric_HandSolder" V 4930 4350 50  0001 C CNN
-F 3 "~" H 5000 4350 50  0001 C CNN
-	1    5000 4350
-	0    1    1    0
-$EndComp
+Text HLabel 5450 4150 0    50   Input ~ 0
+COLLECTOR
 Wire Wire Line
 	5450 4150 5800 4150
@@
 	1    6200 4000
 	0    -1   -1   0
-$EndComp
-$Comp
-L power:GND #PWR?
-U 1 1 5EB39A74
-P 5450 4650
-AR Path="/5E9E304D/5EB39A74" Ref="#PWR?"  Part="1"
-AR Path="/5E9E5DE1/5EB39A74" Ref="#PWR?"  Part="1"
-AR Path="/5E9E5DDE/5EB39A74" Ref="#PWR?"  Part="1"
-AR Path="/5E9E4A6B/5EB39A74" Ref="#PWR?"  Part="1"
-AR Path="/5E9D240B/5EB39A74" Ref="#PWR?"  Part="1"
-AR Path="/5ED17BA0/5ED2A301/5EB39A74" Ref="#PWR035"  Part="1"
-AR Path="/5ED17BA0/5ED2A304/5EB39A74" Ref="#PWR037"  Part="1"
-AR Path="/5ED17BA0/5ED2A307/5EB39A74" Ref="#PWR039"  Part="1"
-AR Path="/5ED17BA0/5ED2A30A/5EB39A74" Ref="#PWR041"  Part="1"
-AR Path="/5ED17BA0/5ED2A30D/5EB39A74" Ref="#PWR043"  Part="1"
-F 0 "#PWR043" H 5450 4400 50  0001 C CNN
-F 1 "GND" H 5455 4477 50  0000 C CNN
-F 2 "" H 5450 4650 50  0001 C CNN
-F 3 "" H 5450 4650 50  0001 C CNN
-	1    5450 4650
-	1    0    0    -1
 $EndComp
 $Comp
@@
 Wire Wire Line
 	5450 3500 5450 3550
-$Comp
-L Frequently_Used:BCW65ALT1G Q4
-U 1 1 5EE78858
-P 5350 4350
-AR Path="/5ED17BA0/5ED2A30D/5EE78858" Ref="Q4"  Part="1"
-AR Path="/5ED17BA0/5ED2A301/5EE78858" Ref="Q5"  Part="1"
-AR Path="/5ED17BA0/5ED2A304/5EE78858" Ref="Q6"  Part="1"
-AR Path="/5ED17BA0/5ED2A307/5EE78858" Ref="Q7"  Part="1"
-AR Path="/5ED17BA0/5ED2A30A/5EE78858" Ref="Q8"  Part="1"
-F 0 "Q4" H 5541 4396 50  0000 L CNN
-F 1 "BCW65ALT1G" H 5541 4305 50  0000 L CNN
-F 2 "Package_TO_SOT_SMD:SOT-23" H 5400 3700 50  0001 C CIN
-F 3 "https://www.onsemi.com/pub/Collateral/BCW65ALT1-D.PDF" H 5350 4350 50  0001 L CNN
-F 4 "ON Semiconductor" H 5400 3600 50  0001 C CNN "Manufacturer Name"
-F 5 "BCW65ALT1G" H 5400 3900 50  0001 C CNN "Manufacturer Part No."
-F 6 "488-BCW65ALT1GCT-ND" H 5400 3800 50  0001 C CNN "Digikey Part No."
-	1    5350 4350
-	1    0    0    -1
-$EndComp
 $EndSCHEMATC

Commit message: Adding Power Daughter Board
Changed lines of the file:
@@
 AR Path="/5ED17BA0/5ED2A30A/5E9E70EC" Ref="D15"  Part="1"
 AR Path="/5ED17BA0/5ED2A30D/5E9E70EC" Ref="D19"  Part="1"
-F 0 "D19" V 5839 3883 50  0000 R CNN
+F 0 "D7" V 5839 3883 50  0000 R CNN
 F 1 "LED" V 5748 3883 50  0000 R CNN
 F 2 "LED_THT:LED_D5.0mm" H 5800 4000 50  0001 C CNN
@@
 AR Path="/5ED17BA0/5ED2A30A/5E9DC34C" Ref="R20"  Part="1"
 AR Path="/5ED17BA0/5ED2A30D/5E9DC34C" Ref="R25"  Part="1"
-F 0 "R25" H 5870 3746 50  0000 L CNN
+F 0 "R10" H 5870 3746 50  0000 L CNN
 F 1 "330" H 5870 3655 50  0000 L CNN
 F 2 "Frequently_Used:0805_2012Metric_HandSolder" V 5730 3700 50  0001 C CNN
@@
 AR Path="/5ED17BA0/5ED2A30A/5E9DC352" Ref="R21"  Part="1"
 AR Path="/5ED17BA0/5ED2A30D/5E9DC352" Ref="R26"  Part="1"
-F 0 "R26" H 6270 3746 50  0000 L CNN
+F 0 "R11" H 6270 3746 50  0000 L CNN
 F 1 "330" H 6270 3655 50  0000 L CNN
 F 2 "Frequently_Used:0805_2012Metric_HandSolder" V 6130 3700 50  0001 C CNN
@@
 AR Path="/5ED17BA0/5ED2A30A/5E9E70F0" Ref="R22"  Part="1"
 AR Path="/5ED17BA0/5ED2A30D/5E9E70F0" Ref="R27"  Part="1"
-F 0 "R27" H 6670 3746 50  0000 L CNN
+F 0 "R12" H 6670 3746 50  0000 L CNN
 F 1 "330" H 6670 3655 50  0000 L CNN
 F 2 "Frequently_Used:0805_2012Metric_HandSolder" V 6530 3700 50  0001 C CNN
@@
 AR Path="/5ED17BA0/5ED2A30A/5E9E70F2" Ref="R23"  Part="1"
 AR Path="/5ED17BA0/5ED2A30D/5E9E70F2" Ref="R28"  Part="1"
-F 0 "R28" H 7070 3746 50  0000 L CNN
+F 0 "R13" H 7070 3746 50  0000 L CNN
 F 1 "330" H 7070 3655 50  0000 L CNN
 F 2 "Frequently_Used:0805_2012Metric_HandSolder" V 6930 3700 50  0001 C CNN
@@
 AR Path="/5ED17BA0/5ED2A30A/5E9E70F3" Ref="D18"  Part="1"
 AR Path="/5ED17BA0/5ED2A30D/5E9E70F3" Ref="D22"  Part="1"
-F 0 "D22" V 7039 3883 50  0000 R CNN
+F 0 "D10" V 7039 3883 50  0000 R CNN
 F 1 "LED" V 6948 3883 50  0000 R CNN
 F 2 "LED_THT:LED_D5.0mm" H 7000 4000 50  0001 C CNN
@@
 AR Path="/5ED17BA0/5ED2A30A/5E9E70F1" Ref="D17"  Part="1"
 AR Path="/5ED17BA0/5ED2A30D/5E9E70F1" Ref="D21"  Part="1"
-F 0 "D21" V 6639 3883 50  0000 R CNN
+F 0 "D9" V 6639 3883 50  0000 R CNN
 F 1 "LED" V 6548 3883 50  0000 R CNN
 F 2 "LED_THT:LED_D5.0mm" H 6600 4000 50  0001 C CNN
@@
 AR Path="/5ED17BA0/5ED2A30A/5E9E70EF" Ref="D16"  Part="1"
 AR Path="/5ED17BA0/5ED2A30D/5E9E70EF" Ref="D20"  Part="1"
-F 0 "D20" V 6239 3883 50  0000 R CNN
+F 0 "D8" V 6239 3883 50  0000 R CNN
 F 1 "LED" V 6148 3883 50  0000 R CNN
 F 2 "LED_THT:LED_D5.0mm" H 6200 4000 50  0001 C CNN

Commit message: Before updating to two switches
Changed lines of the file:
@@
 AR Path="/5ED17BA0/5ED2A30A/5E9E70EC" Ref="D15"  Part="1"
 AR Path="/5ED17BA0/5ED2A30D/5E9E70EC" Ref="D19"  Part="1"
-F 0 "D7" V 5839 3883 50  0000 R CNN
+F 0 "D19" V 5839 3883 50  0000 R CNN
 F 1 "LED" V 5748 3883 50  0000 R CNN
 F 2 "LED_THT:LED_D5.0mm" H 5800 4000 50  0001 C CNN
@@
 AR Path="/5ED17BA0/5ED2A30A/5E9DC34C" Ref="R20"  Part="1"
 AR Path="/5ED17BA0/5ED2A30D/5E9DC34C" Ref="R25"  Part="1"
-F 0 "R10" H 5870 3746 50  0000 L CNN
+F 0 "R25" H 5870 3746 50  0000 L CNN
 F 1 "330" H 5870 3655 50  0000 L CNN
 F 2 "Frequently_Used:0805_2012Metric_HandSolder" V 5730 3700 50  0001 C CNN
@@
 AR Path="/5ED17BA0/5ED2A30A/5E9DC352" Ref="R21"  Part="1"
 AR Path="/5ED17BA0/5ED2A30D/5E9DC352" Ref="R26"  Part="1"
-F 0 "R11" H 6270 3746 50  0000 L CNN
+F 0 "R26" H 6270 3746 50  0000 L CNN
 F 1 "330" H 6270 3655 50  0000 L CNN
 F 2 "Frequently_Used:0805_2012Metric_HandSolder" V 6130 3700 50  0001 C CNN
@@
 AR Path="/5ED17BA0/5ED2A30A/5E9E70F0" Ref="R22"  Part="1"
 AR Path="/5ED17BA0/5ED2A30D/5E9E70F0" Ref="R27"  Part="1"
-F 0 "R12" H 6670 3746 50  0000 L CNN
+F 0 "R27" H 6670 3746 50  0000 L CNN
 F 1 "330" H 6670 3655 50  0000 L CNN
 F 2 "Frequently_Used:0805_2012Metric_HandSolder" V 6530 3700 50  0001 C CNN
@@
 AR Path="/5ED17BA0/5ED2A30A/5E9E70F2" Ref="R23"  Part="1"
 AR Path="/5ED17BA0/5ED2A30D/5E9E70F2" Ref="R28"  Part="1"
-F 0 "R13" H 7070 3746 50  0000 L CNN
+F 0 "R28" H 7070 3746 50  0000 L CNN
 F 1 "330" H 7070 3655 50  0000 L CNN
 F 2 "Frequently_Used:0805_2012Metric_HandSolder" V 6930 3700 50  0001 C CNN
@@
 AR Path="/5ED17BA0/5ED2A30A/5E9E70F3" Ref="D18"  Part="1"
 AR Path="/5ED17BA0/5ED2A30D/5E9E70F3" Ref="D22"  Part="1"
-F 0 "D10" V 7039 3883 50  0000 R CNN
+F 0 "D22" V 7039 3883 50  0000 R CNN
 F 1 "LED" V 6948 3883 50  0000 R CNN
 F 2 "LED_THT:LED_D5.0mm" H 7000 4000 50  0001 C CNN
@@
 AR Path="/5ED17BA0/5ED2A30A/5E9E70F1" Ref="D17"  Part="1"
 AR Path="/5ED17BA0/5ED2A30D/5E9E70F1" Ref="D21"  Part="1"
-F 0 "D9" V 6639 3883 50  0000 R CNN
+F 0 "D21" V 6639 3883 50  0000 R CNN
 F 1 "LED" V 6548 3883 50  0000 R CNN
 F 2 "LED_THT:LED_D5.0mm" H 6600 4000 50  0001 C CNN
@@
 AR Path="/5ED17BA0/5ED2A30A/5E9E70EF" Ref="D16"  Part="1"
 AR Path="/5ED17BA0/5ED2A30D/5E9E70EF" Ref="D20"  Part="1"
-F 0 "D8" V 6239 3883 50  0000 R CNN
+F 0 "D20" V 6239 3883 50  0000 R CNN
 F 1 "LED" V 6148 3883 50  0000 R CNN
 F 2 "LED_THT:LED_D5.0mm" H 6200 4000 50  0001 C CNN

Commit message: Updates
Parts:
- D3, D4, D5, D6: footprint LED_THT:LED_D5.0mm -> LED_SMD:LED_1812_4532Metric
Changed lines of the file:
@@
 $Descr A4 11693 8268
 encoding utf-8
-Sheet 8 11
+Sheet 6 11
 Title ""
 Date ""
@@
 AR Path="/5ED17BA0/5ED2A30A/5E9E70EC" Ref="D15"  Part="1"
 AR Path="/5ED17BA0/5ED2A30D/5E9E70EC" Ref="D19"  Part="1"
-F 0 "D19" V 5839 3883 50  0000 R CNN
+F 0 "D15" V 5839 3883 50  0000 R CNN
 F 1 "LED" V 5748 3883 50  0000 R CNN
-F 2 "LED_THT:LED_D5.0mm" H 5800 4000 50  0001 C CNN
+F 2 "LED_SMD:LED_1812_4532Metric" H 5800 4000 50  0001 C CNN
 F 3 "~" H 5800 4000 50  0001 C CNN
 	1    5800 4000
@@
 AR Path="/5ED17BA0/5ED2A30A/5E9DC34C" Ref="R20"  Part="1"
 AR Path="/5ED17BA0/5ED2A30D/5E9DC34C" Ref="R25"  Part="1"
-F 0 "R25" H 5870 3746 50  0000 L CNN
+F 0 "R20" H 5870 3746 50  0000 L CNN
 F 1 "330" H 5870 3655 50  0000 L CNN
 F 2 "Frequently_Used:0805_2012Metric_HandSolder" V 5730 3700 50  0001 C CNN
@@
 AR Path="/5ED17BA0/5ED2A30A/5E9DC352" Ref="R21"  Part="1"
 AR Path="/5ED17BA0/5ED2A30D/5E9DC352" Ref="R26"  Part="1"
-F 0 "R26" H 6270 3746 50  0000 L CNN
+F 0 "R21" H 6270 3746 50  0000 L CNN
 F 1 "330" H 6270 3655 50  0000 L CNN
 F 2 "Frequently_Used:0805_2012Metric_HandSolder" V 6130 3700 50  0001 C CNN
@@
 AR Path="/5ED17BA0/5ED2A30A/5E9E70F0" Ref="R22"  Part="1"
 AR Path="/5ED17BA0/5ED2A30D/5E9E70F0" Ref="R27"  Part="1"
-F 0 "R27" H 6670 3746 50  0000 L CNN
+F 0 "R22" H 6670 3746 50  0000 L CNN
 F 1 "330" H 6670 3655 50  0000 L CNN
 F 2 "Frequently_Used:0805_2012Metric_HandSolder" V 6530 3700 50  0001 C CNN
@@
 AR Path="/5ED17BA0/5ED2A30A/5E9E70F2" Ref="R23"  Part="1"
 AR Path="/5ED17BA0/5ED2A30D/5E9E70F2" Ref="R28"  Part="1"
-F 0 "R28" H 7070 3746 50  0000 L CNN
+F 0 "R23" H 7070 3746 50  0000 L CNN
 F 1 "330" H 7070 3655 50  0000 L CNN
 F 2 "Frequently_Used:0805_2012Metric_HandSolder" V 6930 3700 50  0001 C CNN
@@
 AR Path="/5ED17BA0/5ED2A30A/5E9E70F3" Ref="D18"  Part="1"
 AR Path="/5ED17BA0/5ED2A30D/5E9E70F3" Ref="D22"  Part="1"
-F 0 "D22" V 7039 3883 50  0000 R CNN
+F 0 "D18" V 7039 3883 50  0000 R CNN
 F 1 "LED" V 6948 3883 50  0000 R CNN
-F 2 "LED_THT:LED_D5.0mm" H 7000 4000 50  0001 C CNN
+F 2 "LED_SMD:LED_1812_4532Metric" H 7000 4000 50  0001 C CNN
 F 3 "~" H 7000 4000 50  0001 C CNN
 	1    7000 4000
@@
 AR Path="/5ED17BA0/5ED2A30A/5E9E70F1" Ref="D17"  Part="1"
 AR Path="/5ED17BA0/5ED2A30D/5E9E70F1" Ref="D21"  Part="1"
-F 0 "D21" V 6639 3883 50  0000 R CNN
+F 0 "D17" V 6639 3883 50  0000 R CNN
 F 1 "LED" V 6548 3883 50  0000 R CNN
-F 2 "LED_THT:LED_D5.0mm" H 6600 4000 50  0001 C CNN
+F 2 "LED_SMD:LED_1812_4532Metric" H 6600 4000 50  0001 C CNN
 F 3 "~" H 6600 4000 50  0001 C CNN
 	1    6600 4000
@@
 AR Path="/5ED17BA0/5ED2A30A/5E9E70EF" Ref="D16"  Part="1"
 AR Path="/5ED17BA0/5ED2A30D/5E9E70EF" Ref="D20"  Part="1"
-F 0 "D20" V 6239 3883 50  0000 R CNN
+F 0 "D16" V 6239 3883 50  0000 R CNN
 F 1 "LED" V 6148 3883 50  0000 R CNN
-F 2 "LED_THT:LED_D5.0mm" H 6200 4000 50  0001 C CNN
+F 2 "LED_SMD:LED_1812_4532Metric" H 6200 4000 50  0001 C CNN
 F 3 "~" H 6200 4000 50  0001 C CNN
 	1    6200 4000
