File: Naquadah Generator Main/BlueLights.sch (KiCad schematic (older format))
At the start: 8 parts

Commit message: Updates
Changed lines of the file:
@@
 $Descr A4 11693 8268
 encoding utf-8
-Sheet 6 11
+Sheet 3 11
 Title ""
 Date ""
@@
 AR Path="/5ED17BA0/5ED2A30A/5E9E70EC" Ref="D15"  Part="1"
 AR Path="/5ED17BA0/5ED2A30D/5E9E70EC" Ref="D19"  Part="1"
-F 0 "D15" V 5839 3883 50  0000 R CNN
+F 0 "D3" V 5839 3883 50  0000 R CNN
 F 1 "LED" V 5748 3883 50  0000 R CNN
 F 2 "LED_SMD:LED_1812_4532Metric" H 5800 4000 50  0001 C CNN
@@
 AR Path="/5ED17BA0/5ED2A30A/5E9DC34C" Ref="R20"  Part="1"
 AR Path="/5ED17BA0/5ED2A30D/5E9DC34C" Ref="R25"  Part="1"
-F 0 "R20" H 5870 3746 50  0000 L CNN
+F 0 "R5" H 5870 3746 50  0000 L CNN
 F 1 "330" H 5870 3655 50  0000 L CNN
 F 2 "Frequently_Used:0805_2012Metric_HandSolder" V 5730 3700 50  0001 C CNN
@@
 AR Path="/5ED17BA0/5ED2A30A/5E9DC352" Ref="R21"  Part="1"
 AR Path="/5ED17BA0/5ED2A30D/5E9DC352" Ref="R26"  Part="1"
-F 0 "R21" H 6270 3746 50  0000 L CNN
+F 0 "R6" H 6270 3746 50  0000 L CNN
 F 1 "330" H 6270 3655 50  0000 L CNN
 F 2 "Frequently_Used:0805_2012Metric_HandSolder" V 6130 3700 50  0001 C CNN
@@
 AR Path="/5ED17BA0/5ED2A30A/5E9E70F0" Ref="R22"  Part="1"
 AR Path="/5ED17BA0/5ED2A30D/5E9E70F0" Ref="R27"  Part="1"
-F 0 "R22" H 6670 3746 50  0000 L CNN
+F 0 "R7" H 6670 3746 50  0000 L CNN
 F 1 "330" H 6670 3655 50  0000 L CNN
 F 2 "Frequently_Used:0805_2012Metric_HandSolder" V 6530 3700 50  0001 C CNN
@@
 AR Path="/5ED17BA0/5ED2A30A/5E9E70F2" Ref="R23"  Part="1"
 AR Path="/5ED17BA0/5ED2A30D/5E9E70F2" Ref="R28"  Part="1"
-F 0 "R23" H 7070 3746 50  0000 L CNN
+F 0 "R8" H 7070 3746 50  0000 L CNN
 F 1 "330" H 7070 3655 50  0000 L CNN
 F 2 "Frequently_Used:0805_2012Metric_HandSolder" V 6930 3700 50  0001 C CNN
@@
 AR Path="/5ED17BA0/5ED2A30A/5E9E70F3" Ref="D18"  Part="1"
 AR Path="/5ED17BA0/5ED2A30D/5E9E70F3" Ref="D22"  Part="1"
-F 0 "D18" V 7039 3883 50  0000 R CNN
+F 0 "D6" V 7039 3883 50  0000 R CNN
 F 1 "LED" V 6948 3883 50  0000 R CNN
 F 2 "LED_SMD:LED_1812_4532Metric" H 7000 4000 50  0001 C CNN
@@
 AR Path="/5ED17BA0/5ED2A30A/5E9E70F1" Ref="D17"  Part="1"
 AR Path="/5ED17BA0/5ED2A30D/5E9E70F1" Ref="D21"  Part="1"
-F 0 "D17" V 6639 3883 50  0000 R CNN
+F 0 "D5" V 6639 3883 50  0000 R CNN
 F 1 "LED" V 6548 3883 50  0000 R CNN
 F 2 "LED_SMD:LED_1812_4532Metric" H 6600 4000 50  0001 C CNN
@@
 AR Path="/5ED17BA0/5ED2A30A/5E9E70EF" Ref="D16"  Part="1"
 AR Path="/5ED17BA0/5ED2A30D/5E9E70EF" Ref="D20"  Part="1"
-F 0 "D16" V 6239 3883 50  0000 R CNN
+F 0 "D4" V 6239 3883 50  0000 R CNN
 F 1 "LED" V 6148 3883 50  0000 R CNN
 F 2 "LED_SMD:LED_1812_4532Metric" H 6200 4000 50  0001 C CNN
@@
 AR Path="/5ED17BA0/5ED2A30A/5EB3A90A" Ref="#PWR040"  Part="1"
 AR Path="/5ED17BA0/5ED2A30D/5EB3A90A" Ref="#PWR042"  Part="1"
-F 0 "#PWR042" H 5450 3350 50  0001 C CNN
+F 0 "#PWR034" H 5450 3350 50  0001 C CNN
 F 1 "+5V" H 5465 3673 50  0000 C CNN
 F 2 "" H 5450 3500 50  0001 C CNN

Commit message: Move libraries and added configuration path.
Moved Li-Ion library to common KiCad library.  Added variables to configuration paths to reference my KiCad libraries.  Moved all 3D components to my common library.
Parts:
- R5, R6, R7, R8: footprint Frequently_Used:0805_2012Metric_HandSolder -> FrequentlyUsed:0805_2012Metric_HandSolder
Changed lines of the file:
@@
 F 0 "R5" H 5870 3746 50  0000 L CNN
 F 1 "330" H 5870 3655 50  0000 L CNN
-F 2 "Frequently_Used:0805_2012Metric_HandSolder" V 5730 3700 50  0001 C CNN
+F 2 "FrequentlyUsed:0805_2012Metric_HandSolder" V 5730 3700 50  0001 C CNN
 F 3 "~" H 5800 3700 50  0001 C CNN
 	1    5800 3700
@@
 F 0 "R6" H 6270 3746 50  0000 L CNN
 F 1 "330" H 6270 3655 50  0000 L CNN
-F 2 "Frequently_Used:0805_2012Metric_HandSolder" V 6130 3700 50  0001 C CNN
+F 2 "FrequentlyUsed:0805_2012Metric_HandSolder" V 6130 3700 50  0001 C CNN
 F 3 "~" H 6200 3700 50  0001 C CNN
 	1    6200 3700
@@
 F 0 "R7" H 6670 3746 50  0000 L CNN
 F 1 "330" H 6670 3655 50  0000 L CNN
-F 2 "Frequently_Used:0805_2012Metric_HandSolder" V 6530 3700 50  0001 C CNN
+F 2 "FrequentlyUsed:0805_2012Metric_HandSolder" V 6530 3700 50  0001 C CNN
 F 3 "~" H 6600 3700 50  0001 C CNN
 	1    6600 3700
@@
 F 0 "R8" H 7070 3746 50  0000 L CNN
 F 1 "330" H 7070 3655 50  0000 L CNN
-F 2 "Frequently_Used:0805_2012Metric_HandSolder" V 6930 3700 50  0001 C CNN
+F 2 "FrequentlyUsed:0805_2012Metric_HandSolder" V 6930 3700 50  0001 C CNN
 F 3 "~" H 7000 3700 50  0001 C CNN
 	1    7000 3700
@@
 AR Path="/5ED17BA0/5ED2A30A/5EB3A90A" Ref="#PWR040"  Part="1"
 AR Path="/5ED17BA0/5ED2A30D/5EB3A90A" Ref="#PWR042"  Part="1"
-F 0 "#PWR034" H 5450 3350 50  0001 C CNN
+F 0 "#PWR042" H 5450 3350 50  0001 C CNN
 F 1 "+5V" H 5465 3673 50  0000 C CNN
 F 2 "" H 5450 3500 50  0001 C CNN

Commit message: Updates
Changed lines of the file:
@@
 $Descr A4 11693 8268
 encoding utf-8
-Sheet 3 11
+Sheet 3 12
 Title ""
 Date ""
@@
 AR Path="/5ED17BA0/5ED2A30A/5E9E70EC" Ref="D15"  Part="1"
 AR Path="/5ED17BA0/5ED2A30D/5E9E70EC" Ref="D19"  Part="1"
-F 0 "D3" V 5839 3883 50  0000 R CNN
+F 0 "D19" V 5839 3883 50  0000 R CNN
 F 1 "LED" V 5748 3883 50  0000 R CNN
 F 2 "LED_SMD:LED_1812_4532Metric" H 5800 4000 50  0001 C CNN
@@
 AR Path="/5ED17BA0/5ED2A30A/5E9DC34C" Ref="R20"  Part="1"
 AR Path="/5ED17BA0/5ED2A30D/5E9DC34C" Ref="R25"  Part="1"
-F 0 "R5" H 5870 3746 50  0000 L CNN
+F 0 "R25" H 5870 3746 50  0000 L CNN
 F 1 "330" H 5870 3655 50  0000 L CNN
 F 2 "FrequentlyUsed:0805_2012Metric_HandSolder" V 5730 3700 50  0001 C CNN
@@
 AR Path="/5ED17BA0/5ED2A30A/5E9DC352" Ref="R21"  Part="1"
 AR Path="/5ED17BA0/5ED2A30D/5E9DC352" Ref="R26"  Part="1"
-F 0 "R6" H 6270 3746 50  0000 L CNN
+F 0 "R26" H 6270 3746 50  0000 L CNN
 F 1 "330" H 6270 3655 50  0000 L CNN
 F 2 "FrequentlyUsed:0805_2012Metric_HandSolder" V 6130 3700 50  0001 C CNN
@@
 AR Path="/5ED17BA0/5ED2A30A/5E9E70F0" Ref="R22"  Part="1"
 AR Path="/5ED17BA0/5ED2A30D/5E9E70F0" Ref="R27"  Part="1"
-F 0 "R7" H 6670 3746 50  0000 L CNN
+F 0 "R27" H 6670 3746 50  0000 L CNN
 F 1 "330" H 6670 3655 50  0000 L CNN
 F 2 "FrequentlyUsed:0805_2012Metric_HandSolder" V 6530 3700 50  0001 C CNN
@@
 AR Path="/5ED17BA0/5ED2A30A/5E9E70F2" Ref="R23"  Part="1"
 AR Path="/5ED17BA0/5ED2A30D/5E9E70F2" Ref="R28"  Part="1"
-F 0 "R8" H 7070 3746 50  0000 L CNN
+F 0 "R28" H 7070 3746 50  0000 L CNN
 F 1 "330" H 7070 3655 50  0000 L CNN
 F 2 "FrequentlyUsed:0805_2012Metric_HandSolder" V 6930 3700 50  0001 C CNN
@@
 AR Path="/5ED17BA0/5ED2A30A/5E9E70F3" Ref="D18"  Part="1"
 AR Path="/5ED17BA0/5ED2A30D/5E9E70F3" Ref="D22"  Part="1"
-F 0 "D6" V 7039 3883 50  0000 R CNN
+F 0 "D22" V 7039 3883 50  0000 R CNN
 F 1 "LED" V 6948 3883 50  0000 R CNN
 F 2 "LED_SMD:LED_1812_4532Metric" H 7000 4000 50  0001 C CNN
@@
 AR Path="/5ED17BA0/5ED2A30A/5E9E70F1" Ref="D17"  Part="1"
 AR Path="/5ED17BA0/5ED2A30D/5E9E70F1" Ref="D21"  Part="1"
-F 0 "D5" V 6639 3883 50  0000 R CNN
+F 0 "D21" V 6639 3883 50  0000 R CNN
 F 1 "LED" V 6548 3883 50  0000 R CNN
 F 2 "LED_SMD:LED_1812_4532Metric" H 6600 4000 50  0001 C CNN
@@
 AR Path="/5ED17BA0/5ED2A30A/5E9E70EF" Ref="D16"  Part="1"
 AR Path="/5ED17BA0/5ED2A30D/5E9E70EF" Ref="D20"  Part="1"
-F 0 "D4" V 6239 3883 50  0000 R CNN
+F 0 "D20" V 6239 3883 50  0000 R CNN
 F 1 "LED" V 6148 3883 50  0000 R CNN
 F 2 "LED_SMD:LED_1812_4532Metric" H 6200 4000 50  0001 C CNN

Commit message: Start of audio
Changed lines of the file:
@@
 AR Path="/5ED17BA0/5ED2A30A/5E9E70EC" Ref="D15"  Part="1"
 AR Path="/5ED17BA0/5ED2A30D/5E9E70EC" Ref="D19"  Part="1"
-F 0 "D19" V 5839 3883 50  0000 R CNN
+F 0 "D3" V 5839 3883 50  0000 R CNN
 F 1 "LED" V 5748 3883 50  0000 R CNN
 F 2 "LED_SMD:LED_1812_4532Metric" H 5800 4000 50  0001 C CNN
@@
 AR Path="/5ED17BA0/5ED2A30A/5E9DC34C" Ref="R20"  Part="1"
 AR Path="/5ED17BA0/5ED2A30D/5E9DC34C" Ref="R25"  Part="1"
-F 0 "R25" H 5870 3746 50  0000 L CNN
+F 0 "R5" H 5870 3746 50  0000 L CNN
 F 1 "330" H 5870 3655 50  0000 L CNN
 F 2 "FrequentlyUsed:0805_2012Metric_HandSolder" V 5730 3700 50  0001 C CNN
@@
 AR Path="/5ED17BA0/5ED2A30A/5E9DC352" Ref="R21"  Part="1"
 AR Path="/5ED17BA0/5ED2A30D/5E9DC352" Ref="R26"  Part="1"
-F 0 "R26" H 6270 3746 50  0000 L CNN
+F 0 "R6" H 6270 3746 50  0000 L CNN
 F 1 "330" H 6270 3655 50  0000 L CNN
 F 2 "FrequentlyUsed:0805_2012Metric_HandSolder" V 6130 3700 50  0001 C CNN
@@
 AR Path="/5ED17BA0/5ED2A30A/5E9E70F0" Ref="R22"  Part="1"
 AR Path="/5ED17BA0/5ED2A30D/5E9E70F0" Ref="R27"  Part="1"
-F 0 "R27" H 6670 3746 50  0000 L CNN
+F 0 "R7" H 6670 3746 50  0000 L CNN
 F 1 "330" H 6670 3655 50  0000 L CNN
 F 2 "FrequentlyUsed:0805_2012Metric_HandSolder" V 6530 3700 50  0001 C CNN
@@
 AR Path="/5ED17BA0/5ED2A30A/5E9E70F2" Ref="R23"  Part="1"
 AR Path="/5ED17BA0/5ED2A30D/5E9E70F2" Ref="R28"  Part="1"
-F 0 "R28" H 7070 3746 50  0000 L CNN
+F 0 "R8" H 7070 3746 50  0000 L CNN
 F 1 "330" H 7070 3655 50  0000 L CNN
 F 2 "FrequentlyUsed:0805_2012Metric_HandSolder" V 6930 3700 50  0001 C CNN
@@
 AR Path="/5ED17BA0/5ED2A30A/5E9E70F3" Ref="D18"  Part="1"
 AR Path="/5ED17BA0/5ED2A30D/5E9E70F3" Ref="D22"  Part="1"
-F 0 "D22" V 7039 3883 50  0000 R CNN
+F 0 "D6" V 7039 3883 50  0000 R CNN
 F 1 "LED" V 6948 3883 50  0000 R CNN
 F 2 "LED_SMD:LED_1812_4532Metric" H 7000 4000 50  0001 C CNN
@@
 AR Path="/5ED17BA0/5ED2A30A/5E9E70F1" Ref="D17"  Part="1"
 AR Path="/5ED17BA0/5ED2A30D/5E9E70F1" Ref="D21"  Part="1"
-F 0 "D21" V 6639 3883 50  0000 R CNN
+F 0 "D5" V 6639 3883 50  0000 R CNN
 F 1 "LED" V 6548 3883 50  0000 R CNN
 F 2 "LED_SMD:LED_1812_4532Metric" H 6600 4000 50  0001 C CNN
@@
 AR Path="/5ED17BA0/5ED2A30A/5E9E70EF" Ref="D16"  Part="1"
 AR Path="/5ED17BA0/5ED2A30D/5E9E70EF" Ref="D20"  Part="1"
-F 0 "D20" V 6239 3883 50  0000 R CNN
+F 0 "D4" V 6239 3883 50  0000 R CNN
 F 1 "LED" V 6148 3883 50  0000 R CNN
 F 2 "LED_SMD:LED_1812_4532Metric" H 6200 4000 50  0001 C CNN
@@
 AR Path="/5ED17BA0/5ED2A30A/5EB3A90A" Ref="#PWR040"  Part="1"
 AR Path="/5ED17BA0/5ED2A30D/5EB3A90A" Ref="#PWR042"  Part="1"
-F 0 "#PWR042" H 5450 3350 50  0001 C CNN
+F 0 "#PWR034" H 5450 3350 50  0001 C CNN
 F 1 "+5V" H 5465 3673 50  0000 C CNN
 F 2 "" H 5450 3500 50  0001 C CNN

Commit message: Audio update
Parts:
- R5, R6, R7, R8: footprint FrequentlyUsed:0805_2012Metric_HandSolder -> Frequently_Used_LE:0805_2012Metric_HandSolder; Manufacturer Name (none) -> KOA Speer Electronics, Inc.; Source (none) -> Digikey
Changed lines of the file:
@@
 $Descr A4 11693 8268
 encoding utf-8
-Sheet 3 12
+Sheet 7 12
 Title ""
 Date ""
@@
 AR Path="/5ED17BA0/5ED2A30A/5E9E70EC" Ref="D15"  Part="1"
 AR Path="/5ED17BA0/5ED2A30D/5E9E70EC" Ref="D19"  Part="1"
-F 0 "D3" V 5839 3883 50  0000 R CNN
+F 0 "D19" V 5839 3883 50  0000 R CNN
 F 1 "LED" V 5748 3883 50  0000 R CNN
 F 2 "LED_SMD:LED_1812_4532Metric" H 5800 4000 50  0001 C CNN
@@
 AR Path="/5ED17BA0/5ED2A30A/5E9DC34C" Ref="R20"  Part="1"
 AR Path="/5ED17BA0/5ED2A30D/5E9DC34C" Ref="R25"  Part="1"
-F 0 "R5" H 5870 3746 50  0000 L CNN
+F 0 "R25" H 5870 3746 50  0000 L CNN
 F 1 "330" H 5870 3655 50  0000 L CNN
-F 2 "FrequentlyUsed:0805_2012Metric_HandSolder" V 5730 3700 50  0001 C CNN
-F 3 "~" H 5800 3700 50  0001 C CNN
+F 2 "Frequently_Used_LE:0805_2012Metric_HandSolder" V 5730 3700 50  0001 C CNN
+F 3 "http://www.koaspeer.com/pdfs/RK73H.pdf" H 5800 3700 50  0001 C CNN
+F 4 "KOA Speer Electronics, Inc." H 5800 3700 50  0001 C CNN "Manufacturer Name"
+F 5 "Digikey" H 5800 3700 50  0001 C CNN "Source"
 	1    5800 3700
 	1    0    0    -1
@@
 AR Path="/5ED17BA0/5ED2A30A/5E9DC352" Ref="R21"  Part="1"
 AR Path="/5ED17BA0/5ED2A30D/5E9DC352" Ref="R26"  Part="1"
-F 0 "R6" H 6270 3746 50  0000 L CNN
+F 0 "R26" H 6270 3746 50  0000 L CNN
 F 1 "330" H 6270 3655 50  0000 L CNN
-F 2 "FrequentlyUsed:0805_2012Metric_HandSolder" V 6130 3700 50  0001 C CNN
-F 3 "~" H 6200 3700 50  0001 C CNN
+F 2 "Frequently_Used_LE:0805_2012Metric_HandSolder" V 6130 3700 50  0001 C CNN
+F 3 "http://www.koaspeer.com/pdfs/RK73H.pdf" H 6200 3700 50  0001 C CNN
+F 4 "KOA Speer Electronics, Inc." H 6200 3700 50  0001 C CNN "Manufacturer Name"
+F 5 "Digikey" H 6200 3700 50  0001 C CNN "Source"
 	1    6200 3700
 	1    0    0    -1
@@
 AR Path="/5ED17BA0/5ED2A30A/5E9E70F0" Ref="R22"  Part="1"
 AR Path="/5ED17BA0/5ED2A30D/5E9E70F0" Ref="R27"  Part="1"
-F 0 "R7" H 6670 3746 50  0000 L CNN
+F 0 "R27" H 6670 3746 50  0000 L CNN
 F 1 "330" H 6670 3655 50  0000 L CNN
-F 2 "FrequentlyUsed:0805_2012Metric_HandSolder" V 6530 3700 50  0001 C CNN
-F 3 "~" H 6600 3700 50  0001 C CNN
+F 2 "Frequently_Used_LE:0805_2012Metric_HandSolder" V 6530 3700 50  0001 C CNN
+F 3 "http://www.koaspeer.com/pdfs/RK73H.pdf" H 6600 3700 50  0001 C CNN
+F 4 "KOA Speer Electronics, Inc." H 6600 3700 50  0001 C CNN "Manufacturer Name"
+F 5 "Digikey" H 6600 3700 50  0001 C CNN "Source"
 	1    6600 3700
 	1    0    0    -1
@@
 AR Path="/5ED17BA0/5ED2A30A/5E9E70F2" Ref="R23"  Part="1"
 AR Path="/5ED17BA0/5ED2A30D/5E9E70F2" Ref="R28"  Part="1"
-F 0 "R8" H 7070 3746 50  0000 L CNN
+F 0 "R28" H 7070 3746 50  0000 L CNN
 F 1 "330" H 7070 3655 50  0000 L CNN
-F 2 "FrequentlyUsed:0805_2012Metric_HandSolder" V 6930 3700 50  0001 C CNN
-F 3 "~" H 7000 3700 50  0001 C CNN
+F 2 "Frequently_Used_LE:0805_2012Metric_HandSolder" V 6930 3700 50  0001 C CNN
+F 3 "http://www.koaspeer.com/pdfs/RK73H.pdf" H 7000 3700 50  0001 C CNN
+F 4 "KOA Speer Electronics, Inc." H 7000 3700 50  0001 C CNN "Manufacturer Name"
+F 5 "Digikey" H 7000 3700 50  0001 C CNN "Source"
 	1    7000 3700
 	1    0    0    -1
@@
 AR Path="/5ED17BA0/5ED2A30A/5E9E70F3" Ref="D18"  Part="1"
 AR Path="/5ED17BA0/5ED2A30D/5E9E70F3" Ref="D22"  Part="1"
-F 0 "D6" V 7039 3883 50  0000 R CNN
+F 0 "D22" V 7039 3883 50  0000 R CNN
 F 1 "LED" V 6948 3883 50  0000 R CNN
 F 2 "LED_SMD:LED_1812_4532Metric" H 7000 4000 50  0001 C CNN
@@
 AR Path="/5ED17BA0/5ED2A30A/5E9E70F1" Ref="D17"  Part="1"
 AR Path="/5ED17BA0/5ED2A30D/5E9E70F1" Ref="D21"  Part="1"
-F 0 "D5" V 6639 3883 50  0000 R CNN
+F 0 "D21" V 6639 3883 50  0000 R CNN
 F 1 "LED" V 6548 3883 50  0000 R CNN
 F 2 "LED_SMD:LED_1812_4532Metric" H 6600 4000 50  0001 C CNN
@@
 AR Path="/5ED17BA0/5ED2A30A/5E9E70EF" Ref="D16"  Part="1"
 AR Path="/5ED17BA0/5ED2A30D/5E9E70EF" Ref="D20"  Part="1"
-F 0 "D4" V 6239 3883 50  0000 R CNN
+F 0 "D20" V 6239 3883 50  0000 R CNN
 F 1 "LED" V 6148 3883 50  0000 R CNN
 F 2 "LED_SMD:LED_1812_4532Metric" H 6200 4000 50  0001 C CNN
@@
 AR Path="/5ED17BA0/5ED2A30A/5EB3A90A" Ref="#PWR040"  Part="1"
 AR Path="/5ED17BA0/5ED2A30D/5EB3A90A" Ref="#PWR042"  Part="1"
-F 0 "#PWR034" H 5450 3350 50  0001 C CNN
+F 0 "#PWR042" H 5450 3350 50  0001 C CNN
 F 1 "+5V" H 5465 3673 50  0000 C CNN
 F 2 "" H 5450 3500 50  0001 C CNN

Commit message: Before switching buttons on daughter board
Changed lines of the file:
@@
 $Descr A4 11693 8268
 encoding utf-8
-Sheet 7 15
+Sheet 3 15
 Title ""
 Date ""
@@
 AR Path="/5ED17BA0/5ED2A30A/5E9E70EC" Ref="D15"  Part="1"
 AR Path="/5ED17BA0/5ED2A30D/5E9E70EC" Ref="D19"  Part="1"
-F 0 "D19" V 5839 3883 50  0000 R CNN
+F 0 "D3" V 5839 3883 50  0000 R CNN
 F 1 "LED" V 5748 3883 50  0000 R CNN
 F 2 "LED_SMD:LED_1812_4532Metric" H 5800 4000 50  0001 C CNN
@@
 AR Path="/5ED17BA0/5ED2A30A/5E9DC34C" Ref="R20"  Part="1"
 AR Path="/5ED17BA0/5ED2A30D/5E9DC34C" Ref="R25"  Part="1"
-F 0 "R25" H 5870 3746 50  0000 L CNN
+F 0 "R5" H 5870 3746 50  0000 L CNN
 F 1 "330" H 5870 3655 50  0000 L CNN
 F 2 "Frequently_Used_LE:0805_2012Metric_HandSolder" V 5730 3700 50  0001 C CNN
@@
 AR Path="/5ED17BA0/5ED2A30A/5E9DC352" Ref="R21"  Part="1"
 AR Path="/5ED17BA0/5ED2A30D/5E9DC352" Ref="R26"  Part="1"
-F 0 "R26" H 6270 3746 50  0000 L CNN
+F 0 "R6" H 6270 3746 50  0000 L CNN
 F 1 "330" H 6270 3655 50  0000 L CNN
 F 2 "Frequently_Used_LE:0805_2012Metric_HandSolder" V 6130 3700 50  0001 C CNN
@@
 AR Path="/5ED17BA0/5ED2A30A/5E9E70F0" Ref="R22"  Part="1"
 AR Path="/5ED17BA0/5ED2A30D/5E9E70F0" Ref="R27"  Part="1"
-F 0 "R27" H 6670 3746 50  0000 L CNN
+F 0 "R7" H 6670 3746 50  0000 L CNN
 F 1 "330" H 6670 3655 50  0000 L CNN
 F 2 "Frequently_Used_LE:0805_2012Metric_HandSolder" V 6530 3700 50  0001 C CNN
@@
 AR Path="/5ED17BA0/5ED2A30A/5E9E70F2" Ref="R23"  Part="1"
 AR Path="/5ED17BA0/5ED2A30D/5E9E70F2" Ref="R28"  Part="1"
-F 0 "R28" H 7070 3746 50  0000 L CNN
+F 0 "R8" H 7070 3746 50  0000 L CNN
 F 1 "330" H 7070 3655 50  0000 L CNN
 F 2 "Frequently_Used_LE:0805_2012Metric_HandSolder" V 6930 3700 50  0001 C CNN
@@
 AR Path="/5ED17BA0/5ED2A30A/5E9E70F3" Ref="D18"  Part="1"
 AR Path="/5ED17BA0/5ED2A30D/5E9E70F3" Ref="D22"  Part="1"
-F 0 "D22" V 7039 3883 50  0000 R CNN
+F 0 "D6" V 7039 3883 50  0000 R CNN
 F 1 "LED" V 6948 3883 50  0000 R CNN
 F 2 "LED_SMD:LED_1812_4532Metric" H 7000 4000 50  0001 C CNN
@@
 AR Path="/5ED17BA0/5ED2A30A/5E9E70F1" Ref="D17"  Part="1"
 AR Path="/5ED17BA0/5ED2A30D/5E9E70F1" Ref="D21"  Part="1"
-F 0 "D21" V 6639 3883 50  0000 R CNN
+F 0 "D5" V 6639 3883 50  0000 R CNN
 F 1 "LED" V 6548 3883 50  0000 R CNN
 F 2 "LED_SMD:LED_1812_4532Metric" H 6600 4000 50  0001 C CNN
@@
 AR Path="/5ED17BA0/5ED2A30A/5E9E70EF" Ref="D16"  Part="1"
 AR Path="/5ED17BA0/5ED2A30D/5E9E70EF" Ref="D20"  Part="1"
-F 0 "D20" V 6239 3883 50  0000 R CNN
+F 0 "D4" V 6239 3883 50  0000 R CNN
 F 1 "LED" V 6148 3883 50  0000 R CNN
 F 2 "LED_SMD:LED_1812_4532Metric" H 6200 4000 50  0001 C CNN
@@
 AR Path="/5ED17BA0/5ED2A30A/5EB3A90A" Ref="#PWR040"  Part="1"
 AR Path="/5ED17BA0/5ED2A30D/5EB3A90A" Ref="#PWR042"  Part="1"
-F 0 "#PWR042" H 5450 3350 50  0001 C CNN
+F 0 "#PWR034" H 5450 3350 50  0001 C CNN
 F 1 "+5V" H 5465 3673 50  0000 C CNN
 F 2 "" H 5450 3500 50  0001 C CNN

Commit message: Audio updates, switching to separate USB schematic
Audio updates, switching to separate USB schematic
Changed lines of the file:
@@
 $Descr A4 11693 8268
 encoding utf-8
-Sheet 3 15
+Sheet 3 16
 Title ""
 Date ""
@@
 AR Path="/5ED17BA0/5ED2A30A/5E9E70EC" Ref="D15"  Part="1"
 AR Path="/5ED17BA0/5ED2A30D/5E9E70EC" Ref="D19"  Part="1"
-F 0 "D3" V 5839 3883 50  0000 R CNN
+F 0 "D19" V 5839 3883 50  0000 R CNN
 F 1 "LED" V 5748 3883 50  0000 R CNN
 F 2 "LED_SMD:LED_1812_4532Metric" H 5800 4000 50  0001 C CNN
@@
 AR Path="/5ED17BA0/5ED2A30A/5E9DC34C" Ref="R20"  Part="1"
 AR Path="/5ED17BA0/5ED2A30D/5E9DC34C" Ref="R25"  Part="1"
-F 0 "R5" H 5870 3746 50  0000 L CNN
+F 0 "R25" H 5870 3746 50  0000 L CNN
 F 1 "330" H 5870 3655 50  0000 L CNN
 F 2 "Frequently_Used_LE:0805_2012Metric_HandSolder" V 5730 3700 50  0001 C CNN
@@
 AR Path="/5ED17BA0/5ED2A30A/5E9DC352" Ref="R21"  Part="1"
 AR Path="/5ED17BA0/5ED2A30D/5E9DC352" Ref="R26"  Part="1"
-F 0 "R6" H 6270 3746 50  0000 L CNN
+F 0 "R26" H 6270 3746 50  0000 L CNN
 F 1 "330" H 6270 3655 50  0000 L CNN
 F 2 "Frequently_Used_LE:0805_2012Metric_HandSolder" V 6130 3700 50  0001 C CNN
@@
 AR Path="/5ED17BA0/5ED2A30A/5E9E70F0" Ref="R22"  Part="1"
 AR Path="/5ED17BA0/5ED2A30D/5E9E70F0" Ref="R27"  Part="1"
-F 0 "R7" H 6670 3746 50  0000 L CNN
+F 0 "R27" H 6670 3746 50  0000 L CNN
 F 1 "330" H 6670 3655 50  0000 L CNN
 F 2 "Frequently_Used_LE:0805_2012Metric_HandSolder" V 6530 3700 50  0001 C CNN
@@
 AR Path="/5ED17BA0/5ED2A30A/5E9E70F2" Ref="R23"  Part="1"
 AR Path="/5ED17BA0/5ED2A30D/5E9E70F2" Ref="R28"  Part="1"
-F 0 "R8" H 7070 3746 50  0000 L CNN
+F 0 "R28" H 7070 3746 50  0000 L CNN
 F 1 "330" H 7070 3655 50  0000 L CNN
 F 2 "Frequently_Used_LE:0805_2012Metric_HandSolder" V 6930 3700 50  0001 C CNN
@@
 AR Path="/5ED17BA0/5ED2A30A/5E9E70F3" Ref="D18"  Part="1"
 AR Path="/5ED17BA0/5ED2A30D/5E9E70F3" Ref="D22"  Part="1"
-F 0 "D6" V 7039 3883 50  0000 R CNN
+F 0 "D22" V 7039 3883 50  0000 R CNN
 F 1 "LED" V 6948 3883 50  0000 R CNN
 F 2 "LED_SMD:LED_1812_4532Metric" H 7000 4000 50  0001 C CNN
@@
 AR Path="/5ED17BA0/5ED2A30A/5E9E70F1" Ref="D17"  Part="1"
 AR Path="/5ED17BA0/5ED2A30D/5E9E70F1" Ref="D21"  Part="1"
-F 0 "D5" V 6639 3883 50  0000 R CNN
+F 0 "D21" V 6639 3883 50  0000 R CNN
 F 1 "LED" V 6548 3883 50  0000 R CNN
 F 2 "LED_SMD:LED_1812_4532Metric" H 6600 4000 50  0001 C CNN
@@
 AR Path="/5ED17BA0/5ED2A30A/5E9E70EF" Ref="D16"  Part="1"
 AR Path="/5ED17BA0/5ED2A30D/5E9E70EF" Ref="D20"  Part="1"
-F 0 "D4" V 6239 3883 50  0000 R CNN
+F 0 "D20" V 6239 3883 50  0000 R CNN
 F 1 "LED" V 6148 3883 50  0000 R CNN
 F 2 "LED_SMD:LED_1812_4532Metric" H 6200 4000 50  0001 C CNN
@@
 AR Path="/5ED17BA0/5ED2A30A/5EB3A90A" Ref="#PWR040"  Part="1"
 AR Path="/5ED17BA0/5ED2A30D/5EB3A90A" Ref="#PWR042"  Part="1"
-F 0 "#PWR034" H 5450 3350 50  0001 C CNN
+F 0 "#PWR042" H 5450 3350 50  0001 C CNN
 F 1 "+5V" H 5465 3673 50  0000 C CNN
 F 2 "" H 5450 3500 50  0001 C CNN
