File: Naquadah Generator Main/BlueLights.sch (KiCad schematic (older format))
At the start: 8 parts

Commit message: Added level shifter, moved user interface connector location
Added level shifter, moved user interface connector location
Parts:
- R5, R6, R7, R8: footprint Frequently_Used_LE:0805_2012Metric_HandSolder -> Frequently_Used_LE:0805_2012Metric; Description (none) -> 330 Ohms ±1% 0.25W, 1/4W Chip Resistor 1206 (3216 Metric); Manufacturer Part No. (none) -> RK73H2ATTD3300F; Source Part No. (none) -> 2019-RK73H2ATTD3300FCT-ND
Changed lines of the file:
@@
 $Descr A4 11693 8268
 encoding utf-8
-Sheet 3 16
+Sheet 3 17
 Title ""
 Date ""
@@
 F 0 "R25" H 5870 3746 50  0000 L CNN
 F 1 "330" H 5870 3655 50  0000 L CNN
-F 2 "Frequently_Used_LE:0805_2012Metric_HandSolder" V 5730 3700 50  0001 C CNN
+F 2 "Frequently_Used_LE:0805_2012Metric" V 5730 3700 50  0001 C CNN
 F 3 "http://www.koaspeer.com/pdfs/RK73H.pdf" H 5800 3700 50  0001 C CNN
 F 4 "KOA Speer Electronics, Inc." H 5800 3700 50  0001 C CNN "Manufacturer Name"
 F 5 "Digikey" H 5800 3700 50  0001 C CNN "Source"
+F 6 "330 Ohms ±1% 0.25W, 1/4W Chip Resistor 1206 (3216 Metric)" H 5800 3700 50  0001 C CNN "Description"
+F 7 "RK73H2ATTD3300F" H 5800 3700 50  0001 C CNN "Manufacturer Part No."
+F 8 "2019-RK73H2ATTD3300FCT-ND" H 5800 3700 50  0001 C CNN "Source Part No."
 	1    5800 3700
 	1    0    0    -1
@@
 F 0 "R26" H 6270 3746 50  0000 L CNN
 F 1 "330" H 6270 3655 50  0000 L CNN
-F 2 "Frequently_Used_LE:0805_2012Metric_HandSolder" V 6130 3700 50  0001 C CNN
+F 2 "Frequently_Used_LE:0805_2012Metric" V 6130 3700 50  0001 C CNN
 F 3 "http://www.koaspeer.com/pdfs/RK73H.pdf" H 6200 3700 50  0001 C CNN
 F 4 "KOA Speer Electronics, Inc." H 6200 3700 50  0001 C CNN "Manufacturer Name"
 F 5 "Digikey" H 6200 3700 50  0001 C CNN "Source"
+F 6 "330 Ohms ±1% 0.25W, 1/4W Chip Resistor 1206 (3216 Metric)" H 6200 3700 50  0001 C CNN "Description"
+F 7 "RK73H2ATTD3300F" H 6200 3700 50  0001 C CNN "Manufacturer Part No."
+F 8 "2019-RK73H2ATTD3300FCT-ND" H 6200 3700 50  0001 C CNN "Source Part No."
 	1    6200 3700
 	1    0    0    -1
@@
 F 0 "R27" H 6670 3746 50  0000 L CNN
 F 1 "330" H 6670 3655 50  0000 L CNN
-F 2 "Frequently_Used_LE:0805_2012Metric_HandSolder" V 6530 3700 50  0001 C CNN
+F 2 "Frequently_Used_LE:0805_2012Metric" V 6530 3700 50  0001 C CNN
 F 3 "http://www.koaspeer.com/pdfs/RK73H.pdf" H 6600 3700 50  0001 C CNN
 F 4 "KOA Speer Electronics, Inc." H 6600 3700 50  0001 C CNN "Manufacturer Name"
 F 5 "Digikey" H 6600 3700 50  0001 C CNN "Source"
+F 6 "330 Ohms ±1% 0.25W, 1/4W Chip Resistor 1206 (3216 Metric)" H 6600 3700 50  0001 C CNN "Description"
+F 7 "RK73H2ATTD3300F" H 6600 3700 50  0001 C CNN "Manufacturer Part No."
+F 8 "2019-RK73H2ATTD3300FCT-ND" H 6600 3700 50  0001 C CNN "Source Part No."
 	1    6600 3700
 	1    0    0    -1
@@
 F 0 "R28" H 7070 3746 50  0000 L CNN
 F 1 "330" H 7070 3655 50  0000 L CNN
-F 2 "Frequently_Used_LE:0805_2012Metric_HandSolder" V 6930 3700 50  0001 C CNN
+F 2 "Frequently_Used_LE:0805_2012Metric" V 6930 3700 50  0001 C CNN
 F 3 "http://www.koaspeer.com/pdfs/RK73H.pdf" H 7000 3700 50  0001 C CNN
 F 4 "KOA Speer Electronics, Inc." H 7000 3700 50  0001 C CNN "Manufacturer Name"
 F 5 "Digikey" H 7000 3700 50  0001 C CNN "Source"
+F 6 "330 Ohms ±1% 0.25W, 1/4W Chip Resistor 1206 (3216 Metric)" H 7000 3700 50  0001 C CNN "Description"
+F 7 "RK73H2ATTD3300F" H 7000 3700 50  0001 C CNN "Manufacturer Part No."
+F 8 "2019-RK73H2ATTD3300FCT-ND" H 7000 3700 50  0001 C CNN "Source Part No."
 	1    7000 3700
 	1    0    0    -1

Commit message: PCB Update
Changed lines of the file:
@@
 $Descr A4 11693 8268
 encoding utf-8
-Sheet 3 17
+Sheet 6 17
 Title ""
 Date ""
@@
 AR Path="/5ED17BA0/5ED2A30A/5E9E70EC" Ref="D15"  Part="1"
 AR Path="/5ED17BA0/5ED2A30D/5E9E70EC" Ref="D19"  Part="1"
-F 0 "D19" V 5839 3883 50  0000 R CNN
+F 0 "D15" V 5839 3883 50  0000 R CNN
 F 1 "LED" V 5748 3883 50  0000 R CNN
 F 2 "LED_SMD:LED_1812_4532Metric" H 5800 4000 50  0001 C CNN
@@
 AR Path="/5ED17BA0/5ED2A30A/5E9DC34C" Ref="R20"  Part="1"
 AR Path="/5ED17BA0/5ED2A30D/5E9DC34C" Ref="R25"  Part="1"
-F 0 "R25" H 5870 3746 50  0000 L CNN
+F 0 "R20" H 5870 3746 50  0000 L CNN
 F 1 "330" H 5870 3655 50  0000 L CNN
 F 2 "Frequently_Used_LE:0805_2012Metric" V 5730 3700 50  0001 C CNN
@@
 AR Path="/5ED17BA0/5ED2A30A/5E9DC352" Ref="R21"  Part="1"
 AR Path="/5ED17BA0/5ED2A30D/5E9DC352" Ref="R26"  Part="1"
-F 0 "R26" H 6270 3746 50  0000 L CNN
+F 0 "R21" H 6270 3746 50  0000 L CNN
 F 1 "330" H 6270 3655 50  0000 L CNN
 F 2 "Frequently_Used_LE:0805_2012Metric" V 6130 3700 50  0001 C CNN
@@
 AR Path="/5ED17BA0/5ED2A30A/5E9E70F0" Ref="R22"  Part="1"
 AR Path="/5ED17BA0/5ED2A30D/5E9E70F0" Ref="R27"  Part="1"
-F 0 "R27" H 6670 3746 50  0000 L CNN
+F 0 "R22" H 6670 3746 50  0000 L CNN
 F 1 "330" H 6670 3655 50  0000 L CNN
 F 2 "Frequently_Used_LE:0805_2012Metric" V 6530 3700 50  0001 C CNN
@@
 AR Path="/5ED17BA0/5ED2A30A/5E9E70F2" Ref="R23"  Part="1"
 AR Path="/5ED17BA0/5ED2A30D/5E9E70F2" Ref="R28"  Part="1"
-F 0 "R28" H 7070 3746 50  0000 L CNN
+F 0 "R23" H 7070 3746 50  0000 L CNN
 F 1 "330" H 7070 3655 50  0000 L CNN
 F 2 "Frequently_Used_LE:0805_2012Metric" V 6930 3700 50  0001 C CNN
@@
 AR Path="/5ED17BA0/5ED2A30A/5E9E70F3" Ref="D18"  Part="1"
 AR Path="/5ED17BA0/5ED2A30D/5E9E70F3" Ref="D22"  Part="1"
-F 0 "D22" V 7039 3883 50  0000 R CNN
+F 0 "D18" V 7039 3883 50  0000 R CNN
 F 1 "LED" V 6948 3883 50  0000 R CNN
 F 2 "LED_SMD:LED_1812_4532Metric" H 7000 4000 50  0001 C CNN
@@
 AR Path="/5ED17BA0/5ED2A30A/5E9E70F1" Ref="D17"  Part="1"
 AR Path="/5ED17BA0/5ED2A30D/5E9E70F1" Ref="D21"  Part="1"
-F 0 "D21" V 6639 3883 50  0000 R CNN
+F 0 "D17" V 6639 3883 50  0000 R CNN
 F 1 "LED" V 6548 3883 50  0000 R CNN
 F 2 "LED_SMD:LED_1812_4532Metric" H 6600 4000 50  0001 C CNN
@@
 AR Path="/5ED17BA0/5ED2A30A/5E9E70EF" Ref="D16"  Part="1"
 AR Path="/5ED17BA0/5ED2A30D/5E9E70EF" Ref="D20"  Part="1"
-F 0 "D20" V 6239 3883 50  0000 R CNN
+F 0 "D16" V 6239 3883 50  0000 R CNN
 F 1 "LED" V 6148 3883 50  0000 R CNN
 F 2 "LED_SMD:LED_1812_4532Metric" H 6200 4000 50  0001 C CNN
@@
 AR Path="/5ED17BA0/5ED2A30A/5EB3A90A" Ref="#PWR040"  Part="1"
 AR Path="/5ED17BA0/5ED2A30D/5EB3A90A" Ref="#PWR042"  Part="1"
-F 0 "#PWR042" H 5450 3350 50  0001 C CNN
+F 0 "#PWR040" H 5450 3350 50  0001 C CNN
 F 1 "+5V" H 5465 3673 50  0000 C CNN
 F 2 "" H 5450 3500 50  0001 C CNN

Commit message: Switched to 0603_1608M size for passives
Parts:
- R5, R6, R7, R8: footprint Frequently_Used_LE:0805_2012Metric -> Frequently_Used_LE:0603_1608Metric; Description 330 Ohms ±1% 0.25W, 1/4W Chip Resistor 1206 (3216 Metric) -> 330 Ohms ±1% 0.25W, 1/4W Chip Resistor 0603 (1608 Metric) A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; Manufacturer Name KOA Speer Electronics, Inc. -> Vishay Dale; Manufacturer Part No. RK73H2ATTD3300F -> RCS0603330RFKEA; Source Part No. 2019-RK73H2ATTD3300FCT-ND -> 541-10456-1-ND
Changed lines of the file:
@@
 $Descr A4 11693 8268
 encoding utf-8
-Sheet 6 17
+Sheet 6 18
 Title ""
 Date ""
@@
 AR Path="/5ED17BA0/5ED2A30A/5E9E70EC" Ref="D15"  Part="1"
 AR Path="/5ED17BA0/5ED2A30D/5E9E70EC" Ref="D19"  Part="1"
-F 0 "D15" V 5839 3883 50  0000 R CNN
+F 0 "D19" V 5839 3883 50  0000 R CNN
 F 1 "LED" V 5748 3883 50  0000 R CNN
 F 2 "LED_SMD:LED_1812_4532Metric" H 5800 4000 50  0001 C CNN
@@
 AR Path="/5ED17BA0/5ED2A30A/5E9DC34C" Ref="R20"  Part="1"
 AR Path="/5ED17BA0/5ED2A30D/5E9DC34C" Ref="R25"  Part="1"
-F 0 "R20" H 5870 3746 50  0000 L CNN
+F 0 "R25" H 5870 3746 50  0000 L CNN
 F 1 "330" H 5870 3655 50  0000 L CNN
-F 2 "Frequently_Used_LE:0805_2012Metric" V 5730 3700 50  0001 C CNN
-F 3 "http://www.koaspeer.com/pdfs/RK73H.pdf" H 5800 3700 50  0001 C CNN
-F 4 "KOA Speer Electronics, Inc." H 5800 3700 50  0001 C CNN "Manufacturer Name"
+F 2 "Frequently_Used_LE:0603_1608Metric" V 5730 3700 50  0001 C CNN
+F 3 "https://www.vishay.com/docs/20065/rcse3.pdf" H 5800 3700 50  0001 C CNN
+F 4 "Vishay Dale" H 5800 3700 50  0001 C CNN "Manufacturer Name"
 F 5 "Digikey" H 5800 3700 50  0001 C CNN "Source"
-F 6 "330 Ohms ±1% 0.25W, 1/4W Chip Resistor 1206 (3216 Metric)" H 5800 3700 50  0001 C CNN "Description"
-F 7 "RK73H2ATTD3300F" H 5800 3700 50  0001 C CNN "Manufacturer Part No."
-F 8 "2019-RK73H2ATTD3300FCT-ND" H 5800 3700 50  0001 C CNN "Source Part No."
+F 6 "330 Ohms ±1% 0.25W, 1/4W Chip Resistor 0603 (1608 Metric) Automotive AEC-Q200, Pulse Withstanding Thick Film" H 5800 3700 50  0001 C CNN "Description"
+F 7 "RCS0603330RFKEA" H 5800 3700 50  0001 C CNN "Manufacturer Part No."
+F 8 "541-10456-1-ND" H 5800 3700 50  0001 C CNN "Source Part No."
 	1    5800 3700
 	1    0    0    -1
@@
 AR Path="/5ED17BA0/5ED2A30A/5E9DC352" Ref="R21"  Part="1"
 AR Path="/5ED17BA0/5ED2A30D/5E9DC352" Ref="R26"  Part="1"
-F 0 "R21" H 6270 3746 50  0000 L CNN
+F 0 "R26" H 6270 3746 50  0000 L CNN
 F 1 "330" H 6270 3655 50  0000 L CNN
-F 2 "Frequently_Used_LE:0805_2012Metric" V 6130 3700 50  0001 C CNN
-F 3 "http://www.koaspeer.com/pdfs/RK73H.pdf" H 6200 3700 50  0001 C CNN
-F 4 "KOA Speer Electronics, Inc." H 6200 3700 50  0001 C CNN "Manufacturer Name"
+F 2 "Frequently_Used_LE:0603_1608Metric" V 6130 3700 50  0001 C CNN
+F 3 "https://www.vishay.com/docs/20065/rcse3.pdf" H 6200 3700 50  0001 C CNN
+F 4 "Vishay Dale" H 6200 3700 50  0001 C CNN "Manufacturer Name"
 F 5 "Digikey" H 6200 3700 50  0001 C CNN "Source"
-F 6 "330 Ohms ±1% 0.25W, 1/4W Chip Resistor 1206 (3216 Metric)" H 6200 3700 50  0001 C CNN "Description"
-F 7 "RK73H2ATTD3300F" H 6200 3700 50  0001 C CNN "Manufacturer Part No."
-F 8 "2019-RK73H2ATTD3300FCT-ND" H 6200 3700 50  0001 C CNN "Source Part No."
+F 6 "330 Ohms ±1% 0.25W, 1/4W Chip Resistor 0603 (1608 Metric) Automotive AEC-Q200, Pulse Withstanding Thick Film" H 6200 3700 50  0001 C CNN "Description"
+F 7 "RCS0603330RFKEA" H 6200 3700 50  0001 C CNN "Manufacturer Part No."
+F 8 "541-10456-1-ND" H 6200 3700 50  0001 C CNN "Source Part No."
 	1    6200 3700
 	1    0    0    -1
@@
 AR Path="/5ED17BA0/5ED2A30A/5E9E70F0" Ref="R22"  Part="1"
 AR Path="/5ED17BA0/5ED2A30D/5E9E70F0" Ref="R27"  Part="1"
-F 0 "R22" H 6670 3746 50  0000 L CNN
+F 0 "R27" H 6670 3746 50  0000 L CNN
 F 1 "330" H 6670 3655 50  0000 L CNN
-F 2 "Frequently_Used_LE:0805_2012Metric" V 6530 3700 50  0001 C CNN
-F 3 "http://www.koaspeer.com/pdfs/RK73H.pdf" H 6600 3700 50  0001 C CNN
-F 4 "KOA Speer Electronics, Inc." H 6600 3700 50  0001 C CNN "Manufacturer Name"
+F 2 "Frequently_Used_LE:0603_1608Metric" V 6530 3700 50  0001 C CNN
+F 3 "https://www.vishay.com/docs/20065/rcse3.pdf" H 6600 3700 50  0001 C CNN
+F 4 "Vishay Dale" H 6600 3700 50  0001 C CNN "Manufacturer Name"
 F 5 "Digikey" H 6600 3700 50  0001 C CNN "Source"
-F 6 "330 Ohms ±1% 0.25W, 1/4W Chip Resistor 1206 (3216 Metric)" H 6600 3700 50  0001 C CNN "Description"
-F 7 "RK73H2ATTD3300F" H 6600 3700 50  0001 C CNN "Manufacturer Part No."
-F 8 "2019-RK73H2ATTD3300FCT-ND" H 6600 3700 50  0001 C CNN "Source Part No."
+F 6 "330 Ohms ±1% 0.25W, 1/4W Chip Resistor 0603 (1608 Metric) Automotive AEC-Q200, Pulse Withstanding Thick Film" H 6600 3700 50  0001 C CNN "Description"
+F 7 "RCS0603330RFKEA" H 6600 3700 50  0001 C CNN "Manufacturer Part No."
+F 8 "541-10456-1-ND" H 6600 3700 50  0001 C CNN "Source Part No."
 	1    6600 3700
 	1    0    0    -1
@@
 AR Path="/5ED17BA0/5ED2A30A/5E9E70F2" Ref="R23"  Part="1"
 AR Path="/5ED17BA0/5ED2A30D/5E9E70F2" Ref="R28"  Part="1"
-F 0 "R23" H 7070 3746 50  0000 L CNN
+F 0 "R28" H 7070 3746 50  0000 L CNN
 F 1 "330" H 7070 3655 50  0000 L CNN
-F 2 "Frequently_Used_LE:0805_2012Metric" V 6930 3700 50  0001 C CNN
-F 3 "http://www.koaspeer.com/pdfs/RK73H.pdf" H 7000 3700 50  0001 C CNN
-F 4 "KOA Speer Electronics, Inc." H 7000 3700 50  0001 C CNN "Manufacturer Name"
+F 2 "Frequently_Used_LE:0603_1608Metric" V 6930 3700 50  0001 C CNN
+F 3 "https://www.vishay.com/docs/20065/rcse3.pdf" H 7000 3700 50  0001 C CNN
+F 4 "Vishay Dale" H 7000 3700 50  0001 C CNN "Manufacturer Name"
 F 5 "Digikey" H 7000 3700 50  0001 C CNN "Source"
-F 6 "330 Ohms ±1% 0.25W, 1/4W Chip Resistor 1206 (3216 Metric)" H 7000 3700 50  0001 C CNN "Description"
-F 7 "RK73H2ATTD3300F" H 7000 3700 50  0001 C CNN "Manufacturer Part No."
-F 8 "2019-RK73H2ATTD3300FCT-ND" H 7000 3700 50  0001 C CNN "Source Part No."
+F 6 "330 Ohms ±1% 0.25W, 1/4W Chip Resistor 0603 (1608 Metric) Automotive AEC-Q200, Pulse Withstanding Thick Film" H 7000 3700 50  0001 C CNN "Description"
+F 7 "RCS0603330RFKEA" H 7000 3700 50  0001 C CNN "Manufacturer Part No."
+F 8 "541-10456-1-ND" H 7000 3700 50  0001 C CNN "Source Part No."
 	1    7000 3700
 	1    0    0    -1
@@
 AR Path="/5ED17BA0/5ED2A30A/5E9E70F3" Ref="D18"  Part="1"
 AR Path="/5ED17BA0/5ED2A30D/5E9E70F3" Ref="D22"  Part="1"
-F 0 "D18" V 7039 3883 50  0000 R CNN
+F 0 "D22" V 7039 3883 50  0000 R CNN
 F 1 "LED" V 6948 3883 50  0000 R CNN
 F 2 "LED_SMD:LED_1812_4532Metric" H 7000 4000 50  0001 C CNN
@@
 AR Path="/5ED17BA0/5ED2A30A/5E9E70F1" Ref="D17"  Part="1"
 AR Path="/5ED17BA0/5ED2A30D/5E9E70F1" Ref="D21"  Part="1"
-F 0 "D17" V 6639 3883 50  0000 R CNN
+F 0 "D21" V 6639 3883 50  0000 R CNN
 F 1 "LED" V 6548 3883 50  0000 R CNN
 F 2 "LED_SMD:LED_1812_4532Metric" H 6600 4000 50  0001 C CNN
@@
 AR Path="/5ED17BA0/5ED2A30A/5E9E70EF" Ref="D16"  Part="1"
 AR Path="/5ED17BA0/5ED2A30D/5E9E70EF" Ref="D20"  Part="1"
-F 0 "D16" V 6239 3883 50  0000 R CNN
+F 0 "D20" V 6239 3883 50  0000 R CNN
 F 1 "LED" V 6148 3883 50  0000 R CNN
 F 2 "LED_SMD:LED_1812_4532Metric" H 6200 4000 50  0001 C CNN
@@
 AR Path="/5ED17BA0/5ED2A30A/5EB3A90A" Ref="#PWR040"  Part="1"
 AR Path="/5ED17BA0/5ED2A30D/5EB3A90A" Ref="#PWR042"  Part="1"
-F 0 "#PWR040" H 5450 3350 50  0001 C CNN
+F 0 "#PWR042" H 5450 3350 50  0001 C CNN
 F 1 "+5V" H 5465 3673 50  0000 C CNN
 F 2 "" H 5450 3500 50  0001 C CNN
