File: Naquadah Generator Main/GreenRedLights.sch (KiCad schematic (older format))
At the start: 4 parts

Commit message: Updates
Changed lines of the file:
@@
 $Descr A4 11693 8268
 encoding utf-8
-Sheet 8 11
+Sheet 9 11
 Title ""
 Date ""
@@
 AR Path="/5ED17BA0/5ED2A32F/5EEF3073" Ref="D2"  Part="1"
 AR Path="/5ED17BA0/5ED2A36D/5EEF3073" Ref="D26"  Part="1"
-F 0 "D2" V 5889 3983 50  0000 R CNN
+F 0 "D26" V 5889 3983 50  0000 R CNN
 F 1 "LED" V 5798 3983 50  0000 R CNN
 F 2 "LED_SMD:LED_1812_4532Metric" H 5850 4100 50  0001 C CNN
@@
 AR Path="/5ED17BA0/5ED2A32F/5EEF307B" Ref="R3"  Part="1"
 AR Path="/5ED17BA0/5ED2A36D/5EEF307B" Ref="R35"  Part="1"
-F 0 "R3" H 5920 3846 50  0000 L CNN
+F 0 "R35" H 5920 3846 50  0000 L CNN
 F 1 "330" H 5920 3755 50  0000 L CNN
 F 2 "Frequently_Used:0805_2012Metric_HandSolder" V 5780 3800 50  0001 C CNN
@@
 AR Path="/5ED17BA0/5ED2A32F/5EEF3083" Ref="R34"  Part="1"
 AR Path="/5ED17BA0/5ED2A36D/5EEF3083" Ref="R36"  Part="1"
-F 0 "R34" H 6320 3846 50  0000 L CNN
+F 0 "R36" H 6320 3846 50  0000 L CNN
 F 1 "330" H 6320 3755 50  0000 L CNN
 F 2 "Frequently_Used:0805_2012Metric_HandSolder" V 6180 3800 50  0001 C CNN
@@
 AR Path="/5ED17BA0/5ED2A32F/5EEF308D" Ref="D25"  Part="1"
 AR Path="/5ED17BA0/5ED2A36D/5EEF308D" Ref="D27"  Part="1"
-F 0 "D25" V 6289 3983 50  0000 R CNN
+F 0 "D27" V 6289 3983 50  0000 R CNN
 F 1 "LED" V 6198 3983 50  0000 R CNN
 F 2 "LED_SMD:LED_1812_4532Metric" H 6250 4100 50  0001 C CNN

Commit message: Move libraries and added configuration path.
Moved Li-Ion library to common KiCad library.  Added variables to configuration paths to reference my KiCad libraries.  Moved all 3D components to my common library.
Parts:
- R3, R34: footprint Frequently_Used:0805_2012Metric_HandSolder -> FrequentlyUsed:0805_2012Metric_HandSolder
Changed lines of the file:
@@
 F 0 "R35" H 5920 3846 50  0000 L CNN
 F 1 "330" H 5920 3755 50  0000 L CNN
-F 2 "Frequently_Used:0805_2012Metric_HandSolder" V 5780 3800 50  0001 C CNN
+F 2 "FrequentlyUsed:0805_2012Metric_HandSolder" V 5780 3800 50  0001 C CNN
 F 3 "~" H 5850 3800 50  0001 C CNN
 	1    5850 3800
@@
 F 0 "R36" H 6320 3846 50  0000 L CNN
 F 1 "330" H 6320 3755 50  0000 L CNN
-F 2 "Frequently_Used:0805_2012Metric_HandSolder" V 6180 3800 50  0001 C CNN
+F 2 "FrequentlyUsed:0805_2012Metric_HandSolder" V 6180 3800 50  0001 C CNN
 F 3 "~" H 6250 3800 50  0001 C CNN
 	1    6250 3800

Commit message: PCB Updates
Changed lines of the file:
@@
 $Descr A4 11693 8268
 encoding utf-8
-Sheet 9 11
+Sheet 8 11
 Title ""
 Date ""
@@
 AR Path="/5ED17BA0/5ED2A32F/5EEF3073" Ref="D2"  Part="1"
 AR Path="/5ED17BA0/5ED2A36D/5EEF3073" Ref="D26"  Part="1"
-F 0 "D26" V 5889 3983 50  0000 R CNN
+F 0 "D2" V 5889 3983 50  0000 R CNN
 F 1 "LED" V 5798 3983 50  0000 R CNN
 F 2 "LED_SMD:LED_1812_4532Metric" H 5850 4100 50  0001 C CNN
@@
 AR Path="/5ED17BA0/5ED2A32F/5EEF307B" Ref="R3"  Part="1"
 AR Path="/5ED17BA0/5ED2A36D/5EEF307B" Ref="R35"  Part="1"
-F 0 "R35" H 5920 3846 50  0000 L CNN
+F 0 "R3" H 5920 3846 50  0000 L CNN
 F 1 "330" H 5920 3755 50  0000 L CNN
 F 2 "FrequentlyUsed:0805_2012Metric_HandSolder" V 5780 3800 50  0001 C CNN
@@
 AR Path="/5ED17BA0/5ED2A32F/5EEF3083" Ref="R34"  Part="1"
 AR Path="/5ED17BA0/5ED2A36D/5EEF3083" Ref="R36"  Part="1"
-F 0 "R36" H 6320 3846 50  0000 L CNN
+F 0 "R34" H 6320 3846 50  0000 L CNN
 F 1 "330" H 6320 3755 50  0000 L CNN
 F 2 "FrequentlyUsed:0805_2012Metric_HandSolder" V 6180 3800 50  0001 C CNN
@@
 AR Path="/5ED17BA0/5ED2A32F/5EEF308D" Ref="D25"  Part="1"
 AR Path="/5ED17BA0/5ED2A36D/5EEF308D" Ref="D27"  Part="1"
-F 0 "D27" V 6289 3983 50  0000 R CNN
+F 0 "D25" V 6289 3983 50  0000 R CNN
 F 1 "LED" V 6198 3983 50  0000 R CNN
 F 2 "LED_SMD:LED_1812_4532Metric" H 6250 4100 50  0001 C CNN

Commit message: Updates
Changed lines of the file:
@@
 $Descr A4 11693 8268
 encoding utf-8
-Sheet 8 11
+Sheet 8 12
 Title ""
 Date ""
@@
 AR Path="/5ED17BA0/5ED2A32F/5EEF3073" Ref="D2"  Part="1"
 AR Path="/5ED17BA0/5ED2A36D/5EEF3073" Ref="D26"  Part="1"
-F 0 "D2" V 5889 3983 50  0000 R CNN
+F 0 "D26" V 5889 3983 50  0000 R CNN
 F 1 "LED" V 5798 3983 50  0000 R CNN
 F 2 "LED_SMD:LED_1812_4532Metric" H 5850 4100 50  0001 C CNN
@@
 AR Path="/5ED17BA0/5ED2A32F/5EEF307B" Ref="R3"  Part="1"
 AR Path="/5ED17BA0/5ED2A36D/5EEF307B" Ref="R35"  Part="1"
-F 0 "R3" H 5920 3846 50  0000 L CNN
+F 0 "R35" H 5920 3846 50  0000 L CNN
 F 1 "330" H 5920 3755 50  0000 L CNN
 F 2 "FrequentlyUsed:0805_2012Metric_HandSolder" V 5780 3800 50  0001 C CNN
@@
 AR Path="/5ED17BA0/5ED2A32F/5EEF3083" Ref="R34"  Part="1"
 AR Path="/5ED17BA0/5ED2A36D/5EEF3083" Ref="R36"  Part="1"
-F 0 "R34" H 6320 3846 50  0000 L CNN
+F 0 "R36" H 6320 3846 50  0000 L CNN
 F 1 "330" H 6320 3755 50  0000 L CNN
 F 2 "FrequentlyUsed:0805_2012Metric_HandSolder" V 6180 3800 50  0001 C CNN
@@
 AR Path="/5ED17BA0/5ED2A32F/5EEF308D" Ref="D25"  Part="1"
 AR Path="/5ED17BA0/5ED2A36D/5EEF308D" Ref="D27"  Part="1"
-F 0 "D25" V 6289 3983 50  0000 R CNN
+F 0 "D27" V 6289 3983 50  0000 R CNN
 F 1 "LED" V 6198 3983 50  0000 R CNN
 F 2 "LED_SMD:LED_1812_4532Metric" H 6250 4100 50  0001 C CNN

Commit message: Audio update
Parts:
- R3, R34: footprint FrequentlyUsed:0805_2012Metric_HandSolder -> Frequently_Used_LE:0805_2012Metric_HandSolder; Manufacturer Name (none) -> KOA Speer Electronics, Inc.; Source (none) -> Digikey
Changed lines of the file:
@@
 F 0 "R35" H 5920 3846 50  0000 L CNN
 F 1 "330" H 5920 3755 50  0000 L CNN
-F 2 "FrequentlyUsed:0805_2012Metric_HandSolder" V 5780 3800 50  0001 C CNN
-F 3 "~" H 5850 3800 50  0001 C CNN
+F 2 "Frequently_Used_LE:0805_2012Metric_HandSolder" V 5780 3800 50  0001 C CNN
+F 3 "http://www.koaspeer.com/pdfs/RK73H.pdf" H 5850 3800 50  0001 C CNN
+F 4 "KOA Speer Electronics, Inc." H 5850 3800 50  0001 C CNN "Manufacturer Name"
+F 5 "Digikey" H 5850 3800 50  0001 C CNN "Source"
 	1    5850 3800
 	1    0    0    -1
@@
 F 0 "R36" H 6320 3846 50  0000 L CNN
 F 1 "330" H 6320 3755 50  0000 L CNN
-F 2 "FrequentlyUsed:0805_2012Metric_HandSolder" V 6180 3800 50  0001 C CNN
-F 3 "~" H 6250 3800 50  0001 C CNN
+F 2 "Frequently_Used_LE:0805_2012Metric_HandSolder" V 6180 3800 50  0001 C CNN
+F 3 "http://www.koaspeer.com/pdfs/RK73H.pdf" H 6250 3800 50  0001 C CNN
+F 4 "KOA Speer Electronics, Inc." H 6250 3800 50  0001 C CNN "Manufacturer Name"
+F 5 "Digikey" H 6250 3800 50  0001 C CNN "Source"
 	1    6250 3800
 	1    0    0    -1
