File: Naquadah Generator Main/GreenRedLights.sch (KiCad schematic (older format))
At the start: 4 parts

Commit message: Added level shifter, moved user interface connector location
Added level shifter, moved user interface connector location
Parts:
- R3, R34: footprint Frequently_Used_LE:0805_2012Metric_HandSolder -> Frequently_Used_LE:0805_2012Metric; Description (none) -> 330 Ohms ±1% 0.25W, 1/4W Chip Resistor 1206 (3216 Metric); Manufacturer Part No. (none) -> RK73H2ATTD3300F; Source Part No. (none) -> 2019-RK73H2ATTD3300FCT-ND
Changed lines of the file:
@@
 $Descr A4 11693 8268
 encoding utf-8
-Sheet 9 16
+Sheet 9 17
 Title ""
 Date ""
@@
 F 0 "R35" H 5920 3846 50  0000 L CNN
 F 1 "330" H 5920 3755 50  0000 L CNN
-F 2 "Frequently_Used_LE:0805_2012Metric_HandSolder" V 5780 3800 50  0001 C CNN
+F 2 "Frequently_Used_LE:0805_2012Metric" V 5780 3800 50  0001 C CNN
 F 3 "http://www.koaspeer.com/pdfs/RK73H.pdf" H 5850 3800 50  0001 C CNN
 F 4 "KOA Speer Electronics, Inc." H 5850 3800 50  0001 C CNN "Manufacturer Name"
 F 5 "Digikey" H 5850 3800 50  0001 C CNN "Source"
+F 6 "330 Ohms ±1% 0.25W, 1/4W Chip Resistor 1206 (3216 Metric)" H 5850 3800 50  0001 C CNN "Description"
+F 7 "RK73H2ATTD3300F" H 5850 3800 50  0001 C CNN "Manufacturer Part No."
+F 8 "2019-RK73H2ATTD3300FCT-ND" H 5850 3800 50  0001 C CNN "Source Part No."
 	1    5850 3800
 	1    0    0    -1
@@
 F 0 "R36" H 6320 3846 50  0000 L CNN
 F 1 "330" H 6320 3755 50  0000 L CNN
-F 2 "Frequently_Used_LE:0805_2012Metric_HandSolder" V 6180 3800 50  0001 C CNN
+F 2 "Frequently_Used_LE:0805_2012Metric" V 6180 3800 50  0001 C CNN
 F 3 "http://www.koaspeer.com/pdfs/RK73H.pdf" H 6250 3800 50  0001 C CNN
 F 4 "KOA Speer Electronics, Inc." H 6250 3800 50  0001 C CNN "Manufacturer Name"
 F 5 "Digikey" H 6250 3800 50  0001 C CNN "Source"
+F 6 "330 Ohms ±1% 0.25W, 1/4W Chip Resistor 1206 (3216 Metric)" H 6250 3800 50  0001 C CNN "Description"
+F 7 "RK73H2ATTD3300F" H 6250 3800 50  0001 C CNN "Manufacturer Part No."
+F 8 "2019-RK73H2ATTD3300FCT-ND" H 6250 3800 50  0001 C CNN "Source Part No."
 	1    6250 3800
 	1    0    0    -1

Commit message: Switched to 0603_1608M size for passives
Parts:
- R3, R34: footprint Frequently_Used_LE:0805_2012Metric -> Frequently_Used_LE:0603_1608Metric; Description 330 Ohms ±1% 0.25W, 1/4W Chip Resistor 1206 (3216 Metric) -> 330 Ohms ±1% 0.25W, 1/4W Chip Resistor 0603 (1608 Metric) A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; Manufacturer Name KOA Speer Electronics, Inc. -> Vishay Dale; Manufacturer Part No. RK73H2ATTD3300F -> RCS0603330RFKEA; Source Part No. 2019-RK73H2ATTD3300FCT-ND -> 541-10456-1-ND
Changed lines of the file:
@@
 $Descr A4 11693 8268
 encoding utf-8
-Sheet 9 17
+Sheet 9 18
 Title ""
 Date ""
@@
 F 0 "R35" H 5920 3846 50  0000 L CNN
 F 1 "330" H 5920 3755 50  0000 L CNN
-F 2 "Frequently_Used_LE:0805_2012Metric" V 5780 3800 50  0001 C CNN
-F 3 "http://www.koaspeer.com/pdfs/RK73H.pdf" H 5850 3800 50  0001 C CNN
-F 4 "KOA Speer Electronics, Inc." H 5850 3800 50  0001 C CNN "Manufacturer Name"
+F 2 "Frequently_Used_LE:0603_1608Metric" V 5780 3800 50  0001 C CNN
+F 3 "https://www.vishay.com/docs/20065/rcse3.pdf" H 5850 3800 50  0001 C CNN
+F 4 "Vishay Dale" H 5850 3800 50  0001 C CNN "Manufacturer Name"
 F 5 "Digikey" H 5850 3800 50  0001 C CNN "Source"
-F 6 "330 Ohms ±1% 0.25W, 1/4W Chip Resistor 1206 (3216 Metric)" H 5850 3800 50  0001 C CNN "Description"
-F 7 "RK73H2ATTD3300F" H 5850 3800 50  0001 C CNN "Manufacturer Part No."
-F 8 "2019-RK73H2ATTD3300FCT-ND" H 5850 3800 50  0001 C CNN "Source Part No."
+F 6 "330 Ohms ±1% 0.25W, 1/4W Chip Resistor 0603 (1608 Metric) Automotive AEC-Q200, Pulse Withstanding Thick Film" H 5850 3800 50  0001 C CNN "Description"
+F 7 "RCS0603330RFKEA" H 5850 3800 50  0001 C CNN "Manufacturer Part No."
+F 8 "541-10456-1-ND" H 5850 3800 50  0001 C CNN "Source Part No."
 	1    5850 3800
 	1    0    0    -1
@@
 F 0 "R36" H 6320 3846 50  0000 L CNN
 F 1 "330" H 6320 3755 50  0000 L CNN
-F 2 "Frequently_Used_LE:0805_2012Metric" V 6180 3800 50  0001 C CNN
-F 3 "http://www.koaspeer.com/pdfs/RK73H.pdf" H 6250 3800 50  0001 C CNN
-F 4 "KOA Speer Electronics, Inc." H 6250 3800 50  0001 C CNN "Manufacturer Name"
+F 2 "Frequently_Used_LE:0603_1608Metric" V 6180 3800 50  0001 C CNN
+F 3 "https://www.vishay.com/docs/20065/rcse3.pdf" H 6250 3800 50  0001 C CNN
+F 4 "Vishay Dale" H 6250 3800 50  0001 C CNN "Manufacturer Name"
 F 5 "Digikey" H 6250 3800 50  0001 C CNN "Source"
-F 6 "330 Ohms ±1% 0.25W, 1/4W Chip Resistor 1206 (3216 Metric)" H 6250 3800 50  0001 C CNN "Description"
-F 7 "RK73H2ATTD3300F" H 6250 3800 50  0001 C CNN "Manufacturer Part No."
-F 8 "2019-RK73H2ATTD3300FCT-ND" H 6250 3800 50  0001 C CNN "Source Part No."
+F 6 "330 Ohms ±1% 0.25W, 1/4W Chip Resistor 0603 (1608 Metric) Automotive AEC-Q200, Pulse Withstanding Thick Film" H 6250 3800 50  0001 C CNN "Description"
+F 7 "RCS0603330RFKEA" H 6250 3800 50  0001 C CNN "Manufacturer Part No."
+F 8 "541-10456-1-ND" H 6250 3800 50  0001 C CNN "Source Part No."
 	1    6250 3800
 	1    0    0    -1
