File: Naquadah Generator Main/Connectors.sch (KiCad schematic (older format))
At the start: 20 parts, among them J0 Conn_ISP_Prog, J1 State_Sensing_Conn, J2 State_Sensing_Conn, J8 USB Solder Pads, P1 USB_C_Plug_USB2.0

Commit message: Added real power schematic
Parts:
- renumbered D25 to D1
Changed lines of the file:
@@
 $EndComp
 $Comp
-L Power_LE:PRTR5V0U2X D25
+L Power_LE:PRTR5V0U2X D1
 U 1 1 5ED3FF2E
 P 4700 1450
-F 0 "D25" H 4800 1900 50  0000 L CNN
+F 0 "D1" H 4800 1900 50  0000 L CNN
 F 1 "RED" H 4800 1800 50  0000 L CNN
 F 2 "Frequently_Used:LED_0805_2012Metric_HandSolder" H 4800 1100 50  0001 L CNN

Commit message: Symbol field corrections and additions
Parts:
- J8: Description (none) -> None; Digikey Part No. (none) -> None; Manufacturer Name (none) -> None; Manufacturer Part No. (none) -> None
Changed lines of the file:
@@
 F 2 "Naquadah_Generator:WireSoldPads_1x4_WOL" H 4550 4050 50  0001 C CNN
 F 3 "None" H 4550 4050 50  0001 C CNN
+F 4 "None" H 4550 4050 50  0001 C CNN "Description"
+F 5 "None" H 4550 4050 50  0001 C CNN "Digikey Part No."
+F 6 "None" H 4550 4050 50  0001 C CNN "Manufacturer Name"
+F 7 "None" H 4550 4050 50  0001 C CNN "Manufacturer Part No."
 	1    4550 4050
 	-1   0    0    1

Commit message: Adding Power Daughter Board
Parts:
- added TP? (x4): TestPoint, Frequently_Used:Pad_2.5-2.5, symbol Frequently_Used:TestPoint
- D1: value RED -> SDP; footprint Frequently_Used:LED_0805_2012Metric_HandSolder -> Package_TO_SOT_SMD:SOT-143; Digikey Part No. 732-4984-1-ND -> (none); Source (none) -> Digikey; Source Part No. (none) -> 732-4984-1-ND
- H1, H2, H3, H4, H5, H6, H7, H8, J0: Digikey Part No. None -> (none); Source (none) -> None; Source Part No. (none) -> None
- J1, J2: Digikey Part No. 455-1804-1-ND -> (none); Source (none) -> Digikey; Source Part No. (none) -> 455-1804-1-ND
- J8: Digikey Part No. None -> (none); Source Part No. (none) -> None
- P1: Digikey Part No. 2073-USB4110-GF-A-1-ND -> (none); Source (none) -> Digikey; Source Part No. (none) -> 2073-USB4110-GF-A-1-ND
Connections:
- wire segments 75 -> 83
Other:
- moved on the sheet: J1, J2

Commit message: Before updating to two switches
Parts:
- gave numbers to parts that had none: 4
Changed lines of the file:
@@
 	5150 4150 5150 4250
 $Comp
-L Frequently_Used:TestPoint TP?
+L Frequently_Used:TestPoint TP3
 U 1 1 5ED8A970
 P 7050 3650
-F 0 "TP?" H 7050 3950 50  0000 C CNN
+F 0 "TP3" H 7050 3950 50  0000 C CNN
 F 1 "TestPoint" H 6950 3400 50  0001 L CNN
 F 2 "Frequently_Used:Pad_2.5-2.5" H 7250 3650 50  0001 C CNN
@@
 $EndComp
 $Comp
-L Frequently_Used:TestPoint TP?
+L Frequently_Used:TestPoint TP4
 U 1 1 5ED8C4D5
 P 7300 3650
-F 0 "TP?" H 7300 3950 50  0000 C CNN
+F 0 "TP4" H 7300 3950 50  0000 C CNN
 F 1 "TestPoint" H 7200 3400 50  0001 L CNN
 F 2 "Frequently_Used:Pad_2.5-2.5" H 7500 3650 50  0001 C CNN
@@
 	7300 3750 7000 3750
 $Comp
-L Frequently_Used:TestPoint TP?
+L Frequently_Used:TestPoint TP5
 U 1 1 5ED9FCBB
 P 9450 3650
-F 0 "TP?" H 9450 3950 50  0000 C CNN
+F 0 "TP5" H 9450 3950 50  0000 C CNN
 F 1 "TestPoint" H 9350 3400 50  0001 L CNN
 F 2 "Frequently_Used:Pad_2.5-2.5" H 9650 3650 50  0001 C CNN
@@
 $EndComp
 $Comp
-L Frequently_Used:TestPoint TP?
+L Frequently_Used:TestPoint TP6
 U 1 1 5ED9FCC2
 P 9700 3650
-F 0 "TP?" H 9700 3950 50  0000 C CNN
+F 0 "TP6" H 9700 3950 50  0000 C CNN
 F 1 "TestPoint" H 9600 3400 50  0001 L CNN
 F 2 "Frequently_Used:Pad_2.5-2.5" H 9900 3650 50  0001 C CNN

Commit message: Updates
Parts:
- J0: footprint Naquadah_Generator:PinHeader_2x03_P2.54mm_Vertical -> Arduino:Connector_ISP; symbol Naquadah_Generator:Conn_ISP -> Arduino:Conn_ISP
Changed lines of the file:
@@
 $Descr A4 11693 8268
 encoding utf-8
-Sheet 11 11
+Sheet 10 11
 Title ""
 Date ""
@@
 Sensing Board 2
 $Comp
-L Naquadah_Generator:Conn_ISP J?
+L Arduino:Conn_ISP J?
 U 1 1 5EDC6C09
 P 8050 1950
@@
 F 0 "J0" H 8050 2275 50  0000 C CNN
 F 1 "Conn_ISP_Prog" H 8050 2184 50  0000 C CNN
-F 2 "Naquadah_Generator:PinHeader_2x03_P2.54mm_Vertical" H 8100 1950 50  0001 C CNN
+F 2 "Arduino:Connector_ISP" H 8100 1950 50  0001 C CNN
 F 3 "None" H 8100 1950 50  0001 C CNN
 F 4 "None" H 8050 1950 50  0001 C CNN "Source Part No."

Commit message: Updates
Parts:
- J1, J2: footprint Naquadah_Generator:State_Sensing_Mother_Board_JST_Conn -> Naquadah_Generator:Mother_Board_Hor_4_Pin_JST_Conn
Changed lines of the file:
@@
 F 0 "J1" H 6850 3600 50  0000 C CNN
 F 1 "State_Sensing_Conn" H 6850 4200 50  0000 C CNN
-F 2 "Naquadah_Generator:State_Sensing_Mother_Board_JST_Conn" H 6850 3250 50  0001 C CNN
+F 2 "Naquadah_Generator:Mother_Board_Hor_4_Pin_JST_Conn" H 6850 3250 50  0001 C CNN
 F 3 "http://www.jst-mfg.com/product/pdf/eng/eSH.pdf" H 6850 3950 50  0001 C CNN
 F 4 "455-1804-1-ND" H 6850 3550 50  0001 C CNN "Source Part No."
@@
 F 0 "J2" H 9250 3600 50  0000 C CNN
 F 1 "State_Sensing_Conn" H 9250 4200 50  0000 C CNN
-F 2 "Naquadah_Generator:State_Sensing_Mother_Board_JST_Conn" H 9250 3250 50  0001 C CNN
+F 2 "Naquadah_Generator:Mother_Board_Hor_4_Pin_JST_Conn" H 9250 3250 50  0001 C CNN
 F 3 "http://www.jst-mfg.com/product/pdf/eng/eSH.pdf" H 9250 3950 50  0001 C CNN
 F 4 "455-1804-1-ND" H 9250 3550 50  0001 C CNN "Source Part No."

Commit message: Move libraries and added configuration path.
Moved Li-Ion library to common KiCad library.  Added variables to configuration paths to reference my KiCad libraries.  Moved all 3D components to my common library.
Parts:
- C8: footprint Frequently_Used:0805_2012Metric_HandSolder -> FrequentlyUsed:0805_2012Metric_HandSolder; symbol Frequently_Used:C -> Frequently_Used_LE:C
- J0: symbol Arduino:Conn_ISP -> Arduino_LE:Conn_ISP
- R14, R19, R24, R29, R30: footprint Frequently_Used:0805_2012Metric_HandSolder -> FrequentlyUsed:0805_2012Metric_HandSolder; symbol Frequently_Used:R -> Frequently_Used_LE:R
- TP3, TP4, TP5, TP6: footprint Frequently_Used:Pad_2.5-2.5 -> FrequentlyUsed:Pad_2.5-2.5; symbol Frequently_Used:TestPoint -> Frequently_Used_LE:TestPoint
Changed lines of the file:
@@
 	7400 3750 7300 3750
 $Comp
-L Frequently_Used:GND #PWR?
+L Frequently_Used_LE:GND #PWR?
 U 1 1 5EDC6BCE
 P 7950 4150
@@
 	7950 3950 7950 3850
 $Comp
-L Frequently_Used:+5V #PWR?
+L Frequently_Used_LE:+5V #PWR?
 U 1 1 5EDC6BD8
 P 7950 3850
@@
 	9800 3750 9700 3750
 $Comp
-L Frequently_Used:GND #PWR?
+L Frequently_Used_LE:GND #PWR?
 U 1 1 5EDC6BEB
 P 10350 4150
@@
 	10350 3950 10350 3850
 $Comp
-L Frequently_Used:+5V #PWR?
+L Frequently_Used_LE:+5V #PWR?
 U 1 1 5EDC6BF5
 P 10350 3850
@@
 Sensing Board 2
 $Comp
-L Arduino:Conn_ISP J?
+L Arduino_LE:Conn_ISP J?
 U 1 1 5EDC6C09
 P 8050 1950
@@
 	7600 1950 7700 1950
 $Comp
-L Frequently_Used:GND #PWR?
+L Frequently_Used_LE:GND #PWR?
 U 1 1 5EDC6C17
 P 8800 2150
@@
 	8800 1850 8800 1750
 $Comp
-L Frequently_Used:+5V #PWR?
+L Frequently_Used_LE:+5V #PWR?
 U 1 1 5EDC6C21
 P 8800 1750
@@
 	2350 1200 2350 1250
 $Comp
-L Frequently_Used:VBUS #PWR0112
+L Frequently_Used_LE:VBUS #PWR0112
 U 1 1 5EDE054B
 P 2450 1100
@@
 	2350 2900 2350 2950
 $Comp
-L Frequently_Used:GND #PWR?
+L Frequently_Used_LE:GND #PWR?
 U 1 1 5EDE1EB1
 P 1600 4250
@@
 NoConn ~ 2200 2250
 $Comp
-L Frequently_Used:R R19
+L Frequently_Used_LE:R R19
 U 1 1 5EE65B3E
 P 3250 4000
 F 0 "R19" H 3180 3954 50  0000 R CNN
 F 1 "5.1k" H 3180 4045 50  0000 R CNN
-F 2 "Frequently_Used:0805_2012Metric_HandSolder" V 3180 4000 50  0001 C CNN
+F 2 "FrequentlyUsed:0805_2012Metric_HandSolder" V 3180 4000 50  0001 C CNN
 F 3 "" H 3250 4000 50  0001 C CNN
 	1    3250 4000
@@
 $EndComp
 $Comp
-L Frequently_Used:R R24
+L Frequently_Used_LE:R R24
 U 1 1 5EE68FFD
 P 3600 4000
 F 0 "R24" H 3530 3954 50  0000 R CNN
 F 1 "5.1k" H 3530 4045 50  0000 R CNN
-F 2 "Frequently_Used:0805_2012Metric_HandSolder" V 3530 4000 50  0001 C CNN
+F 2 "FrequentlyUsed:0805_2012Metric_HandSolder" V 3530 4000 50  0001 C CNN
 F 3 "" H 3600 4000 50  0001 C CNN
 	1    3600 4000
@@
 	3600 4150 3600 4250
 $Comp
-L Frequently_Used:GND #PWR?
+L Frequently_Used_LE:GND #PWR?
 U 1 1 5EE6DEDB
 P 3250 4250
@@
 $EndComp
 $Comp
-L Frequently_Used:GND #PWR?
+L Frequently_Used_LE:GND #PWR?
 U 1 1 5EE6E61C
 P 3600 4250
@@
 	5550 2550 5700 2550
 $Comp
-L Frequently_Used:R R30
+L Frequently_Used_LE:R R30
 U 1 1 5EE7B03D
 P 5400 2550
 F 0 "R30" V 5350 2650 50  0000 L CNN
 F 1 "5.1k" V 5450 2650 50  0000 L CNN
-F 2 "Frequently_Used:0805_2012Metric_HandSolder" V 5330 2550 50  0001 C CNN
+F 2 "FrequentlyUsed:0805_2012Metric_HandSolder" V 5330 2550 50  0001 C CNN
 F 3 "" H 5400 2550 50  0001 C CNN
 	1    5400 2550
@@
 	5250 2550 5200 2550
 $Comp
-L Frequently_Used:R R29
+L Frequently_Used_LE:R R29
 U 1 1 5EE722B8
 P 5400 2300
 F 0 "R29" V 5350 2400 50  0000 L CNN
 F 1 "5.1k" V 5450 2400 50  0000 L CNN
-F 2 "Frequently_Used:0805_2012Metric_HandSolder" V 5330 2300 50  0001 C CNN
+F 2 "FrequentlyUsed:0805_2012Metric_HandSolder" V 5330 2300 50  0001 C CNN
 F 3 "" H 5400 2300 50  0001 C CNN
 	1    5400 2300
@@
 	4700 1050 4700 950
 $Comp
-L Frequently_Used:VBUS #PWR0116
+L Frequently_Used_LE:VBUS #PWR0116
 U 1 1 5ED508DF
 P 4700 950
@@
 $EndComp
 $Comp
-L Frequently_Used:GND #PWR?
+L Frequently_Used_LE:GND #PWR?
 U 1 1 5ED510AF
 P 4700 1950
@@
 $EndComp
 $Comp
-L Frequently_Used:C C8
+L Frequently_Used_LE:C C8
 U 1 1 5ED51CE6
 P 1600 4000
 F 0 "C8" H 1650 4100 50  0000 L CNN
 F 1 "4.7uF" H 1650 3900 50  0000 L CNN
-F 2 "Frequently_Used:0805_2012Metric_HandSolder" H 1638 3850 50  0001 C CNN
+F 2 "FrequentlyUsed:0805_2012Metric_HandSolder" H 1638 3850 50  0001 C CNN
 F 3 "" H 1600 4000 50  0001 C CNN
 	1    1600 4000
@@
 $EndComp
 $Comp
-L Frequently_Used:R R14
+L Frequently_Used_LE:R R14
 U 1 1 5ED52CB7
 P 2000 4000
 F 0 "R14" H 2070 4046 50  0000 L CNN
 F 1 "1M" H 2070 3955 50  0000 L CNN
-F 2 "Frequently_Used:0805_2012Metric_HandSolder" V 1930 4000 50  0001 C CNN
+F 2 "FrequentlyUsed:0805_2012Metric_HandSolder" V 1930 4000 50  0001 C CNN
 F 3 "" H 2000 4000 50  0001 C CNN
 	1    2000 4000
@@
 	2000 4150 2000 4250
 $Comp
-L Frequently_Used:GND #PWR?
+L Frequently_Used_LE:GND #PWR?
 U 1 1 5ED57050
 P 2000 4250
@@
 	2450 2900 2450 3000
 $Comp
-L Frequently_Used:GND #PWR?
+L Frequently_Used_LE:GND #PWR?
 U 1 1 5ED5A3E8
 P 2450 3000
@@
 $EndComp
 $Comp
-L Frequently_Used:VBUS #PWR0120
+L Frequently_Used_LE:VBUS #PWR0120
 U 1 1 5EE6129E
 P 5150 3750
@@
 $EndComp
 $Comp
-L Frequently_Used:GND #PWR?
+L Frequently_Used_LE:GND #PWR?
 U 1 1 5EE62115
 P 5150 4250
@@
 	5150 4150 5150 4250
 $Comp
-L Frequently_Used:TestPoint TP3
+L Frequently_Used_LE:TestPoint TP3
 U 1 1 5ED8A970
 P 7050 3650
 F 0 "TP3" H 7050 3950 50  0000 C CNN
 F 1 "TestPoint" H 6950 3400 50  0001 L CNN
-F 2 "Frequently_Used:Pad_2.5-2.5" H 7250 3650 50  0001 C CNN
+F 2 "FrequentlyUsed:Pad_2.5-2.5" H 7250 3650 50  0001 C CNN
 F 3 "None" H 7250 3650 50  0001 C CNN
 F 4 "HE1" H 7050 3850 50  0000 C CNN "Name"
@@
 $EndComp
 $Comp
-L Frequently_Used:TestPoint TP4
+L Frequently_Used_LE:TestPoint TP4
 U 1 1 5ED8C4D5
 P 7300 3650
 F 0 "TP4" H 7300 3950 50  0000 C CNN
 F 1 "TestPoint" H 7200 3400 50  0001 L CNN
-F 2 "Frequently_Used:Pad_2.5-2.5" H 7500 3650 50  0001 C CNN
+F 2 "FrequentlyUsed:Pad_2.5-2.5" H 7500 3650 50  0001 C CNN
 F 3 "None" H 7500 3650 50  0001 C CNN
 F 4 "HE2" H 7300 3850 50  0000 C CNN "Name"
@@
 	7300 3750 7000 3750
 $Comp
-L Frequently_Used:TestPoint TP5
+L Frequently_Used_LE:TestPoint TP5
 U 1 1 5ED9FCBB
 P 9450 3650
 F 0 "TP5" H 9450 3950 50  0000 C CNN
 F 1 "TestPoint" H 9350 3400 50  0001 L CNN
-F 2 "Frequently_Used:Pad_2.5-2.5" H 9650 3650 50  0001 C CNN
+F 2 "FrequentlyUsed:Pad_2.5-2.5" H 9650 3650 50  0001 C CNN
 F 3 "None" H 9650 3650 50  0001 C CNN
 F 4 "HE1" H 9450 3850 50  0000 C CNN "Name"
@@
 $EndComp
 $Comp
-L Frequently_Used:TestPoint TP6
+L Frequently_Used_LE:TestPoint TP6
 U 1 1 5ED9FCC2
 P 9700 3650
 F 0 "TP6" H 9700 3950 50  0000 C CNN
 F 1 "TestPoint" H 9600 3400 50  0001 L CNN
-F 2 "Frequently_Used:Pad_2.5-2.5" H 9900 3650 50  0001 C CNN
+F 2 "FrequentlyUsed:Pad_2.5-2.5" H 9900 3650 50  0001 C CNN
 F 3 "None" H 9900 3650 50  0001 C CNN
 F 4 "HE2" H 9700 3850 50  0000 C CNN "Name"

Commit message: PCB Updates
Parts:
- J1, J2: footprint Naquadah_Generator:Mother_Board_Hor_4_Pin_JST_Conn -> Naquadah_Generator:Daughter_Board_Hor_4_Pin_JST_Conn
- P1: footprint Connectors LE:GCT_USB4110-GF-A -> Connectors_LE:2047110001; symbol Connectors_LE:USB_C_Plug_USB2.0 -> Connectors_LE:USB_C_Plug_2_USB2.0; Manufacturer Name GCT -> Molex; Manufacturer Part No. USB4110-GF-A -> 2047110001; Source Part No. 2073-USB4110-GF-A-1-ND -> 900-2047110001CT-ND
Connections:
- wire segments 83 -> 103
- no-connect marks 5 -> 10
Changed lines of the file:
@@
 F 0 "J1" H 6850 3600 50  0000 C CNN
 F 1 "State_Sensing_Conn" H 6850 4200 50  0000 C CNN
-F 2 "Naquadah_Generator:Mother_Board_Hor_4_Pin_JST_Conn" H 6850 3250 50  0001 C CNN
+F 2 "Naquadah_Generator:Daughter_Board_Hor_4_Pin_JST_Conn" H 6850 3250 50  0001 C CNN
 F 3 "http://www.jst-mfg.com/product/pdf/eng/eSH.pdf" H 6850 3950 50  0001 C CNN
 F 4 "455-1804-1-ND" H 6850 3550 50  0001 C CNN "Source Part No."
@@
 F 0 "J2" H 9250 3600 50  0000 C CNN
 F 1 "State_Sensing_Conn" H 9250 4200 50  0000 C CNN
-F 2 "Naquadah_Generator:Mother_Board_Hor_4_Pin_JST_Conn" H 9250 3250 50  0001 C CNN
+F 2 "Naquadah_Generator:Daughter_Board_Hor_4_Pin_JST_Conn" H 9250 3250 50  0001 C CNN
 F 3 "http://www.jst-mfg.com/product/pdf/eng/eSH.pdf" H 9250 3950 50  0001 C CNN
 F 4 "455-1804-1-ND" H 9250 3550 50  0001 C CNN "Source Part No."
@@
 HALLEFF4
 $Comp
-L Connectors_LE:USB_C_Plug_USB2.0 P1
+L Connectors_LE:USB_C_Plug_2_USB2.0 P1
 U 1 1 5EDDB911
-P 1600 2050
-F 0 "P1" H 1350 3200 50  0000 L CNN
-F 1 "USB_C_Plug_USB2.0" H 1350 3100 50  0000 L CNN
-F 2 "Connectors LE:GCT_USB4110-GF-A" H 1700 1550 50  0001 C CNN
-F 3 "https://gct.co/files/drawings/usb4110.pdf" H 1700 1550 50  0001 C CNN
-F 4 "USB-C 2.0 Female SMD Connector" H 1600 2050 50  0001 C CNN "Description"
-F 5 "2073-USB4110-GF-A-1-ND" H 1600 2050 50  0001 C CNN "Source Part No."
-F 6 "GCT" H 1600 2050 50  0001 C CNN "Manufacturer Name"
-F 7 "USB4110-GF-A" H 1600 2050 50  0001 C CNN "Manufacturer Part No."
-F 8 "Digikey" H 1600 2050 50  0001 C CNN "Source"
-	1    1600 2050
-	1    0    0    -1
-$EndComp
-Wire Wire Line
-	2350 1150 2200 1150
-Wire Wire Line
-	2350 1250 2200 1250
-Wire Wire Line
-	2350 1150 2350 1200
-Wire Wire Line
-	2350 1200 2450 1200
-Wire Wire Line
-	2450 1200 2450 1100
-Connection ~ 2350 1200
-Wire Wire Line
-	2350 1200 2350 1250
+P 1700 2050
+AR Path="/5EDDB911" Ref="P1"  Part="1"
+AR Path="/5EDBBDC8/5EDDB911" Ref="P1"  Part="1"
+F 0 "P1" H 1450 3200 50  0000 L CNN
+F 1 "USB_C_Plug_USB2.0" H 1450 3100 50  0000 L CNN
+F 2 "Connectors_LE:2047110001" H 1800 1550 50  0001 C CNN
+F 3 "https://www.molex.com/pdm_docs/sd/2047110001_sd.pdf" H 1800 1550 50  0001 C CNN
+F 4 "USB-C 2.0 Female SMD Connector" H 1700 2050 50  0001 C CNN "Description"
+F 5 "Digikey" H 1700 2050 50  0001 C CNN "Source"
+F 6 "900-2047110001CT-ND" H 1700 2050 50  0001 C CNN "Source Part No."
+F 7 "Molex" H 1700 2050 50  0001 C CNN "Manufacturer Name"
+F 8 "2047110001" H 1700 2050 50  0001 C CNN "Manufacturer Part No."
+	1    1700 2050
+	1    0    0    -1
+$EndComp
+Wire Wire Line
+	1050 1250 1150 1250
+Wire Wire Line
+	1050 1350 1150 1350
+Wire Wire Line
+	1050 1250 1050 1300
+Wire Wire Line
+	1050 1300 900  1300
+Wire Wire Line
+	900  1300 900  1200
+Connection ~ 1050 1300
+Wire Wire Line
+	1050 1300 1050 1350
 $Comp
 L Frequently_Used_LE:VBUS #PWR0112
 U 1 1 5EDE054B
-P 2450 1100
-F 0 "#PWR0112" H 2450 950 50  0001 C CNN
-F 1 "VBUS" H 2465 1273 50  0000 C CNN
-F 2 "" H 2450 1100 50  0001 C CNN
-F 3 "" H 2450 1100 50  0001 C CNN
-	1    2450 1100
-	1    0    0    -1
-$EndComp
-Wire Wire Line
-	2200 2850 2350 2850
-Wire Wire Line
-	2350 2850 2350 2900
-Wire Wire Line
-	2350 2950 2200 2950
-Wire Wire Line
-	2350 2900 2450 2900
+P 900 1200
+F 0 "#PWR0112" H 900 1050 50  0001 C CNN
+F 1 "VBUS" H 915 1373 50  0000 C CNN
+F 2 "" H 900 1200 50  0001 C CNN
+F 3 "" H 900 1200 50  0001 C CNN
+	1    900  1200
+	-1   0    0    -1
+$EndComp
+Wire Wire Line
+	1150 2800 1050 2800
+Wire Wire Line
+	1050 2800 1050 2850
+Wire Wire Line
+	1050 2900 1150 2900
 Wire Wire Line
 	1600 4150 1600 4250
-Connection ~ 2350 2900
-Wire Wire Line
-	2350 2900 2350 2950
+Connection ~ 1050 2850
+Wire Wire Line
+	1050 2850 1050 2900
 $Comp
 L Frequently_Used_LE:GND #PWR?
@@
 $EndComp
 Wire Wire Line
-	2200 1400 2350 1400
-Wire Wire Line
-	2350 1500 2200 1500
-Wire Wire Line
-	2200 1650 2350 1650
-Wire Wire Line
-	2350 1750 2200 1750
-NoConn ~ 2200 2150
-NoConn ~ 2200 2250
+	2200 1900 2350 1900
+Wire Wire Line
+	2350 2000 2200 2000
+Wire Wire Line
+	2200 2150 2350 2150
+Wire Wire Line
+	2350 2250 2200 2250
+NoConn ~ 2200 2900
+NoConn ~ 2200 3000
 $Comp
 L Frequently_Used_LE:R R19
@@
 $EndComp
 Wire Wire Line
-	2450 2900 2450 3000
-$Comp
-L Frequently_Used_LE:GND #PWR?
-U 1 1 5ED5A3E8
-P 2450 3000
-AR Path="/5ED5A3E8" Ref="#PWR?"  Part="1"
-AR Path="/5EDBBDC8/5ED5A3E8" Ref="#PWR0119"  Part="1"
-F 0 "#PWR0119" H 2450 2750 50  0001 C CNN
-F 1 "GND" H 2450 2850 50  0000 C CNN
-F 2 "" H 2450 3000 50  0001 C CNN
-F 3 "" H 2450 3000 50  0001 C CNN
-	1    2450 3000
-	1    0    0    -1
-$EndComp
-Wire Wire Line
-	2200 2400 2600 2400
-Wire Wire Line
 	1350 3750 1600 3750
 Wire Wire Line
@@
 	1600 3750 2000 3750
 Wire Wire Line
-	2350 1400 2350 1450
-Wire Wire Line
-	2350 1650 2350 1700
-Wire Wire Line
-	2350 1450 2600 1450
-Connection ~ 2350 1450
-Wire Wire Line
-	2350 1450 2350 1500
-Wire Wire Line
-	2350 1700 2600 1700
-Connection ~ 2350 1700
-Wire Wire Line
-	2350 1700 2350 1750
-Text Label 2400 1450 0    50   ~ 0
+	2350 1900 2350 1950
+Wire Wire Line
+	2350 2150 2350 2200
+Wire Wire Line
+	2350 1950 2600 1950
+Connection ~ 2350 1950
+Wire Wire Line
+	2350 1950 2350 2000
+Wire Wire Line
+	2350 2200 2600 2200
+Connection ~ 2350 2200
+Wire Wire Line
+	2350 2200 2350 2250
+Text Label 2400 1950 0    50   ~ 0
 D+
-Text Label 2400 1700 0    50   ~ 0
+Text Label 2400 2200 0    50   ~ 0
 D-
 Text Label 3750 2300 0    50   ~ 0
@@
 D-
 Wire Wire Line
-	2200 1900 2600 1900
-Wire Wire Line
-	2200 2000 2600 2000
-Text Label 2400 1900 0    50   ~ 0
+	2200 1650 2600 1650
+Wire Wire Line
+	2200 1750 2600 1750
+Text Label 2400 1650 0    50   ~ 0
 CC1
-Text Label 2400 2000 0    50   ~ 0
+Text Label 2400 1750 0    50   ~ 0
 CC2
 Text Label 3000 3650 0    50   ~ 0
@@
 Text Label 3000 3750 0    50   ~ 0
 CC2
-Text Label 2400 2400 0    50   ~ 0
-SHLD
 NoConn ~ 2200 2500
 NoConn ~ 2200 2600
@@
 Wire Wire Line
 	9700 3750 9400 3750
+Wire Wire Line
+	1050 1250 1050 1150
+Wire Wire Line
+	1050 1150 1150 1150
+Connection ~ 1050 1250
+Wire Wire Line
+	1050 1350 1050 1450
+Wire Wire Line
+	1050 1450 1150 1450
+Connection ~ 1050 1350
+Wire Wire Line
+	1050 2800 1050 2700
+Wire Wire Line
+	1050 2700 1150 2700
+Connection ~ 1050 2800
+Wire Wire Line
+	1050 2900 1050 3000
+Wire Wire Line
+	1050 3000 1150 3000
+Connection ~ 1050 2900
+$Comp
+L Frequently_Used_LE:GND #PWR?
+U 1 1 5ED5A3E8
+P 900 2950
+AR Path="/5ED5A3E8" Ref="#PWR?"  Part="1"
+AR Path="/5EDBBDC8/5ED5A3E8" Ref="#PWR0119"  Part="1"
+F 0 "#PWR0119" H 900 2700 50  0001 C CNN
+F 1 "GND" H 900 2800 50  0000 C CNN
+F 2 "" H 900 2950 50  0001 C CNN
+F 3 "" H 900 2950 50  0001 C CNN
+	1    900  2950
+	-1   0    0    -1
+$EndComp
+Wire Wire Line
+	1050 2850 900  2850
+Wire Wire Line
+	900  2850 900  2950
+Text Label 650  2050 0    50   ~ 0
+SHLD
+Wire Wire Line
+	650  2050 1050 2050
+Wire Wire Line
+	1150 1800 1050 1800
+Wire Wire Line
+	1050 2050 1050 2100
+Wire Wire Line
+	1050 2300 1150 2300
+Connection ~ 1050 2050
+Wire Wire Line
+	1150 2200 1050 2200
+Connection ~ 1050 2200
+Wire Wire Line
+	1050 2200 1050 2300
+Wire Wire Line
+	1150 2100 1050 2100
+Connection ~ 1050 2100
+Wire Wire Line
+	1050 2100 1050 2200
+Wire Wire Line
+	1150 2000 1050 2000
+Wire Wire Line
+	1050 1800 1050 1900
+Connection ~ 1050 2000
+Wire Wire Line
+	1050 2000 1050 2050
+Wire Wire Line
+	1150 1900 1050 1900
+Connection ~ 1050 1900
+Wire Wire Line
+	1050 1900 1050 2000
+NoConn ~ 2200 2400
+NoConn ~ 2200 1500
+NoConn ~ 2200 1400
+NoConn ~ 2200 1250
+NoConn ~ 2200 1150
 $EndSCHEMATC
