File: Naquadah Generator Main/Connectors.sch (KiCad schematic (older format))
At the start: 24 parts, among them J0 Conn_ISP_Prog, J1 State_Sensing_Conn, J2 State_Sensing_Conn, J8 USB Solder Pads, P1 USB_C_Plug_USB2.0

Commit message: Separated digital and analog ground.
Connections:
- net labels added: GNDD
- net labels removed: GND
Changed lines of the file:
@@
 	7400 3750 7300 3750
 $Comp
-L Frequently_Used_LE:GND #PWR?
+L Frequently_Used_LE:GNDD #PWR?
 U 1 1 5EDC6BCE
 P 7950 4150
@@
 AR Path="/5EDBBDC8/5EDC6BCE" Ref="#PWR0106"  Part="1"
 F 0 "#PWR0106" H 7950 3900 50  0001 C CNN
-F 1 "GND" H 7950 4000 50  0000 C CNN
+F 1 "GNDD" H 7950 4000 50  0000 C CNN
 F 2 "" H 7950 4150 50  0001 C CNN
 F 3 "" H 7950 4150 50  0001 C CNN
@@
 	9800 3750 9700 3750
 $Comp
-L Frequently_Used_LE:GND #PWR?
+L Frequently_Used_LE:GNDD #PWR?
 U 1 1 5EDC6BEB
 P 10350 4150
@@
 AR Path="/5EDBBDC8/5EDC6BEB" Ref="#PWR0108"  Part="1"
 F 0 "#PWR0108" H 10350 3900 50  0001 C CNN
-F 1 "GND" H 10350 4000 50  0000 C CNN
+F 1 "GNDD" H 10350 4000 50  0000 C CNN
 F 2 "" H 10350 4150 50  0001 C CNN
 F 3 "" H 10350 4150 50  0001 C CNN
@@
 	7600 1950 7700 1950
 $Comp
-L Frequently_Used_LE:GND #PWR?
+L Frequently_Used_LE:GNDD #PWR?
 U 1 1 5EDC6C17
 P 8800 2150
@@
 AR Path="/5EDBBDC8/5EDC6C17" Ref="#PWR0110"  Part="1"
 F 0 "#PWR0110" H 8800 1900 50  0001 C CNN
-F 1 "GND" H 8800 2000 50  0000 C CNN
+F 1 "GNDD" H 8800 2000 50  0000 C CNN
 F 2 "" H 8800 2150 50  0001 C CNN
 F 3 "" H 8800 2150 50  0001 C CNN
@@
 	1050 2850 1050 2900
 $Comp
-L Frequently_Used_LE:GND #PWR?
+L Frequently_Used_LE:GNDD #PWR?
 U 1 1 5EDE1EB1
 P 1600 4250
@@
 AR Path="/5EDBBDC8/5EDE1EB1" Ref="#PWR0113"  Part="1"
 F 0 "#PWR0113" H 1600 4000 50  0001 C CNN
-F 1 "GND" H 1600 4100 50  0000 C CNN
+F 1 "GNDD" H 1600 4100 50  0000 C CNN
 F 2 "" H 1600 4250 50  0001 C CNN
 F 3 "" H 1600 4250 50  0001 C CNN
@@
 	3600 4150 3600 4250
 $Comp
-L Frequently_Used_LE:GND #PWR?
+L Frequently_Used_LE:GNDD #PWR?
 U 1 1 5EE6DEDB
 P 3250 4250
@@
 AR Path="/5EDBBDC8/5EE6DEDB" Ref="#PWR0114"  Part="1"
 F 0 "#PWR0114" H 3250 4000 50  0001 C CNN
-F 1 "GND" H 3250 4100 50  0000 C CNN
+F 1 "GNDD" H 3250 4100 50  0000 C CNN
 F 2 "" H 3250 4250 50  0001 C CNN
 F 3 "" H 3250 4250 50  0001 C CNN
@@
 $EndComp
 $Comp
-L Frequently_Used_LE:GND #PWR?
+L Frequently_Used_LE:GNDD #PWR?
 U 1 1 5EE6E61C
 P 3600 4250
@@
 AR Path="/5EDBBDC8/5EE6E61C" Ref="#PWR0115"  Part="1"
 F 0 "#PWR0115" H 3600 4000 50  0001 C CNN
-F 1 "GND" H 3600 4100 50  0000 C CNN
+F 1 "GNDD" H 3600 4100 50  0000 C CNN
 F 2 "" H 3600 4250 50  0001 C CNN
 F 3 "" H 3600 4250 50  0001 C CNN
@@
 $EndComp
 $Comp
-L Frequently_Used_LE:GND #PWR?
+L Frequently_Used_LE:GNDD #PWR?
 U 1 1 5ED510AF
 P 4700 1950
@@
 AR Path="/5EDBBDC8/5ED510AF" Ref="#PWR0117"  Part="1"
 F 0 "#PWR0117" H 4700 1700 50  0001 C CNN
-F 1 "GND" H 4700 1800 50  0000 C CNN
+F 1 "GNDD" H 4700 1800 50  0000 C CNN
 F 2 "" H 4700 1950 50  0001 C CNN
 F 3 "" H 4700 1950 50  0001 C CNN
@@
 	2000 4150 2000 4250
 $Comp
-L Frequently_Used_LE:GND #PWR?
+L Frequently_Used_LE:GNDD #PWR?
 U 1 1 5ED57050
 P 2000 4250
@@
 AR Path="/5EDBBDC8/5ED57050" Ref="#PWR0118"  Part="1"
 F 0 "#PWR0118" H 2000 4000 50  0001 C CNN
-F 1 "GND" H 2000 4100 50  0000 C CNN
+F 1 "GNDD" H 2000 4100 50  0000 C CNN
 F 2 "" H 2000 4250 50  0001 C CNN
 F 3 "" H 2000 4250 50  0001 C CNN
@@
 $EndComp
 $Comp
-L Frequently_Used_LE:GND #PWR?
+L Frequently_Used_LE:GNDD #PWR?
 U 1 1 5EE62115
 P 5150 4250
@@
 AR Path="/5EDBBDC8/5EE62115" Ref="#PWR0121"  Part="1"
 F 0 "#PWR0121" H 5150 4000 50  0001 C CNN
-F 1 "GND" H 5150 4100 50  0000 C CNN
+F 1 "GNDD" H 5150 4100 50  0000 C CNN
 F 2 "" H 5150 4250 50  0001 C CNN
 F 3 "" H 5150 4250 50  0001 C CNN
@@
 Connection ~ 1050 2900
 $Comp
-L Frequently_Used_LE:GND #PWR?
+L Frequently_Used_LE:GNDD #PWR?
 U 1 1 5ED5A3E8
 P 900 2950
@@
 AR Path="/5EDBBDC8/5ED5A3E8" Ref="#PWR0119"  Part="1"
 F 0 "#PWR0119" H 900 2700 50  0001 C CNN
-F 1 "GND" H 900 2800 50  0000 C CNN
+F 1 "GNDD" H 900 2800 50  0000 C CNN
 F 2 "" H 900 2950 50  0001 C CNN
 F 3 "" H 900 2950 50  0001 C CNN

Commit message: Audio update
Parts:
- C8: footprint FrequentlyUsed:0805_2012Metric_HandSolder -> Frequently_Used_LE:0805_2012Metric_HandSolder
- R14: footprint FrequentlyUsed:0805_2012Metric_HandSolder -> Frequently_Used_LE:0805_2012Metric_HandSolder; Description (none) -> 1 MOhms ±1% 0.25W, 1/4W Chip Resistor 0805 (2012 Metric); Manufacturer Name (none) -> KOA Speer Electronics, Inc.; Manufacturer Part No. (none) -> RK73H2ATTD1004F; Source (none) -> Digikey; Source Part No. (none) -> 2019-RK73H2ATTD1004FCT-ND
- R19, R24, R29, R30: footprint FrequentlyUsed:0805_2012Metric_HandSolder -> Frequently_Used_LE:0805_2012Metric_HandSolder; Description (none) -> 5.1 kOhms ±1% 0.25W, 1/4W Chip Resistor 0805 (2012 Metric); Manufacturer Name (none) -> KOA Speer Electronics, Inc.; Manufacturer Part No. (none) -> RK73H2ATTD5101F; Source (none) -> Digikey; Source Part No. (none) -> 2019-RK73H2ATTD5101FCT-ND
- TP3, TP4, TP5, TP6: footprint FrequentlyUsed:Pad_2.5-2.5 -> Frequently_Used_LE:Pad_2.5-2.5
Connections:
- net labels added: DGND
- net labels removed: GNDD
Other:
- note added: "ATMega USB"
- moved on the sheet: C8, D1, H1, H2, H3, H4, H5, H6, H7, H8, J0, J1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

Commit message: Power updates
Parts:
- TP3, TP4, TP5, TP6: symbol Frequently_Used_LE:TestPoint -> Frequently_Used_LE:TestPoint_1
Changed lines of the file:
@@
 $Descr A4 11693 8268
 encoding utf-8
-Sheet 10 12
+Sheet 10 15
 Title ""
 Date ""
@@
 	5500 6750 5500 6850
 $Comp
-L Frequently_Used_LE:TestPoint TP3
+L Frequently_Used_LE:TestPoint_1 TP3
 U 1 1 5ED8A970
 P 5550 1250
@@
 $EndComp
 $Comp
-L Frequently_Used_LE:TestPoint TP4
+L Frequently_Used_LE:TestPoint_1 TP4
 U 1 1 5ED8C4D5
 P 5800 1250
@@
 	5800 1350 5500 1350
 $Comp
-L Frequently_Used_LE:TestPoint TP5
+L Frequently_Used_LE:TestPoint_1 TP5
 U 1 1 5ED9FCBB
 P 8150 1250
@@
 $EndComp
 $Comp
-L Frequently_Used_LE:TestPoint TP6
+L Frequently_Used_LE:TestPoint_1 TP6
 U 1 1 5ED9FCC2
 P 8400 1250

Commit message: Audio updates, switching to separate USB schematic
Audio updates, switching to separate USB schematic
Connections:
- wire segments 103 -> 105
Changed lines of the file:
@@
 $Descr A4 11693 8268
 encoding utf-8
-Sheet 10 15
+Sheet 10 16
 Title ""
 Date ""
@@
 CC2
 NoConn ~ 2700 5150
-NoConn ~ 2700 5250
-NoConn ~ 2700 5350
+NoConn ~ 2700 5300
+NoConn ~ 2700 5400
 Text Label 1700 6350 0    50   ~ 0
 SHLD
@@
 U 1 1 5EE457C4
 P 4900 6650
-F 0 "J8" H 4818 6225 50  0000 C CNN
-F 1 "USB Solder Pads" H 4818 6316 50  0000 C CNN
+F 0 "J8" H 4900 6350 50  0000 C CNN
+F 1 "USB Solder Pads" H 4750 6850 50  0000 C CNN
 F 2 "Naquadah_Generator:WireSoldPads_1x4_WOL" H 4900 6650 50  0001 C CNN
 F 3 "None" H 4900 6650 50  0001 C CNN
@@
 L Frequently_Used_LE:VBUS #PWR0120
 U 1 1 5EE6129E
-P 5500 6350
-F 0 "#PWR0120" H 5500 6200 50  0001 C CNN
-F 1 "VBUS" H 5515 6523 50  0000 C CNN
-F 2 "" H 5500 6350 50  0001 C CNN
-F 3 "" H 5500 6350 50  0001 C CNN
-	1    5500 6350
+P 5700 6350
+F 0 "#PWR0120" H 5700 6200 50  0001 C CNN
+F 1 "VBUS" H 5715 6523 50  0000 C CNN
+F 2 "" H 5700 6350 50  0001 C CNN
+F 3 "" H 5700 6350 50  0001 C CNN
+	1    5700 6350
 	1    0    0    -1
 $EndComp
@@
 D-
 Wire Wire Line
-	5100 6450 5500 6450
-Wire Wire Line
-	5500 6450 5500 6350
+	5700 6450 5700 6350
 Wire Wire Line
 	5100 6750 5500 6750
@@
 Text Notes 3000 7400 0    79   ~ 16
 ATMega USB
+Wire Wire Line
+	5300 6350 5300 6450
+$Comp
+L Frequently_Used_LE:PWR_FLAG #FLG?
+U 1 1 5FBCCA10
+P 5300 6350
+AR Path="/5FBCCA10" Ref="#FLG?"  Part="1"
+AR Path="/5EA6751D/5FBCCA10" Ref="#FLG?"  Part="1"
+AR Path="/5EDBBDC8/5FBCCA10" Ref="#FLG0105"  Part="1"
+F 0 "#FLG0105" H 5300 6425 50  0001 C CNN
+F 1 "PWR_FLAG" H 5300 6523 50  0000 C CNN
+F 2 "" H 5300 6350 50  0001 C CNN
+F 3 "~" H 5300 6350 50  0001 C CNN
+	1    5300 6350
+	1    0    0    -1
+$EndComp
+Wire Wire Line
+	5100 6450 5300 6450
+Connection ~ 5300 6450
+Wire Wire Line
+	5300 6450 5700 6450
 $EndSCHEMATC

Commit message: Added level shifter, moved user interface connector location
Added level shifter, moved user interface connector location
Parts:
- removed C8: 4.7uF, Frequently_Used_LE:0805_2012Metric_HandSolder, symbol Frequently_Used_LE:C
- removed D1: SDP, Package_TO_SOT_SMD:SOT-143, symbol Power_LE:PRTR5V0U2X
- removed J8: USB Solder Pads, Naquadah_Generator:WireSoldPads_1x4_WOL, symbol Connector_Generic:Conn_01x04
- removed P1: USB_C_Plug_USB2.0, Connectors_LE:2047110001, symbol Connectors_LE:USB_C_Plug_2_USB2.0
- removed R14: 1M, Frequently_Used_LE:0805_2012Metric_HandSolder, symbol Frequently_Used_LE:R
- removed R19, R24, R29, R30: 5.1k, Frequently_Used_LE:0805_2012Metric_HandSolder, symbol Frequently_Used_LE:R
- added D31: 5A 100V, Li_Ion_LE:DO-214AC, symbol Frequently_Used_LE:D
- added J10: Power Board Conn, Naquadah_Generator:Daughter_Board_Vert_5_Pin_JST_Conn, symbol Naquadah_Generator:Power_Daughter_5_Pin_Conn
- added JP4: Bridged, Jumper_LE:SolderJumper-2_P1.3mm_Bridged_RoundedPad1.0x1.5mm, symbol Jumper:SolderJumper_2_Bridged
- added TP10, TP2, TP7, TP8, TP9: TestPoint, Frequently_Used_LE:Pad_2.5-2.5, symbol Frequently_Used_LE:TestPoint_1
Connections:
- net labels added: BATT+, BATT-, MODE, READY, SWITCH
- net labels removed: CC1, CC2, SHLD
- wire segments 105 -> 55
- no-connect marks 10 -> 0
Other:
- note added: "ATMega ISP Breakout"
- note added: "User Interface Board Connector"
- note removed: "ISP Breakout"
- moved on the sheet: J0, J1, J2, TP3, TP4, TP5, TP6

Commit message: Switched to 0603_1608M size for passives
Parts:
- removed J10: Power Board Conn, Naquadah_Generator:Daughter_Board_Vert_5_Pin_JST_Conn, symbol Naquadah_Generator:Power_Daughter_5_Pin_Conn
- added J10: User_Interface_6_Pin_Conn, Naquadah_Generator:Daughter_Board_Vert_6_Pin_JST_Conn, symbol Naquadah_Generator:User_Interface_6_Pin_Conn
- added J3: Conn_01x02, Connector_LE:JST_SH_BM02B-SRSS-TB_1x02-1MP_P1.00mm_Vertical, symbol Connector_Generic:Conn_01x02
- added TP10: TestPoint, Frequently_Used_LE:Pad_2.5-2.5, symbol Frequently_Used_LE:TestPoint_1
- J1, J2: Description State sensing daughter board connector -> Connector Header Surface Mount, Right Angle 4 position 0.03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
- TP2, TP3, TP4, TP5, TP6, TP8, TP9: Description None -> Test point
- TP20: renamed from TP10; Description None -> Test point; Name MODE -> VOLUME
- TP7: Description None -> Test point; Name SW -> SWITCH
Connections:
- net +5V: now also J3.2 (Pin_2)
- net BATT+: now also J10.2 (BATT+)
- net BATT-: now also J10.1 (BATT-)
- net MODE: now also J10.4 (MODE), TP10.1; no longer TP20.1
- net READY: now also J10.5 (READY)
- net SWITCH: now also J10.6 (SWITCH)
- new net VOLUME: J10.3 (VOLUME), TP20.1
- new net WHITELT: J3.1 (Pin_1)
Other:
- note added: "White Lights"
- moved on the sheet: TP2, TP20, TP7, TP8, TP9

Commit message: Update JST connectors
Parts:
- added WA1: WireAssembly, Mechanical_LE:Wire_Assembly, symbol Mechanical_LE:WireAssembly
- J1, J2: footprint Naquadah_Generator:Daughter_Board_Hor_4_Pin_JST_Conn -> Connector_JST:JST_SH_SM04B-SRSS-TB_1x04-1MP_P1.00mm_Horizontal
- J10: footprint Naquadah_Generator:Daughter_Board_Vert_6_Pin_JST_Conn -> Connector_JST:JST_SH_BM06B-SRSS-TB_1x06-1MP_P1.00mm_Vertical
