File: Naquadah Generator Main/Shift Registers.sch (KiCad schematic (older format))
At the start: 4 parts, among them U201 74HC595, U202 74HC595

Commit message: Partial Update
Parts:
- D2: renamed from D?; symbol Device:LED -> Frequently_Used:LED
- R3: renamed from R?; footprint Resistor_THT:R_Axial_DIN0207_L6.3mm_D2.5mm_P10.16mm_Horizontal -> Frequently_Used:0805_2012Metric_HandSolder; symbol Device:R -> Frequently_Used:R
- renumbered U201 to U2, U202 to U3
Connections:
- net labels added: SRBLUELT1, SRBLUELT2, SRBLUELT3, SRBLUELT4, SRBLUELT5, SRGRNLT, SRRDLT, SRWHTLT
- net labels removed: BLUELT1, BLUELT2, BLUELT3, BLUELT4, BLUELT5, GRNLT, RDLT, WHTLT
Other:
- moved on the sheet: D2, R3, U2, U3

Commit message: Resize to correct for scale
Parts:
- added J3: Conn_01x02, Connector_Wire:SolderWirePad_1x02_P3.81mm_Drill1.2mm, symbol Connector_Generic:Conn_01x02
- added U4: ULN2803ADWRG4, Naquadah_Generator:SOIC127P1030X265-18N, symbol Naquadah_Generator:ULN2803ADWRG4
- U2, U3: footprint Package_DIP:DIP-16_W7.62mm -> Naquadah_Generator:SOIC-16_3.9x9.9mm_P1.27mm_Hand_Solder; Digikey Part No. (none) -> 296-14857-1-ND; Manufacturer Name (none) -> Texas Instruments; Manufacturer Part No. (none) -> SN74HC595DR
Connections:
- net labels added: BLUELT1, BLUELT2, BLUELT3, BLUELT4, BLUELT5, GRNLT, RDLT, WHTLT
- wire segments 36 -> 56
Other:
- note added: "Transistor Array"
- moved on the sheet: D2, R3, U2, U3

Commit message: Updates
Parts:
- U2, U3, U4: Description (none) -> Texas Instruments
Changed lines of the file:
@@
 $Descr A4 11693 8268
 encoding utf-8
-Sheet 3 10
+Sheet 3 11
 Title ""
 Date ""
@@
 F 5 "Texas Instruments" H 2400 1950 50  0001 C CNN "Manufacturer Name"
 F 6 "SN74HC595DR" H 2400 1950 50  0001 C CNN "Manufacturer Part No."
+F 7 "Texas Instruments" H 2400 1950 50  0001 C CNN "Description"
 	1    2400 1950
 	1    0    0    -1
@@
 F 5 "Texas Instruments" H 4850 1950 50  0001 C CNN "Manufacturer Name"
 F 6 "ULN2803ADWR" H 4850 1950 50  0001 C CNN "Manufacturer Part No."
+F 7 "Texas Instruments" H 4850 1950 50  0001 C CNN "Description"
 	1    4850 1950
 	1    0    0    -1
@@
 F 5 "Texas Instruments" H 2350 5300 50  0001 C CNN "Manufacturer Name"
 F 6 "SN74HC595DR" H 2350 5300 50  0001 C CNN "Manufacturer Part No."
+F 7 "Texas Instruments" H 2350 5300 50  0001 C CNN "Description"
 	1    2350 5300
 	1    0    0    -1

Commit message: Adding Power Daughter Board
Parts:
- U2, U3: Digikey Part No. 296-14857-1-ND -> (none); Source (none) -> Digikey; Source Part No. (none) -> 296-14857-1-ND
- U4: Digikey Part No. 296-15777-1-ND -> (none); Source (none) -> Digikey; Source Part No. (none) -> 296-15777-1-ND
Changed lines of the file:
@@
 F 2 "Naquadah_Generator:SOIC-16_3.9x9.9mm_P1.27mm_Hand_Solder" H 2400 1950 50  0001 C CNN
 F 3 "http://www.ti.com/lit/ds/symlink/sn74hc595.pdf?HQS=TI-null-null-digikeymode-df-pf-null-wwe&ts=1590028307018" H 2400 1950 50  0001 C CNN
-F 4 "296-14857-1-ND" H 2400 1950 50  0001 C CNN "Digikey Part No."
+F 4 "296-14857-1-ND" H 2400 1950 50  0001 C CNN "Source Part No."
 F 5 "Texas Instruments" H 2400 1950 50  0001 C CNN "Manufacturer Name"
 F 6 "SN74HC595DR" H 2400 1950 50  0001 C CNN "Manufacturer Part No."
 F 7 "Texas Instruments" H 2400 1950 50  0001 C CNN "Description"
+F 8 "Digikey" H 2400 1950 50  0001 C CNN "Source"
 	1    2400 1950
 	1    0    0    -1
@@
 F 2 "Naquadah_Generator:SOIC127P1030X265-18N" H 4550 1050 50  0001 L BNN
 F 3 "http://www.ti.com/lit/ds/symlink/uln2803a.pdf?HQS=TI-null-null-digikeymode-df-pf-null-wwe&ts=1590002980089" H 4850 1950 50  0001 L BNN
-F 4 "296-15777-1-ND" H 4850 1950 50  0001 C CNN "Digikey Part No."
+F 4 "296-15777-1-ND" H 4850 1950 50  0001 C CNN "Source Part No."
 F 5 "Texas Instruments" H 4850 1950 50  0001 C CNN "Manufacturer Name"
 F 6 "ULN2803ADWR" H 4850 1950 50  0001 C CNN "Manufacturer Part No."
 F 7 "Texas Instruments" H 4850 1950 50  0001 C CNN "Description"
+F 8 "Digikey" H 4850 1950 50  0001 C CNN "Source"
 	1    4850 1950
 	1    0    0    -1
@@
 F 2 "Naquadah_Generator:SOIC-16_3.9x9.9mm_P1.27mm_Hand_Solder" H 2350 5300 50  0001 C CNN
 F 3 "http://www.ti.com/lit/ds/symlink/sn74hc595.pdf?HQS=TI-null-null-digikeymode-df-pf-null-wwe&ts=1590028307018" H 2350 5300 50  0001 C CNN
-F 4 "296-14857-1-ND" H 2350 5300 50  0001 C CNN "Digikey Part No."
+F 4 "296-14857-1-ND" H 2350 5300 50  0001 C CNN "Source Part No."
 F 5 "Texas Instruments" H 2350 5300 50  0001 C CNN "Manufacturer Name"
 F 6 "SN74HC595DR" H 2350 5300 50  0001 C CNN "Manufacturer Part No."
 F 7 "Texas Instruments" H 2350 5300 50  0001 C CNN "Description"
+F 8 "Digikey" H 2350 5300 50  0001 C CNN "Source"
 	1    2350 5300
 	1    0    0    -1

Commit message: Updates
Parts:
- removed D2: LED, LED_THT:LED_D5.0mm, symbol Frequently_Used:LED
- removed R3: 330, Frequently_Used:0805_2012Metric_HandSolder, symbol Frequently_Used:R
Connections:
- net labels removed: IND
- wire segments 56 -> 53
- no-connect marks 8 -> 9
Other:
- moved on the sheet: J3, U2, U3, U4

Commit message: Updates
Parts:
- U4: Description Texas Instruments -> Bipolar (BJT) Transistor Array 8 NPN Darlington 50V 500mA S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
Changed lines of the file:
@@
 F 5 "Texas Instruments" H 6650 3700 50  0001 C CNN "Manufacturer Name"
 F 6 "ULN2803ADWR" H 6650 3700 50  0001 C CNN "Manufacturer Part No."
-F 7 "Texas Instruments" H 6650 3700 50  0001 C CNN "Description"
+F 7 "Bipolar (BJT) Transistor Array 8 NPN Darlington 50V 500mA Surface Mount 18-SOIC" H 6650 3700 50  0001 C CNN "Description"
 F 8 "Digikey" H 6650 3700 50  0001 C CNN "Source"
 	1    6650 3700

Commit message: Move libraries and added configuration path.
Moved Li-Ion library to common KiCad library.  Added variables to configuration paths to reference my KiCad libraries.  Moved all 3D components to my common library.
Connections:
- wire segments 53 -> 55
Changed lines of the file:
@@
 $EndDescr
 $Comp
-L Frequently_Used:GND #PWR028
+L Frequently_Used_LE:GND #PWR028
 U 1 1 5ED2A2E7
 P 3650 4400
@@
 $EndComp
 $Comp
-L Frequently_Used:GND #PWR032
+L Frequently_Used_LE:GND #PWR032
 U 1 1 5ED2A2ED
 P 2400 6900
@@
 NoConn ~ 2800 6700
 $Comp
-L Frequently_Used:GND #PWR026
+L Frequently_Used_LE:GND #PWR026
 U 1 1 5ED2A2FE
 P 2400 4000
@@
 WHTLT
 Wire Wire Line
+	4050 3900 4550 3900
+Wire Wire Line
+	4050 3300 4550 3300
+Wire Wire Line
+	4050 3400 4550 3400
+Wire Wire Line
 	4050 3500 4550 3500
 Wire Wire Line
-	4050 3400 4550 3400
-Wire Wire Line
 	4050 3600 4550 3600
 Wire Wire Line
 	4050 3700 4550 3700
 Wire Wire Line
+	4050 4000 4550 4000
+Wire Wire Line
 	4050 3800 4550 3800
 Wire Wire Line
-	4050 3900 4550 3900
-Wire Wire Line
-	4050 3300 4550 3300
-Wire Wire Line
-	4050 4000 4550 4000
-Wire Wire Line
 	3250 3900 2400 3900
 Wire Wire Line
 	2400 3900 2400 4000
 $Comp
-L Frequently_Used:+5V #PWR027
+L Frequently_Used_LE:+5V #PWR027
 U 1 1 5ED2A354
 P 3650 3050
@@
 Wire Wire Line
 	1500 5800 2000 5800
+Text Label 4100 3800 0    50   ~ 0
+SRBLUELT5
+Text Label 4100 3700 0    50   ~ 0
+SRBLUELT4
+Text Label 4100 3600 0    50   ~ 0
+SRBLUELT3
+Text Label 4100 3500 0    50   ~ 0
+SRBLUELT2
+Text Label 4100 3400 0    50   ~ 0
+SRBLUELT1
 Text Label 4100 4000 0    50   ~ 0
-SRBLUELT5
+SRGRNLT
+Text Label 4100 3300 0    50   ~ 0
+SRRDLT
 Text Label 4100 3900 0    50   ~ 0
-SRBLUELT4
-Text Label 4100 3800 0    50   ~ 0
-SRBLUELT3
-Text Label 4100 3700 0    50   ~ 0
-SRBLUELT2
-Text Label 4100 3600 0    50   ~ 0
-SRBLUELT1
-Text Label 4100 3300 0    50   ~ 0
-SRGRNLT
-Text Label 4100 3400 0    50   ~ 0
-SRRDLT
-Text Label 4100 3500 0    50   ~ 0
 SRWHTLT
 $Sheet
@@
 	3650 3050 3650 3100
 $Comp
-L Frequently_Used:+5V #PWR025
+L Frequently_Used_LE:+5V #PWR025
 U 1 1 5ED69E0B
 P 2400 3500
@@
 SRLATCH
 $Comp
-L Frequently_Used:GND #PWR030
+L Frequently_Used_LE:GND #PWR030
 U 1 1 5ED706AF
 P 1150 6500
@@
 	1150 6400 1150 6500
 $Comp
-L Frequently_Used:+5V #PWR029
+L Frequently_Used_LE:+5V #PWR029
 U 1 1 5ED7340D
 P 1150 6000
@@
 	1150 6100 2000 6100
 $Comp
-L Frequently_Used:+5V #PWR031
+L Frequently_Used_LE:+5V #PWR031
 U 1 1 5ED747C1
 P 2400 5550
@@
 Shift Register 1
 Wire Wire Line
-	5750 4100 6250 4100
+	5750 3900 6250 3900
+Wire Wire Line
+	5750 3800 6250 3800
+Wire Wire Line
+	5750 3700 6250 3700
+Wire Wire Line
+	5750 3600 6250 3600
+Wire Wire Line
+	5750 3500 6250 3500
 Wire Wire Line
 	5750 4000 6250 4000
 Wire Wire Line
-	5750 3900 6250 3900
-Wire Wire Line
-	5750 3800 6250 3800
-Wire Wire Line
-	5750 3700 6250 3700
-Wire Wire Line
-	5750 3600 6250 3600
-Wire Wire Line
-	5750 3500 6250 3500
+	5750 3400 6250 3400
 $Comp
 L Naquadah_Generator:ULN2803ADWRG4 U4
@@
 $EndComp
 Wire Wire Line
-	5750 3400 6250 3400
+	5750 4100 6250 4100
+Text Label 5750 3900 0    50   ~ 0
+SRBLUELT5
+Text Label 5750 3800 0    50   ~ 0
+SRBLUELT4
+Text Label 5750 3700 0    50   ~ 0
+SRBLUELT3
+Text Label 5750 3600 0    50   ~ 0
+SRBLUELT2
+Text Label 5750 3500 0    50   ~ 0
+SRBLUELT1
+Text Label 5750 4000 0    50   ~ 0
+SRWHTLT
+Text Label 5750 3400 0    50   ~ 0
+SRRDLT
 Text Label 5750 4100 0    50   ~ 0
-SRBLUELT5
-Text Label 5750 4000 0    50   ~ 0
-SRBLUELT4
-Text Label 5750 3900 0    50   ~ 0
-SRBLUELT3
-Text Label 5750 3800 0    50   ~ 0
-SRBLUELT2
-Text Label 5750 3700 0    50   ~ 0
-SRBLUELT1
-Text Label 5750 3600 0    50   ~ 0
-SRWHTLT
-Text Label 5750 3500 0    50   ~ 0
-SRRDLT
-Text Label 5750 3400 0    50   ~ 0
 SRGRNLT
 $Comp
-L Frequently_Used:GND #PWR0101
+L Frequently_Used_LE:GND #PWR0101
 U 1 1 5ED4DB66
 P 7150 4400
@@
 	-1   0    0    1
 $EndComp
+Text Label 7100 3900 0    50   ~ 0
+BLUELT5
+Text Label 7100 3800 0    50   ~ 0
+BLUELT4
+Text Label 7100 3700 0    50   ~ 0
+BLUELT3
+Text Label 7100 3600 0    50   ~ 0
+BLUELT2
+Text Label 7100 3500 0    50   ~ 0
+BLUELT1
 Text Label 7100 4100 0    50   ~ 0
-BLUELT5
-Text Label 7100 4000 0    50   ~ 0
-BLUELT4
-Text Label 7100 3900 0    50   ~ 0
-BLUELT3
-Text Label 7100 3800 0    50   ~ 0
-BLUELT2
-Text Label 7100 3700 0    50   ~ 0
-BLUELT1
+GRNLT
 Text Label 7100 3400 0    50   ~ 0
-GRNLT
-Text Label 7100 3500 0    50   ~ 0
 RDLT
-Text Label 7100 3600 0    50   ~ 0
-WHTLT
-Wire Wire Line
-	7550 3400 7050 3400
+Wire Wire Line
+	7550 4100 7050 4100
+Wire Wire Line
+	7050 3400 7550 3400
+Wire Wire Line
+	7050 3900 7550 3900
+Wire Wire Line
+	7050 3800 7550 3800
+Wire Wire Line
+	7050 3700 7550 3700
+Wire Wire Line
+	7050 3600 7550 3600
 Wire Wire Line
 	7050 3500 7550 3500
-Wire Wire Line
-	7050 4100 7550 4100
-Wire Wire Line
-	7050 4000 7550 4000
-Wire Wire Line
-	7050 3900 7550 3900
-Wire Wire Line
-	7050 3800 7550 3800
-Wire Wire Line
-	7050 3700 7550 3700
-Wire Wire Line
-	7050 3600 7550 3600
 $Comp
 L 74xx:74HC595 U3
@@
 Transistor Array
 NoConn ~ 2800 5900
+Wire Wire Line
+	7050 4000 7550 4000
+Text Label 7100 4000 0    50   ~ 0
+WHTLT
+Wire Wire Line
+	7050 3200 7150 3200
+Wire Wire Line
+	7150 3200 7150 3100
+$Comp
+L Frequently_Used_LE:+5V #PWR?
+U 1 1 5EE819EA
+P 7150 3100
+F 0 "#PWR?" H 7150 2950 50  0001 C CNN
+F 1 "+5V" H 7165 3273 50  0000 C CNN
+F 2 "" H 7150 3100 50  0001 C CNN
+F 3 "" H 7150 3100 50  0001 C CNN
+	1    7150 3100
+	1    0    0    -1
+$EndComp
 $EndSCHEMATC
