File: Naquadah Generator Main/Shift Registers.sch (KiCad schematic (older format))
At the start: 4 parts, among them J3 Conn_01x02, U2 74HC595, U3 74HC595, U4 ULN2803ADWRG4

Commit message: Separated digital and analog ground.
Connections:
- net labels added: GNDD
- net labels removed: GND
Changed lines of the file:
@@
 $EndDescr
 $Comp
-L Frequently_Used_LE:GND #PWR028
+L Frequently_Used_LE:GNDD #PWR028
 U 1 1 5ED2A2E7
 P 3650 4400
 F 0 "#PWR028" H 3650 4150 50  0001 C CNN
-F 1 "GND" H 3655 4227 50  0000 C CNN
+F 1 "GNDD" H 3655 4227 50  0000 C CNN
 F 2 "" H 3650 4400 50  0001 C CNN
 F 3 "" H 3650 4400 50  0001 C CNN
@@
 $EndComp
 $Comp
-L Frequently_Used_LE:GND #PWR032
+L Frequently_Used_LE:GNDD #PWR032
 U 1 1 5ED2A2ED
 P 2400 6900
 F 0 "#PWR032" H 2400 6650 50  0001 C CNN
-F 1 "GND" H 2405 6727 50  0000 C CNN
+F 1 "GNDD" H 2405 6727 50  0000 C CNN
 F 2 "" H 2400 6900 50  0001 C CNN
 F 3 "" H 2400 6900 50  0001 C CNN
@@
 NoConn ~ 2800 6700
 $Comp
-L Frequently_Used_LE:GND #PWR026
+L Frequently_Used_LE:GNDD #PWR026
 U 1 1 5ED2A2FE
 P 2400 4000
 F 0 "#PWR026" H 2400 3750 50  0001 C CNN
-F 1 "GND" V 2405 3872 50  0000 R CNN
+F 1 "GNDD" V 2405 3872 50  0000 R CNN
 F 2 "" H 2400 4000 50  0001 C CNN
 F 3 "" H 2400 4000 50  0001 C CNN
@@
 SRLATCH
 $Comp
-L Frequently_Used_LE:GND #PWR030
+L Frequently_Used_LE:GNDD #PWR030
 U 1 1 5ED706AF
 P 1150 6500
 F 0 "#PWR030" H 1150 6250 50  0001 C CNN
-F 1 "GND" V 1155 6372 50  0000 R CNN
+F 1 "GNDD" V 1155 6372 50  0000 R CNN
 F 2 "" H 1150 6500 50  0001 C CNN
 F 3 "" H 1150 6500 50  0001 C CNN
@@
 SRGRNLT
 $Comp
-L Frequently_Used_LE:GND #PWR0101
+L Frequently_Used_LE:GNDD #PWR0101
 U 1 1 5ED4DB66
 P 7150 4400
 F 0 "#PWR0101" H 7150 4150 50  0001 C CNN
-F 1 "GND" H 7155 4227 50  0000 C CNN
+F 1 "GNDD" H 7155 4227 50  0000 C CNN
 F 2 "" H 7150 4400 50  0001 C CNN
 F 3 "" H 7150 4400 50  0001 C CNN

Commit message: Audio update
Connections:
- net labels added: DGND
- net labels removed: GNDD
Changed lines of the file:
@@
 $EndDescr
 $Comp
-L Frequently_Used_LE:GNDD #PWR028
+L Frequently_Used_LE:DGND #PWR028
 U 1 1 5ED2A2E7
 P 3650 4400
 F 0 "#PWR028" H 3650 4150 50  0001 C CNN
-F 1 "GNDD" H 3655 4227 50  0000 C CNN
+F 1 "DGND" H 3655 4227 50  0000 C CNN
 F 2 "" H 3650 4400 50  0001 C CNN
 F 3 "" H 3650 4400 50  0001 C CNN
@@
 $EndComp
 $Comp
-L Frequently_Used_LE:GNDD #PWR032
+L Frequently_Used_LE:DGND #PWR032
 U 1 1 5ED2A2ED
 P 2400 6900
 F 0 "#PWR032" H 2400 6650 50  0001 C CNN
-F 1 "GNDD" H 2405 6727 50  0000 C CNN
+F 1 "DGND" H 2405 6727 50  0000 C CNN
 F 2 "" H 2400 6900 50  0001 C CNN
 F 3 "" H 2400 6900 50  0001 C CNN
@@
 NoConn ~ 2800 6700
 $Comp
-L Frequently_Used_LE:GNDD #PWR026
+L Frequently_Used_LE:DGND #PWR026
 U 1 1 5ED2A2FE
 P 2400 4000
 F 0 "#PWR026" H 2400 3750 50  0001 C CNN
-F 1 "GNDD" V 2405 3872 50  0000 R CNN
+F 1 "DGND" V 2405 3872 50  0000 R CNN
 F 2 "" H 2400 4000 50  0001 C CNN
 F 3 "" H 2400 4000 50  0001 C CNN
@@
 WHTLT
 Wire Wire Line
+	4050 3500 4550 3500
+Wire Wire Line
+	4050 3300 4550 3300
+Wire Wire Line
+	4050 4000 4550 4000
+Wire Wire Line
 	4050 3900 4550 3900
 Wire Wire Line
-	4050 3300 4550 3300
+	4050 3800 4550 3800
+Wire Wire Line
+	4050 3700 4550 3700
 Wire Wire Line
 	4050 3400 4550 3400
 Wire Wire Line
-	4050 3500 4550 3500
-Wire Wire Line
 	4050 3600 4550 3600
-Wire Wire Line
-	4050 3700 4550 3700
-Wire Wire Line
-	4050 4000 4550 4000
-Wire Wire Line
-	4050 3800 4550 3800
 Wire Wire Line
 	3250 3900 2400 3900
@@
 Wire Wire Line
 	1500 5800 2000 5800
-Text Label 4100 3800 0    50   ~ 0
+Text Label 4100 3600 0    50   ~ 0
 SRBLUELT5
 Text Label 4100 3700 0    50   ~ 0
 SRBLUELT4
-Text Label 4100 3600 0    50   ~ 0
+Text Label 4100 3800 0    50   ~ 0
 SRBLUELT3
-Text Label 4100 3500 0    50   ~ 0
+Text Label 4100 3900 0    50   ~ 0
 SRBLUELT2
+Text Label 4100 4000 0    50   ~ 0
+SRBLUELT1
 Text Label 4100 3400 0    50   ~ 0
-SRBLUELT1
-Text Label 4100 4000 0    50   ~ 0
 SRGRNLT
 Text Label 4100 3300 0    50   ~ 0
 SRRDLT
-Text Label 4100 3900 0    50   ~ 0
+Text Label 4100 3500 0    50   ~ 0
 SRWHTLT
 $Sheet
@@
 SRLATCH
 $Comp
-L Frequently_Used_LE:GNDD #PWR030
+L Frequently_Used_LE:DGND #PWR030
 U 1 1 5ED706AF
 P 1150 6500
 F 0 "#PWR030" H 1150 6250 50  0001 C CNN
-F 1 "GNDD" V 1155 6372 50  0000 R CNN
+F 1 "DGND" V 1155 6372 50  0000 R CNN
 F 2 "" H 1150 6500 50  0001 C CNN
 F 3 "" H 1150 6500 50  0001 C CNN
@@
 SRGRNLT
 $Comp
-L Frequently_Used_LE:GNDD #PWR0101
+L Frequently_Used_LE:DGND #PWR0101
 U 1 1 5ED4DB66
 P 7150 4400
 F 0 "#PWR0101" H 7150 4150 50  0001 C CNN
-F 1 "GNDD" H 7155 4227 50  0000 C CNN
+F 1 "DGND" H 7155 4227 50  0000 C CNN
 F 2 "" H 7150 4400 50  0001 C CNN
 F 3 "" H 7150 4400 50  0001 C CNN

Commit message: Audio updates, switching to separate USB schematic
Audio updates, switching to separate USB schematic
Parts:
- U4: symbol Naquadah_Generator:ULN2803ADWRG4 -> Transistor_Array:ULN2803A
Connections:
- wire segments 55 -> 54
Changed lines of the file:
@@
 $Descr A4 11693 8268
 encoding utf-8
-Sheet 2 15
+Sheet 2 16
 Title ""
 Date ""
@@
 Wire Wire Line
 	2400 3900 2400 4000
-$Comp
-L Frequently_Used_LE:+5V #PWR027
-U 1 1 5ED2A354
-P 3650 3050
-F 0 "#PWR027" H 3650 2900 50  0001 C CNN
-F 1 "+5V" H 3665 3223 50  0000 C CNN
-F 2 "" H 3650 3050 50  0001 C CNN
-F 3 "" H 3650 3050 50  0001 C CNN
-	1    3650 3050
-	1    0    0    -1
-$EndComp
 Text Label 4100 4200 0    50   ~ 0
 SR1OUT2IN
@@
 Text HLabel 3100 3500 0    50   Input ~ 0
 SRCLK
-Wire Wire Line
-	3650 3050 3650 3100
 $Comp
 L Frequently_Used_LE:+5V #PWR025
@@
 Wire Wire Line
 	2400 5550 2400 5600
-Text Notes 2000 7400 0    79   ~ 16
+Text Notes 1950 7400 0    79   ~ 16
 Shift Register 2
 Text Notes 3200 4900 0    79   ~ 16
@@
 	5750 3400 6250 3400
 $Comp
-L Naquadah_Generator:ULN2803ADWRG4 U4
+L Transistor_Array:ULN2803A U4
 U 1 1 5ED3FEF3
-P 6650 3700
-F 0 "U4" H 6650 4465 50  0000 C CNN
-F 1 "ULN2803ADWRG4" H 6650 4374 50  0000 C CNN
-F 2 "Naquadah_Generator:SOIC127P1030X265-18N" H 6350 2800 50  0001 L BNN
-F 3 "http://www.ti.com/lit/ds/symlink/uln2803a.pdf?HQS=TI-null-null-digikeymode-df-pf-null-wwe&ts=1590002980089" H 6650 3700 50  0001 L BNN
-F 4 "296-15777-1-ND" H 6650 3700 50  0001 C CNN "Source Part No."
-F 5 "Texas Instruments" H 6650 3700 50  0001 C CNN "Manufacturer Name"
-F 6 "ULN2803ADWR" H 6650 3700 50  0001 C CNN "Manufacturer Part No."
-F 7 "Bipolar (BJT) Transistor Array 8 NPN Darlington 50V 500mA Surface Mount 18-SOIC" H 6650 3700 50  0001 C CNN "Description"
-F 8 "Digikey" H 6650 3700 50  0001 C CNN "Source"
-	1    6650 3700
+P 6650 3600
+F 0 "U4" H 6650 4365 50  0000 C CNN
+F 1 "ULN2803ADWRG4" H 6650 4274 50  0000 C CNN
+F 2 "Naquadah_Generator:SOIC127P1030X265-18N" H 6350 2700 50  0001 L BNN
+F 3 "http://www.ti.com/lit/ds/symlink/uln2803a.pdf?HQS=TI-null-null-digikeymode-df-pf-null-wwe&ts=1590002980089" H 6650 3600 50  0001 L BNN
+F 4 "296-15777-1-ND" H 6650 3600 50  0001 C CNN "Source Part No."
+F 5 "Texas Instruments" H 6650 3600 50  0001 C CNN "Manufacturer Name"
+F 6 "ULN2803ADWR" H 6650 3600 50  0001 C CNN "Manufacturer Part No."
+F 7 "Bipolar (BJT) Transistor Array 8 NPN Darlington 50V 500mA Surface Mount 18-SOIC" H 6650 3600 50  0001 C CNN "Description"
+F 8 "Digikey" H 6650 3600 50  0001 C CNN "Source"
+	1    6650 3600
 	1    0    0    -1
 $EndComp
@@
 L Frequently_Used_LE:DGND #PWR0101
 U 1 1 5ED4DB66
-P 7150 4400
-F 0 "#PWR0101" H 7150 4150 50  0001 C CNN
-F 1 "DGND" H 7155 4227 50  0000 C CNN
-F 2 "" H 7150 4400 50  0001 C CNN
-F 3 "" H 7150 4400 50  0001 C CNN
-	1    7150 4400
-	1    0    0    -1
-$EndComp
-Wire Wire Line
-	7050 4300 7150 4300
-Wire Wire Line
-	7150 4300 7150 4400
+P 6650 4400
+F 0 "#PWR0101" H 6650 4150 50  0001 C CNN
+F 1 "DGND" H 6655 4227 50  0000 C CNN
+F 2 "" H 6650 4400 50  0001 C CNN
+F 3 "" H 6650 4400 50  0001 C CNN
+	1    6650 4400
+	1    0    0    -1
+$EndComp
+Wire Wire Line
+	6650 4300 6650 4400
 Wire Wire Line
 	9800 3200 9800 3400
@@
 WHTLT
 Wire Wire Line
-	7050 3200 7150 3200
-Wire Wire Line
-	7150 3200 7150 3100
+	3650 3050 3650 3100
+$Comp
+L Frequently_Used_LE:+5V #PWR027
+U 1 1 5ED2A354
+P 3650 3050
+F 0 "#PWR027" H 3650 2900 50  0001 C CNN
+F 1 "+5V" H 3665 3223 50  0000 C CNN
+F 2 "" H 3650 3050 50  0001 C CNN
+F 3 "" H 3650 3050 50  0001 C CNN
+	1    3650 3050
+	1    0    0    -1
+$EndComp
 $Comp
 L Frequently_Used_LE:+5V #PWR0122
 U 1 1 5EE819EA
-P 7150 3100
-F 0 "#PWR0122" H 7150 2950 50  0001 C CNN
-F 1 "+5V" H 7165 3273 50  0000 C CNN
-F 2 "" H 7150 3100 50  0001 C CNN
-F 3 "" H 7150 3100 50  0001 C CNN
-	1    7150 3100
-	1    0    0    -1
-$EndComp
+P 7150 3200
+F 0 "#PWR0122" H 7150 3050 50  0001 C CNN
+F 1 "+5V" H 7165 3373 50  0000 C CNN
+F 2 "" H 7150 3200 50  0001 C CNN
+F 3 "" H 7150 3200 50  0001 C CNN
+	1    7150 3200
+	1    0    0    -1
+$EndComp
+Wire Wire Line
+	7150 3300 7150 3200
+Wire Wire Line
+	7050 3300 7150 3300
 $EndSCHEMATC

Commit message: Added level shifter, moved user interface connector location
Added level shifter, moved user interface connector location
Parts:
- added U12: CD74HC4050PWR, Package_SO:TSSOP-16_4.4x5mm_P0.65mm, symbol 74xx~LE:CD74HC4050PWR
- J3: Description (none) -> None; Manufacturer Name (none) -> None; Manufacturer Part No. (none) -> None; Source (none) -> None; Source Part No. (none) -> None
- U2, U3: Description Texas Instruments -> Shift Register 1 Element 8 Bit 16-SOIC
Connections:
- net labels added: +3.3V, AUDIORESET, AUDIORESET5V, READY, SNDLATCH, SNDLATCH5V, SNDON, SNDON5V, SNDRANDOM, SNDRANDOM5V
- wire segments 54 -> 71
- no-connect marks 9 -> 8
Other:
- note added: "Level Shifter"
- moved on the sheet: J3, U2, U3, U4

Commit message: Switched to 0603_1608M size for passives
Parts:
- removed J3: Conn_01x02, Connector_Wire:SolderWirePad_1x02_P3.81mm_Drill1.2mm, symbol Connector_Generic:Conn_01x02
- U12: symbol 74xx~LE:CD74HC4050PWR -> 74xx_LE:CD74HC4050PWR
Connections:
- net labels added: WHITELT
- wire segments 71 -> 69
Changed lines of the file:
@@
 $Descr A4 11693 8268
 encoding utf-8
-Sheet 2 17
+Sheet 2 18
 Title ""
 Date ""
@@
 $EndComp
 $Sheet
-S 9900 3550 500  200
+S 9900 3450 500  200
 U 5ED2A301
 F0 "Blue Lights 2" 50
 F1 "BlueLights.sch" 50
-F2 "COLLECTOR" I L 9900 3650 50
-$EndSheet
-$Sheet
-S 9900 4000 500  200
+F2 "COLLECTOR" I L 9900 3550 50
+$EndSheet
+$Sheet
+S 9900 3900 500  200
 U 5ED2A304
 F0 "Blue Lights 3" 50
 F1 "BlueLights.sch" 50
-F2 "COLLECTOR" I L 9900 4100 50
-$EndSheet
-$Sheet
-S 9900 4450 500  200
+F2 "COLLECTOR" I L 9900 4000 50
+$EndSheet
+$Sheet
+S 9900 4350 500  200
 U 5ED2A307
 F0 "Blue Lights 4" 50
 F1 "BlueLights.sch" 50
-F2 "COLLECTOR" I L 9900 4550 50
-$EndSheet
-$Sheet
-S 9900 4900 500  200
+F2 "COLLECTOR" I L 9900 4450 50
+$EndSheet
+$Sheet
+S 9900 4800 500  200
 U 5ED2A30A
 F0 "Blue Lights 5" 50
 F1 "BlueLights.sch" 50
-F2 "COLLECTOR" I L 9900 5000 50
-$EndSheet
-$Sheet
-S 9900 3100 500  200
+F2 "COLLECTOR" I L 9900 4900 50
+$EndSheet
+$Sheet
+S 9900 3000 500  200
 U 5ED2A30D
 F0 "Blue Lights 1" 50
 F1 "BlueLights.sch" 50
-F2 "COLLECTOR" I L 9900 3200 50
+F2 "COLLECTOR" I L 9900 3100 50
 $EndSheet
 NoConn ~ 3150 4700
 NoConn ~ 3150 4600
 NoConn ~ 3150 4500
-Text Label 9450 5000 0    50   ~ 0
+Text Label 9450 4900 0    50   ~ 0
 BLUELT5
-Text Label 9450 4550 0    50   ~ 0
+Text Label 9450 4450 0    50   ~ 0
 BLUELT4
-Text Label 9450 4100 0    50   ~ 0
+Text Label 9450 4000 0    50   ~ 0
 BLUELT3
-Text Label 9450 3650 0    50   ~ 0
+Text Label 9450 3550 0    50   ~ 0
 BLUELT2
-Text Label 9450 3200 0    50   ~ 0
+Text Label 9450 3100 0    50   ~ 0
 BLUELT1
 $Sheet
-S 9900 1950 500  200
+S 9900 2050 500  200
 U 5ED2A32F
 F0 "Red Lights" 50
 F1 "GreenRedLights.sch" 50
-F2 "COLLECTOR" I L 9900 2050 50
-$EndSheet
-Text Label 9450 1600 0    50   ~ 0
+F2 "COLLECTOR" I L 9900 2150 50
+$EndSheet
+Text Label 9450 1700 0    50   ~ 0
 GRNLT
-Text Label 9450 2050 0    50   ~ 0
+Text Label 9450 2150 0    50   ~ 0
 RDLT
-Text Label 9450 2850 0    50   ~ 0
-WHTLT
 Wire Wire Line
 	3150 1900 3650 1900
@@
 SRWHTLT
 $Sheet
-S 9900 1500 500  200
+S 9900 1600 500  200
 U 5ED2A36D
 F0 "Green Lights" 50
 F1 "GreenRedLights.sch" 50
-F2 "COLLECTOR" I L 9900 1600 50
-$EndSheet
-Wire Wire Line
-	9900 1600 9450 1600
-Wire Wire Line
-	10400 2850 9450 2850
-Wire Wire Line
-	9900 2050 9450 2050
-Wire Wire Line
-	9900 3200 9450 3200
-Wire Wire Line
-	9900 3650 9450 3650
-Wire Wire Line
-	9900 5000 9450 5000
-Wire Wire Line
-	9900 4550 9450 4550
-Wire Wire Line
-	9900 4100 9450 4100
-$Comp
-L 74xx:74HC595 U2
-U 1 1 5ED2A2DB
-P 2750 2100
-F 0 "U2" H 2950 2750 50  0000 L CNN
-F 1 "74HC595" H 2950 2650 50  0000 L CNN
-F 2 "Naquadah_Generator:SOIC-16_3.9x9.9mm_P1.27mm_Hand_Solder" H 2750 2100 50  0001 C CNN
-F 3 "http://www.ti.com/lit/ds/symlink/sn74hc595.pdf?HQS=TI-null-null-digikeymode-df-pf-null-wwe&ts=1590028307018" H 2750 2100 50  0001 C CNN
-F 4 "296-14857-1-ND" H 2750 2100 50  0001 C CNN "Source Part No."
-F 5 "Texas Instruments" H 2750 2100 50  0001 C CNN "Manufacturer Name"
-F 6 "SN74HC595DR" H 2750 2100 50  0001 C CNN "Manufacturer Part No."
-F 7 "Shift Register 1 Element 8 Bit 16-SOIC" H 2750 2100 50  0001 C CNN "Description"
-F 8 "Digikey" H 2750 2100 50  0001 C CNN "Source"
-	1    2750 2100
-	1    0    0    -1
-$EndComp
+F2 "COLLECTOR" I L 9900 1700 50
+$EndSheet
+Wire Wire Line
+	9900 1700 9450 1700
+Wire Wire Line
+	9900 2150 9450 2150
+Wire Wire Line
+	9900 3100 9450 3100
+Wire Wire Line
+	9900 3550 9450 3550
+Wire Wire Line
+	9900 4900 9450 4900
+Wire Wire Line
+	9900 4450 9450 4450
+Wire Wire Line
+	9900 4000 9450 4000
 Text HLabel 2200 2200 0    50   Input ~ 0
 SRLATCH
@@
 U 1 1 5ED3FEF3
 P 5750 2000
-F 0 "U4" H 5750 2765 50  0000 C CNN
-F 1 "ULN2803ADWRG4" H 5750 2674 50  0000 C CNN
+F 0 "U4" H 5750 2550 50  0000 C CNN
+F 1 "ULN2803ADWRG4" H 5750 2450 50  0000 C CNN
 F 2 "Naquadah_Generator:SOIC127P1030X265-18N" H 5450 1100 50  0001 L BNN
 F 3 "http://www.ti.com/lit/ds/symlink/uln2803a.pdf?HQS=TI-null-null-digikeymode-df-pf-null-wwe&ts=1590002980089" H 5750 2000 50  0001 L BNN
@@
 Wire Wire Line
 	5750 2700 5750 2800
-Wire Wire Line
-	10400 2650 10400 2850
-$Comp
-L power:+5V #PWR?
-U 1 1 5ED5733C
-P 10400 2500
-AR Path="/5ED17BA0/5ED2A32C/5ED5733C" Ref="#PWR?"  Part="1"
-AR Path="/5ED17BA0/5ED5733C" Ref="#PWR0102"  Part="1"
-F 0 "#PWR0102" H 10400 2350 50  0001 C CNN
-F 1 "+5V" H 10415 2673 50  0000 C CNN
-F 2 "" H 10400 2500 50  0001 C CNN
-F 3 "" H 10400 2500 50  0001 C CNN
-	1    10400 2500
-	1    0    0    -1
-$EndComp
-Wire Wire Line
-	10400 2500 10400 2550
-$Comp
-L Connector_Generic:Conn_01x02 J?
-U 1 1 5ED57335
-P 10200 2650
-AR Path="/5EA45E37/5ED57335" Ref="J?"  Part="1"
-AR Path="/5EA4676F/5ED57335" Ref="J?"  Part="1"
-AR Path="/5EA46A2B/5ED57335" Ref="J?"  Part="1"
-AR Path="/5ED17BA0/5ED2A32C/5ED57335" Ref="J?"  Part="1"
-AR Path="/5ED17BA0/5ED57335" Ref="J3"  Part="1"
-F 0 "J3" H 10750 2550 50  0000 R CNN
-F 1 "Conn_01x02" H 10750 2650 50  0000 R CNN
-F 2 "Connector_Wire:SolderWirePad_1x02_P3.81mm_Drill1.2mm" H 10200 2650 50  0001 C CNN
-F 3 "None" H 10200 2650 50  0001 C CNN
-F 4 "None" H 10200 2650 50  0001 C CNN "Description"
-F 5 "None" H 10200 2650 50  0001 C CNN "Manufacturer Name"
-F 6 "None" H 10200 2650 50  0001 C CNN "Manufacturer Part No."
-F 7 "None" H 10200 2650 50  0001 C CNN "Source"
-F 8 "None" H 10200 2650 50  0001 C CNN "Source Part No."
-	1    10200 2650
-	-1   0    0    1
-$EndComp
 Text Label 6200 2300 0    50   ~ 0
 BLUELT5
@@
 U 1 1 5ED2A2E1
 P 2750 4400
-F 0 "U3" H 2950 5050 50  0000 L CNN
-F 1 "74HC595" H 2950 4950 50  0000 L CNN
+F 0 "U3" H 2850 5050 50  0000 L CNN
+F 1 "74HC595" H 2850 4950 50  0000 L CNN
 F 2 "Naquadah_Generator:SOIC-16_3.9x9.9mm_P1.27mm_Hand_Solder" H 2750 4400 50  0001 C CNN
 F 3 "http://www.ti.com/lit/ds/symlink/sn74hc595.pdf?HQS=TI-null-null-digikeymode-df-pf-null-wwe&ts=1590028307018" H 2750 4400 50  0001 C CNN
@@
 	6150 1700 6250 1700
 $Comp
-L 74xx~LE:CD74HC4050PWR U12
+L 74xx_LE:CD74HC4050PWR U12
 U 1 1 6075B9A1
 P 5750 4550
-F 0 "U12" H 5750 5165 50  0000 C CNN
-F 1 "CD74HC4050PWR" H 5750 5074 50  0000 C CNN
+F 0 "U12" H 5750 5150 50  0000 C CNN
+F 1 "CD74HC4050PWR" H 5750 5050 50  0000 C CNN
 F 2 "Package_SO:TSSOP-16_4.4x5mm_P0.65mm" H 5750 3950 50  0001 C CNN
 F 3 "https://www.ti.com/lit/ds/symlink/cd74hc4049.pdf?HQS=TI-null-null-digikeymode-df-pf-null-wwe&ts=1598393766631" H 5200 4900 50  0001 C CNN
@@
 NoConn ~ 5200 4700
 NoConn ~ 5200 4800
+Text Label 9450 2650 0    50   ~ 0
+WHTLT
+Wire Wire Line
+	10050 2650 9450 2650
+Text HLabel 10050 2650 2    50   Input ~ 0
+WHITELT
+$Comp
+L 74xx:74HC595 U2
+U 1 1 5ED2A2DB
+P 2750 2100
+F 0 "U2" H 2850 2750 50  0000 L CNN
+F 1 "74HC595" H 2850 2650 50  0000 L CNN
+F 2 "Naquadah_Generator:SOIC-16_3.9x9.9mm_P1.27mm_Hand_Solder" H 2750 2100 50  0001 C CNN
+F 3 "http://www.ti.com/lit/ds/symlink/sn74hc595.pdf?HQS=TI-null-null-digikeymode-df-pf-null-wwe&ts=1590028307018" H 2750 2100 50  0001 C CNN
+F 4 "296-14857-1-ND" H 2750 2100 50  0001 C CNN "Source Part No."
+F 5 "Texas Instruments" H 2750 2100 50  0001 C CNN "Manufacturer Name"
+F 6 "SN74HC595DR" H 2750 2100 50  0001 C CNN "Manufacturer Part No."
+F 7 "Shift Register 1 Element 8 Bit 16-SOIC" H 2750 2100 50  0001 C CNN "Description"
+F 8 "Digikey" H 2750 2100 50  0001 C CNN "Source"
+	1    2750 2100
+	1    0    0    -1
+$EndComp
 $EndSCHEMATC

Commit message: Update JST connectors
Parts:
- U12: Source Texas Instruments -> Digikey
Changed lines of the file:
@@
 F 5 "Texas Instruments" H 5750 3750 50  0001 C CNN "Manufacturer Name"
 F 6 "CD74HC4050PWR" H 5750 3650 50  0001 C CNN "Manufacturer Part No."
-F 7 "Texas Instruments" H 5750 3550 50  0001 C CNN "Source"
+F 7 "Digikey" H 5750 3550 50  0001 C CNN "Source"
 F 8 "296-9215-1-ND" H 5750 3450 50  0001 C CNN "Source Part No."
 	1    5750 4550
