File: Naquadah Generator Main/WhiteLights.sch (KiCad schematic (older format))
At the start: 3 parts, among them J2 Conn_01x02, Q1 BC337

Commit message: Before changing BOM
Connections:
- net labels added: +5V, GND
- net labels removed: 5V, VGND
- wire segments 6 -> 5
Other:
- moved on the sheet: R34
Changed lines of the file:
@@
 $Descr A4 11693 8268
 encoding utf-8
-Sheet 13 14
+Sheet 8 10
 Title ""
 Date ""
@@
 $EndDescr
 Wire Wire Line
-	5450 4750 5400 4750
+	5450 4550 5450 4650
 Wire Wire Line
-	5450 4550 5450 4750
-Wire Wire Line
-	4650 4350 4850 4350
+	4650 4350 4750 4350
 Text HLabel 4650 4350 0    50   Input ~ 0
 SIGNAL
@@
 L Device:R R?
 U 1 1 5EAB22CD
-P 5000 4350
+P 4900 4350
 AR Path="/5E9E5DDE/5EAB22CD" Ref="R?"  Part="1"
 AR Path="/5E9E304D/5EAB22CD" Ref="R?"  Part="1"
@@
 AR Path="/5EA4676F/5EAB22CD" Ref="R33"  Part="1"
 AR Path="/5EA46A2B/5EAB22CD" Ref="R34"  Part="1"
-F 0 "R34" V 4793 4350 50  0000 C CNN
-F 1 "2.7k" V 4884 4350 50  0000 C CNN
-F 2 "Resistor_THT:R_Axial_DIN0207_L6.3mm_D2.5mm_P10.16mm_Horizontal" V 4930 4350 50  0001 C CNN
-F 3 "~" H 5000 4350 50  0001 C CNN
-	1    5000 4350
+F 0 "R34" V 4800 4350 50  0000 C CNN
+F 1 "2.7k" V 5000 4350 50  0000 C CNN
+F 2 "Resistor_THT:R_Axial_DIN0207_L6.3mm_D2.5mm_P10.16mm_Horizontal" V 4830 4350 50  0001 C CNN
+F 3 "~" H 4900 4350 50  0001 C CNN
+	1    4900 4350
 	0    1    1    0
 $EndComp
-Text GLabel 5400 4750 0    50   Input ~ 0
-VGND
 $Comp
 L Transistor_BJT:BC337 Q?
@@
 	1    0    0    -1
 $EndComp
-Text GLabel 5400 3450 0    50   Input ~ 0
-5V
 $Comp
 L Connector_Generic:Conn_01x02 J2
@@
 AR Path="/5EA4676F/5EAB22CE" Ref="J3"  Part="1"
 AR Path="/5EA46A2B/5EAB22CE" Ref="J4"  Part="1"
-F 0 "J4" H 5750 3750 50  0000 C CNN
-F 1 "Conn_01x02" H 5600 3850 50  0000 C CNN
+F 0 "J4" H 5800 3800 50  0000 R CNN
+F 1 "Conn_01x02" H 5800 3900 50  0000 R CNN
 F 2 "Connector_Wire:SolderWirePad_1x02_P3.81mm_Drill1.2mm" H 5250 3900 50  0001 C CNN
 F 3 "~" H 5250 3900 50  0001 C CNN
@@
 $EndComp
 Wire Wire Line
-	5400 3450 5450 3450
+	5450 3900 5450 4150
 Wire Wire Line
-	5450 3450 5450 3800
+	5050 4350 5150 4350
+$Comp
+L power:+5V #PWR?
+U 1 1 5EC230EA
+P 5450 3750
+F 0 "#PWR?" H 5450 3600 50  0001 C CNN
+F 1 "+5V" H 5465 3923 50  0000 C CNN
+F 2 "" H 5450 3750 50  0001 C CNN
+F 3 "" H 5450 3750 50  0001 C CNN
+	1    5450 3750
+	1    0    0    -1
+$EndComp
 Wire Wire Line
-	5450 3900 5450 4150
+	5450 3750 5450 3800
+$Comp
+L power:GND #PWR?
+U 1 1 5EC23FDA
+P 5450 4650
+F 0 "#PWR?" H 5450 4400 50  0001 C CNN
+F 1 "GND" H 5455 4477 50  0000 C CNN
+F 2 "" H 5450 4650 50  0001 C CNN
+F 3 "" H 5450 4650 50  0001 C CNN
+	1    5450 4650
+	1    0    0    -1
+$EndComp
 $EndSCHEMATC

Commit message: Changed name of libraries to remove underscore
Changed lines of the file:
@@
 $Descr A4 11693 8268
 encoding utf-8
-Sheet 8 10
+Sheet 8 11
 Title ""
 Date ""
@@
 AR Path="/5EA4676F/5EAB22CD" Ref="R33"  Part="1"
 AR Path="/5EA46A2B/5EAB22CD" Ref="R34"  Part="1"
-F 0 "R34" V 4800 4350 50  0000 C CNN
+AR Path="/5ED17BA0/5ED2A32C/5EAB22CD" Ref="R?"  Part="1"
+F 0 "R?" V 4800 4350 50  0000 C CNN
 F 1 "2.7k" V 5000 4350 50  0000 C CNN
 F 2 "Resistor_THT:R_Axial_DIN0207_L6.3mm_D2.5mm_P10.16mm_Horizontal" V 4830 4350 50  0001 C CNN
@@
 AR Path="/5EA4676F/5E9E70EA" Ref="Q2"  Part="1"
 AR Path="/5EA46A2B/5E9E70EA" Ref="Q3"  Part="1"
-F 0 "Q3" H 5541 4396 50  0000 L CNN
+AR Path="/5ED17BA0/5ED2A32C/5E9E70EA" Ref="Q?"  Part="1"
+F 0 "Q?" H 5541 4396 50  0000 L CNN
 F 1 "BC337" H 5541 4305 50  0000 L CNN
 F 2 "Package_TO_SOT_THT:TO-92_Inline" H 5550 4275 50  0001 L CIN
@@
 AR Path="/5EA4676F/5EAB22CE" Ref="J3"  Part="1"
 AR Path="/5EA46A2B/5EAB22CE" Ref="J4"  Part="1"
-F 0 "J4" H 5800 3800 50  0000 R CNN
+AR Path="/5ED17BA0/5ED2A32C/5EAB22CE" Ref="J?"  Part="1"
+F 0 "J?" H 5800 3800 50  0000 R CNN
 F 1 "Conn_01x02" H 5800 3900 50  0000 R CNN
 F 2 "Connector_Wire:SolderWirePad_1x02_P3.81mm_Drill1.2mm" H 5250 3900 50  0001 C CNN

Commit message: Partial Update
Parts:
- removed Q1: BC337, Package_TO_SOT_THT:TO-92_Inline, symbol Transistor_BJT:BC337
- added Q3: BCW65ALT1G, Package_TO_SOT_SMD:SOT-23, symbol Frequently_Used:BCW65ALT1G
- R29: renamed from R32; footprint Resistor_THT:R_Axial_DIN0207_L6.3mm_D2.5mm_P10.16mm_Horizontal -> Frequently_Used:0805_2012Metric_HandSolder
- renumbered J2 to J3
Changed lines of the file:
@@
 $Descr A4 11693 8268
 encoding utf-8
-Sheet 8 11
+Sheet 9 11
 Title ""
 Date ""
@@
 AR Path="/5E9E5DE1/5EAB22CD" Ref="R?"  Part="1"
 AR Path="/5E9E4A6B/5EAB22CD" Ref="R?"  Part="1"
-AR Path="/5EA45E37/5EAB22CD" Ref="R32"  Part="1"
-AR Path="/5EA4676F/5EAB22CD" Ref="R33"  Part="1"
-AR Path="/5EA46A2B/5EAB22CD" Ref="R34"  Part="1"
-AR Path="/5ED17BA0/5ED2A32C/5EAB22CD" Ref="R?"  Part="1"
-F 0 "R?" V 4800 4350 50  0000 C CNN
+AR Path="/5EA45E37/5EAB22CD" Ref="R?"  Part="1"
+AR Path="/5EA4676F/5EAB22CD" Ref="R?"  Part="1"
+AR Path="/5EA46A2B/5EAB22CD" Ref="R?"  Part="1"
+AR Path="/5ED17BA0/5ED2A32C/5EAB22CD" Ref="R29"  Part="1"
+F 0 "R29" V 4800 4350 50  0000 C CNN
 F 1 "2.7k" V 5000 4350 50  0000 C CNN
-F 2 "Resistor_THT:R_Axial_DIN0207_L6.3mm_D2.5mm_P10.16mm_Horizontal" V 4830 4350 50  0001 C CNN
+F 2 "Frequently_Used:0805_2012Metric_HandSolder" V 4830 4350 50  0001 C CNN
 F 3 "~" H 4900 4350 50  0001 C CNN
 	1    4900 4350
@@
 $EndComp
 $Comp
-L Transistor_BJT:BC337 Q?
-U 1 1 5E9E70EA
-P 5350 4350
-AR Path="/5E9E5DDE/5E9E70EA" Ref="Q?"  Part="1"
-AR Path="/5E9E304D/5E9E70EA" Ref="Q?"  Part="1"
-AR Path="/5E9D240B/5E9E70EA" Ref="Q?"  Part="1"
-AR Path="/5E9E5DE1/5E9E70EA" Ref="Q?"  Part="1"
-AR Path="/5E9E4A6B/5E9E70EA" Ref="Q?"  Part="1"
-AR Path="/5EA45E37/5E9E70EA" Ref="Q1"  Part="1"
-AR Path="/5EA4676F/5E9E70EA" Ref="Q2"  Part="1"
-AR Path="/5EA46A2B/5E9E70EA" Ref="Q3"  Part="1"
-AR Path="/5ED17BA0/5ED2A32C/5E9E70EA" Ref="Q?"  Part="1"
-F 0 "Q?" H 5541 4396 50  0000 L CNN
-F 1 "BC337" H 5541 4305 50  0000 L CNN
-F 2 "Package_TO_SOT_THT:TO-92_Inline" H 5550 4275 50  0001 L CIN
-F 3 "https://diotec.com/tl_files/diotec/files/pdf/datasheets/bc337.pdf" H 5350 4350 50  0001 L CNN
-	1    5350 4350
-	1    0    0    -1
-$EndComp
-$Comp
-L Connector_Generic:Conn_01x02 J2
+L Connector_Generic:Conn_01x02 J?
 U 1 1 5EAB22CE
 P 5250 3900
-AR Path="/5EA45E37/5EAB22CE" Ref="J2"  Part="1"
-AR Path="/5EA4676F/5EAB22CE" Ref="J3"  Part="1"
-AR Path="/5EA46A2B/5EAB22CE" Ref="J4"  Part="1"
-AR Path="/5ED17BA0/5ED2A32C/5EAB22CE" Ref="J?"  Part="1"
-F 0 "J?" H 5800 3800 50  0000 R CNN
+AR Path="/5EA45E37/5EAB22CE" Ref="J?"  Part="1"
+AR Path="/5EA4676F/5EAB22CE" Ref="J?"  Part="1"
+AR Path="/5EA46A2B/5EAB22CE" Ref="J?"  Part="1"
+AR Path="/5ED17BA0/5ED2A32C/5EAB22CE" Ref="J3"  Part="1"
+F 0 "J3" H 5800 3800 50  0000 R CNN
 F 1 "Conn_01x02" H 5800 3900 50  0000 R CNN
 F 2 "Connector_Wire:SolderWirePad_1x02_P3.81mm_Drill1.2mm" H 5250 3900 50  0001 C CNN
@@
 	5050 4350 5150 4350
 $Comp
-L power:+5V #PWR?
+L power:+5V #PWR044
 U 1 1 5EC230EA
 P 5450 3750
-F 0 "#PWR?" H 5450 3600 50  0001 C CNN
+F 0 "#PWR044" H 5450 3600 50  0001 C CNN
 F 1 "+5V" H 5465 3923 50  0000 C CNN
 F 2 "" H 5450 3750 50  0001 C CNN
@@
 	5450 3750 5450 3800
 $Comp
-L power:GND #PWR?
+L power:GND #PWR045
 U 1 1 5EC23FDA
 P 5450 4650
-F 0 "#PWR?" H 5450 4400 50  0001 C CNN
+F 0 "#PWR045" H 5450 4400 50  0001 C CNN
 F 1 "GND" H 5455 4477 50  0000 C CNN
 F 2 "" H 5450 4650 50  0001 C CNN
@@
 	1    0    0    -1
 $EndComp
+$Comp
+L Frequently_Used:BCW65ALT1G Q3
+U 1 1 5EE768A7
+P 5350 4350
+F 0 "Q3" H 5541 4396 50  0000 L CNN
+F 1 "BCW65ALT1G" H 5541 4305 50  0000 L CNN
+F 2 "Package_TO_SOT_SMD:SOT-23" H 5400 3700 50  0001 C CIN
+F 3 "https://www.onsemi.com/pub/Collateral/BCW65ALT1-D.PDF" H 5350 4350 50  0001 L CNN
+F 4 "ON Semiconductor" H 5400 3600 50  0001 C CNN "Manufacturer Name"
+F 5 "BCW65ALT1G" H 5400 3900 50  0001 C CNN "Manufacturer Part No."
+F 6 "488-BCW65ALT1GCT-ND" H 5400 3800 50  0001 C CNN "Digikey Part No."
+	1    5350 4350
+	1    0    0    -1
+$EndComp

Commit message: Adding Power Daughter Board
Parts:
- Q3: Digikey Part No. 488-BCW65ALT1GCT-ND -> (none); Source Part No. (none) -> 488-BCW65ALT1GCT-ND
Changed lines of the file:
@@
 F 4 "ON Semiconductor" H 5400 3600 50  0001 C CNN "Manufacturer Name"
 F 5 "BCW65ALT1G" H 5400 3900 50  0001 C CNN "Manufacturer Part No."
-F 6 "488-BCW65ALT1GCT-ND" H 5400 3800 50  0001 C CNN "Digikey Part No."
+F 6 "488-BCW65ALT1GCT-ND" H 5400 3800 50  0001 C CNN "Source Part No."
 	1    5350 4350
 	1    0    0    -1

Commit message: Move libraries and added configuration path.
Moved Li-Ion library to common KiCad library.  Added variables to configuration paths to reference my KiCad libraries.  Moved all 3D components to my common library.
Parts:
- Q3: symbol Frequently_Used:BCW65ALT1G -> Frequently_Used_LE:BCW65ALT1G
- R29: footprint Frequently_Used:0805_2012Metric_HandSolder -> FrequentlyUsed:0805_2012Metric_HandSolder
Changed lines of the file:
@@
 F 0 "R29" V 4800 4350 50  0000 C CNN
 F 1 "2.7k" V 5000 4350 50  0000 C CNN
-F 2 "Frequently_Used:0805_2012Metric_HandSolder" V 4830 4350 50  0001 C CNN
+F 2 "FrequentlyUsed:0805_2012Metric_HandSolder" V 4830 4350 50  0001 C CNN
 F 3 "~" H 4900 4350 50  0001 C CNN
 	1    4900 4350
@@
 $EndComp
 $Comp
-L Frequently_Used:BCW65ALT1G Q3
+L Frequently_Used_LE:BCW65ALT1G Q3
 U 1 1 5EE768A7
 P 5350 4350

Commit message: Separated digital and analog ground.
Connections:
- net labels added: GNDD
- net labels removed: GND
Changed lines of the file:
@@
 	5450 3750 5450 3800
 $Comp
-L power:GND #PWR045
+L power:GNDD #PWR045
 U 1 1 5EC23FDA
 P 5450 4650
 F 0 "#PWR045" H 5450 4400 50  0001 C CNN
-F 1 "GND" H 5455 4477 50  0000 C CNN
+F 1 "GNDD" H 5455 4477 50  0000 C CNN
 F 2 "" H 5450 4650 50  0001 C CNN
 F 3 "" H 5450 4650 50  0001 C CNN

Commit message: Audio update
Parts:
- R29: footprint FrequentlyUsed:0805_2012Metric_HandSolder -> Frequently_Used_LE:0805_2012Metric_HandSolder
Changed lines of the file:
@@
 F 0 "R29" V 4800 4350 50  0000 C CNN
 F 1 "2.7k" V 5000 4350 50  0000 C CNN
-F 2 "FrequentlyUsed:0805_2012Metric_HandSolder" V 4830 4350 50  0001 C CNN
+F 2 "Frequently_Used_LE:0805_2012Metric_HandSolder" V 4830 4350 50  0001 C CNN
 F 3 "~" H 4900 4350 50  0001 C CNN
 	1    4900 4350
