File: Naquadah Generator Main/Audio.sch (KiCad schematic (older format))
At the start: 1 part, among them U7 VS1000

Commit message: Start of audio
Parts:
- added C? (x2): 22pF, FrequentlyUsed:0805_2012Metric_HandSolder, symbol Frequently_Used_LE:C
- added R?: 1M, symbol Frequently_Used_LE:R
- added Y?: 12MHz, Naquadah_Generator:Oscillator_ABM3-16.000MHZ-B2-T, symbol Frequently_Used_LE:Crystal
Connections:
- net labels added: GND, GNDA, GNDD, XTALI, XTALO
- wire segments 3 -> 33
Changed lines of the file:
@@
 Comment4 ""
 $EndDescr
+Wire Wire Line
+	5200 2500 4750 2500
+Wire Wire Line
+	6450 4050 6900 4050
+Wire Wire Line
+	6450 4150 6900 4150
+Text HLabel 4750 2500 0    50   Input ~ 0
+RESET
+Text HLabel 6900 4050 2    50   Input ~ 0
+RX
+Text HLabel 6900 4150 2    50   Input ~ 0
+TX
+$Comp
+L Frequently_Used_LE:C C?
+U 1 1 5F255A01
+P 1600 1300
+AR Path="/5F255A01" Ref="C?"  Part="1"
+AR Path="/5F06C1CA/5F255A01" Ref="C?"  Part="1"
+F 0 "C?" V 1650 1250 50  0000 R CNN
+F 1 "22pF" V 1650 1350 50  0000 L CNN
+F 2 "FrequentlyUsed:0805_2012Metric_HandSolder" H 1638 1150 50  0001 C CNN
+F 3 "" H 1600 1300 50  0001 C CNN
+F 4 "" H 1600 1300 50  0001 C CNN "Source Part No."
+F 5 "" H 1600 1300 50  0001 C CNN "Manufacturer Name"
+F 6 "" H 1600 1300 50  0001 C CNN "Manufacturer Part No."
+F 7 "Digikey" H 1600 1300 50  0001 C CNN "Source"
+	1    1600 1300
+	0    1    1    0
+$EndComp
+$Comp
+L Frequently_Used_LE:C C?
+U 1 1 5F255A0B
+P 1600 1000
+AR Path="/5F255A0B" Ref="C?"  Part="1"
+AR Path="/5F06C1CA/5F255A0B" Ref="C?"  Part="1"
+F 0 "C?" V 1550 950 50  0000 R CNN
+F 1 "22pF" V 1550 1050 50  0000 L CNN
+F 2 "FrequentlyUsed:0805_2012Metric_HandSolder" H 1638 850 50  0001 C CNN
+F 3 "" H 1600 1000 50  0001 C CNN
+F 4 "" H 1600 1000 50  0001 C CNN "Source Part No."
+F 5 "" H 1600 1000 50  0001 C CNN "Manufacturer Name"
+F 6 "" H 1600 1000 50  0001 C CNN "Manufacturer Part No."
+F 7 "Digikey" H 1600 1000 50  0001 C CNN "Source"
+	1    1600 1000
+	0    1    1    0
+$EndComp
+$Comp
+L Frequently_Used_LE:Crystal Y?
+U 1 1 5F255A16
+P 1900 1150
+AR Path="/5F255A16" Ref="Y?"  Part="1"
+AR Path="/5F06C1CA/5F255A16" Ref="Y?"  Part="1"
+F 0 "Y?" H 1900 1000 50  0000 C CNN
+F 1 "12MHz" H 1900 1300 50  0000 C CNN
+F 2 "Naquadah_Generator:Oscillator_ABM3-16.000MHZ-B2-T" H 1900 1150 50  0001 C CNN
+F 3 "https://abracon.com/Resonators/abm3.pdf" H 1900 1150 50  0001 C CNN
+F 4 "535-9103-1-ND" H 1900 1150 50  0001 C CNN "Source Part No."
+F 5 "Abracon " H 1900 1150 50  0001 C CNN "Manufacturer Name"
+F 6 "ABM3-16.000MHZ-B2-T" H 1900 1150 50  0001 C CNN "Manufacturer Part No."
+F 7 "Abracon LLC" H 1900 1150 50  0001 C CNN "Description"
+F 8 "Digikey" H 1900 1150 50  0001 C CNN "Source"
+	1    1900 1150
+	0    1    1    0
+$EndComp
+Wire Wire Line
+	1750 1000 1900 1000
+Connection ~ 1900 1000
+Wire Wire Line
+	1900 1000 2250 1000
+Wire Wire Line
+	1750 1300 1900 1300
+Wire Wire Line
+	1900 1300 2250 1300
+Wire Wire Line
+	1450 1300 1350 1300
+Wire Wire Line
+	1350 1300 1350 1150
+Wire Wire Line
+	1350 1000 1450 1000
+Wire Wire Line
+	1350 1150 1150 1150
+Wire Wire Line
+	1150 1150 1150 1250
+Connection ~ 1350 1150
+Wire Wire Line
+	1350 1150 1350 1000
+$Comp
+L Frequently_Used_LE:GND #PWR?
+U 1 1 5F255A2A
+P 1150 1250
+AR Path="/5F255A2A" Ref="#PWR?"  Part="1"
+AR Path="/5F06C1CA/5F255A2A" Ref="#PWR?"  Part="1"
+F 0 "#PWR?" H 1150 1000 50  0001 C CNN
+F 1 "GND" H 1150 1100 50  0000 C CNN
+F 2 "" H 1150 1250 50  0001 C CNN
+F 3 "" H 1150 1250 50  0001 C CNN
+	1    1150 1250
+	1    0    0    -1
+$EndComp
+Text Label 2700 1300 2    50   ~ 0
+XTALO
+Text Label 4700 2700 0    50   ~ 0
+XTALI
+Text Label 4700 2800 0    50   ~ 0
+XTALO
+Text Label 2700 1000 2    50   ~ 0
+XTALI
+Connection ~ 1900 1300
+$Comp
+L Frequently_Used_LE:R R?
+U 1 1 5F25855F
+P 2250 1150
+F 0 "R?" H 2320 1196 50  0000 L CNN
+F 1 "1M" H 2320 1105 50  0000 L CNN
+F 2 "" V 2180 1150 50  0001 C CNN
+F 3 "" H 2250 1150 50  0001 C CNN
+	1    2250 1150
+	1    0    0    -1
+$EndComp
+Connection ~ 2250 1000
+Wire Wire Line
+	2250 1000 2700 1000
+Connection ~ 2250 1300
+Wire Wire Line
+	2250 1300 2700 1300
+Wire Wire Line
+	4450 2600 4450 2700
+Wire Wire Line
+	4700 2700 5200 2700
+Wire Wire Line
+	4700 2800 5200 2800
+Wire Wire Line
+	4450 2600 5200 2600
 $Comp
 L Audio~LE:VS1000 U7
@@
 $EndComp
 Wire Wire Line
-	5200 2500 4750 2500
-Wire Wire Line
-	6450 4050 6900 4050
-Wire Wire Line
-	6450 4150 6900 4150
-Text HLabel 4750 2500 0    50   Input ~ 0
-RESET
-Text HLabel 6900 4050 2    50   Input ~ 0
-RX
-Text HLabel 6900 4150 2    50   Input ~ 0
-TX
+	4700 4800 4700 4900
+Wire Wire Line
+	4700 5000 5200 5000
+Connection ~ 4700 4900
+Wire Wire Line
+	4700 4900 4700 5000
+Wire Wire Line
+	4700 5000 4700 5100
+Connection ~ 4700 5000
+Wire Wire Line
+	5200 4800 4700 4800
+Wire Wire Line
+	5200 4900 4700 4900
+Wire Wire Line
+	5200 4400 4450 4400
+Wire Wire Line
+	4450 4700 5200 4700
+Wire Wire Line
+	5200 4600 4450 4600
+Connection ~ 4450 4600
+Wire Wire Line
+	4450 4600 4450 4700
+Wire Wire Line
+	5200 4500 4450 4500
+Wire Wire Line
+	4450 4400 4450 4500
+Connection ~ 4450 4500
+Wire Wire Line
+	4450 4500 4450 4600
+Wire Wire Line
+	4450 4700 4450 4800
+Connection ~ 4450 4700
+$Comp
+L Frequently_Used_LE:GNDA #PWR?
+U 1 1 5F265ADA
+P 4450 4800
+F 0 "#PWR?" H 4450 4550 50  0001 C CNN
+F 1 "GNDA" H 4455 4627 50  0000 C CNN
+F 2 "" H 4450 4800 50  0001 C CNN
+F 3 "" H 4450 4800 50  0001 C CNN
+	1    4450 4800
+	1    0    0    -1
+$EndComp
+$Comp
+L Frequently_Used_LE:GNDD #PWR?
+U 1 1 5F2663C3
+P 4450 2700
+F 0 "#PWR?" H 4450 2450 50  0001 C CNN
+F 1 "GNDD" H 4455 2527 50  0000 C CNN
+F 2 "" H 4450 2700 50  0001 C CNN
+F 3 "" H 4450 2700 50  0001 C CNN
+	1    4450 2700
+	1    0    0    -1
+$EndComp
+$Comp
+L Frequently_Used_LE:GNDD #PWR?
+U 1 1 5F266BA0
+P 4700 5100
+F 0 "#PWR?" H 4700 4850 50  0001 C CNN
+F 1 "GNDD" H 4705 4927 50  0000 C CNN
+F 2 "" H 4700 5100 50  0001 C CNN
+F 3 "" H 4700 5100 50  0001 C CNN
+	1    4700 5100
+	1    0    0    -1
+$EndComp
 $EndSCHEMATC

Commit message: Separated digital and analog ground.
Parts:
- added L?: Ferrite, symbol Device:L_Core_Ferrite_Small
Connections:
- wire segments 33 -> 35
Changed lines of the file:
@@
 	1    0    0    -1
 $EndComp
+$Comp
+L Frequently_Used_LE:GNDD #PWR?
+U 1 1 5F28FF9A
+P 3050 4750
+F 0 "#PWR?" H 3050 4500 50  0001 C CNN
+F 1 "GNDD" H 3055 4577 50  0000 C CNN
+F 2 "" H 3050 4750 50  0001 C CNN
+F 3 "" H 3050 4750 50  0001 C CNN
+	1    3050 4750
+	1    0    0    -1
+$EndComp
+$Comp
+L Frequently_Used_LE:GNDA #PWR?
+U 1 1 5F29074F
+P 2550 4750
+F 0 "#PWR?" H 2550 4500 50  0001 C CNN
+F 1 "GNDA" H 2555 4577 50  0000 C CNN
+F 2 "" H 2550 4750 50  0001 C CNN
+F 3 "" H 2550 4750 50  0001 C CNN
+	1    2550 4750
+	1    0    0    -1
+$EndComp
+$Comp
+L Device:L_Core_Ferrite_Small L?
+U 1 1 5F291B0D
+P 2800 4750
+F 0 "L?" V 2619 4750 50  0000 C CNN
+F 1 "Ferrite" V 2710 4750 50  0000 C CNN
+F 2 "" H 2800 4750 50  0001 C CNN
+F 3 "~" H 2800 4750 50  0001 C CNN
+	1    2800 4750
+	0    1    1    0
+$EndComp
+Wire Wire Line
+	2550 4750 2700 4750
+Wire Wire Line
+	2900 4750 3050 4750
 $EndSCHEMATC

Commit message: Audio update
Parts:
- added C20, C?: 1.0uF, Frequently_Used_LE:0805_2012Metric_HandSolder, symbol Frequently_Used_LE:C
- added C21: 0.1uF, Frequently_Used_LE:0805_2012Metric_HandSolder, symbol Frequently_Used_LE:C
- added JP1, JP3: Open, Jumper_LE:SolderJumper-2_P1.3mm_Open_RoundedPad1.0x1.5mm, symbol Jumper:SolderJumper_2_Open
- added JP2: Bridged, Jumper_LE:SolderJumper-2_P1.3mm_Bridged_RoundedPad1.0x1.5mm, symbol Jumper:SolderJumper_2_Bridged
- added L2: Ferrite, symbol Device:L_Core_Ferrite_Small
- added R39, R42, R43, R44, R45, R46, R? (x9): 100k, Frequently_Used_LE:0805_2012Metric_HandSolder, symbol Frequently_Used_LE:R
- added R47: 1M, Frequently_Used_LE:0805_2012Metric_HandSolder, symbol Frequently_Used_LE:R
- added TP12, TP13: TestPoint, Frequently_Used_LE:Pad_2.5-2.5, symbol Frequently_Used_LE:TestPoint
- added U9: MX25L1606EM1I-12G, Package_SO:SOP-8_3.9x4.9mm_P1.27mm, symbol Memory~LE:MX25L1606EM1I-12G
- C10, C16: renamed from C?; footprint FrequentlyUsed:0805_2012Metric_HandSolder -> Frequently_Used_LE:0805_2012Metric_HandSolder
- R37: renamed from R?; footprint (none) -> Frequently_Used_LE:0805_2012Metric_HandSolder; Description (none) -> 1 MOhms ±1% 0.25W, 1/4W Chip Resistor 0805 (2012 Metric); Manufacturer Name (none) -> KOA Speer Electronics, Inc.; Manufacturer Part No. (none) -> RK73H2ATTD1004F; Source (none) -> Digikey; Source Part No. (none) -> 2019-RK73H2ATTD1004FCT-ND
- U7: symbol Audio~LE:VS1000 -> Audio_LE:VS1000
- gave numbers to parts that had none: 2
Connections:
- net labels added: +3.3V, +5V, AGND, AVDD, CVDD, DGND, IO_0, IO_1, IO_2, IO_3, IO_4, IO_5, IO_6, IO_7, MISO, MOSI, SCLK, SDCD, SDCLK, SDDI, SDDO, SDXCS, VSRX, XCS
- net labels removed: GND, GNDA, GNDD
- wire segments 35 -> 158
Other:
- note added: "Crystal"
- note added: "Flash Memory"
- note added: "Pull Up and Pull Down"
- moved on the sheet: L3

Commit message: Power updates
Parts:
- added C23, C24: 1UF, Frequently_Used_LE:0805_2012Metric_HandSolder, symbol Frequently_Used_LE:C
- added C25, C28, C29: 1.0uF, Frequently_Used_LE:0805_2012Metric_HandSolder, symbol Frequently_Used_LE:C
- added C26, C27, C33: 22pF, Frequently_Used_LE:0805_2012Metric_HandSolder, symbol Frequently_Used_LE:C
- added C34: 10uF, Frequently_Used_LE:0805_2012Metric_HandSolder, symbol Frequently_Used_LE:C
- added C35: 47nF, Frequently_Used_LE:0805_2012Metric_HandSolder, symbol Frequently_Used_LE:C
- added D28: YELLOW, Frequently_Used_LE:LED_0805_2012Metric_HandSolder, symbol Frequently_Used_LE:LED
- added L4, L5: Ferrite, symbol Device:L_Core_Ferrite_Small
- added R57, R61: 100k, Frequently_Used_LE:0805_2012Metric_HandSolder, symbol Frequently_Used_LE:R
- added R58, R59: 100, Frequently_Used_LE:0805_2012Metric_HandSolder, symbol Frequently_Used_LE:R
- added R60: 10k, Frequently_Used_LE:0805_2012Metric_HandSolder, symbol Frequently_Used_LE:R
- added R62: 470, Frequently_Used_LE:0805_2012Metric_HandSolder, symbol Frequently_Used_LE:R
- added R63: 10, Frequently_Used_LE:0805_2012Metric_HandSolder, symbol Frequently_Used_LE:R
- added RV1: 10k, symbol Device:R_POT
- added U10: PAM8302AAD, Package_SO:SOP-8_3.9x4.9mm_P1.27mm, symbol Amplifier_Audio:PAM8302AAD
- TP12, TP13: symbol Frequently_Used_LE:TestPoint -> Frequently_Used_LE:TestPoint_1
- U9: footprint Package_SO:SOP-8_3.9x4.9mm_P1.27mm -> Package_SO_LE:SOP-8_3.9x4.9mm_P1.27mm; symbol Memory~LE:MX25L1606EM1I-12G -> Memory_LE:MX25L1606EM1I-12G
- gave numbers to parts that had none: 10
Connections:
- net labels added: AO+, AO-, AUDLEFT, AUDPRE+, CBUF, POWBTN, RCAP
- wire segments 158 -> 213
- no-connect marks 0 -> 1
Other:
- note added: "Amplifier"
- note added: "Audio"
- note added: "Audio IC"
- note added: "Decoupling"
- note added: "Digital to Analog Connections"
- note added: "Power"
- note added: "Reset"
- moved on the sheet: C10, C16, C20, C21, C22, JP1, JP2, JP3, L2, L3, R37, R39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

Commit message: Fixed analog  and digital power symbol names.
Parts:
- L2, L3, L4, L5: footprint (none) -> Frequently_Used_LE:0603_1608Metric; Description (none) -> 120 Ohms @ 100MHz 1 Ferrite Bead 0603 (1608 Metric) 800mA 1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; Manufacturer Name (none) -> Murata Electronics; Manufacturer Part No. (none) -> BLM18AG121SN1D; Source (none) -> Digikey; Source Part No. (none) -> 490-1011-1-ND
Changed lines of the file:
@@
 F 0 "L3" V 1369 7150 50  0000 C CNN
 F 1 "Ferrite" V 1460 7150 50  0000 C CNN
-F 2 "" H 1550 7150 50  0001 C CNN
-F 3 "~" H 1550 7150 50  0001 C CNN
+F 2 "Frequently_Used_LE:0603_1608Metric" H 1550 7150 50  0001 C CNN
+F 3 "https://www.murata.com/en-us/products/productdata/8796738650142/ENFA0003.pdf" H 1550 7150 50  0001 C CNN
+F 4 "120 Ohms @ 100MHz 1 Ferrite Bead 0603 (1608 Metric) 800mA 180mOhm" H 1550 7150 50  0001 C CNN "Description"
+F 5 "Murata Electronics" H 1550 7150 50  0001 C CNN "Manufacturer Name"
+F 6 "BLM18AG121SN1D" H 1550 7150 50  0001 C CNN "Manufacturer Part No."
+F 7 "Digikey" H 1550 7150 50  0001 C CNN "Source"
+F 8 "490-1011-1-ND" H 1550 7150 50  0001 C CNN "Source Part No."
 	1    1550 7150
 	0    1    1    0
@@
 F 0 "L2" V 1369 6200 50  0000 C CNN
 F 1 "Ferrite" V 1460 6200 50  0000 C CNN
-F 2 "" H 1550 6200 50  0001 C CNN
-F 3 "~" H 1550 6200 50  0001 C CNN
+F 2 "Frequently_Used_LE:0603_1608Metric" H 1550 6200 50  0001 C CNN
+F 3 "https://www.murata.com/en-us/products/productdata/8796738650142/ENFA0003.pdf" H 1550 6200 50  0001 C CNN
+F 4 "120 Ohms @ 100MHz 1 Ferrite Bead 0603 (1608 Metric) 800mA 180mOhm" H 1550 6200 50  0001 C CNN "Description"
+F 5 "Murata Electronics" H 1550 6200 50  0001 C CNN "Manufacturer Name"
+F 6 "BLM18AG121SN1D" H 1550 6200 50  0001 C CNN "Manufacturer Part No."
+F 7 "Digikey" H 1550 6200 50  0001 C CNN "Source"
+F 8 "490-1011-1-ND" H 1550 6200 50  0001 C CNN "Source Part No."
 	1    1550 6200
 	0    1    1    0
@@
 $EndComp
 $Comp
-L Frequently_Used_LE:AGND #PWR
+L Frequently_Used_LE:AGND #PWR0136
 U 1 1 5F9072C6
 P 5650 7050
-F 0 "#PWR" H 5650 6800 50  0001 C CNN
+F 0 "#PWR0136" H 5650 6800 50  0001 C CNN
 F 1 "AGND" H 5650 6900 50  0000 C CNN
 F 2 "" H 5650 7050 50  0001 C CNN
@@
 F 0 "L4" V 5400 6500 50  0000 C CNN
 F 1 "Ferrite" V 5550 6500 50  0000 C CNN
-F 2 "" H 5450 6500 50  0001 C CNN
-F 3 "~" H 5450 6500 50  0001 C CNN
+F 2 "Frequently_Used_LE:0603_1608Metric" H 5450 6500 50  0001 C CNN
+F 3 "https://www.murata.com/en-us/products/productdata/8796738650142/ENFA0003.pdf" H 5450 6500 50  0001 C CNN
+F 4 "120 Ohms @ 100MHz 1 Ferrite Bead 0603 (1608 Metric) 800mA 180mOhm" H 5450 6500 50  0001 C CNN "Description"
+F 5 "Murata Electronics" H 5450 6500 50  0001 C CNN "Manufacturer Name"
+F 6 "BLM18AG121SN1D" H 5450 6500 50  0001 C CNN "Manufacturer Part No."
+F 7 "Digikey" H 5450 6500 50  0001 C CNN "Source"
+F 8 "490-1011-1-ND" H 5450 6500 50  0001 C CNN "Source Part No."
 	1    5450 6500
 	0    1    1    0
@@
 F 0 "L5" V 5800 6300 50  0000 C CNN
 F 1 "Ferrite" V 5950 6300 50  0000 C CNN
-F 2 "" H 5850 6300 50  0001 C CNN
-F 3 "~" H 5850 6300 50  0001 C CNN
+F 2 "Frequently_Used_LE:0603_1608Metric" H 5850 6300 50  0001 C CNN
+F 3 "https://www.murata.com/en-us/products/productdata/8796738650142/ENFA0003.pdf" H 5850 6300 50  0001 C CNN
+F 4 "120 Ohms @ 100MHz 1 Ferrite Bead 0603 (1608 Metric) 800mA 180mOhm" H 5850 6300 50  0001 C CNN "Description"
+F 5 "Murata Electronics" H 5850 6300 50  0001 C CNN "Manufacturer Name"
+F 6 "BLM18AG121SN1D" H 5850 6300 50  0001 C CNN "Manufacturer Part No."
+F 7 "Digikey" H 5850 6300 50  0001 C CNN "Source"
+F 8 "490-1011-1-ND" H 5850 6300 50  0001 C CNN "Source Part No."
 	1    5850 6300
 	0    1    1    0

Commit message: Before switching buttons on daughter board
Other:
- moved on the sheet: C20, C21
Changed lines of the file:
@@
 L Frequently_Used_LE:C C?
 U 1 1 5F3A06EA
-P 8750 1000
+P 9200 1000
 AR Path="/5F3A06EA" Ref="C?"  Part="1"
 AR Path="/5F06C1CA/5F3A06EA" Ref="C20"  Part="1"
-F 0 "C20" H 8900 1100 50  0000 R CNN
-F 1 "1.0uF" H 8800 900 50  0000 L CNN
+F 0 "C20" H 9350 1100 50  0000 R CNN
+F 1 "1.0uF" H 9250 900 50  0000 L CNN
+F 2 "Frequently_Used_LE:0805_2012Metric_HandSolder" H 9238 850 50  0001 C CNN
+F 3 "" H 9200 1000 50  0001 C CNN
+F 4 "" H 9200 1000 50  0001 C CNN "Source Part No."
+F 5 "" H 9200 1000 50  0001 C CNN "Manufacturer Name"
+F 6 "" H 9200 1000 50  0001 C CNN "Manufacturer Part No."
+F 7 "Digikey" H 9200 1000 50  0001 C CNN "Source"
+	1    9200 1000
+	1    0    0    -1
+$EndComp
+Wire Wire Line
+	8750 1250 8750 1150
+$Comp
+L Frequently_Used_LE:C C?
+U 1 1 5F3A6FC5
+P 8750 1000
+AR Path="/5F3A6FC5" Ref="C?"  Part="1"
+AR Path="/5F06C1CA/5F3A6FC5" Ref="C21"  Part="1"
+F 0 "C21" H 8900 1100 50  0000 R CNN
+F 1 "0.1uF" H 8800 900 50  0000 L CNN
 F 2 "Frequently_Used_LE:0805_2012Metric_HandSolder" H 8788 850 50  0001 C CNN
 F 3 "" H 8750 1000 50  0001 C CNN
@@
 	1    0    0    -1
 $EndComp
-Wire Wire Line
-	8750 1250 8750 1150
-$Comp
-L Frequently_Used_LE:C C?
-U 1 1 5F3A6FC5
-P 9200 1000
-AR Path="/5F3A6FC5" Ref="C?"  Part="1"
-AR Path="/5F06C1CA/5F3A6FC5" Ref="C21"  Part="1"
-F 0 "C21" H 9350 1100 50  0000 R CNN
-F 1 "0.1uF" H 9250 900 50  0000 L CNN
-F 2 "Frequently_Used_LE:0805_2012Metric_HandSolder" H 9238 850 50  0001 C CNN
-F 3 "" H 9200 1000 50  0001 C CNN
-F 4 "" H 9200 1000 50  0001 C CNN "Source Part No."
-F 5 "" H 9200 1000 50  0001 C CNN "Manufacturer Name"
-F 6 "" H 9200 1000 50  0001 C CNN "Manufacturer Part No."
-F 7 "Digikey" H 9200 1000 50  0001 C CNN "Source"
-	1    9200 1000
-	1    0    0    -1
-$EndComp

Commit message: Audio updates, switching to separate USB schematic
Audio updates, switching to separate USB schematic
Parts:
- removed R48, R49, R50, R51, R52, R55: 100k, Frequently_Used_LE:0805_2012Metric_HandSolder, symbol Frequently_Used_LE:R
- U10: symbol Amplifier_Audio:PAM8302AAD -> Amplifier_Audio_LE:PAM8302AAD
Connections:
- net labels added: D+, D-, VBUS
- net labels removed: SDCD, SDCLK, SDDI, SDDO, SDXCS, VSRX
- wire segments 213 -> 209
- no-connect marks 1 -> 8
Other:
- note added: "Pull Down"
- note added: "Pull Up"
- note added: "VS1000 USB"
- note removed: "Pull Up and Pull Down"
- moved on the sheet: C10, C16, C20, C21, C22, C29, C33, C34, D28, JP1, JP2, JP3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
