File: Naquadah Generator Main/Boost 3.0A 5V 0805_2012.sch (KiCad schematic (older format))
At the start: 14 parts, among them U8 PAM2421AECADJR

Commit message: Audio updates, switching to separate USB schematic
Audio updates, switching to separate USB schematic
Connections:
- wire segments 62 -> 60
Changed lines of the file:
@@
 $Descr A 11000 8500
 encoding utf-8
-Sheet 12 15
+Sheet 12 16
 Title "Li-ion 3A Charge"
 Date ""
@@
 Text Notes 4850 4400 0    79   ~ 16
 3.0A 5V Boost
-$Comp
-L power:PWR_FLAG #FLG07
-U 1 1 5EC7BC40
-P 3950 2750
-F 0 "#FLG07" H 3950 2825 50  0001 C CNN
-F 1 "PWR_FLAG" H 3950 2923 50  0000 C CNN
-F 2 "" H 3950 2750 50  0001 C CNN
-F 3 "~" H 3950 2750 50  0001 C CNN
-	1    3950 2750
-	1    0    0    -1
-$EndComp
-Wire Wire Line
-	3950 2750 3950 2800
 Wire Wire Line
 	5900 3950 5900 4000
@@
 	-1   0    0    1
 $EndComp
-Connection ~ 3950 2800
 $Comp
 L Frequently_Used_LE:L L1
@@
 Wire Wire Line
 	4750 2800 5050 2800
-Wire Wire Line
-	3950 2800 4750 2800
 Connection ~ 4750 2800
 Wire Wire Line
@@
 Wire Wire Line
 	4750 3350 4750 3200
-Wire Wire Line
-	3750 2800 3950 2800
 Connection ~ 3750 2800
 Wire Wire Line
@@
 Text HLabel 7150 4000 2    50   Input ~ 0
 GND
+Wire Wire Line
+	3750 2800 4750 2800
 $EndSCHEMATC

Commit message: Switched to 0603_1608M size for passives
Parts:
- C12, C18: footprint Frequently_Used_LE:0805_2012Metric -> Frequently_Used_LE:0603_1608Metric; Description 10µF ±10% 6.3V Ceramic Capacitor X5R 0805 (2012 Metric) -> 10µF ±20% 6.3V Ceramic Capacitor X5R 0603 (1608 Metric); Manufacturer Part No. CL21A106KQCLRNC -> CL10A106MQ8NNNC; Source Part No. 1276-2405-1-ND -> 1276-1119-1-ND
- C13: footprint Frequently_Used_LE:0805_2012Metric -> Frequently_Used_LE:0603_1608Metric; Description 2200pF ±10% 50V Ceramic Capacitor X7R 0805 (2012 Metric) -> 2200pF ±10% 50V Ceramic Capacitor X7R 0603 (1608 Metric); Manufacturer Part No. CL21B222KBANNNC -> CL10B222KB8NNNC; Source Part No. 1276-1171-1-ND -> 1276-1110-1-ND
- C14: footprint Frequently_Used_LE:0805_2012Metric -> Frequently_Used_LE:0603_1608Metric; Description 1µF ±10% 16V Ceramic Capacitor X7R 0805 (2012 Metric) -> 1µF ±10% 10V Ceramic Capacitor X5R 0603 (1608 Metric); Manufacturer Part No. CL21B105KOFNNWE -> CL10A105KP8NNNC; Source Part No. 1276-2931-1-ND -> 1276-1182-1-ND
- C15: footprint Frequently_Used_LE:0805_2012Metric -> Frequently_Used_LE:0603_1608Metric; Description 47pF ±5% 50V Ceramic Capacitor C0G, NP0 0805 (2012 Metric) -> 47pF ±5% 50V Ceramic Capacitor C0G, NP0 0603 (1608 Metric); Manufacturer Part No. CL21C470JBANNNC -> CL10C470JB8NNNC; Source Part No. 1276-1156-1-ND -> 1276-1037-1-ND
- C17: footprint Frequently_Used_LE:0805_2012Metric -> Frequently_Used_LE:0603_1608Metric; Description 10000pF ±10% 50V Ceramic Capacitor X7R 0805 (2012 Metric) -> 10000pF ±10% 50V Ceramic Capacitor X7R 0603 (1608 Metric); Manufacturer Part No. CL21B103KBANNNC -> CL10B103KB8NNNC; Source Part No. 1276-1015-1-ND -> 1276-1009-1-ND
- R38: footprint Frequently_Used_LE:0805_2012Metric -> Frequently_Used_LE:0603_1608Metric; Description 51 kOhms ±1% 0.25W, 1/4W Chip Resistor 1206 (3216 Metric) -> 100 Ohms ±1% 0.1W, 1/10W Chip Resistor 0603 (1608 Metric) T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; Manufacturer Name KOA Speer Electronics, Inc. -> Yageo; Manufacturer Part No. RK73H2ATTD5102F -> RC0603FR-07100RL; Source Part No. 2019-RK73H2ATTD5102FCT-ND -> 311-100HRCT-ND
- R40: footprint Frequently_Used_LE:0805_2012Metric -> Frequently_Used_LE:0603_1608Metric; Description 30 kOhms ±1% 0.25W, 1/4W Chip Resistor 1206 (3216 Metric) -> 30 kOhms ±1% 0.1W, 1/10W Chip Resistor 0603 (1608 Metric) A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; Manufacturer Name KOA Speer Electronics, Inc. -> Vishay Dale; Manufacturer Part No. RK73H2ATTD3002F -> CRCW060330K0FKEA; Source Part No. 2019-RK73H2ATTD3002FCT-ND -> 541-30.0KHCT-ND
- R41: footprint Frequently_Used_LE:0805_2012Metric -> Frequently_Used_LE:0603_1608Metric; Description 10 kOhms ±1% 0.25W, 1/4W Chip Resistor 1206 (3216 Metric) -> 10 kOhms ±1% 0.25W, 1/4W Chip Resistor 0603 (1608 Metric) A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; Manufacturer Name KOA Speer Electronics, Inc. -> Rohm Semiconductor; Manufacturer Part No. RK73H2ATTD1002F -> ESR03EZPF1002; Source Part No. 2019-RK73H2ATTD1002FCT-ND -> RHM10KADCT-ND
