File: Power Daughter Board/Power Daughter Board.sch (KiCad schematic (older format))
At the start: 29 parts, among them J1 End_Sphere_Conn, J2 Jack-DC, SW1 MHPS2283, U1 MCP73833T

Commit message: Changer power daughter board directory name
Parts:
- H2, H3, H4: Manufacturer Name (none) -> None
- J1: footprint Naquadah Generator:Power_Daughter_Board_Conn -> Naquadah_Generator:State_Sensing_Mother_Board_JST_Conn; symbol Naquadah_Generator:End_Sphere_Conn -> Naquadah_Generator:Power_Daughter_Conn; Digikey Part No. (none) -> 455-1792-1-ND
- J2: footprint Naquadah Generator:PJ-006A-SMT -> CUI_PJ-006A-SMT
- TP1: Manufacturer (none) -> None; Name RDY -> Name
- TP2: Manufacturer (none) -> None; Manufacturer Part No. (none) -> None; Name SW -> Name
- TP3: Manufacturer (none) -> None; Manufacturer Part No. (none) -> None; Name BATT+ -> Name
- TP4: Manufacturer (none) -> None; Manufacturer Part No. (none) -> None; Name GND -> Name
- U1: footprint Li-ion 5A Boost 1A Charge Protect:MCP73833 -> High Power Lipo 18650 Boost Charge Protect:Charger_MCP73833
Changed lines of the file:
@@
 F 0 "U1" H 5525 2437 60  0000 C CNN
 F 1 "MCP73833T" H 5525 2331 60  0000 C CNN
-F 2 "Li-ion 5A Boost 1A Charge Protect:MCP73833" H 5550 1350 60  0001 C CNN
+F 2 "High Power Lipo 18650 Boost Charge Protect:Charger_MCP73833" H 5550 1350 60  0001 C CNN
 F 3 "http://ww1.microchip.com/downloads/en/DeviceDoc/22005b.pdf" H 5525 2331 60  0001 C CNN
 F 4 "Charger IC" H 5550 1950 50  0001 C CNN "Description"
@@
 	3950 1750 5000 1750
 $Comp
-L Naquadah_Generator:End_Sphere_Conn J1
+L Naquadah_Generator:Power_Daughter_Conn J1
 U 1 1 5EDA477E
 P 6400 4650
 F 0 "J1" H 6400 4350 50  0000 C CNN
 F 1 "End_Sphere_Conn" H 6400 5050 50  0000 C CNN
-F 2 "Naquadah Generator:Power_Daughter_Board_Conn" H 6450 4000 50  0001 C CNN
+F 2 "Naquadah_Generator:State_Sensing_Mother_Board_JST_Conn" H 6450 4000 50  0001 C CNN
 F 3 "http://www.jst-mfg.com/product/pdf/eng/eSH.pdf" H 6400 4700 50  0001 C CNN
 F 4 "Digikey" H 6400 4650 50  0001 C CNN "Source"
@@
 F 7 "BM06B-SRSS-TB(LF)(SN)" H 6450 4100 50  0001 C CNN "Manufacturer Part No."
 F 8 "Connector Header Surface Mount 6 position 0.039\" (1.00mm)" H 6400 4650 50  0001 C CNN "Description"
+F 9 "455-1792-1-ND" H 0   0   50  0001 C CNN "Digikey Part No."
 	1    6400 4650
 	-1   0    0    1
@@
 F 0 "J2" H 8650 5150 50  0000 L CNN
 F 1 "Jack-DC" H 8650 5050 50  0000 L CNN
-F 2 "Naquadah Generator:PJ-006A-SMT" H 8950 4760 50  0001 C CNN
-F 3 "https://www.cuidevices.com/product/resource/pj-006a-smt.pdf" H 8950 4760 50  0001 C CNN
+F 2 "CUI_PJ-006A-SMT" H 8950 4760 50  0001 C CNN
+F 3 "Manufacturer recommendations" H 8950 4760 50  0001 C CNN
 F 4 "Power Barrel Connector Jack 2.10mm ID (0.083\"), 5.50mm OD (0.217\") Surface Mount" H 8900 4800 50  0001 C CNN "Description"
 F 5 "Digikey" H 8900 4800 50  0001 C CNN "Source"
@@
 F 2 "Frequently_Used:Pad_2.5-2.5" H 6800 4300 50  0001 C CNN
 F 3 "None" H 6800 4300 50  0001 C CNN
-F 4 "RDY" H 6600 4500 50  0000 C CNN "Name"
+F 4 "Name" H 6600 4500 50  0000 C CNN "Name"
 F 5 "Test point" H 6600 4300 50  0001 C CNN "Description"
 F 6 "None" H 6600 4300 50  0001 C CNN "Source"
@@
 F 8 "None" H 6600 4300 50  0001 C CNN "Manufacturer Name"
 F 9 "None" H 6600 4300 50  0001 C CNN "Manufacturer Part No."
+F 10 "None" H 0   0   50  0001 C CNN "Manufacturer"
 	1    6600 4300
 	1    0    0    -1
@@
 F 2 "Frequently_Used:Pad_2.5-2.5" H 7050 4300 50  0001 C CNN
 F 3 "None" H 7050 4300 50  0001 C CNN
-F 4 "SW" H 6850 4500 50  0000 C CNN "Name"
+F 4 "Name" H 6850 4500 50  0000 C CNN "Name"
 F 5 "Test point" H 6850 4300 50  0001 C CNN "Description"
 F 6 "None" H 6850 4300 50  0001 C CNN "Source"
 F 7 "None" H 6850 4300 50  0001 C CNN "Source Part No."
 F 8 "None" H 6850 4300 50  0001 C CNN "Manufacturer Name"
+F 9 "None" H 0   0   50  0001 C CNN "Manufacturer"
+F 10 "None" H 0   0   50  0001 C CNN "Manufacturer Part No."
 	1    6850 4300
 	1    0    0    -1
@@
 F 2 "Frequently_Used:Pad_2.5-2.5" H 7050 4950 50  0001 C CNN
 F 3 "None" H 7050 4950 50  0001 C CNN
-F 4 "BATT+" H 6850 5150 50  0000 C CNN "Name"
+F 4 "Name" H 6850 5150 50  0000 C CNN "Name"
 F 5 "Test point" H 6850 4950 50  0001 C CNN "Description"
 F 6 "None" H 6850 4950 50  0001 C CNN "Source Part No."
 F 7 "None" H 6850 4950 50  0001 C CNN "Manufacturer Name"
 F 8 "None" H 6850 4950 50  0001 C CNN "Source"
+F 9 "None" H 0   0   50  0001 C CNN "Manufacturer"
+F 10 "None" H 0   0   50  0001 C CNN "Manufacturer Part No."
 	1    6850 4950
 	-1   0    0    1
@@
 F 2 "Frequently_Used:Pad_2.5-2.5" H 7300 4950 50  0001 C CNN
 F 3 "None" H 7300 4950 50  0001 C CNN
-F 4 "GND" H 7100 5150 50  0000 C CNN "Name"
+F 4 "Name" H 7100 5150 50  0000 C CNN "Name"
 F 5 "Test point" H 7100 4950 50  0001 C CNN "Description"
 F 6 "None" H 7100 4950 50  0001 C CNN "Source Part No."
 F 7 "None" H 7100 4950 50  0001 C CNN "Manufacturer Name"
 F 8 "None" H 7100 4950 50  0001 C CNN "Source"
+F 9 "None" H 0   0   50  0001 C CNN "Manufacturer"
+F 10 "None" H 0   0   50  0001 C CNN "Manufacturer Part No."
 	1    7100 4950
 	-1   0    0    1
@@
 F 1 "WireAssembly" H 3378 7055 50  0000 L CNN
 F 2 "Naquadah Generator:Wire_Assembly_Four" H 3000 7200 50  0001 C CNN
-F 3 "http://www.jst-mfg.com/product/pdf/eng/eSR.pdf" H 3000 7200 50  0001 C CNN
+F 3 "~" H 3000 7200 50  0001 C CNN
 F 4 "Digikey" H 3000 7100 50  0001 C CNN "Source"
 F 5 "6 Position Cable Assembly Rectangular Socket to Socket, Reversed 1.00' (304.80mm)" H 3000 7100 50  0001 C CNN "Description"
@@
 F 6 "None" H 805 7075 50  0001 C CNN "Source"
 F 7 "None" H 805 7075 50  0001 C CNN "Source Part No."
+F 8 "None" H 0   0   50  0001 C CNN "Manufacturer Name"
 	1    800  7200
 	1    0    0    -1
@@
 F 6 "None" H 1755 6825 50  0001 C CNN "Source"
 F 7 "None" H 1755 6825 50  0001 C CNN "Source Part No."
+F 8 "None" H 0   0   50  0001 C CNN "Manufacturer Name"
 	1    1750 6950
 	1    0    0    -1
@@
 F 6 "None" H 1755 7075 50  0001 C CNN "Source"
 F 7 "None" H 1755 7075 50  0001 C CNN "Source Part No."
+F 8 "None" H 0   0   50  0001 C CNN "Manufacturer Name"
 	1    1750 7200
 	1    0    0    -1

Commit message: Clean up
Parts:
- J1: Digikey Part No. 455-1792-1-ND -> (none)
- SW1: Manufacturer Apem -> (none); Manufacturer Name (none) -> Apem; Source (none) -> Digikey; Source Part No. (none) -> 679-3532-ND
- TP1, TP2, TP3, TP4: Manufacturer None -> (none)
Changed lines of the file:
@@
 F 3 "http://ww1.microchip.com/downloads/en/DeviceDoc/22005b.pdf" H 5525 2331 60  0001 C CNN
 F 4 "Charger IC" H 5550 1950 50  0001 C CNN "Description"
-F 5 "MCP73833T-AMI/UNCT-ND" H 5550 1950 50  0001 C CNN "Source Part No."
-F 6 "MCP73833T-AMI/UN" H 5550 1950 50  0001 C CNN "Manufacturer Part No."
-F 7 "Microchip Technology" H 5550 1950 50  0001 C CNN "Manufacturer Name"
-F 8 "Digikey" H 5550 1950 50  0001 C CNN "Source"
+F 5 "Digikey" H 5550 1950 50  0001 C CNN "Source"
+F 6 "MCP73833T-AMI/UNCT-ND" H 5550 1950 50  0001 C CNN "Source Part No."
+F 7 "MCP73833T-AMI/UN" H 5550 1950 50  0001 C CNN "Manufacturer Part No."
+F 8 "Microchip Technology" H 5550 1950 50  0001 C CNN "Manufacturer Name"
 	1    5550 1950
 	1    0    0    -1
@@
 U 1 1 5EDA477E
 P 6400 4650
-F 0 "J1" H 6400 4350 50  0000 C CNN
+F 0 "J1" H 6400 4300 50  0000 C CNN
 F 1 "End_Sphere_Conn" H 6400 5050 50  0000 C CNN
 F 2 "Naquadah_Generator:State_Sensing_Mother_Board_JST_Conn" H 6450 4000 50  0001 C CNN
@@
 F 7 "BM06B-SRSS-TB(LF)(SN)" H 6450 4100 50  0001 C CNN "Manufacturer Part No."
 F 8 "Connector Header Surface Mount 6 position 0.039\" (1.00mm)" H 6400 4650 50  0001 C CNN "Description"
-F 9 "455-1792-1-ND" H 0   0   50  0001 C CNN "Digikey Part No."
 	1    6400 4650
 	-1   0    0    1
@@
 F 8 "None" H 6600 4300 50  0001 C CNN "Manufacturer Name"
 F 9 "None" H 6600 4300 50  0001 C CNN "Manufacturer Part No."
-F 10 "None" H 0   0   50  0001 C CNN "Manufacturer"
 	1    6600 4300
 	1    0    0    -1
@@
 F 7 "None" H 6850 4300 50  0001 C CNN "Source Part No."
 F 8 "None" H 6850 4300 50  0001 C CNN "Manufacturer Name"
-F 9 "None" H 0   0   50  0001 C CNN "Manufacturer"
-F 10 "None" H 0   0   50  0001 C CNN "Manufacturer Part No."
+F 9 "None" H 0   0   50  0001 C CNN "Manufacturer Part No."
 	1    6850 4300
 	1    0    0    -1
@@
 F 4 "Name" H 6850 5150 50  0000 C CNN "Name"
 F 5 "Test point" H 6850 4950 50  0001 C CNN "Description"
-F 6 "None" H 6850 4950 50  0001 C CNN "Source Part No."
-F 7 "None" H 6850 4950 50  0001 C CNN "Manufacturer Name"
-F 8 "None" H 6850 4950 50  0001 C CNN "Source"
-F 9 "None" H 0   0   50  0001 C CNN "Manufacturer"
-F 10 "None" H 0   0   50  0001 C CNN "Manufacturer Part No."
+F 6 "None" H 6850 4950 50  0001 C CNN "Source"
+F 7 "None" H 6850 4950 50  0001 C CNN "Source Part No."
+F 8 "None" H 6850 4950 50  0001 C CNN "Manufacturer Name"
+F 9 "None" H 0   0   50  0001 C CNN "Manufacturer Part No."
 	1    6850 4950
 	-1   0    0    1
@@
 F 4 "Name" H 7100 5150 50  0000 C CNN "Name"
 F 5 "Test point" H 7100 4950 50  0001 C CNN "Description"
-F 6 "None" H 7100 4950 50  0001 C CNN "Source Part No."
-F 7 "None" H 7100 4950 50  0001 C CNN "Manufacturer Name"
-F 8 "None" H 7100 4950 50  0001 C CNN "Source"
-F 9 "None" H 0   0   50  0001 C CNN "Manufacturer"
-F 10 "None" H 0   0   50  0001 C CNN "Manufacturer Part No."
+F 6 "None" H 7100 4950 50  0001 C CNN "Source"
+F 7 "None" H 7100 4950 50  0001 C CNN "Source Part No."
+F 8 "None" H 7100 4950 50  0001 C CNN "Manufacturer Name"
+F 9 "None" H 0   0   50  0001 C CNN "Manufacturer Part No."
 	1    7100 4950
 	-1   0    0    1
@@
 F 1 "WireAssembly" H 3378 7055 50  0000 L CNN
 F 2 "Naquadah Generator:Wire_Assembly_Four" H 3000 7200 50  0001 C CNN
-F 3 "~" H 3000 7200 50  0001 C CNN
-F 4 "Digikey" H 3000 7100 50  0001 C CNN "Source"
-F 5 "6 Position Cable Assembly Rectangular Socket to Socket, Reversed 1.00' (304.80mm)" H 3000 7100 50  0001 C CNN "Description"
+F 3 "http://www.jst-mfg.com/product/pdf/eng/eSR.pdf" H 3000 7200 50  0001 C CNN
+F 4 "6 Position Cable Assembly Rectangular Socket to Socket, Reversed 1.00' (304.80mm)" H 3000 7100 50  0001 C CNN "Description"
+F 5 "Digikey" H 3000 7100 50  0001 C CNN "Source"
 F 6 "455-3019-ND" H 3000 7100 50  0001 C CNN "Source Part No."
 F 7 "JST Sales America Inc." H 3000 7100 50  0001 C CNN "Manufacturer Name"
@@
 F 3 "https://media.digikey.com/pdf/Data%20Sheets/APEM%20Components%20PDFs/MHPS_Series.pdf" H 5150 5100 50  0001 L CNN
 F 4 "APEM - MHPS2283 - Pushbutton Switch,STRAIGHT,DPDT,PC TAIL Terminal,PCB Hole Count:6" H 4350 4350 50  0001 L CNN "Description"
-F 5 "Apem" H 4350 4250 50  0001 L CNN "Manufacturer"
-F 6 "MHPS2283" H 4350 4150 50  0001 L CNN "Manufacturer Part No."
+F 5 "Digikey" H 4850 4900 50  0001 C CNN "Source"
+F 6 "679-3532-ND" H 4850 4900 50  0001 C CNN "Source Part No."
+F 7 "Apem" H 4850 4900 50  0001 C CNN "Manufacturer Name"
+F 8 "MHPS2283" H 4350 4150 50  0001 L CNN "Manufacturer Part No."
 	1    4850 4900
 	1    0    0    -1
@@
 F 2 "Naquadah Generator:MountingHole_2.2mm_M2" H 800 6950 50  0001 C CNN
 F 3 "None" H 800 6950 50  0001 C CNN
-F 4 "None" H 800 6950 50  0001 C CNN "Manufacturer Name"
-F 5 "None" H 805 6825 50  0001 C CNN "Manufacturer Part No."
-F 6 "None" H 805 6825 50  0001 C CNN "Source"
-F 7 "None" H 805 6825 50  0001 C CNN "Source Part No."
+F 4 "None" H 805 6825 50  0001 C CNN "Source"
+F 5 "None" H 805 6825 50  0001 C CNN "Source Part No."
+F 6 "None" H 800 6950 50  0001 C CNN "Manufacturer Name"
+F 7 "None" H 805 6825 50  0001 C CNN "Manufacturer Part No."
 	1    800  6950
 	1    0    0    -1
@@
 F 2 "Naquadah Generator:MountingHole_2.2mm_M2" H 800 7200 50  0001 C CNN
 F 3 "None" H 800 7200 50  0001 C CNN
-F 4 "" H 805 7075 50  0001 C CNN "Manufacturer"
-F 5 "None" H 805 7075 50  0001 C CNN "Manufacturer Part No."
-F 6 "None" H 805 7075 50  0001 C CNN "Source"
-F 7 "None" H 805 7075 50  0001 C CNN "Source Part No."
-F 8 "None" H 0   0   50  0001 C CNN "Manufacturer Name"
+F 4 "None" H 805 7075 50  0001 C CNN "Source"
+F 5 "None" H 805 7075 50  0001 C CNN "Source Part No."
+F 6 "None" H 0   0   50  0001 C CNN "Manufacturer Name"
+F 7 "None" H 805 7075 50  0001 C CNN "Manufacturer Part No."
 	1    800  7200
 	1    0    0    -1
@@
 F 2 "Naquadah Generator:MountingHole_2.2mm_M2" H 1750 6950 50  0001 C CNN
 F 3 "None" H 1750 6950 50  0001 C CNN
-F 4 "" H 1755 6825 50  0001 C CNN "Manufacturer"
-F 5 "None" H 1755 6825 50  0001 C CNN "Manufacturer Part No."
-F 6 "None" H 1755 6825 50  0001 C CNN "Source"
-F 7 "None" H 1755 6825 50  0001 C CNN "Source Part No."
-F 8 "None" H 0   0   50  0001 C CNN "Manufacturer Name"
+F 4 "None" H 1755 6825 50  0001 C CNN "Source"
+F 5 "None" H 1755 6825 50  0001 C CNN "Source Part No."
+F 6 "None" H 0   0   50  0001 C CNN "Manufacturer Name"
+F 7 "None" H 1755 6825 50  0001 C CNN "Manufacturer Part No."
 	1    1750 6950
 	1    0    0    -1
@@
 F 2 "Naquadah Generator:MountingHole_2.2mm_M2" H 1750 7200 50  0001 C CNN
 F 3 "None" H 1750 7200 50  0001 C CNN
-F 4 "" H 1755 7075 50  0001 C CNN "Manufacturer"
-F 5 "None" H 1755 7075 50  0001 C CNN "Manufacturer Part No."
-F 6 "None" H 1755 7075 50  0001 C CNN "Source"
-F 7 "None" H 1755 7075 50  0001 C CNN "Source Part No."
-F 8 "None" H 0   0   50  0001 C CNN "Manufacturer Name"
+F 4 "None" H 1755 7075 50  0001 C CNN "Source"
+F 5 "None" H 1755 7075 50  0001 C CNN "Source Part No."
+F 6 "None" H 0   0   50  0001 C CNN "Manufacturer Name"
+F 7 "None" H 1755 7075 50  0001 C CNN "Manufacturer Part No."
 	1    1750 7200
 	1    0    0    -1

Commit message: Switched to 4 pin power board connector
Parts:
- H1, H2, H3, H4: Description (none) -> None
- J1: value End_Sphere_Conn -> Power Board Conn; footprint Naquadah_Generator:State_Sensing_Mother_Board_JST_Conn -> Naquadah_Generator:Daughter_Board_Vert_4_Pin_JST_Conn; symbol Naquadah_Generator:Power_Daughter_Conn -> Naquadah_Generator:Power_Daughter_4_Pin_Conn; Description Connector Header Surface Mount 6 position 0.039\" (1.00mm) -> Connector Header Surface Mount 4 position 0.039\" (1.00mm); Manufacturer Part No. BM06B-SRSS-TB(LF)(SN) -> BM04B-SRSS-TB(LF)(SN); Source Part No. 455-1792-1-ND -> 455-1790-1-ND
- J2: footprint CUI_PJ-006A-SMT -> Naquadah_Generator:PJ-006A-SMT
- TP1: Name Name -> RDY
- TP2: Name Name -> SW
- TP3: Name Name -> B+
- TP4: Name Name -> GND
- U1: footprint High Power Lipo 18650 Boost Charge Protect:Charger_MCP73833 -> Li-ion 5A Boost 1A Charge Protect:MCP73833
Connections:
- wire segments 82 -> 74
Other:
- moved on the sheet: H1, H2, H3, H4, TP1, TP2, TP3, TP4, WA1

Commit message: Before updating to two switches
Parts:
- added SW2: MHPS2283N, Naquadah_Generator:MHPS2283, symbol Naquadah_Generator:MHPS2283
- added TP5: TestPoint, Frequently_Used:Pad_2.5-2.5, symbol Frequently_Used:TestPoint
- J1: footprint Naquadah_Generator:Daughter_Board_Vert_4_Pin_JST_Conn -> Naquadah_Generator:Daughter_Board_Vert_5_Pin_JST_Conn; symbol Naquadah_Generator:Power_Daughter_4_Pin_Conn -> Naquadah_Generator:Power_Daughter_5_Pin_Conn
- SW1: footprint Naquadah Generator:MHPS2283 -> Naquadah_Generator:MHPS2283
Connections:
- net labels added: MODE
- wire segments 74 -> 84
- no-connect marks 3 -> 5
Other:
- note added: "Mode Button"
- moved on the sheet: D1, D5, J2, R1, R5, SW1, TP1, TP2, TP3, TP4
