File: Power Daughter Board/Power Daughter Board.sch (KiCad schematic (older format))
At the start: 31 parts, among them J1 Power Board Conn, J2 Jack-DC, SW1 MHPS2283, SW2 MHPS2283N, U1 MCP73833T

Commit message: Power updates
Parts:
- removed C1, C2: 22uF, Li-ion:0805_2012Metric_HandSolder, symbol Li_Ion_LE:C
- removed D2, D3: GREEN, Li-ion:LED_0805_2012Metric_HandSolder, symbol Li_Ion_LE:LED
- removed D4: RED, Li-ion:LED_0805_2012Metric_HandSolder, symbol Li_Ion_LE:LED
- removed R2, R3, R4, R8: 1k, Li-ion:0805_2012Metric_HandSolder, symbol Li_Ion_LE:R
- removed R6: 1.54k, Li-ion:0805_2012Metric_HandSolder, symbol Li_Ion_LE:R
- removed R7: 69.8k, Li-ion:0805_2012Metric_HandSolder, symbol Li_Ion_LE:R
- removed TH1: 10k, Li-ion:0805_2012Metric_HandSolder, symbol Li_Ion_LE:Thermistor_NTC
- removed U1: MCP73833T, Li-ion:MCP73833, symbol Li_Ion_LE:MCP73833T
- D1, D5: symbol Li_Ion_LE:LED -> Frequently_Used_LE:LED
- R1, R5: symbol Li_Ion_LE:R -> Frequently_Used_LE:R
- TP1, TP2, TP3, TP4, TP5: symbol Frequently_Used_LE:TestPoint -> Frequently_Used_LE:TestPoint_1
Connections:
- net labels added: DGND
- net labels removed: GND, PG, PROG, ST1, ST2, THRM, THRMIC
- wire segments 84 -> 46
Other:
- moved on the sheet: J1, J2, SW1, SW2

Commit message: Before switching buttons on daughter board
Parts:
- D1, D5: footprint Li-ion:LED_0805_2012Metric_HandSolder -> Frequently_Used_LE:LED_0805_2012Metric
- R1, R5: footprint Li-ion:0805_2012Metric_HandSolder -> Frequently_Used_LE:0805_2012Metric
Changed lines of the file:
@@
 F 0 "D1" H 7900 2300 50  0000 L CNN
 F 1 "GREEN" H 7900 2100 50  0000 L CNN
-F 2 "Li-ion:LED_0805_2012Metric_HandSolder" H 8000 2200 50  0001 C CNN
+F 2 "Frequently_Used_LE:LED_0805_2012Metric" H 8000 2200 50  0001 C CNN
 F 3 "https://www.we-online.de/katalog/datasheet/150080VS75000.pdf" H 8000 2200 50  0001 C CNN
 F 4 "Green 570nm LED Indication - Discrete 2V 0805 (2012 Metric)" H 8000 2200 50  0001 C CNN "Description"
@@
 F 0 "R1" V 7900 1500 59  0000 L CNN
 F 1 "1k" V 8100 1500 59  0000 L CNN
-F 2 "Li-ion:0805_2012Metric_HandSolder" H 8000 1600 50  0001 C CNN
+F 2 "Frequently_Used_LE:0805_2012Metric" H 8000 1600 50  0001 C CNN
 F 3 "http://www.koaspeer.com/pdfs/RK73H.pdf" H 8000 1600 50  0001 C CNN
 F 4 "1 kOhms ±1% 0.25W, 1/4W Chip Resistor 1206 (3216 Metric) " H 8000 1600 50  0001 C CNN "Description"
@@
 F 0 "D5" H 6550 2300 50  0000 L CNN
 F 1 "RED" H 6550 2100 50  0000 L CNN
-F 2 "Li-ion:LED_0805_2012Metric_HandSolder" H 6650 2200 50  0001 C CNN
+F 2 "Frequently_Used_LE:LED_0805_2012Metric" H 6650 2200 50  0001 C CNN
 F 3 "https://www.we-online.de/katalog/datasheet/150080RS75000.pdf" H 6650 2200 50  0001 C CNN
 F 4 "Red 625nm LED Indication - Discrete 2V 0805 (2012 Metric)" H 6650 2200 50  0001 C CNN "Description"
@@
 F 0 "R5" V 6550 1500 59  0000 L CNN
 F 1 "1k" V 6750 1500 59  0000 L CNN
-F 2 "Li-ion:0805_2012Metric_HandSolder" H 6650 1600 50  0001 C CNN
+F 2 "Frequently_Used_LE:0805_2012Metric" H 6650 1600 50  0001 C CNN
 F 3 "http://www.koaspeer.com/pdfs/RK73H.pdf" H 6650 1600 50  0001 C CNN
 F 4 "1 kOhms ±1% 0.25W, 1/4W Chip Resistor 1206 (3216 Metric) " H 6650 1600 50  0001 C CNN "Description"
@@
 $EndSheet
 $Comp
-L Frequently_Used_LE:DGND #PWR?
+L Frequently_Used_LE:DGND #PWR0101
 U 1 1 5F3CF85B
 P 2850 2450
-F 0 "#PWR?" H 2850 2200 50  0001 C CNN
+F 0 "#PWR0101" H 2850 2200 50  0001 C CNN
 F 1 "DGND" H 2855 2277 50  0000 C CNN
 F 2 "" H 2850 2450 50  0001 C CNN
@@
 	2850 2350 2850 2450
 $Comp
-L Frequently_Used_LE:DGND #PWR?
+L Frequently_Used_LE:DGND #PWR0102
 U 1 1 5F3DA09E
 P 9000 4950
-F 0 "#PWR?" H 9000 4700 50  0001 C CNN
+F 0 "#PWR0102" H 9000 4700 50  0001 C CNN
 F 1 "DGND" H 9005 4777 50  0000 C CNN
 F 2 "" H 9000 4950 50  0001 C CNN
@@
 $EndComp
 $Comp
-L Frequently_Used_LE:DGND #PWR?
+L Frequently_Used_LE:DGND #PWR0103
 U 1 1 5F3DB069
 P 7300 4850
-F 0 "#PWR?" H 7300 4600 50  0001 C CNN
+F 0 "#PWR0103" H 7300 4600 50  0001 C CNN
 F 1 "DGND" H 7305 4677 50  0000 C CNN
 F 2 "" H 7300 4850 50  0001 C CNN
@@
 $EndComp
 $Comp
-L Frequently_Used_LE:DGND #PWR?
+L Frequently_Used_LE:DGND #PWR0104
 U 1 1 5F3DBFD7
 P 3600 5000
-F 0 "#PWR?" H 3600 4750 50  0001 C CNN
+F 0 "#PWR0104" H 3600 4750 50  0001 C CNN
 F 1 "DGND" H 3605 4827 50  0000 C CNN
 F 2 "" H 3600 5000 50  0001 C CNN
@@
 $EndComp
 $Comp
-L Frequently_Used_LE:DGND #PWR?
+L Frequently_Used_LE:DGND #PWR0105
 U 1 1 5F3DCE48
 P 8000 2450
-F 0 "#PWR?" H 8000 2200 50  0001 C CNN
+F 0 "#PWR0105" H 8000 2200 50  0001 C CNN
 F 1 "DGND" H 8005 2277 50  0000 C CNN
 F 2 "" H 8000 2450 50  0001 C CNN
@@
 $EndComp
 $Comp
-L Frequently_Used_LE:DGND #PWR?
+L Frequently_Used_LE:DGND #PWR0106
 U 1 1 5F3DDAC4
 P 6650 2450
-F 0 "#PWR?" H 6650 2200 50  0001 C CNN
+F 0 "#PWR0106" H 6650 2200 50  0001 C CNN
 F 1 "DGND" H 6655 2277 50  0000 C CNN
 F 2 "" H 6650 2450 50  0001 C CNN

Commit message: Audio updates, switching to separate USB schematic
Audio updates, switching to separate USB schematic
Parts:
- removed SW1: MHPS2283, Naquadah_Generator:MHPS2283, symbol Naquadah_Generator:MHPS2283
- removed SW2: MHPS2283N, Naquadah_Generator:MHPS2283, symbol Naquadah_Generator:MHPS2283
- added H5, H6: MountingHole, Naquadah_Generator:MountingHole_2.7mm_M2.5, symbol Naquadah_Generator:MountingHole
- added SW1: SW_Push_DPDT_2-5_3-4_1-4, Button_Switches_LE:ESB-33535A, symbol Buttons_Switches_LE:SW_Push_DPDT_2-5_3-4_1-4
- added SW2: SW_Push_Dual_1-3_2-4, Button_Switches_LE:PTS647SK38SMTR2LFS, symbol Buttons_Switches_LE:SW_Push_Dual_1-3_2-4
Connections:
- net BATT+: now also SW1.2 (C), SW1.5 (C)
- net DGND: now also SW2.1, SW2.3
- net MODE: now also SW2.2, SW2.4
- net SWITCH: now also SW1.1 (NO), SW1.4 (NO)
- no-connect marks 5 -> 3
Other:
- moved on the sheet: H1, H2, H3, H4, J1, J2, TP1, TP2, TP3, TP4, TP5, WA1

Commit message: Switched to 0603_1608M size for passives
Parts:
- added R10, R11, R12, R9: 2.7k, Frequently_Used_LE:0805_2012Metric, symbol Frequently_Used_LE:R
- added SW3, SW4: SW_Push_Dual_1-3_2-4, Button_Switches_LE:PTS647SK38SMTR2LFS, symbol Buttons_Switches_LE:SW_Push_Dual_1-3_2-4
- added TP6: TestPoint, Frequently_Used_LE:Pad_2.5-2.5, symbol Frequently_Used_LE:TestPoint_1
- J1: value Power Board Conn -> Mother Board Conn; footprint Naquadah_Generator:Daughter_Board_Vert_5_Pin_JST_Conn -> Naquadah_Generator:Daughter_Board_Vert_6_Pin_JST_Conn; symbol Naquadah_Generator:Power_Daughter_5_Pin_Conn -> Naquadah_Generator:User_Interface_6_Pin_Conn
- TP5: Name SW -> SWITCH
Connections:
- net DGND: now also R9.2
- net MODE: now also J1.4 (MODE); no longer J1.3 (MODE)
- net READY: now also J1.5 (READY), R12.1; no longer J1.4 (READY)
- net SWITCH: now also J1.6 (SWITCH); no longer J1.5 (SW)
- new net: R10.2, R9.1, SW3.1, SW3.3
- new net: R11.1, R12.2, SW4.2, SW4.4
- new net VOLUME: J1.3 (VOLUME), R10.1, R11.2, SW3.2, SW3.4, SW4.1, SW4.3, TP6.1
Other:
- note added: "Volume Down / Up"
- moved on the sheet: D1, D5, J2, R1, R5, SW1, SW2, TP1, TP2, TP3, TP4, TP5
