File: Power Daughter Board/Power Daughter Board.kicad_pcb (KiCad board)
At the start: 2 copper layers, 34.8 x 39.1 mm, 29 parts, among them J1 End_Sphere_Conn, J2 Jack-DC, SW1 MHPS2283, U1 MCP73833T

Commit message: Switched to 4 pin power board connector
Parts:
- added ?: , , F.Cu at (151.9, 106.8)
- J1: value End_Sphere_Conn -> Power Board Conn; footprint Naquadah Generator:Power_Daughter_Board_Conn -> Naquadah_Generator:Daughter_Board_Vert_4_Pin_JST_Conn
- J2: footprint Naquadah Generator:PJ-006A-SMT -> Naquadah_Generator:PJ-006A-SMT
Connections:
- J1 pad 2: GND -> /BATT+
- J1 pad 3: /BATT+ -> /SWITCH
- J1 pad 4: /BATT+ -> /READY
Routing:
- net /READY: track 26.6 -> 24.2 mm
- net /BATT+: track 13.5 -> 12.1 mm
Other:
- board text added: "1"
- board text added: "2"
- board text added: "G B S R"
- board text added: "P"
- board text removed: "B+"
- board text removed: "G"
- board text removed: "RDY"
- board text removed: "SW"

Commit message: Before updating to two switches
Parts:
- removed ?: , 
- added SW2: MHPS2283N, Naquadah_Generator:MHPS2283, F.Cu at (157.2, 94.0)
- added TP5: TestPoint, Frequently_Used:Pad_2.5-2.5, B.Cu at (136.7, 80.3)
- J1: footprint Naquadah_Generator:Daughter_Board_Vert_4_Pin_JST_Conn -> Naquadah_Generator:Daughter_Board_Vert_5_Pin_JST_Conn
- SW1: footprint Naquadah Generator:MHPS2283 -> Naquadah_Generator:MHPS2283
- moved D1 12.2 mm to (145.9, 93.2)
- moved D5 11.3 mm to (145.8, 97.0)
- moved SW1 9.51 mm to (136.0, 95.5)
Other:
- board text added: "CHARGING"
- board text added: "COMPLETE"
- board text added: "FAULT"
- board text added: "NC B SW"
- board text added: "SHUTDOWN"
- board text added: "STANDBY"
- board text added: "TEST"

Commit message: Power board 2 switch V1
Parts:
- moved R8 20.1 mm to (151.1, 98.1), turned to 90 degrees
- moved TP5 19.7 mm to (138.7, 99.9)
- moved TP4 18.5 mm to (131.4, 110.6)
- moved TP3 14.2 mm to (131.4, 105.5)
- moved TP1 13.8 mm to (145.5, 93.7)
- moved TP2 8.27 mm to (152.2, 100.0)
- moved R1 8.07 mm to (139.9, 95.8), turned to 270 degrees
- moved R5 6.45 mm to (151.1, 92.7), turned to 90 degrees
- moved D5 5.38 mm to (145.5, 91.7), turned to 0 degrees
- moved D1 3.66 mm to (145.5, 96.8), turned to 180 degrees
- moved H2 3.32 mm to (156.3, 102.9)
- moved H1 3.32 mm to (134.7, 102.9)
- moved SW1 2.51 mm to (133.8, 94.2), turned to 0 degrees
- moved C1 1.89 mm to (155.2, 110.3), turned to 180 degrees
- moved C2 1.79 mm to (155.2, 107.8), turned to 180 degrees
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Connections:
- D1 pad 1: /ON -> GND
- D1 pad 2: /SWITCH -> /ONIND
- D5 pad 1: /RDYIND -> GND
- D5 pad 2: /READY -> /RDYIND
- J1 pad 3: /SWITCH -> /MODE
- J1 pad 5: /MODE -> /SWITCH
- R1 pad 1: /ON -> /SWITCH
- R1 pad 2: GND -> /ONIND
- R5 pad 1: /RDYIND -> /READY
- R5 pad 2: GND -> /RDYIND
- TP2 pad 1: /SWITCH -> /MODE
- TP5 pad 1: /MODE -> /SWITCH
Routing:
- net /MODE: track 0.00 -> 22.1 mm
- net /SWITCH: track 43.7 -> 26.1 mm
- net /PROG: track 29.8 -> 15.8 mm
- net /READY: track 24.2 -> 18.5 mm
- net /ON: track 5.34 -> 0.00 mm
- net /ONIND: track 0.00 -> 4.06 mm
- net GND: track 30.0 -> 27.1 mm, vias 10 -> 9
- net /PG: track 28.0 -> 28.9 mm
- net /RDYIND: track 5.32 -> 4.54 mm
- net /ST1: track 17.9 -> 18.7 mm
- net /BATT+: track 12.1 -> 12.6 mm
Other:
- board text added: "B"
- board text added: "G"
- board text added: "GBMRS"
- board text added: "NC G M"
- board text added: "NQH-PCB-003"
- board text added: "S B NC"
- board text added: "V1.0.0"
- board text removed: "+"
- board text removed: "-"
- board text removed: "G B S R"
- board text removed: "NC B SW"

Commit message: Updates
Parts:
- H1, H2, H3, H4: footprint Naquadah Generator:MountingHole_2.2mm_M2 -> Naquadah_Generator:MountingHole_2.7mm_M2.5
- WA1: footprint Naquadah Generator:Wire_Assembly_Four -> Naquadah_Generator:Wire_Assembly_Four
- moved TP4 2.38 mm to (131.4, 113.0)
- moved TP3 2.26 mm to (131.4, 107.8)
- moved TP2 0.51 mm to (151.7, 100.0)
- moved TP5 0.49 mm to (139.2, 99.9)
Routing:
- net /BATT+: track 12.6 -> 14.9 mm

Commit message: Move libraries and added configuration path.
Moved Li-Ion library to common KiCad library.  Added variables to configuration paths to reference my KiCad libraries.  Moved all 3D components to my common library.
Parts:
- C1, C2, R1, R2, R3, R4, R5, R6, R7, R8, TH1: footprint Li-ion 5A Boost 1A Charge Protect:0805_2012Metric_HandSolder -> Li-ion:0805_2012Metric_HandSolder
- D1, D2, D3, D4, D5: footprint Li-ion 5A Boost 1A Charge Protect:LED_0805_2012Metric_HandSolder -> Li-ion:LED_0805_2012Metric_HandSolder
- TP1, TP2, TP3, TP4, TP5: footprint Frequently_Used:Pad_2.5-2.5 -> FrequentlyUsed:Pad_2.5-2.5
- U1: footprint Li-ion 5A Boost 1A Charge Protect:MCP73833 -> Li-ion:MCP73833
