File: Power Daughter Board/Power Daughter Board.kicad_pcb (KiCad board)
At the start: 2 copper layers, 34.8 x 39.1 mm, 31 parts, among them J1 Power Board Conn, J2 Jack-DC, SW1 MHPS2283, SW2 MHPS2283N, U1 MCP73833T

Commit message: Before switching buttons on daughter board
Parts:
- C1, C2, R1, R2, R3, R4, R5, R6, R7, TH1: footprint Li-ion:0805_2012Metric_HandSolder -> Frequently_Used_LE:0805_2012Metric
- D1, D2, D3, D4, D5: footprint Li-ion:LED_0805_2012Metric_HandSolder -> Frequently_Used_LE:LED_0805_2012Metric
- R8: value 1k -> 1.33k; footprint Li-ion:0805_2012Metric_HandSolder -> Frequently_Used_LE:0805_2012Metric
- TP1, TP2, TP3, TP4, TP5: footprint FrequentlyUsed:Pad_2.5-2.5 -> Frequently_Used_LE:Pad_2.5-2.5
- U1: footprint Li-ion:MCP73833 -> Li_Ion_LE:MCP73833
Connections:
- net /PG renamed /Charge 750mA/PG
- net /PROG renamed /Charge 750mA/PROG
- net /ST1 renamed /Charge 750mA/ST1
- net /ST2 renamed /Charge 750mA/ST2
- net /THRM renamed /Charge 750mA/THRM
- net /THRMIC renamed /Charge 750mA/THRMIC
- net GND renamed DGND

Commit message: Audio updates, switching to separate USB schematic
Audio updates, switching to separate USB schematic
Parts:
- SW1: value MHPS2283 -> SW_Push_DPDT_2-5_3-4_1-4; footprint Naquadah_Generator:MHPS2283 -> Button_Switches_LE:ESB-33535A
- SW2: value MHPS2283N -> SW_Push_Dual_1-3_2-4; footprint Naquadah_Generator:MHPS2283 -> Button_Switches_LE:PTS647SK38SMTR2LFS
Connections:
- SW1 pad 1: (no net) -> /SWITCH
- SW1 pad 3: /SWITCH -> (no net)
- SW2 pad 1: (no net) -> DGND
- SW2 pad 2: DGND -> /MODE
- SW2 pad 3: /MODE -> DGND
Routing:
- net /BATT+: track 14.9 -> 13.4 mm
- net /Charge 750mA/PROG: track 15.8 -> 17.1 mm, vias 2 -> 0
- net /Charge 750mA/THRMIC: track 30.9 -> 31.6 mm

Commit message: Switched to 0603_1608M size for passives
Parts:
- added H5: MountingHole, Naquadah_Generator:MountingHole_2.7mm_M2.5, F.Cu at (184.6, 109.6)
- added H6: MountingHole, Naquadah_Generator:MountingHole_2.7mm_M2.5, F.Cu at (108.1, 110.0)
- added R10: 2.7k, Frequently_Used_LE:0805_2012Metric, F.Cu at (136.3, 90.1)
- added R11: 2.7k, Frequently_Used_LE:0805_2012Metric, F.Cu at (159.4, 90.1)
- added R12: 2.7k, Frequently_Used_LE:0805_2012Metric, F.Cu at (154.6, 90.1)
- added R9: 2.7k, Frequently_Used_LE:0805_2012Metric, F.Cu at (131.4, 90.2)
- added SW3: SW_Push_Dual_1-3_2-4, Button_Switches_LE:PTS647SK38SMTR2LFS, F.Cu at (133.8, 94.2)
- added SW4: SW_Push_Dual_1-3_2-4, Button_Switches_LE:PTS647SK38SMTR2LFS, F.Cu at (157.1, 94.2)
- added TP6: TestPoint, Frequently_Used_LE:Pad_2.5-2.5, B.Cu at (168.6, 90.0)
- J1: value Power Board Conn -> Mother Board Conn; footprint Naquadah_Generator:Daughter_Board_Vert_5_Pin_JST_Conn -> Naquadah_Generator:Daughter_Board_Vert_6_Pin_JST_Conn
- moved D1 43.0 mm to (102.5, 99.0)
- moved R1 43.0 mm to (96.9, 97.9)
- moved D5 22.5 mm to (165.2, 102.7), turned to 180 degrees
- moved R5 17.5 mm to (157.2, 109.1)
- moved SW1 17.1 mm to (126.0, 109.4), turned to 90 degrees
- moved SW2 17.1 mm to (165.0, 109.4)
- moved R6 15.9 mm to (140.7, 94.7)
- moved R7 15.9 mm to (140.8, 98.2)
- moved TH1 15.9 mm to (140.7, 101.8)
- moved U1 14.9 mm to (150.2, 98.0)
- moved C1 14.8 mm to (145.5, 99.2)
- moved C2 14.8 mm to (145.5, 96.7)
- moved R8 9.49 mm to (145.5, 90.4), turned to 180 degrees
- moved R3 0.78 mm to (160.8, 118.6)
Connections:
- J1 pad 3: /MODE -> /VOLUME
- J1 pad 4: /READY -> /MODE
- J1 pad 5: /SWITCH -> /READY
Routing:
- net /Charge 750mA/THRMIC: track 31.6 -> 0.00 mm, vias 2 -> 0
- net /Charge 750mA/PROG: track 17.1 -> 0.00 mm
- net /MODE: track 22.4 -> 11.8 mm
- net DGND: track 27.3 -> 20.7 mm, vias 9 -> 7
- net /SWITCH: track 26.2 -> 20.2 mm
- net /READY: track 18.5 -> 12.9 mm, vias 1 -> 0
- net /RDYIND: track 4.54 -> 0.00 mm
- net /ONIND: track 4.06 -> 0.00 mm
- net /Charge 750mA/ST1: track 18.7 -> 14.9 mm
- net /Charge 750mA/ST2: track 5.74 -> 2.88 mm
- net Net-(D3-Pad1): track 6.30 -> 5.63 mm
- net /BATT+: vias 3 -> 0
Other:
- board text added: "GBVMRS"
- board text removed: "GBMRS"
