File: User Interface Daughter Board/User Interface Daughter Board.kicad_pcb (KiCad board)
At the start: 2 copper layers, 34.8 x 39.1 mm, 40 parts, among them J1 Mother Board Conn, J2 Jack-DC, SW1 SW_Push_DPDT_2-5_3-4_1-4, SW2 SW_Push_Dual_1-3_2-4, SW3 SW_Push_Dual_1-3_2-4, SW4 SW_Push_Dual_1-3_2-4, U1 MCP73833T

Commit message: Update JST connectors
Parts:
- J1: footprint Naquadah_Generator:Daughter_Board_Vert_6_Pin_JST_Conn -> Connector_JST:JST_SH_BM06B-SRSS-TB_1x06-1MP_P1.00mm_Vertical
- WA1: footprint Naquadah_Generator:Wire_Assembly_Four -> Mechanical_LE:Wire_Assembly
Routing:
- net /READY: track 12.9 -> 0.00 mm
- net /MODE: track 11.8 -> 0.03 mm
- net /SWITCH: track 20.2 -> 10.4 mm
- net /BATT+: track 13.4 -> 12.7 mm

Commit message: Updated fiducials.
Parts:
- added FID1: Fiducial, Fiducial_LE:Fiducial_1mm_Mask2mm, F.Cu at (169.2, 126.2)
- added FID2: Fiducial, Fiducial_LE:Fiducial_1mm_Mask2mm, F.Cu at (172.8, 126.2)
- added FID3: Fiducial, Fiducial_LE:Fiducial_1mm_Mask2mm, F.Cu at (176.3, 126.2)
Changed lines of the file:
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@@
     (tracks 75)
     (zones 0)
-    (modules 40)
+    (modules 43)
     (nets 21)
   )
@@
     (uvia_drill 0.1)
   )
+  (module Fiducial_LE:Fiducial_1mm_Mask2mm (layer F.Cu)
+    (at 176.33 126.24)
+    (descr "Circular Fiducial, 1mm bare copper, 2mm soldermask opening (Level A)")
+    (tags fiducial)
+    (attr smd)
+    (fp_text reference FID3 (at 0 -2) (layer F.Fab)
+      (effects (font (size 1 1) (thickness 0.15)))
+    )
+    (fp_text value Fiducial (at 0 2) (layer F.Fab)
+      (effects (font (size 1 1) (thickness 0.15)))
+    )
+    (fp_circle (center 0 0) (end 1 0) (layer F.Fab) (width 0.1))
+    (fp_text user %R (at 0 0) (layer F.Fab)
+      (effects (font (size 0.4 0.4) (thickness 0.06)))
+    )
+    (fp_circle (center 0 0) (end 1.25 0) (layer F.CrtYd) (width 0.05))
+    (pad "" smd circle (at 0 0) (size 1 1) (layers F.Cu F.Mask)
+      (solder_mask_margin 0.5) (clearance 0.5))
+  )
+  (module Fiducial_LE:Fiducial_1mm_Mask2mm (layer F.Cu)
+    (at 172.78 126.24)
+    (descr "Circular Fiducial, 1mm bare copper, 2mm soldermask opening (Level A)")
+    (tags fiducial)
+    (attr smd)
+    (fp_text reference FID2 (at 0 -2) (layer F.Fab)
+      (effects (font (size 1 1) (thickness 0.15)))
+    )
+    (fp_text value Fiducial (at 0 2) (layer F.Fab)
+      (effects (font (size 1 1) (thickness 0.15)))
+    )
+    (fp_circle (center 0 0) (end 1 0) (layer F.Fab) (width 0.1))
+    (fp_text user %R (at 0 0) (layer F.Fab)
+      (effects (font (size 0.4 0.4) (thickness 0.06)))
+    )
+    (fp_circle (center 0 0) (end 1.25 0) (layer F.CrtYd) (width 0.05))
+    (pad "" smd circle (at 0 0) (size 1 1) (layers F.Cu F.Mask)
+      (solder_mask_margin 0.5) (clearance 0.5))
+  )
+  (module Fiducial_LE:Fiducial_1mm_Mask2mm (layer F.Cu)
+    (at 169.23 126.24)
+    (descr "Circular Fiducial, 1mm bare copper, 2mm soldermask opening (Level A)")
+    (tags fiducial)
+    (attr smd)
+    (fp_text reference FID1 (at 0 -2) (layer F.Fab)
+      (effects (font (size 1 1) (thickness 0.15)))
+    )
+    (fp_text value Fiducial (at 0 2) (layer F.Fab)
+      (effects (font (size 1 1) (thickness 0.15)))
+    )
+    (fp_circle (center 0 0) (end 1 0) (layer F.Fab) (width 0.1))
+    (fp_text user %R (at 0 0) (layer F.Fab)
+      (effects (font (size 0.4 0.4) (thickness 0.06)))
+    )
+    (fp_circle (center 0 0) (end 1.25 0) (layer F.CrtYd) (width 0.05))
+    (pad "" smd circle (at 0 0) (size 1 1) (layers F.Cu F.Mask)
+      (solder_mask_margin 0.5) (clearance 0.5))
+  )
   (module Connector_JST:JST_SH_BM06B-SRSS-TB_1x06-1MP_P1.00mm_Vertical (layer B.Cu)
